Commit message: dvrk_arm_rviz: fixed to use either Classic or Si, added missing "mimic" in PSM Si xacro, added "simulated" argument, dos2unix, formatting...

File: urdf/Si/psm.base.urdf.xacro (robot description, xacro)
@@ -1,308 +1,314 @@
 <?xml version="1.0"?>
 <robot name="dvrk_si" xmlns:xacro="http://www.ros.org/wiki/xacro">
-    <xacro:macro name="psm_arm_active" params="prefix parent_link xyz rpy">
-        <link
-            name="${prefix}link_0">
-            <inertial>
-            <origin
-                xyz="-0.080771 2.1131E-08 1.8613E-07"
-                rpy="0 0 0" />
-            <mass
-                value="1.5188" />
-            <inertia
-                ixx="0.002395"
-                ixy="-2.6476E-18"
-                ixz="-1.3484E-18"
-                iyy="0.0040794"
-                iyz="4.2598E-10"
-                izz="0.0043778" />
-            </inertial>
-            <visual>
-            <origin
-                xyz="0 0 0"
-                rpy="0 0 0" />
-            <geometry>
-                <mesh
-                filename="package://dvrk_model/meshes/Si/PSM_ECM/link_0.STL" />
-            </geometry>
-            <material
-                name="">
-                <color
-                rgba="0.79216 0.81961 0.93333 1" />
-            </material>
-            </visual>
-            <collision>
-            <origin
-                xyz="0 0 0"
-                rpy="0 0 0" />
-            <geometry>
-                <mesh
-                filename="package://dvrk_model/meshes/Si/PSM_ECM/link_0.STL" />
-            </geometry>
-            </collision>
-        </link>
-        <joint name="${prefix}fixed" type="fixed">
-            <parent link="${parent_link}"/>
-            <child link="${prefix}link_0"/>
-            <origin rpy="${rpy}" xyz="${xyz}"/>
-        </joint>
-        <link
-            name="${prefix}link_1">
-            <inertial>
-            <origin
-                xyz="0.1461 0.090363 -0.024957"
-                rpy="0 0 0" />
-            <mass
-                value="1.7571" />
-            <inertia
-                ixx="0.0049404"
-                ixy="-0.0035267"
-                ixz="0.0045945"
-                iyy="0.019686"
-                iyz="0.00070407"
-                izz="0.020795" />
-            </inertial>
-            <visual>
-            <origin
-                xyz="0 0 0"
-                rpy="0 0 0" />
-            <geometry>
-                <mesh
-                filename="package://dvrk_model/meshes/Si/PSM_ECM/link_1.STL" />
-            </geometry>
-            <material
-                name="">
-                <color
-                rgba="0.79216 0.81961 0.93333 1" />
-            </material>
-            </visual>
-            <collision>
-            <origin
-                xyz="0 0 0"
-                rpy="0 0 0" />
-            <geometry>
-                <mesh
-                filename="package://dvrk_model/meshes/Si/PSM_ECM/link_1.STL" />
-            </geometry>
-            </collision>
-        </link>
-        <joint
-            name="${prefix}j1"
-            type="revolute">
-            <origin
-            xyz="0.158 0 0"
-            rpy="0 0 0" />
-            <parent
-            link="${prefix}link_0" />
-            <child
-            link="${prefix}link_1" />
-            <axis
-            xyz="1 0 0" />
-            <limit
-            lower="-3.14"
-            upper="3.14"
-            effort="0"
-            velocity="0" />
-        </joint>
-        <link
-            name="${prefix}link_2">
-            <inertial>
-            <origin
-                xyz="0.083895 -0.00073113 -0.028998"
-                rpy="0 0 0" />
-            <mass
-                value="4.017" />
-            <inertia
-                ixx="0.012797"
-                ixy="-0.0002464"
-                ixz="0.0011164"
-                iyy="0.026307"
-                iyz="8.5164E-05"
-                izz="0.025616" />
-            </inertial>
-            <visual>
-            <origin
-                xyz="0 0 0"
-                rpy="0 0 0" />
-            <geometry>
-                <mesh
-                filename="package://dvrk_model/meshes/Si/PSM_ECM/link_2.STL" />
-            </geometry>
-            <material
-                name="">
-                <color
-                rgba="0.79216 0.81961 0.93333 1" />
-            </material>
-            </visual>
-            <collision>
-            <origin
-                xyz="0 0 0"
-                rpy="0 0 0" />
-            <geometry>
-                <mesh
-                filename="package://dvrk_model/meshes/Si/PSM_ECM/link_2.STL" />
-            </geometry>
-            </collision>
-        </link>
-        <joint
-            name="${prefix}j2"
-            type="revolute">
-            <origin
-            xyz="0.2987 0 -0.071222"
-            rpy="0 -1.1345 -3.1416" />
-            <parent
-            link="${prefix}link_1" />
-            <child
-            link="${prefix}link_2" />
-            <axis
-            xyz="0 -1 0" />
-            <limit
-            lower="-3.14"
-            upper="3.14"
-            effort="0"
-            velocity="0" />
-        </joint>
-        <link
-            name="${prefix}link_3">
-            <inertial>
-            <origin
-                xyz="0.11824 1.9336E-19 0.12932"
-                rpy="0 0 0" />
-            <mass
-                value="2.1982" />
-            <inertia
-                ixx="0.0076428"
-                ixy="-2.8207E-19"
-                ixz="-0.0074855"
-                iyy="0.032839"
-                iyz="-1.4256E-19"
-                izz="0.026585" />
-            </inertial>
-            <visual>
-            <origin
-                xyz="0 0 0"
-                rpy="0 0 0" />
-            <geometry>
-                <mesh
-                filename="package://dvrk_model/meshes/Si/PSM_ECM/link_3.STL" />
-            </geometry>
-            <material
-                name="">
-                <color
-                rgba="0.79216 0.81961 0.93333 1" />
-            </material>
-            </visual>
-            <collision>
-            <origin
-                xyz="0 0 0"
-                rpy="0 0 0" />
-            <geometry>
-                <mesh
-                filename="package://dvrk_model/meshes/Si/PSM_ECM/link_3.STL" />
-            </geometry>
-            </collision>
-        </link>
-        <joint
-            name="${prefix}j3"
-            type="revolute">
-            <origin
-            xyz="0.2032 0 0"
-            rpy="0 -0.90761 -3.1416" />
-            <parent
-            link="${prefix}link_2" />
-            <child
-            link="${prefix}link_3" />
-            <axis
-            xyz="0 1 0" />
-            <limit
-            lower="-3.14"
-            upper="3.14"
-            effort="0"
-            velocity="0" />
-        </joint>
-        <link
-            name="${prefix}link_4">
-            <inertial>
-            <origin
-                xyz="0.041219 -9.0734E-08 0.13651"
-                rpy="0 0 0" />
-            <mass
-                value="0.75206" />
-            <inertia
-                ixx="0.018546"
-                ixy="3.3933E-09"
-                ixz="0.00048607"
-                iyy="0.018573"
-                iyz="-1.7077E-08"
-                izz="0.00039277" />
-            </inertial>
-            <visual>
-            <origin
-                xyz="0 0 0"
-                rpy="0 0 0" />
-            <geometry>
-                <mesh
-                filename="package://dvrk_model/meshes/Si/PSM_ECM/link_4.STL" />
-            </geometry>
-            <material
-                name="">
-                <color
-                rgba="0.79216 0.81961 0.93333 1" />
-            </material>
-            </visual>
-            <collision>
-            <origin
-                xyz="0 0 0"
-                rpy="0 0 0" />
-            <geometry>
-                <mesh
-                filename="package://dvrk_model/meshes/Si/PSM_ECM/link_4.STL" />
-            </geometry>
-            </collision>
-        </link>
-        <joint
-            name="${prefix}j4"
-            type="revolute">
-            <origin
-            xyz="0.35966 0 0.16013"
-            rpy="0 -0.063963 0" />
-            <parent
-            link="${prefix}link_3" />
-            <child
-            link="${prefix}link_4" />
-            <axis
-            xyz="0 1 0" />
-            <limit
-            lower="-3.14"
-            upper="3.14"
-            effort="0"
-            velocity="0" />
-        </joint>
-        <link name="${prefix}tool_parent"/>
-        <joint
-            name="${prefix}outer_insertion_ref"
-            type="fixed">
-            <origin
-            xyz="0.05061 0 0.41911"
-            rpy="0 0 0" />
-            <parent
-            link="${prefix}link_4" />
-            <child
-            link="${prefix}tool_parent" />
-        </joint>
-        <link name="${prefix}RCM"/>
-        <joint
-            name="${prefix}jrcm"
-            type="fixed">
-            <origin
-            xyz="0.10643 0 -0.1731"
-            rpy="3.1416 0 -1.5708" />
-            <parent
-            link="${prefix}link_4" />
-            <child
-            link="${prefix}RCM" />
-            <axis
-            xyz="0 0 0" />
-        </joint>
-    </xacro:macro>
+  <xacro:macro name="psm_arm_active" params="prefix parent_link xyz rpy">
+    <link
+        name="${prefix}link_0">
+      <inertial>
+        <origin
+            xyz="-0.080771 2.1131E-08 1.8613E-07"
+            rpy="0 0 0" />
+        <mass
+            value="1.5188" />
+        <inertia
+            ixx="0.002395"
+            ixy="-2.6476E-18"
+            ixz="-1.3484E-18"
+            iyy="0.0040794"
+            iyz="4.2598E-10"
+            izz="0.0043778" />
+      </inertial>
+      <visual>
+        <origin
+            xyz="0 0 0"
+            rpy="0 0 0" />
+        <geometry>
+          <mesh
+              filename="package://dvrk_model/meshes/Si/PSM_ECM/link_0.STL" />
+        </geometry>
+        <material
+            name="">
+          <color
+              rgba="0.79216 0.81961 0.93333 1" />
+        </material>
+      </visual>
+      <collision>
+        <origin
+            xyz="0 0 0"
+            rpy="0 0 0" />
+        <geometry>
+          <mesh
+              filename="package://dvrk_model/meshes/Si/PSM_ECM/link_0.STL" />
+        </geometry>
+      </collision>
+    </link>
+    <joint name="${prefix}fixed" type="fixed">
+      <parent link="${parent_link}"/>
+      <child link="${prefix}link_0"/>
+      <origin rpy="${rpy}" xyz="${xyz}"/>
+    </joint>
+    <link
+        name="${prefix}link_1">
+      <inertial>
+        <origin
+            xyz="0.1461 0.090363 -0.024957"
+            rpy="0 0 0" />
+        <mass
+            value="1.7571" />
+        <inertia
+            ixx="0.0049404"
+            ixy="-0.0035267"
+            ixz="0.0045945"
+            iyy="0.019686"
+            iyz="0.00070407"
+            izz="0.020795" />
+      </inertial>
+      <visual>
+        <origin
+            xyz="0 0 0"
+            rpy="0 0 0" />
+        <geometry>
+          <mesh
+              filename="package://dvrk_model/meshes/Si/PSM_ECM/link_1.STL" />
+        </geometry>
+        <material
+            name="">
+          <color
+              rgba="0.79216 0.81961 0.93333 1" />
+        </material>
+      </visual>
+      <collision>
+        <origin
+            xyz="0 0 0"
+            rpy="0 0 0" />
+        <geometry>
+          <mesh
+              filename="package://dvrk_model/meshes/Si/PSM_ECM/link_1.STL" />
+        </geometry>
+      </collision>
+    </link>
+    <joint
+        name="yaw"
+        type="revolute">
+      <origin
+          xyz="0.158 0 0"
+          rpy="0 0 0" />
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