Commit message: Squash commits. Currently parent_link parameterization used for linking to the SUJ.

File: urdf/Si/ECM.urdf.xacro (robot description, xacro)
@@ -1,14 +1,14 @@
 <?xml version="1.0" ?>
 <robot name="ECM" xmlns:xacro="http://www.ros.org/wiki/xacro">
-    <xacro:property name="ECM_" value="ECM_"/>
+    <xacro:property name="ECM" value="ECM_"/>
     <xacro:property name="ECM_tool" value="SF826001"/>
+    <xacro:arg name="parent_link_" default="world"/>
+    <xacro:property name="parent_link" default="$(arg parent_link_)"/>
     <xacro:include filename="$(find dvrk_model)/urdf/Si/psm_base.urdf.xacro"/>
     <xacro:include filename="$(find dvrk_model)/urdf/Si/tools.urdf.xacro"/>
-    <link name="world"/>
+    <link name="${parent_link}"/>
     <xacro:psm_arm_active
-        prefix="${ECM_}"
-        parent_link="world"
-        xyz="0 0 0"
-        rpy="0 0 0"/>
-    <xacro:tool tool_name="SF826001" prefix="${ECM_}" parent_link="${ECM_}tool_parent"/>
+        prefix="${ECM}"
+        parent_link="${parent_link}"/>
+    <xacro:tool tool_name="SF826001" prefix="${ECM}" parent_link="${ECM}tool_parent"/>
 </robot>

File: urdf/Si/PSM1.urdf.xacro (robot description, xacro)
@@ -2,12 +2,13 @@
 <robot name="PSM1" xmlns:xacro="http://www.ros.org/wiki/xacro">
   <xacro:property name="tool_name" value="P420006"/>
+  <xacro:property name="PSM1" value="PSM1_"/>
+  <xacro:arg name="parent_link_" default="world"/>
+  <xacro:property name="parent_link" default="$(arg parent_link_)"/>
   <xacro:include filename="$(find dvrk_model)/urdf/Si/psm_base.urdf.xacro"/>
   <xacro:include filename="$(find dvrk_model)/urdf/Si/tools.urdf.xacro"/>
-  <link name="world"/>
+  <link name="${parent_link}"/>
   <xacro:psm_arm_active
-      prefix="PSM1_"
-      parent_link="world"
-      xyz="0 0 0"
-      rpy="0 0 0"/>
-  <xacro:tool tool_name="${tool_name}" prefix="PSM1_" parent_link="PSM1_tool_parent"/>
+      prefix="${PSM1}"
+      parent_link="${parent_link}"/>
+  <xacro:tool tool_name="${tool_name}" prefix="${PSM1}_" parent_link="${PSM1}tool_parent"/>
 </robot>

File: urdf/Si/PSM2.urdf.xacro (robot description, xacro)
@@ -2,12 +2,13 @@
 <robot name="PSM2" xmlns:xacro="http://www.ros.org/wiki/xacro">
   <xacro:property name="tool_name" value="P420006"/>
+  <xacro:property name="PSM2" value="PSM2_"/>
+  <xacro:arg name="parent_link_" default="world"/>
+  <xacro:property name="parent_link" default="$(arg parent_link_)"/>
   <xacro:include filename="$(find dvrk_model)/urdf/Si/psm_base.urdf.xacro"/>
   <xacro:include filename="$(find dvrk_model)/urdf/Si/tools.urdf.xacro"/>
-  <link name="world"/>
+  <link name="${parent_link}"/>
   <xacro:psm_arm_active
-      prefix="PSM2_"
-      parent_link="world"
-      xyz="0 0 0"
-      rpy="0 0 0"/>
-  <xacro:tool tool_name="${tool_name}" prefix="PSM2_" parent_link="PSM2_tool_parent"/>
+      prefix="${PSM2}"
+      parent_link="${parent_link}"/>
+  <xacro:tool tool_name="${tool_name}" prefix="${PSM2}" parent_link="${PSM2}tool_parent"/>
 </robot>

File: urdf/Si/PSM3.urdf.xacro (robot description, xacro)
@@ -2,12 +2,13 @@
 <robot name="PSM3" xmlns:xacro="http://www.ros.org/wiki/xacro">
   <xacro:property name="tool_name" value="P420006"/>
+  <xacro:property name="PSM3" value="PSM3_">
+  <xacro:arg name="parent_link_" default="world"/>
+  <xacro:property name="parent_link" default="$(arg parent_link_)"/>
   <xacro:include filename="$(find dvrk_model)/urdf/Si/psm_base.urdf.xacro"/>
   <xacro:include filename="$(find dvrk_model)/urdf/Si/tools.urdf.xacro"/>
-  <link name="world"/>
+  <link name="${parent_link}"/>
   <xacro:psm_arm_active
-      prefix="PSM3_"
-      parent_link="world"
-      xyz="0 0 0"
-      rpy="0 0 0"/>
-  <xacro:tool tool_name="${tool_name}" prefix="PSM3_" parent_link="PSM3_tool_parent"/>
+      prefix="${PSM3}"
+      parent_link="${parent_link}"/>
+  <xacro:tool tool_name="${tool_name}" prefix="${PSM3}" parent_link="${PSM3}tool_parent"/>
 </robot>

File: urdf/Si/SUJ.urdf.xacro (robot description, xacro)
@@ -22,5 +22,5 @@
         prefix="ECM_"
         parent_link="SUJ_column"
-        xyz="0.173 0 0.478"
+        xyz="0.223 0 0.528"
         rpy="0 0 0"/>
 </robot>

File: urdf/Si/psm.urdf.xacro (robot description, xacro)
@@ -3,10 +3,12 @@
   <xacro:property name="tool_name" default="P420006"/>
   <xacro:property name="arm" default="$(arg arm)"/>
+  <xacro:arg name="parent_link_" default="world"/>
+  <xacro:property name="parent_link" default="$(arg parent_link_)"/>
   <xacro:include filename="$(find dvrk_model)/urdf/Si/psm_base.urdf.xacro"/>
   <xacro:include filename="$(find dvrk_model)/urdf/Si/tools.urdf.xacro"/>
-  <link name="${arm}_base_link"/>
+  <link name="${parent_link}"/>
   <xacro:psm_arm_active
       prefix="${arm}_"
-      parent_link="${arm}_base_link"/>
-  <xacro:tool tool_name="${tool_name}" prefix="${arm}" parent_link="${arm}_tool_parent"/>
+      parent_link="${parent_link}"/>
+  <xacro:tool tool_name="${tool_name}" prefix="${arm}_" parent_link="${arm}_tool_parent"/>
 </robot>

File: urdf/Si/suj.urdf.xacro (robot description, xacro)
@@ -655,5 +655,5 @@
                 type="revolute">
                 <origin
-                xyz="0.025 0 0.63722"
+                xyz="-0.025 0.0 0.5232"
                 rpy="0 0 0" />
                 <parent
