Commit message: Si patient cart: fixed offsets, removed inertial

File: urdf/Si/SUJ.urdf.xacro (robot description, xacro)
@@ -1,26 +1,27 @@
 <?xml version="1.0" ?>
 <robot name="patient_cart" xmlns:xacro="http://www.ros.org/wiki/xacro">
-    <xacro:include filename="$(find dvrk_model)/urdf/Si/suj.urdf.xacro"/>
-    <xacro:include filename="$(find dvrk_model)/urdf/Si/suj_column.urdf.xacro"/>
-    <xacro:suj_column/>
-    <xacro:suj
-        prefix="PSM1_"
-        parent_link="SUJ_column"
-        xyz="0 0.228 0.528"
-        rpy="0 0 1.5708"/>
-    <xacro:suj
-        prefix="PSM2_"
-        parent_link="SUJ_column"
-        xyz="0 -0.228 0.528"
-        rpy="0 0 -1.5708" />
-    <xacro:suj
-        prefix="PSM3_"
-        parent_link="SUJ_column"
-        xyz="-0.223 0 0.528"
-        rpy="0 0 -3.1416"/>
-    <xacro:suj
-        prefix="ECM_"
-        parent_link="SUJ_column"
-        xyz="0.223 0 0.528"
-        rpy="0 0 0"/>
+  <xacro:include filename="$(find dvrk_model)/urdf/common.urdf.xacro"/>
+  <xacro:include filename="$(find dvrk_model)/urdf/Si/suj.urdf.xacro"/>
+  <xacro:include filename="$(find dvrk_model)/urdf/Si/suj_column.urdf.xacro"/>
+  <xacro:suj_column/>
+  <xacro:suj
+      prefix="PSM1_"
+      parent_link="SUJ_column"
+      xyz="0.0 0.228 0.528"
+      rpy="0.0 0.0 ${PI / 2.0}"/>
+  <xacro:suj
+      prefix="PSM2_"
+      parent_link="SUJ_column"
+      xyz="0.0 -0.228 0.528"
+      rpy="0.0 0.0 ${-PI / 2.0}" />
+  <xacro:suj
+      prefix="PSM3_"
+      parent_link="SUJ_column"
+      xyz="-0.223 0.0 0.528"
+      rpy="0.0 0.0 ${-PI}"/>
+  <xacro:suj
+      prefix="ECM_"
+      parent_link="SUJ_column"
+      xyz="0.223 0.0 0.528"
+      rpy="0.0 0.0 0.0"/>
 </robot>

File: urdf/Si/suj.urdf.xacro (robot description, xacro)
@@ -5,22 +5,8 @@
             <link
                 name="SUJ_${prefix}link_0">
-                <inertial>
-                <origin
-                    xyz="-0.042353 -4.4531E-08 0.24208"
-                    rpy="0 0 0" />
-                <mass
-                    value="12.704" />
-                <inertia
-                    ixx="0.368"
-                    ixy="-6.2028E-09"
-                    ixz="-0.021772"
-                    iyy="0.3714"
-                    iyz="5.3603E-09"
-                    izz="0.047463" />
-                </inertial>
-                <visual>
-                <origin
-                    xyz="0 0 0"
-                    rpy="0 0 0" />
+                <visual>
+                <origin
+                    xyz="0.0 0.0 0.0"
+                    rpy="0.0 0.0 0.0" />
                 <geometry>
                     <mesh
@@ -30,11 +16,11 @@
                     name="">
                     <color
-                    rgba="0.79216 0.81961 0.93333 1" />
-                </material>
-                </visual>
-                <collision>
-                <origin
-                    xyz="0 0 0"
-                    rpy="0 0 0" />
+                    rgba="0.79216 0.81961 0.93333 1.0" />
+                </material>
+                </visual>
+                <collision>
+                <origin
+                    xyz="0.0 0.0 0.0"
+                    rpy="0.0 0.0 0.0" />
                 <geometry>
                     <mesh
@@ -54,31 +40,17 @@
                 link="SUJ_${prefix}link_0" />
                 <axis
-                xyz="0 0 1" />
+                xyz="0.0 0.0 1.0" />
                 <limit
                 lower="0.0"
                 upper="0.512"
-                effort="0"
-                velocity="0" />
+                effort="0.0"
+                velocity="0.0" />
             </joint>
             <link
                 name="SUJ_${prefix}link_1">
-                <inertial>
-                <origin
-                    xyz="0.21712 2.5962E-08 0.072796"
-                    rpy="0 0 0" />
-                <mass
-                    value="7.0906" />
-                <inertia
-                    ixx="0.015346"
-                    ixy="-1.6493E-08"
-                    ixz="-0.0010396"
-                    iyy="0.22426"
-                    iyz="8.2106E-09"
-                    izz="0.2218" />
-                </inertial>
-                <visual>
-                <origin
-                    xyz="0 0 0"
-                    rpy="0 0 0" />
+                <visual>
+                <origin
+                    xyz="0.0 0.0 0.0"
+                    rpy="0.0 0.0 0.0" />
                 <geometry>
                     <mesh
@@ -88,11 +60,11 @@
                     name="">
                     <color
-                    rgba="0.79216 0.81961 0.93333 1" />
-                </material>
-                </visual>
-                <collision>
-                <origin
-                    xyz="0 0 0"
-                    rpy="0 0 0" />
+                    rgba="0.79216 0.81961 0.93333 1.0" />
+                </material>
+                </visual>
+                <collision>
+                <origin
+                    xyz="0.0 0.0 0.0"
+                    rpy="0.0 0.0 0.0" />
                 <geometry>
                     <mesh
@@ -105,6 +77,6 @@
                 type="revolute">
                 <origin
-                xyz="-0.024998 0 0.59"
-                rpy="0 0 0" />
+                xyz="-0.024998 0.0 0.59"
+                rpy="0.0 0.0 0.0" />
                 <parent
                 link="SUJ_${prefix}link_0" />
@@ -112,31 +84,17 @@
                 link="SUJ_${prefix}link_1" />
                 <axis
-                xyz="0 0 1" />
+                xyz="0.0 0.0 1.0" />
                 <limit
                 lower="-3.141"
                 upper="3.141"
-                effort="0"
-                velocity="0" />
+                effort="0.0"
+                velocity="0.0" />
             </joint>
             <link
                 name="SUJ_${prefix}link_2">
-                <inertial>
-                <origin
-                    xyz="0.22659 -1.07E-07 0.065498"
-                    rpy="0 0 0" />
-                <mass
-                    value="5.8282" />
-                <inertia
-                    ixx="0.011467"
-                    ixy="-2.0133E-09"
-                    ixz="0.0026277"
-                    iyy="0.19305"
-                    iyz="2.1385E-09"
-                    izz="0.19056" />
-                </inertial>
-                <visual>
-                <origin
-                    xyz="0 0 0"
-                    rpy="0 0 0" />
+                <visual>
+                <origin
+                    xyz="0.0 0.0 0.0"
+                    rpy="0.0 0.0 0.0" />
                 <geometry>
                     <mesh
@@ -146,11 +104,11 @@
                     name="">
                     <color
-                    rgba="0.79216 0.81961 0.93333 1" />
-                </material>
-                </visual>
-                <collision>
-                <origin
-                    xyz="0 0 0"
-                    rpy="0 0 0" />
+                    rgba="0.79216 0.81961 0.93333 1.0" />
+                </material>
+                </visual>
+                <collision>
+                <origin
+                    xyz="0.0 0.0 0.0"
+                    rpy="0.0 0.0 0.0" />
                 <geometry>
                     <mesh
@@ -163,6 +121,6 @@
                 type="revolute">
                 <origin
-                xyz="0.4575 0 0.144"
-                rpy="0 0 0" />
+                xyz="0.4575 0.0 0.144"
+                rpy="0.0 0.0 0.0" />
                 <parent
                 link="SUJ_${prefix}link_1" />
@@ -170,31 +128,17 @@
                 link="SUJ_${prefix}link_2" />
                 <axis
-                xyz="0 0 1" />
+                xyz="0.0 0.0 1.0" />
                 <limit
                 lower="-3.141"
                 upper="3.141"
-                effort="0"
-                velocity="0" />
+                effort="0.0"
+                velocity="0.0" />
             </joint>
             <link
                 name="SUJ_${prefix}link_3">
-                <inertial>
-                <origin
-                    xyz="0.014738 8.0422E-08 -0.027873"
-                    rpy="0 0 0" />
-                <mass
-                    value="0.5504" />
-                <inertia
-                    ixx="0.00064459"
-                    ixy="2.3418E-09"
-                    ixz="1.1203E-05"
-                    iyy="0.00057105"
-                    iyz="-2.8921E-09"
-                    izz="0.00085397" />
-                </inertial>
-                <visual>
-                <origin
-                    xyz="0 0 0"
-                    rpy="0 0 0" />
+                <visual>
+                <origin
+                    xyz="0.0 0.0 0.0"
+                    rpy="0.0 0.0 0.0" />
                 <geometry>
                     <mesh
@@ -204,11 +148,11 @@
                     name="">
                     <color
-                    rgba="0.79216 0.81961 0.93333 1" />
-                </material>
-                </visual>
-                <collision>
-                <origin
-                    xyz="0 0 0"
-                    rpy="0 0 0" />
+                    rgba="0.79216 0.81961 0.93333 1.0" />
+                </material>
+                </visual>
+                <collision>
+                <origin
+                    xyz="0.0 0.0 0.0"
+                    rpy="0.0 0.0 0.0" />
                 <geometry>
                     <mesh
@@ -221,6 +165,6 @@
                 type="revolute">
                 <origin
-                xyz="0.458 0 -0.01875"
-                rpy="0 0 0" />
+                xyz="0.458 0.0 -0.01875"
+                rpy="0.0 0.0 0.0" />
                 <parent
                 link="SUJ_${prefix}link_2" />
@@ -232,6 +176,6 @@
                 lower="-3.141"
                 upper="3.141"
-                effort="0"
-                velocity="0" />
+                effort="0.0"
+                velocity="0.0" />
             </joint>
             <link name="${prefix}mounting_point"/>
@@ -240,6 +184,6 @@
                 type="fixed">
                 <origin
-                xyz="0.045255 0 -0.045255"
-                rpy="0 0.7854 0" />
+                xyz="0.045255 0.0 -0.045255"
+                rpy="0.0 0.7854 0.0" />
                 <parent
                 link="SUJ_${prefix}link_3" />
@@ -251,22 +195,8 @@
              <link
                 name="SUJ_${prefix}link_0">
-                <inertial>
-                <origin
-                    xyz="-0.043484 -9.4105E-09 0.22013"
-                    rpy="0 0 0" />
-                <mass
-                    value="11.927" />
-                <inertia
-                    ixx="0.27621"
-                    ixy="-5.0682E-09"
-                    ixz="-0.016932"
-                    iyy="0.27936"
-                    iyz="3.4609E-09"
-                    izz="0.046091" />
-                </inertial>
-                <visual>
-                <origin
-                    xyz="0 0 0"
-                    rpy="0 0 0" />
+                <visual>
+                <origin
+                    xyz="0.0 0.0 0.0"
+                    rpy="0.0 0.0 0.0" />
                 <geometry>
                     <mesh
@@ -276,11 +206,11 @@
                     name="">
                     <color
-                    rgba="0.79216 0.81961 0.93333 1" />
-                </material>
-                </visual>
-                <collision>
-                <origin
-                    xyz="0 0 0"
-                    rpy="0 0 0" />
+                    rgba="0.79216 0.81961 0.93333 1.0" />
+                </material>
+                </visual>
+                <collision>
+                <origin
+                    xyz="0.0 0.0 0.0"
+                    rpy="0.0 0.0 0.0" />
                 <geometry>
                     <mesh
@@ -300,31 +230,17 @@
                 link="SUJ_${prefix}link_0" />
                 <axis
-                xyz="0 0 1" />
+                xyz="0.0 0.0 1.0" />
                 <limit
                 lower="0.0"
                 upper="0.512"
-                effort="0"
-                velocity="0" />
+                effort="0.0"
+                velocity="0.0" />
             </joint>
             <link
                 name="SUJ_${prefix}link_1">
-                <inertial>
-                <origin
-                    xyz="0.20518 1.3159E-05 0.040755"
-                    rpy="0 0 0" />
-                <mass
-                    value="7.8622" />
-                <inertia
-                    ixx="0.043421"
-                    ixy="8.2624E-06"
-                    ixz="0.030604"
-                    iyy="0.20282"
-                    iyz="-6.5783E-05"
-                    izz="0.17543" />
-                </inertial>
-                <visual>
-                <origin
-                    xyz="0 0 0"
-                    rpy="0 0 0" />
+                <visual>
+                <origin
+                    xyz="0.0 0.0 0.0"
+                    rpy="0.0 0.0 0.0" />
                 <geometry>
                     <mesh
@@ -334,11 +250,11 @@
                     name="">
                     <color
-                    rgba="0.79216 0.81961 0.93333 1" />
-                </material>
-                </visual>
-                <collision>
-                <origin
-                    xyz="0 0 0"
-                    rpy="0 0 0" />
+                    rgba="0.79216 0.81961 0.93333 1.0" />
+                </material>
+                </visual>
+                <collision>
+                <origin
+                    xyz="0.0 0.0 0.0"
+                    rpy="0.0 0.0 0.0" />
                 <geometry>
                     <mesh
@@ -351,6 +267,6 @@
                 type="revolute">
                 <origin
-                xyz="-0.024998 0 0.513"
-                rpy="0 0 -0.23716" />
+                xyz="-0.024998 0.0 0.513"
+                rpy="0.0 0.0 0.0" />
                 <parent
                 link="SUJ_${prefix}link_0" />
@@ -358,31 +274,17 @@
                 link="SUJ_${prefix}link_1" />
                 <axis
-                xyz="0 0 1" />
+                xyz="0.0 0.0 1.0" />
                 <limit
                 lower="-3.14"
                 upper="3.14"
-                effort="0"
-                velocity="0" />
+                effort="0.0"
+                velocity="0.0" />
             </joint>
             <link
                 name="SUJ_${prefix}link_2">
-                <inertial>
-                <origin
-                    xyz="0.22894 -6.2716E-08 -9.2061E-05"
-                    rpy="0 0 0" />
-                <mass
-                    value="6.7952" />
-                <inertia
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