Commit message: Si: rename shared meshes to USM/USM_*

File: urdf/Si/PSM_base.urdf.xacro (robot description, xacro)
@@ -27,5 +27,5 @@
         <origin xyz="0 0 0" rpy="0 0 0"/>
         <geometry>
-          <mesh filename="package://dvrk_model/meshes/Si/PSM_ECM/PSM_ECM_base.stl"/>
+          <mesh filename="package://dvrk_model/meshes/Si/USM/USM_base.stl"/>
         </geometry>
         <material name=""><color rgba="0.79216 0.81961 0.93333 1"/></material>
@@ -34,5 +34,5 @@
         <origin xyz="0 0 0" rpy="0 0 0"/>
         <geometry>
-          <mesh filename="package://dvrk_model/meshes/Si/PSM_ECM/PSM_ECM_base.stl"/>
+          <mesh filename="package://dvrk_model/meshes/Si/USM/USM_base.stl"/>
         </geometry>
       </collision>
@@ -56,5 +56,5 @@
         <origin xyz="0 0 0" rpy="0 0 0"/>
         <geometry>
-          <mesh filename="package://dvrk_model/meshes/Si/PSM_ECM/PSM_ECM_yaw.stl"/>
+          <mesh filename="package://dvrk_model/meshes/Si/USM/USM_yaw.stl"/>
         </geometry>
         <material name=""><color rgba="0.79216 0.81961 0.93333 1"/></material>
@@ -63,5 +63,5 @@
         <origin xyz="0 0 0" rpy="0 0 0"/>
         <geometry>
-          <mesh filename="package://dvrk_model/meshes/Si/PSM_ECM/PSM_ECM_yaw.stl"/>
+          <mesh filename="package://dvrk_model/meshes/Si/USM/USM_yaw.stl"/>
         </geometry>
       </collision>
@@ -87,5 +87,5 @@
         <origin xyz="0 0 0" rpy="0 0 0"/>
         <geometry>
-          <mesh filename="package://dvrk_model/meshes/Si/PSM_ECM/PSM_ECM_pitch.stl"/>
+          <mesh filename="package://dvrk_model/meshes/Si/USM/USM_pitch.stl"/>
         </geometry>
         <material name=""><color rgba="0.79216 0.81961 0.93333 1"/></material>
@@ -94,5 +94,5 @@
         <origin xyz="0 0 0" rpy="0 0 0"/>
         <geometry>
-          <mesh filename="package://dvrk_model/meshes/Si/PSM_ECM/PSM_ECM_pitch.stl"/>
+          <mesh filename="package://dvrk_model/meshes/Si/USM/USM_pitch.stl"/>
         </geometry>
       </collision>
@@ -118,5 +118,5 @@
         <origin xyz="0 0 0" rpy="0 0 0"/>
         <geometry>
-          <mesh filename="package://dvrk_model/meshes/Si/PSM_ECM/PSM_ECM_pitch_bottom.stl"/>
+          <mesh filename="package://dvrk_model/meshes/Si/USM/USM_pitch_bottom.stl"/>
         </geometry>
         <material name=""><color rgba="0.79216 0.81961 0.93333 1"/></material>
@@ -125,5 +125,5 @@
         <origin xyz="0 0 0" rpy="0 0 0"/>
         <geometry>
-          <mesh filename="package://dvrk_model/meshes/Si/PSM_ECM/PSM_ECM_pitch_bottom.stl"/>
+          <mesh filename="package://dvrk_model/meshes/Si/USM/USM_pitch_bottom.stl"/>
         </geometry>
       </collision>
@@ -149,5 +149,5 @@
         <origin xyz="0 0 0" rpy="0 0 0"/>
         <geometry>
-          <mesh filename="package://dvrk_model/meshes/Si/PSM_ECM/PSM_ECM_pitch_top.stl"/>
+          <mesh filename="package://dvrk_model/meshes/Si/USM/USM_pitch_top.stl"/>
         </geometry>
         <material name=""><color rgba="0.79216 0.81961 0.93333 1"/></material>
@@ -156,5 +156,5 @@
         <origin xyz="0 0 0" rpy="0 0 0"/>
         <geometry>
-          <mesh filename="package://dvrk_model/meshes/Si/PSM_ECM/PSM_ECM_pitch_top.stl"/>
+          <mesh filename="package://dvrk_model/meshes/Si/USM/USM_pitch_top.stl"/>
         </geometry>
       </collision>

Commit message: Si remove all outer

File: urdf/Si/PSM_base.urdf.xacro (robot description, xacro)
@@ -4,6 +4,6 @@
   <!--
     Si PSM arm — 3 actuated DOF:
-      Joint 1: yaw    (revolute, outer yaw)
-      Joint 2: pitch  (revolute, outer pitch, parallelogram linkage ×3)
+      Joint 1: yaw    (revolute, yaw)
+      Joint 2: pitch  (revolute, pitch, parallelogram linkage ×3)
       Joint 3: insertion (prismatic)
     Macro output: ends at ${prefix}PSM_tool_parent_link.
@@ -67,5 +67,5 @@
       </collision>
     </link>
-    <!-- joint 1: yaw (outer yaw) -->
+    <!-- joint 1: yaw -->
     <joint name="yaw" type="revolute">
       <origin xyz="0.158 0 0" rpy="0.0 0.0 0.0"/>
@@ -73,7 +73,7 @@
       <child  link="${prefix}PSM_ECM_yaw_link"/>
       <axis xyz="-1.0 0.0 0.0"/>
-      <limit lower="-3.14" upper="3.14" effort="0.0" velocity="0.0"/> <!--flagged placeholder and limits of ±π-->
+      <limit lower="-3.14" upper="3.14" effort="0.0" velocity="0.0"/>
     </joint>
-    <!-- link 2: outer pitch arm -->
+    <!-- link 2: pitch arm -->
     <link name="${prefix}PSM_ECM_pitch_link">
       <inertial>
@@ -98,5 +98,5 @@
       </collision>
     </link>
-    <!-- joint 2: pitch (outer pitch) -->
+    <!-- joint 2: pitch -->
     <joint name="pitch" type="revolute">
       <origin xyz="0.2987 0 -0.071222" rpy="0 -1.1345 -3.1416"/>
@@ -104,5 +104,5 @@
       <child  link="${prefix}PSM_ECM_pitch_link"/>
       <axis xyz="0 -1 0"/>
-      <limit lower="-3.14" upper="3.14" effort="0" velocity="0"/> <!--flagged placeholder and limits of ±π-->
+      <limit lower="-3.14" upper="3.14" effort="0" velocity="0"/>
     </joint>
     <!-- link 3: pitch parallelogram arm (mimic pitch) -->
@@ -134,5 +134,5 @@
       <child  link="${prefix}PSM_ECM_pitch_bottom_link"/>
       <axis xyz="0 1 0"/>
-      <limit lower="-3.14" upper="3.14" effort="0" velocity="0"/> <!--flagged placeholder and limits of ±π-->
+      <limit lower="-3.14" upper="3.14" effort="0" velocity="0"/>
       <mimic joint="pitch" multiplier="-1"/>
     </joint>
@@ -165,5 +165,5 @@
       <child  link="${prefix}PSM_ECM_pitch_top_link"/>
       <axis xyz="0 1 0"/>
-      <limit lower="-3.14" upper="3.14" effort="0" velocity="0"/> <!--flagged placeholder and limits of ±π-->
+      <limit lower="-3.14" upper="3.14" effort="0" velocity="0"/>
       <mimic joint="pitch" multiplier="1"/>
     </joint>

Commit message: update mesh file names for USM, change PSM_ECM to USM

File: urdf/Si/PSM_base.urdf.xacro (robot description, xacro)
@@ -16,5 +16,5 @@
                        rpy:='0.0 0.0 0.0'">
     <!-- link 0: arm base -->
-    <link name="${prefix}PSM_ECM_base_link">
+    <link name="${prefix}USM_base_link">
       <inertial>
         <origin xyz="-0.080771 2.1131E-08 1.8613E-07" rpy="0 0 0"/>
@@ -41,9 +41,9 @@
     <joint name="${prefix}base_fixed" type="fixed">
       <parent link="${parent_link}"/>
-      <child  link="${prefix}PSM_ECM_base_link"/>
+      <child  link="${prefix}USM_base_link"/>
       <origin rpy="${rpy}" xyz="${xyz}"/>
     </joint>
     <!-- link 1: yaw body -->
-    <link name="${prefix}PSM_ECM_yaw_link">
+    <link name="${prefix}USM_yaw_link">
       <inertial>
         <origin xyz="0.1461 0.090363 -0.024957" rpy="0 0 0"/>
@@ -70,11 +70,11 @@
     <joint name="yaw" type="revolute">
       <origin xyz="0.158 0 0" rpy="0.0 0.0 0.0"/>
-      <parent link="${prefix}PSM_ECM_base_link"/>
-      <child  link="${prefix}PSM_ECM_yaw_link"/>
+      <parent link="${prefix}USM_base_link"/>
+      <child  link="${prefix}USM_yaw_link"/>
       <axis xyz="-1.0 0.0 0.0"/>
       <limit lower="-3.14" upper="3.14" effort="0.0" velocity="0.0"/>
     </joint>
     <!-- link 2: pitch arm -->
-    <link name="${prefix}PSM_ECM_pitch_link">
+    <link name="${prefix}USM_pitch_link">
       <inertial>
         <origin xyz="0.083895 -0.00073113 -0.028998" rpy="0.0 0.0 0.0"/>
@@ -101,11 +101,11 @@
     <joint name="pitch" type="revolute">
       <origin xyz="0.2987 0 -0.071222" rpy="0 -1.1345 -3.1416"/>
-      <parent link="${prefix}PSM_ECM_yaw_link"/>
-      <child  link="${prefix}PSM_ECM_pitch_link"/>
+      <parent link="${prefix}USM_yaw_link"/>
+      <child  link="${prefix}USM_pitch_link"/>
       <axis xyz="0 -1 0"/>
       <limit lower="-3.14" upper="3.14" effort="0" velocity="0"/>
     </joint>
     <!-- link 3: pitch parallelogram arm (mimic pitch) -->
-    <link name="${prefix}PSM_ECM_pitch_bottom_link">
+    <link name="${prefix}USM_pitch_3_link">
       <inertial>
         <origin xyz="0.11824 1.9336E-19 0.12932" rpy="0 0 0"/>
@@ -118,5 +118,5 @@
         <origin xyz="0 0 0" rpy="0 0 0"/>
         <geometry>
-          <mesh filename="package://dvrk_model/meshes/Si/USM/USM_pitch_bottom.stl"/>
+          <mesh filename="package://dvrk_model/meshes/Si/USM/USM_pitch_3.stl"/>
         </geometry>
         <material name=""><color rgba="0.79216 0.81961 0.93333 1"/></material>
@@ -125,5 +125,5 @@
         <origin xyz="0 0 0" rpy="0 0 0"/>
         <geometry>
-          <mesh filename="package://dvrk_model/meshes/Si/USM/USM_pitch_bottom.stl"/>
+          <mesh filename="package://dvrk_model/meshes/Si/USM/USM_pitch_3.stl"/>
         </geometry>
       </collision>
@@ -131,6 +131,6 @@
     <joint name="pitch_2" type="revolute">
       <origin xyz="0.2032 0 0" rpy="0 -0.90761 -3.1416"/>
-      <parent link="${prefix}PSM_ECM_pitch_link"/>
-      <child  link="${prefix}PSM_ECM_pitch_bottom_link"/>
+      <parent link="${prefix}USM_pitch_link"/>
+      <child  link="${prefix}USM_pitch_3_link"/>
       <axis xyz="0 1 0"/>
       <limit lower="-3.14" upper="3.14" effort="0" velocity="0"/>
@@ -138,5 +138,5 @@
     </joint>
     <!-- link 4: pitch parallelogram distal (mimic pitch) -->
-    <link name="${prefix}PSM_ECM_pitch_top_link">
+    <link name="${prefix}USM_pitch_4_link">
       <inertial>
         <origin xyz="0.041219 -9.0734E-08 0.13651" rpy="0 0 0"/>
@@ -149,5 +149,5 @@
         <origin xyz="0 0 0" rpy="0 0 0"/>
         <geometry>
-          <mesh filename="package://dvrk_model/meshes/Si/USM/USM_pitch_top.stl"/>
+          <mesh filename="package://dvrk_model/meshes/Si/USM/USM_pitch_4.stl"/>
         </geometry>
         <material name=""><color rgba="0.79216 0.81961 0.93333 1"/></material>
@@ -156,5 +156,5 @@
         <origin xyz="0 0 0" rpy="0 0 0"/>
         <geometry>
-          <mesh filename="package://dvrk_model/meshes/Si/USM/USM_pitch_top.stl"/>
+          <mesh filename="package://dvrk_model/meshes/Si/USM/USM_pitch_4.stl"/>
         </geometry>
       </collision>
@@ -162,6 +162,6 @@
     <joint name="pitch_3" type="revolute">
       <origin xyz="0.35966 0 0.16013" rpy="0 -0.063963 0"/>
-      <parent link="${prefix}PSM_ECM_pitch_bottom_link"/>
-      <child  link="${prefix}PSM_ECM_pitch_top_link"/>
+      <parent link="${prefix}USM_pitch_3_link"/>
+      <child  link="${prefix}USM_pitch_4_link"/>
       <axis xyz="0 1 0"/>
       <limit lower="-3.14" upper="3.14" effort="0" velocity="0"/>
@@ -175,5 +175,5 @@
     <joint name="insertion" type="prismatic">
       <origin xyz="0.05061 0 0.41911" rpy="${PI} 0 0"/>
-      <parent link="${prefix}PSM_ECM_pitch_top_link"/>
+      <parent link="${prefix}USM_pitch_4_link"/>
       <child  link="${prefix}PSM_tool_parent_link"/>
       <axis xyz="0 0 1"/>
@@ -190,5 +190,5 @@
     <joint name="${prefix}jrcm" type="fixed">
       <origin xyz="0.10643 0 -0.1731" rpy="3.1416 0 -1.5708"/>
-      <parent link="${prefix}PSM_ECM_pitch_top_link"/>
+      <parent link="${prefix}USM_pitch_4_link"/>
       <child  link="${prefix}PSM_RCM_link"/>
       <axis xyz="0 0 0"/>
