Commit message: Updated metallic Si arms

File: urdf/Si/ECM_base.urdf.xacro (robot description, xacro)
@@ -40,5 +40,5 @@
           <mesh filename="package://dvrk_model/meshes/arms/Si/USM/USM_base.stl"/>
         </geometry>
-        <material name=""><color rgba="0.79216 0.81961 0.93333 1"/></material>
+        <material name=""><color rgba="0.80000 0.80000 0.80000 1"/></material>
       </visual>
       <collision>
@@ -69,5 +69,5 @@
           <mesh filename="package://dvrk_model/meshes/arms/Si/USM/USM_yaw.stl"/>
         </geometry>
-        <material name=""><color rgba="0.79216 0.81961 0.93333 1"/></material>
+        <material name=""><color rgba="0.80000 0.80000 0.80000 1"/></material>
       </visual>
       <collision>
@@ -100,5 +100,5 @@
           <mesh filename="package://dvrk_model/meshes/arms/Si/USM/USM_pitch.stl"/>
         </geometry>
-        <material name=""><color rgba="0.79216 0.81961 0.93333 1"/></material>
+        <material name=""><color rgba="0.80000 0.80000 0.80000 1"/></material>
       </visual>
       <collision>
@@ -131,5 +131,5 @@
           <mesh filename="package://dvrk_model/meshes/arms/Si/USM/USM_pitch_3.stl"/>
         </geometry>
-        <material name=""><color rgba="0.79216 0.81961 0.93333 1"/></material>
+        <material name=""><color rgba="0.80000 0.80000 0.80000 1"/></material>
       </visual>
       <collision>
@@ -162,5 +162,5 @@
           <mesh filename="package://dvrk_model/meshes/arms/Si/USM/USM_pitch_4.stl"/>
         </geometry>
-        <material name=""><color rgba="0.79216 0.81961 0.93333 1"/></material>
+        <material name=""><color rgba="0.80000 0.80000 0.80000 1"/></material>
       </visual>
       <collision>

File: urdf/Si/PSM_base.urdf.xacro (robot description, xacro)
@@ -39,5 +39,5 @@
           <mesh filename="package://dvrk_model/meshes/arms/Si/USM/USM_base.stl"/>
         </geometry>
-        <material name=""><color rgba="0.79216 0.81961 0.93333 1"/></material>
+        <material name=""><color rgba="0.80000 0.80000 0.80000 1"/></material>
       </visual>
       <collision>
@@ -68,5 +68,5 @@
           <mesh filename="package://dvrk_model/meshes/arms/Si/USM/USM_yaw.stl"/>
         </geometry>
-        <material name=""><color rgba="0.79216 0.81961 0.93333 1"/></material>
+        <material name=""><color rgba="0.80000 0.80000 0.80000 1"/></material>
       </visual>
       <collision>
@@ -99,5 +99,5 @@
           <mesh filename="package://dvrk_model/meshes/arms/Si/USM/USM_pitch.stl"/>
         </geometry>
-        <material name=""><color rgba="0.79216 0.81961 0.93333 1"/></material>
+        <material name=""><color rgba="0.80000 0.80000 0.80000 1"/></material>
       </visual>
       <collision>
@@ -130,5 +130,5 @@
           <mesh filename="package://dvrk_model/meshes/arms/Si/USM/USM_pitch_3.stl"/>
         </geometry>
-        <material name=""><color rgba="0.79216 0.81961 0.93333 1"/></material>
+        <material name=""><color rgba="0.80000 0.80000 0.80000 1"/></material>
       </visual>
       <collision>
@@ -161,5 +161,5 @@
           <mesh filename="package://dvrk_model/meshes/arms/Si/USM/USM_pitch_4.stl"/>
         </geometry>
-        <material name=""><color rgba="0.79216 0.81961 0.93333 1"/></material>
+        <material name=""><color rgba="0.80000 0.80000 0.80000 1"/></material>
       </visual>
       <collision>

File: urdf/Si/SUJ_base.urdf.xacro (robot description, xacro)
@@ -16,5 +16,5 @@
                     name="">
                     <color
-                    rgba="0.79216 0.81961 0.93333 1.0" />
+                    rgba="0.80000 0.80000 0.80000 1.0" />
                 </material>
                 </visual>
@@ -60,5 +60,5 @@
                     name="">
                     <color
-                    rgba="0.79216 0.81961 0.93333 1.0" />
+                    rgba="0.80000 0.80000 0.80000 1.0" />
                 </material>
                 </visual>
@@ -104,5 +104,5 @@
                     name="">
                     <color
-                    rgba="0.79216 0.81961 0.93333 1.0" />
+                    rgba="0.80000 0.80000 0.80000 1.0" />
                 </material>
                 </visual>
@@ -148,5 +148,5 @@
                     name="">
                     <color
-                    rgba="0.79216 0.81961 0.93333 1.0" />
+                    rgba="0.80000 0.80000 0.80000 1.0" />
                 </material>
                 </visual>
@@ -218,5 +218,5 @@
                     name="">
                     <color
-                    rgba="0.79216 0.81961 0.93333 1.0" />
+                    rgba="0.80000 0.80000 0.80000 1.0" />
                 </material>
                 </visual>
@@ -262,5 +262,5 @@
                     name="">
                     <color
-                    rgba="0.79216 0.81961 0.93333 1.0" />
+                    rgba="0.80000 0.80000 0.80000 1.0" />
                 </material>
                 </visual>
@@ -306,5 +306,5 @@
                     name="">
                     <color
-                    rgba="0.79216 0.81961 0.93333 1.0" />
+                    rgba="0.80000 0.80000 0.80000 1.0" />
                 </material>
                 </visual>
@@ -350,5 +350,5 @@
                     name="">
                     <color
-                    rgba="0.79216 0.81961 0.93333 1.0" />
+                    rgba="0.80000 0.80000 0.80000 1.0" />
                 </material>
                 </visual>
@@ -394,5 +394,5 @@
                     name="">
                     <color
-                    rgba="0.79216 0.81961 0.93333 1.0" />
+                    rgba="0.80000 0.80000 0.80000 1.0" />
                 </material>
                 </visual>
@@ -464,5 +464,5 @@
                     name="">
                     <color
-                    rgba="0.79216 0.81961 0.93333 1.0" />
+                    rgba="0.80000 0.80000 0.80000 1.0" />
                 </material>
                 </visual>
@@ -508,5 +508,5 @@
                     name="">
                     <color
-                    rgba="0.79216 0.81961 0.93333 1.0" />
+                    rgba="0.80000 0.80000 0.80000 1.0" />
                 </material>
                 </visual>
@@ -552,5 +552,5 @@
                     name="">
                     <color
-                    rgba="0.79216 0.81961 0.93333 1.0" />
+                    rgba="0.80000 0.80000 0.80000 1.0" />
                 </material>
                 </visual>
@@ -596,5 +596,5 @@
                     name="">
                     <color
-                    rgba="0.79216 0.81961 0.93333 1.0" />
+                    rgba="0.80000 0.80000 0.80000 1.0" />
                 </material>
                 </visual>

File: urdf/Si/SUJ_cart.urdf.xacro (robot description, xacro)
@@ -35,5 +35,5 @@
                 name="">
                 <color
-                rgba="0.79216 0.81961 0.93333 1" />
+                rgba="0.80000 0.80000 0.80000 1" />
             </material>
             </visual>
