Commit message: Trying to use multiple joint and state publishers to match C++ component.  PSMs should them be attached at end of SUJs.  tf2 static broadcast almost works but there is likely a race condition so this is not a solution.

File: urdf/Classic/ecm.urdf.xacro (robot description, xacro)
@@ -6,36 +6,8 @@
   <xacro:macro name="ecm" params="prefix parent_link xyz rpy">
     <!-- Joint 0: Fixed to World-->
-    <joint name="setup_fixed_joint" type="fixed">
+    <joint name="fixed" type="fixed">
       <parent link="${parent_link}"/>
-      <child link="${prefix}_setup_base_link"/>
+      <child link="${prefix}_base_link"/>
       <origin rpy="${rpy}" xyz="${xyz}"/>
-    </joint>
-    <link name="${prefix}_setup_base_link"/>
-    <joint name="setup_tip_joint" type="fixed">
-      <parent link="${prefix}_setup_base_link"/>
-      <child link="${prefix}_setup_link"/>
-      <origin rpy="-0.87046370379 0 -${PI/2}" xyz="0.91324 -0.02111 0.03166"/>
-      <axis xyz="0 0 1"/>
-    </joint>
-    <link name="${prefix}_setup_link">
-      <visual>
-        <origin rpy="0 0 0" xyz="0 0 0"/>
-        <geometry>
-          <mesh filename="package://dvrk_model/meshes/Classic/ecm/Endo_Arm.STL"/>
-        </geometry>
-	<material name="DaVinciRed"/>
-      </visual>
-      <collision>
-        <origin rpy="0 0 0" xyz="0 0 0"/>
-        <geometry>
-          <mesh filename="package://dvrk_model/meshes/Classic/ecm/Endo_Arm.STL"/>
-        </geometry>
-      </collision>
-    </link>
-    <!-- Joint 0: Fixed to Setup Joint-->
-    <joint name="fixed_joint" type="fixed">
-      <parent link="${prefix}_setup_link"/>
-      <child link="${prefix}_base_link"/>
-      <origin rpy="0 0 0" xyz="0 0.603 0"/>
     </joint>
     <link name="${prefix}_base_link"/>

File: urdf/Si/PSM1.urdf.xacro (robot description, xacro)
@@ -1,14 +1,13 @@
 <?xml version="1.0" ?>
 <robot name="PSM1" xmlns:xacro="http://www.ros.org/wiki/xacro">
-    <xacro:property name="PSM1_" value="PSM1_"/>
-    <xacro:property name="PSM1_tool" value="420006"/>
-    <xacro:include filename="$(find dvrk_model)/urdf/Si/psm_base.urdf.xacro"/>
-    <xacro:include filename="$(find dvrk_model)/urdf/Si/tools.urdf.xacro"/>
-    <link name="world"/>
-    <xacro:psm_arm_active
-        prefix="${PSM1_}"
-        parent_link="world"
-        xyz="0 0 0"
-        rpy="0 0 0"/>
-    <xacro:tool tool_name="P420006" prefix="${PSM1_}" parent_link="${PSM1_}tool_parent"/>
+  <xacro:property name="tool_name" value="P420006"/>
+  <xacro:include filename="$(find dvrk_model)/urdf/Si/psm_base.urdf.xacro"/>
+  <xacro:include filename="$(find dvrk_model)/urdf/Si/tools.urdf.xacro"/>
+  <link name="world"/>
+  <xacro:psm_arm_active
+      prefix="PSM1_"
+      parent_link="world"
+      xyz="0 0 0"
+      rpy="0 0 0"/>
+  <xacro:tool tool_name="${tool_name}" prefix="PSM1_" parent_link="PSM1_tool_parent"/>
 </robot>

File: urdf/Si/PSM2.urdf.xacro (robot description, xacro)
@@ -1,14 +1,13 @@
 <?xml version="1.0" ?>
 <robot name="PSM2" xmlns:xacro="http://www.ros.org/wiki/xacro">
-    <xacro:property name="PSM2_" value="PSM2_"/>
-    <xacro:property name="PSM2_tool" value="420006"/>
-    <xacro:include filename="$(find dvrk_model)/urdf/Si/psm_base.urdf.xacro"/>
-    <xacro:include filename="$(find dvrk_model)/urdf/Si/tools.urdf.xacro"/>
-    <link name="world"/>
-    <xacro:psm_arm_active
-        prefix="${PSM2_}"
-        parent_link="world"
-        xyz="0 0 0"
-        rpy="0 0 0"/>
-    <xacro:tool tool_name="P420006" prefix="${PSM2_}" parent_link="${PSM2_}tool_parent"/>
+  <xacro:property name="tool_name" value="P420006"/>
+  <xacro:include filename="$(find dvrk_model)/urdf/Si/psm_base.urdf.xacro"/>
+  <xacro:include filename="$(find dvrk_model)/urdf/Si/tools.urdf.xacro"/>
+  <link name="world"/>
+  <xacro:psm_arm_active
+      prefix="PSM2_"
+      parent_link="world"
+      xyz="0 0 0"
+      rpy="0 0 0"/>
+  <xacro:tool tool_name="${tool_name}" prefix="PSM2_" parent_link="PSM2_tool_parent"/>
 </robot>

File: urdf/Si/PSM3.urdf.xacro (robot description, xacro)
@@ -1,14 +1,13 @@
 <?xml version="1.0" ?>
 <robot name="PSM3" xmlns:xacro="http://www.ros.org/wiki/xacro">
-    <xacro:property name="PSM3_" value="PSM3_"/>
-    <xacro:property name="PSM3_tool" value="420006"/>
-    <xacro:include filename="$(find dvrk_model)/urdf/Si/psm_base.urdf.xacro"/>
-    <xacro:include filename="$(find dvrk_model)/urdf/Si/tools.urdf.xacro"/>
-    <link name="world"/>
-    <xacro:psm_arm_active
-        prefix="${PSM3_}"
-        parent_link="world"
-        xyz="0 0 0"
-        rpy="0 0 0"/>
-    <xacro:tool tool_name="P420006" prefix="${PSM3_}" parent_link="${PSM3_}tool_parent"/>
+  <xacro:property name="tool_name" value="P420006"/>
+  <xacro:include filename="$(find dvrk_model)/urdf/Si/psm_base.urdf.xacro"/>
+  <xacro:include filename="$(find dvrk_model)/urdf/Si/tools.urdf.xacro"/>
+  <link name="world"/>
+  <xacro:psm_arm_active
+      prefix="PSM3_"
+      parent_link="world"
+      xyz="0 0 0"
+      rpy="0 0 0"/>
+  <xacro:tool tool_name="${tool_name}" prefix="PSM3_" parent_link="PSM3_tool_parent"/>
 </robot>

File: urdf/Si/SUJ.urdf.xacro (robot description, xacro)
@@ -1,801 +1,26 @@
-<?xml version="1.0"?>
-<robot name="dvrk_si" xmlns:xacro="http://www.ros.org/wiki/xacro">
-    <xacro:macro name="suj" params="prefix parent_link xyz rpy">
-        <xacro:if value="${prefix == 'PSM1_' or prefix == 'PSM2_'}">
-            <link
-                name="SUJ_${prefix}link_0">
-                <inertial>
-                <origin
-                    xyz="-0.042353 -4.4531E-08 0.24208"
-                    rpy="0 0 0" />
-                <mass
-                    value="12.704" />
-                <inertia
-                    ixx="0.368"
-                    ixy="-6.2028E-09"
-                    ixz="-0.021772"
-                    iyy="0.3714"
-                    iyz="5.3603E-09"
-                    izz="0.047463" />
-                </inertial>
-                <visual>
-                <origin
-                    xyz="0 0 0"
-                    rpy="0 0 0" />
-                <geometry>
-                    <mesh
-                    filename="package://dvrk_model/meshes/Si/SUJ/PSM/12/link_0.STL" />
-                </geometry>
-                <material
-                    name="">
-                    <color
-                    rgba="0.79216 0.81961 0.93333 1" />
-                </material>
-                </visual>
-                <collision>
-                <origin
-                    xyz="0 0 0"
-                    rpy="0 0 0" />
-                <geometry>
-                    <mesh
-                    filename="package://dvrk_model/meshes/Si/SUJ/PSM/12/link_0.STL" />
-                </geometry>
-                </collision>
-            </link>
-            <joint
-                name="SUJ_${prefix}j0"
-                type="prismatic">
-                <origin
-                xyz="${xyz}"
-                rpy="${rpy}" />
-                <parent
-                link="${parent_link}" />
-                <child
-                link="SUJ_${prefix}link_0" />
-                <axis
-                xyz="0 0 1" />
-                <limit
-                lower="0.0"
-                upper="0.512"
-                effort="0"
-                velocity="0" />
-            </joint>
-            <link
-                name="SUJ_${prefix}link_1">
-                <inertial>
-                <origin
-                    xyz="0.21712 2.5962E-08 0.072796"
-                    rpy="0 0 0" />
-                <mass
-                    value="7.0906" />
-                <inertia
-                    ixx="0.015346"
-                    ixy="-1.6493E-08"
-                    ixz="-0.0010396"
-                    iyy="0.22426"
-                    iyz="8.2106E-09"
-                    izz="0.2218" />
-                </inertial>
-                <visual>
-                <origin
-                    xyz="0 0 0"
-                    rpy="0 0 0" />
-                <geometry>
-                    <mesh
-                    filename="package://dvrk_model/meshes/Si/SUJ/PSM/12/link_1.STL" />
-                </geometry>
-                <material
-                    name="">
-                    <color
-                    rgba="0.79216 0.81961 0.93333 1" />
-                </material>
-                </visual>
-                <collision>
-                <origin
-                    xyz="0 0 0"
-                    rpy="0 0 0" />
-                <geometry>
-                    <mesh
-                    filename="package://dvrk_model/meshes/Si/SUJ/PSM/12/link_1.STL" />
-                </geometry>
-                </collision>
-            </link>
-            <joint
-                name="SUJ_${prefix}j1"
-                type="revolute">
-                <origin
-                xyz="-0.024998 0 0.59"
-                rpy="0 0 0" />
-                <parent
-                link="SUJ_${prefix}link_0" />
-                <child
-                link="SUJ_${prefix}link_1" />
-                <axis
-                xyz="0 0 1" />
-                <limit
-                lower="-3.141"
-                upper="3.141"
-                effort="0"
-                velocity="0" />
-            </joint>
-            <link
-                name="SUJ_${prefix}link_2">
-                <inertial>
-                <origin
-                    xyz="0.22659 -1.07E-07 0.065498"
-                    rpy="0 0 0" />
-                <mass
-                    value="5.8282" />
-                <inertia
-                    ixx="0.011467"
-                    ixy="-2.0133E-09"
-                    ixz="0.0026277"
-                    iyy="0.19305"
-                    iyz="2.1385E-09"
-                    izz="0.19056" />
-                </inertial>
-                <visual>
-                <origin
-                    xyz="0 0 0"
-                    rpy="0 0 0" />
-                <geometry>
-                    <mesh
-                    filename="package://dvrk_model/meshes/Si/SUJ/PSM/12/link_2.STL" />
-                </geometry>
-                <material
-                    name="">
-                    <color
-                    rgba="0.79216 0.81961 0.93333 1" />
-                </material>
-                </visual>
-                <collision>
-                <origin
-                    xyz="0 0 0"
-                    rpy="0 0 0" />
-                <geometry>
-                    <mesh
-                    filename="package://dvrk_model/meshes/Si/SUJ/PSM/12/link_2.STL" />
-                </geometry>
-                </collision>
-            </link>
-            <joint
-                name="SUJ_${prefix}j2"
-                type="revolute">
-                <origin
-                xyz="0.4575 0 0.144"
-                rpy="0 0 0" />
-                <parent
-                link="SUJ_${prefix}link_1" />
-                <child
-                link="SUJ_${prefix}link_2" />
-                <axis
-                xyz="0 0 1" />
-                <limit
-                lower="-3.141"
-                upper="3.141"
-                effort="0"
-                velocity="0" />
-            </joint>
-            <link
-                name="SUJ_${prefix}link_3">
-                <inertial>
-                <origin
-                    xyz="0.014738 8.0422E-08 -0.027873"
-                    rpy="0 0 0" />
-                <mass
-                    value="0.5504" />
-                <inertia
-                    ixx="0.00064459"
-                    ixy="2.3418E-09"
-                    ixz="1.1203E-05"
-                    iyy="0.00057105"
-                    iyz="-2.8921E-09"
-                    izz="0.00085397" />
-                </inertial>
-                <visual>
-                <origin
-                    xyz="0 0 0"
-                    rpy="0 0 0" />
-                <geometry>
-                    <mesh
-                    filename="package://dvrk_model/meshes/Si/SUJ/PSM/12/link_3.STL" />
-                </geometry>
-                <material
-                    name="">
-                    <color
-                    rgba="0.79216 0.81961 0.93333 1" />
-                </material>
-                </visual>
-                <collision>
-                <origin
-                    xyz="0 0 0"
-                    rpy="0 0 0" />
-                <geometry>
-                    <mesh
-                    filename="package://dvrk_model/meshes/Si/SUJ/PSM/12/link_3.STL" />
-                </geometry>
-                </collision>
-            </link>
-            <joint
-                name="SUJ_${prefix}j3"
-                type="revolute">
-                <origin
-                xyz="0.458 0 -0.01875"
-                rpy="0 0 0" />
-                <parent
-                link="SUJ_${prefix}link_2" />
-                <child
-                link="SUJ_${prefix}link_3" />
-                <axis
-                xyz="0 0 -1" />
-                <limit
-                lower="-3.141"
-                upper="3.141"
-                effort="0"
-                velocity="0" />
-            </joint>
-            <link name="${prefix}active_arm_parent"/>
-            <joint
-                name="${prefix}fixed_psm"
-                type="fixed">
-                <origin
-                xyz="0.045255 0 -0.045255"
-                rpy="0 0.7854 0" />
-                <parent
-                link="SUJ_${prefix}link_3" />
-                <child
-                link="${prefix}active_arm_parent" />
-            </joint>
-        </xacro:if>
-        <xacro:if value="${prefix == 'PSM3_'}">
-             <link
-                name="SUJ_${prefix}link_0">
-                <inertial>
-                <origin
-                    xyz="-0.043484 -9.4105E-09 0.22013"
-                    rpy="0 0 0" />
-                <mass
-                    value="11.927" />
-                <inertia
-                    ixx="0.27621"
-                    ixy="-5.0682E-09"
-                    ixz="-0.016932"
-                    iyy="0.27936"
-                    iyz="3.4609E-09"
-                    izz="0.046091" />
-                </inertial>
-                <visual>
-                <origin
-                    xyz="0 0 0"
-                    rpy="0 0 0" />
-                <geometry>
-                    <mesh
-                    filename="package://dvrk_model/meshes/Si/SUJ/PSM/3/link_0.STL" />
-                </geometry>
-                <material
-                    name="">
-                    <color
-                    rgba="0.79216 0.81961 0.93333 1" />
-                </material>
-                </visual>
-                <collision>
-                <origin
-                    xyz="0 0 0"
-                    rpy="0 0 0" />
-                <geometry>
-                    <mesh
-                    filename="package://dvrk_model/meshes/Si/SUJ/PSM/3/link_0.STL" />
-                </geometry>
-                </collision>
-            </link>
-            <joint
-                name="SUJ_${prefix}j0"
-                type="prismatic">
-                <origin
-                xyz="${xyz}"
-                rpy="${rpy}" />
-                <parent
-                link="${parent_link}" />
-                <child
-                link="SUJ_${prefix}link_0" />
-                <axis
-                xyz="0 0 1" />
-                <limit
-                lower="0.0"
-                upper="0.512"
-                effort="0"
-                velocity="0" />
-            </joint>
-            <link
-                name="SUJ_${prefix}link_1">
-                <inertial>
-                <origin
-                    xyz="0.20518 1.3159E-05 0.040755"
-                    rpy="0 0 0" />
-                <mass
-                    value="7.8622" />
-                <inertia
-                    ixx="0.043421"
-                    ixy="8.2624E-06"
-                    ixz="0.030604"
-                    iyy="0.20282"
-                    iyz="-6.5783E-05"
-                    izz="0.17543" />
-                </inertial>
-                <visual>
-                <origin
-                    xyz="0 0 0"
-                    rpy="0 0 0" />
-                <geometry>
-                    <mesh
-                    filename="package://dvrk_model/meshes/Si/SUJ/PSM/3/link_1.STL" />
-                </geometry>
-                <material
-                    name="">
-                    <color
-                    rgba="0.79216 0.81961 0.93333 1" />
-                </material>
-                </visual>
-                <collision>
-                <origin
-                    xyz="0 0 0"
-                    rpy="0 0 0" />
-                <geometry>
-                    <mesh
-                    filename="package://dvrk_model/meshes/Si/SUJ/PSM/3/link_1.STL" />
-                </geometry>
-                </collision>
-            </link>
-            <joint
-                name="SUJ_${prefix}j1"
-                type="revolute">
-                <origin
-                xyz="-0.024998 0 0.513"
-                rpy="0 0 -0.23716" />
-                <parent
-                link="SUJ_${prefix}link_0" />
-                <child
-                link="SUJ_${prefix}link_1" />
-                <axis
-                xyz="0 0 1" />
-                <limit
-                lower="-3.14"
-                upper="3.14"
-                effort="0"
-                velocity="0" />
-            </joint>
-            <link
-                name="SUJ_${prefix}link_2">
-                <inertial>
-                <origin
-                    xyz="0.22894 -6.2716E-08 -9.2061E-05"
-                    rpy="0 0 0" />
-                <mass
-                    value="6.7952" />
-                <inertia
-                    ixx="0.01388"
-                    ixy="-1.0152E-09"
-                    ixz="3.4458E-05"
-                    iyy="0.21125"
-                    iyz="4.6007E-09"
-                    izz="0.20955" />
-                </inertial>
-                <visual>
-                <origin
-                    xyz="0 0 0"
-                    rpy="0 0 0" />
-                <geometry>
-                    <mesh
-                    filename="package://dvrk_model/meshes/Si/SUJ/PSM/3/link_2.STL" />
-                </geometry>
-                <material
-                    name="">
-                    <color
-                    rgba="0.79216 0.81961 0.93333 1" />
-                </material>
-                </visual>
-                <collision>
-                <origin
-                    xyz="0 0 0"
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
File: urdf/Si/suj.urdf.xacro (robot description, xacro)
@@ -44,5 +44,5 @@
             </link>
             <joint
-                name="SUJ_${prefix}j0"
+                name="SUJ_${prefix}J0"
                 type="prismatic">
                 <origin
@@ -102,5 +102,5 @@
             </link>
             <joint
-                name="SUJ_${prefix}j1"
+                name="SUJ_${prefix}J1"
                 type="revolute">
                 <origin
@@ -160,5 +160,5 @@
             </link>
             <joint
-                name="SUJ_${prefix}j2"
+                name="SUJ_${prefix}J2"
                 type="revolute">
                 <origin
@@ -218,5 +218,5 @@
             </link>
             <joint
-                name="SUJ_${prefix}j3"
+                name="SUJ_${prefix}J3"
                 type="revolute">
                 <origin
@@ -235,5 +235,5 @@
                 velocity="0" />
             </joint>
-            <link name="${prefix}active_arm_parent"/>
+            <link name="${prefix}mounting_point"/>
             <joint
                 name="${prefix}fixed_psm"
@@ -245,5 +245,5 @@
                 link="SUJ_${prefix}link_3" />
                 <child
-                link="${prefix}active_arm_parent" />
+                link="${prefix}mounting_point" />
             </joint>
         </xacro:if>
@@ -290,5 +290,5 @@
             </link>
             <joint
-                name="SUJ_${prefix}j0"
+                name="SUJ_${prefix}J0"
                 type="prismatic">
                 <origin
@@ -348,5 +348,5 @@
             </link>
             <joint
-                name="SUJ_${prefix}j1"
+                name="SUJ_${prefix}J1"
                 type="revolute">
                 <origin
@@ -406,5 +406,5 @@
             </link>
             <joint
-                name="SUJ_${prefix}j2"
+                name="SUJ_${prefix}J2"
                 type="revolute">
                 <origin
@@ -464,5 +464,5 @@
             </link>
             <joint
-                name="SUJ_${prefix}j3"
+                name="SUJ_${prefix}J3"
                 type="revolute">
                 <origin
@@ -522,5 +522,5 @@
             </link>
             <joint
-                name="SUJ_${prefix}j4"
+                name="SUJ_${prefix}J4"
                 type="revolute">
                 <origin
@@ -539,5 +539,5 @@
                 velocity="0" />
             </joint>
-            <link name="${prefix}active_arm_parent"/>
+            <link name="${prefix}mounting_point"/>
             <joint
                 name="${prefix}fixed_psm"
@@ -549,5 +549,5 @@
                 link="SUJ_${prefix}link_4" />
                 <child
-                link="${prefix}active_arm_parent" />
+                link="${prefix}mounting_point" />
             </joint>
         </xacro:if>
@@ -594,5 +594,5 @@
             </link>
             <joint
-                name="SUJ_${prefix}j0"
+                name="SUJ_${prefix}J0"
                 type="prismatic">
                 <origin
@@ -652,5 +652,5 @@
             </link>
             <joint
-                name="SUJ_${prefix}j1"
+                name="SUJ_${prefix}J1"
                 type="revolute">
                 <origin
@@ -710,5 +710,5 @@
             </link>
             <joint
-                name="SUJ_${prefix}j2"
+                name="SUJ_${prefix}J2"
                 type="revolute">
                 <origin
@@ -768,5 +768,5 @@
             </link>
             <joint
-                name="SUJ_${prefix}j3"
+                name="SUJ_${prefix}J3"
                 type="revolute">
                 <origin
@@ -785,5 +785,5 @@
                 velocity="0" />
             </joint>
-            <link name="${prefix}active_arm_parent"/>
+            <link name="${prefix}mounting_point"/>
             <joint
                 name="${prefix}fixed_psm"
@@ -795,5 +795,5 @@
                 link="SUJ_${prefix}link_3" />
                 <child
-                link="${prefix}active_arm_parent" />
+                link="${prefix}mounting_point" />
             </joint>
         </xacro:if>
