Commit message: Trying to use multiple joint and state publishers to match C++ component.  PSMs should them be attached at end of SUJs.  tf2 static broadcast almost works but there is likely a race condition so this is not a solution.

File: urdf/Si/suj_column.urdf.xacro (robot description, xacro)
@@ -1,5 +1,5 @@
 <?xml version="1.0"?>
 <robot name="dvrk_si" xmlns:xacro="http://www.ros.org/wiki/xacro">
-    <xacro:macro name="suj_tower">
+    <xacro:macro name="suj_column">
         <link name="world"/>
         <joint
@@ -8,7 +8,7 @@
             <origin xyz="0 0 0" rpy="0 0 0" />
             <parent link="world" />
-            <child link="SUJ_tower" />
+            <child link="SUJ_column" />
         </joint>
-        <link name="SUJ_tower">
+        <link name="SUJ_column">
             <inertial>
             <origin
