Commit message: working version for Si patient cart using multiple urdf

File: urdf/Classic/MTMR.urdf.xacro (robot description, xacro)
@@ -7,4 +7,4 @@
       prefix="MTMR_"
       parent_link="world"
-      xyz="0.25 0.0 1.0" rpy="0.0 0.0 0.0"/>
+      xyz="0.25 0.0 1.0"/>
 </robot>

File: urdf/Classic/mtm.urdf.xacro (robot description, xacro)
@@ -4,5 +4,5 @@
   <xacro:include filename="$(find dvrk_model)/urdf/Classic/common.urdf.xacro"/>
   <!-- Macro for the da Vinci Master Console -->
-  <xacro:macro name="master_console" params="prefix parent_link xyz rpy">
+  <xacro:macro name="master_console" params="prefix parent_link xyz:='0.0 0.0 0.0' rpy:='0.0 0.0 0.0'">
     <joint name="base_fixed" type="fixed">
       <parent link="${parent_link}"/>
@@ -15,5 +15,5 @@
   </xacro:macro>
   <!-- Macros for left and right MTMs -->
-  <xacro:macro name="mtm_left" params="prefix parent_link xyz rpy">
+  <xacro:macro name="mtm_left" params="prefix parent_link xyz:='0.0 0.0 0.0' rpy:='0.0 0.0 0.0'">
     <xacro:mtm
         prefix="${prefix}"
@@ -22,5 +22,5 @@
     <xacro:mtm_platform_left prefix="${prefix}"/>
   </xacro:macro>
-  <xacro:macro name="mtm_right" params="prefix parent_link xyz rpy">
+  <xacro:macro name="mtm_right" params="prefix parent_link xyz:='0.0 0.0 0.0' rpy:='0.0 0.0 0.0'">
     <xacro:mtm
 	prefix="${prefix}"

File: urdf/Si/psm_base.urdf.xacro (robot description, xacro)
@@ -1,5 +1,5 @@
 <?xml version="1.0"?>
 <robot name="dvrk_si" xmlns:xacro="http://www.ros.org/wiki/xacro">
-  <xacro:macro name="psm_arm_active" params="prefix parent_link xyz rpy">
+  <xacro:macro name="psm_arm_active" params="prefix parent_link xyz:='0.0 0.0 0.0' rpy:='0.0 0.0 0.0'">
     <link
         name="${prefix}link_0">
