Commit message: update bugs in urdf/psm files

File: urdf/Classic/PSM_base.urdf.xacro (robot description, xacro)
@@ -33,5 +33,5 @@
     </link>
     <!-- joint 1: yaw -->
-    <joint name="yaw" type="revolute">
+    <joint name="yaw" type="revolute"> <!--outer_yaw-->
       <parent link="${prefix}PSM_base_link"/>
       <child  link="${prefix}PSM_outer_yaw_link"/>
@@ -54,5 +54,5 @@
       across the 5 parallelogram sub-links below.
     -->
-    <joint name="pitch" type="revolute">
+    <joint name="pitch" type="revolute"> <!--outer_pitch-->
       <parent link="${prefix}PSM_outer_yaw_link"/>
       <child  link="${prefix}PSM_outer_pitch_link"/>

File: urdf/Si/PSM_base.urdf.xacro (robot description, xacro)
@@ -68,10 +68,10 @@
     </link>
     <!-- joint 1: yaw (outer yaw) -->
-    <joint name="yaw" type="revolute">
+    <joint name="yaw" type="revolute"> <!--outer_yaw-->
       <origin xyz="0.158 0 0" rpy="0.0 0.0 0.0"/>
       <parent link="${prefix}PSM_ECM_base_link"/>
       <child  link="${prefix}PSM_ECM_outer_yaw_link"/>
       <axis xyz="-1.0 0.0 0.0"/>
-      <limit lower="-3.14" upper="3.14" effort="0.0" velocity="0.0"/>
+      <limit lower="-3.14" upper="3.14" effort="0.0" velocity="0.0"/> <!--flagged placeholder and limits of ±π-->
     </joint>
     <!-- link 2: outer pitch arm -->
@@ -99,10 +99,10 @@
     </link>
     <!-- joint 2: pitch (outer pitch) -->
-    <joint name="pitch" type="revolute">
+    <joint name="pitch" type="revolute"> <!--outer_pitch-->
       <origin xyz="0.2987 0 -0.071222" rpy="0 -1.1345 -3.1416"/>
       <parent link="${prefix}PSM_ECM_outer_yaw_link"/>
       <child  link="${prefix}PSM_ECM_outer_pitch_link"/>
       <axis xyz="0 -1 0"/>
-      <limit lower="-3.14" upper="3.14" effort="0" velocity="0"/>
+      <limit lower="-3.14" upper="3.14" effort="0" velocity="0"/> <!--flagged placeholder and limits of ±π-->
     </joint>
     <!-- link 3: pitch parallelogram arm (mimic pitch) -->
@@ -134,5 +134,5 @@
       <child  link="${prefix}PSM_ECM_outer_pitch_bottom_link"/>
       <axis xyz="0 1 0"/>
-      <limit lower="-3.14" upper="3.14" effort="0" velocity="0"/>
+      <limit lower="-3.14" upper="3.14" effort="0" velocity="0"/> <!--flagged placeholder and limits of ±π-->
       <mimic joint="pitch" multiplier="-1"/>
     </joint>
@@ -165,5 +165,5 @@
       <child  link="${prefix}PSM_ECM_outer_pitch_top_link"/>
       <axis xyz="0 1 0"/>
-      <limit lower="-3.14" upper="3.14" effort="0" velocity="0"/>
+      <limit lower="-3.14" upper="3.14" effort="0" velocity="0"/> <!--flagged placeholder and limits of ±π-->
       <mimic joint="pitch" multiplier="1"/>
     </joint>

File: urdf/common/PSM_instrument.urdf.xacro (robot description, xacro)
@@ -24,5 +24,5 @@
     <xacro:property name="is_si" value="${str(instrument).startswith('42')}"/>
     <!-- Dynamically select the correct shaft length based on generation -->
-    <xacro:property name="shaft_length" value="${0.53559 if is_si else 0.4162}"/>
+    <xacro:property name="shaft_length" value="${0.53559 if is_si else 0.4162}"/> <!--0.4670 for Si as also in strucuture.md-->
     <!-- fixed joint to hold the shaft visual BEFORE the roll joint -->
     <joint name="instrument_base_fixed" type="fixed">
