Commit message: Remove 'outer' from PSM joint/link/mesh names (Classic + Si)

File: urdf/Classic/PSM_base.urdf.xacro (robot description, xacro)
@@ -3,6 +3,6 @@
   <!--
     Classic PSM arm — 3 actuated DOF:
-      Joint 1: outer_yaw   (revolute)
-      Joint 2: outer_pitch  (revolute, parallelogram linkage)
+      Joint 1: yaw   (revolute)
+      Joint 2: pitch  (revolute, parallelogram linkage)
       Joint 3: insertion    (prismatic)
     Macro output: ends at ${prefix}PSM_tool_parent_link.
@@ -33,46 +33,46 @@
     </link>
     <!-- joint 1: yaw -->
-    <joint name="yaw" type="revolute"> <!--outer_yaw-->
+    <joint name="yaw" type="revolute"> <!--yaw-->
       <parent link="${prefix}PSM_base_link"/>
-      <child  link="${prefix}PSM_outer_yaw_link"/>
+      <child  link="${prefix}PSM_yaw_link"/>
       <axis xyz="0 0 1"/>
       <origin rpy="0 -1.5708 1.5708" xyz="0.0 0.0 0.0"/>
       <limit lower="-1.5707" upper="1.5707" velocity=".4" effort="1000"/>
     </joint>
-    <!-- link 1: outer_yaw -->
-    <link name="${prefix}PSM_outer_yaw_link">
+    <!-- link 1: yaw -->
+    <link name="${prefix}PSM_yaw_link">
       <visual>
         <origin rpy="3.1416 0 1.5708" xyz="0.0125 0 0.5265"/>
         <geometry>
-          <mesh filename="package://dvrk_model/meshes/Classic/PSM/PSM_outer_yaw.dae"/>
+          <mesh filename="package://dvrk_model/meshes/Classic/PSM/PSM_yaw.dae"/>
         </geometry>
       </visual>
     </link>
     <!--
-      Joint 2: outer_pitch (revolute) with parallelogram linkage.
-      The outer_pitch_link itself has no mesh; the visual is distributed
+      Joint 2: pitch (revolute) with parallelogram linkage.
+      The pitch_link itself has no mesh; the visual is distributed
       across the 5 parallelogram sub-links below.
     -->
-    <joint name="pitch" type="revolute"> <!--outer_pitch-->
-      <parent link="${prefix}PSM_outer_yaw_link"/>
-      <child  link="${prefix}PSM_outer_pitch_link"/>
+    <joint name="pitch" type="revolute"> <!--pitch-->
+      <parent link="${prefix}PSM_yaw_link"/>
+      <child  link="${prefix}PSM_pitch_link"/>
       <axis xyz="0 0 1"/>
       <origin rpy="-1.5708 -1.5708 0" xyz="0 0 0"/>
       <limit lower="-0.7854" upper="0.7854" velocity=".4" effort="1000"/>
     </joint>
-    <link name="${prefix}PSM_outer_pitch_link"/>
+    <link name="${prefix}PSM_pitch_link"/>
     <!-- parallelogram sub-joint 1 -->
     <joint name="pitch_1" type="continuous">
-      <parent link="${prefix}PSM_outer_yaw_link"/>
-      <child  link="${prefix}PSM_outer_pitch_back_link"/>
+      <parent link="${prefix}PSM_yaw_link"/>
+      <child  link="${prefix}PSM_pitch_back_link"/>
       <axis xyz="0 0 1"/>
       <origin rpy="-1.5708 -1.5708 0" xyz="0 0.0295 0.5185"/>
       <mimic joint="pitch" multiplier="1"/>
     </joint>
-    <link name="${prefix}PSM_outer_pitch_back_link">
+    <link name="${prefix}PSM_pitch_back_link">
       <visual>
         <origin rpy="0 0 -0.27129" xyz="0 0 0"/>
         <geometry>
-          <mesh filename="package://dvrk_model/meshes/Classic/PSM/PSM_outer_pitch_back.dae"/>
+          <mesh filename="package://dvrk_model/meshes/Classic/PSM/PSM_pitch_back.dae"/>
         </geometry>
       </visual>
@@ -80,15 +80,15 @@
     <!-- parallelogram sub-joint 2 -->
     <joint name="pitch_2" type="continuous">
-      <parent link="${prefix}PSM_outer_yaw_link"/>
-      <child  link="${prefix}PSM_outer_pitch_front_link"/>
+      <parent link="${prefix}PSM_yaw_link"/>
+      <child  link="${prefix}PSM_pitch_front_link"/>
       <axis xyz="0 0 1"/>
       <origin rpy="-1.5708 -1.5708 0" xyz="0 0.0295 0.4285"/>
       <mimic joint="pitch" multiplier="1"/>
     </joint>
-    <link name="${prefix}PSM_outer_pitch_front_link">
+    <link name="${prefix}PSM_pitch_front_link">
       <visual>
         <origin rpy="0 0 -0.27129" xyz="0 0 0"/>
         <geometry>
-          <mesh filename="package://dvrk_model/meshes/Classic/PSM/PSM_outer_pitch_front.dae"/>
+          <mesh filename="package://dvrk_model/meshes/Classic/PSM/PSM_pitch_front.dae"/>
         </geometry>
       </visual>
@@ -96,15 +96,15 @@
     <!-- parallelogram sub-joint 3 -->
     <joint name="pitch_3" type="continuous">
-      <parent link="${prefix}PSM_outer_pitch_back_link"/>
-      <child  link="${prefix}PSM_outer_pitch_bottom_link"/>
+      <parent link="${prefix}PSM_pitch_back_link"/>
+      <child  link="${prefix}PSM_pitch_bottom_link"/>
       <axis xyz="0 0 1"/>
       <origin rpy="0 0 0" xyz="0.04178 0.15007 -0.0137"/>
       <mimic joint="pitch" multiplier="-1"/>
     </joint>
-    <link name="${prefix}PSM_outer_pitch_bottom_link">
+    <link name="${prefix}PSM_pitch_bottom_link">
       <visual>
         <origin rpy="0 -1.5708 0" xyz="0.009 0 0"/>
         <geometry>
-          <mesh filename="package://dvrk_model/meshes/Classic/PSM/PSM_outer_pitch_bottom.dae"/>
+          <mesh filename="package://dvrk_model/meshes/Classic/PSM/PSM_pitch_bottom.dae"/>
         </geometry>
       </visual>
@@ -112,15 +112,15 @@
     <!-- parallelogram sub-joint 4 -->
     <joint name="pitch_4" type="continuous">
-      <parent link="${prefix}PSM_outer_pitch_back_link"/>
-      <child  link="${prefix}PSM_outer_pitch_top_link"/>
+      <parent link="${prefix}PSM_pitch_back_link"/>
+      <child  link="${prefix}PSM_pitch_top_link"/>
       <axis xyz="0 0 1"/>
       <origin rpy="0 0 0" xyz="0.04209 0.18695 -0.02412"/>
       <mimic joint="pitch" multiplier="-1"/>
     </joint>
-    <link name="${prefix}PSM_outer_pitch_top_link">
+    <link name="${prefix}PSM_pitch_top_link">
       <visual>
         <origin rpy="0 -1.5708 0" xyz="0.009 0 0"/>
         <geometry>
-          <mesh filename="package://dvrk_model/meshes/Classic/PSM/PSM_outer_pitch_top.dae"/>
+          <mesh filename="package://dvrk_model/meshes/Classic/PSM/PSM_pitch_top.dae"/>
         </geometry>
       </visual>
@@ -128,15 +128,15 @@
     <!-- parallelogram sub-joint 5 -->
     <joint name="pitch_5" type="continuous">
-      <parent link="${prefix}PSM_outer_pitch_bottom_link"/>
-      <child  link="${prefix}PSM_outer_insertion_link"/>
+      <parent link="${prefix}PSM_pitch_bottom_link"/>
+      <child  link="${prefix}PSM_insertion_link"/>
       <axis xyz="0 0 1"/>
       <origin rpy="0 0 0" xyz="-0.520 0 -0.0155"/>
       <mimic joint="pitch" multiplier="1"/>
     </joint>
-    <link name="${prefix}PSM_outer_insertion_link">
+    <link name="${prefix}PSM_insertion_link">
       <visual>
         <origin rpy="0 -1.5708 1.5708" xyz="0.02528 0.429 0"/>
         <geometry>
-          <mesh filename="package://dvrk_model/meshes/Classic/PSM/PSM_outer_insertion.dae"/>
+          <mesh filename="package://dvrk_model/meshes/Classic/PSM/PSM_insertion.dae"/>
         </geometry>
       </visual>
@@ -144,5 +144,5 @@
     <!-- joint 3: insertion (prismatic) -->
     <joint name="insertion" type="prismatic">
-      <parent link="${prefix}PSM_outer_pitch_link"/>
+      <parent link="${prefix}PSM_pitch_link"/>
       <child  link="${prefix}PSM_tool_parent_link"/>
       <axis xyz="0 0 1"/>

File: urdf/Classic/psm_base.urdf.xacro (robot description, xacro)
@@ -20,5 +20,5 @@
     <joint name="yaw" type="revolute">
       <parent link="${prefix}psm_base_link"/>
-      <child link="${prefix}outer_yaw_link"/>
+      <child link="${prefix}yaw_link"/>
       <axis xyz="0 0 1"/>
       <!-- <origin rpy="1.5708 -1.5708 0" xyz="0.0 -0.369 0.0"/> -->
@@ -26,30 +26,30 @@
       <limit lower="-1.5707" upper="1.5707" velocity=".4" effort="1000"/>
     </joint>
-    <!-- link 1: outer_yaw -->
-    <link name="${prefix}outer_yaw_link">
+    <!-- link 1: yaw -->
+    <link name="${prefix}yaw_link">
       <visual>        <!-- <origin rpy="0 0 -1.5708" xyz="0.0125 0 0.1575"/> -->
         <origin rpy="3.1416 0 1.5708" xyz="0.0125 0 0.5265"/>
         <geometry>
-          <mesh filename="package://dvrk_model/meshes/Classic/PSM/outer_yaw.dae"/>
+          <mesh filename="package://dvrk_model/meshes/Classic/PSM/yaw.dae"/>
         </geometry>
       </visual>
     </link>
     <!-- Note: I can not put visual link here as it's parallel -->
-    <!-- mechanism, so the outer_pitch_link does not have visual -->
-    <!-- link, all visual links mimic outer_pitch value -->
-    <!-- joint 2: outer_pitch -->
+    <!-- mechanism, so the pitch_link does not have visual -->
+    <!-- link, all visual links mimic pitch value -->
+    <!-- joint 2: pitch -->
     <joint name="pitch" type="revolute">
-      <parent link="${prefix}outer_yaw_link"/>
-      <child link="${prefix}outer_pitch_link"/>
+      <parent link="${prefix}yaw_link"/>
+      <child link="${prefix}pitch_link"/>
       <axis xyz="0 0 1"/>
       <origin rpy="-1.5708 -1.5708 0" xyz="0 0 0"/>
       <limit lower="-0.7854" upper="0.7854" velocity=".4" effort="1000"/>
     </joint>
-    <!-- link 2: outer_pitch_link -->
-    <link name="${prefix}outer_pitch_link"/>
-    <!-- joint 2-1: outer_pitch_1 -->
+    <!-- link 2: pitch_link -->
+    <link name="${prefix}pitch_link"/>
+    <!-- joint 2-1: pitch_1 -->
     <joint name="pitch_1" type="continuous">
-      <parent link="${prefix}outer_yaw_link"/>
-      <child link="${prefix}outer_pitch_back_link"/>
+      <parent link="${prefix}yaw_link"/>
+      <child link="${prefix}pitch_back_link"/>
       <axis xyz="0 0 1"/>
       <!-- <origin rpy="-1.5708 -1.5708 0" xyz="0 0.0295 0.1495"/> -->
@@ -57,78 +57,78 @@
       <mimic joint="pitch" multiplier="1"/>
     </joint>
-    <!-- link 2-1: outer_pitch_back -->
-    <link name="${prefix}outer_pitch_back_link">
+    <!-- link 2-1: pitch_back -->
+    <link name="${prefix}pitch_back_link">
       <visual>
         <origin rpy="0 0 -0.27129" xyz="0 0 0"/>
         <geometry>
-          <mesh filename="package://dvrk_model/meshes/Classic/PSM/outer_pitch_back.dae"/>
+          <mesh filename="package://dvrk_model/meshes/Classic/PSM/pitch_back.dae"/>
         </geometry>
       </visual>
     </link>
-    <!-- joint 2-2: outer_pitch_2 -->
+    <!-- joint 2-2: pitch_2 -->
     <joint name="pitch_2" type="continuous">
-      <parent link="${prefix}outer_yaw_link"/>
-      <child link="${prefix}outer_pitch_front_link"/>
+      <parent link="${prefix}yaw_link"/>
+      <child link="${prefix}pitch_front_link"/>
       <axis xyz="0 0 1"/>
       <origin rpy="-1.5708 -1.5708 0" xyz="0 0.0295 0.4285"/>
       <mimic joint="pitch" multiplier="1"/>
     </joint>
-    <!-- link 2-2: outer_pitch_front -->
-    <link name="${prefix}outer_pitch_front_link">
+    <!-- link 2-2: pitch_front -->
+    <link name="${prefix}pitch_front_link">
       <visual>
         <origin rpy="0 0 -0.27129" xyz="0 0 0"/>
         <geometry>
-          <mesh filename="package://dvrk_model/meshes/Classic/PSM/outer_pitch_front.dae"/>
+          <mesh filename="package://dvrk_model/meshes/Classic/PSM/pitch_front.dae"/>
         </geometry>
       </visual>
     </link>
-    <!-- joint 2-3: outer_pitch_3 -->
+    <!-- joint 2-3: pitch_3 -->
     <joint name="pitch_3" type="continuous">
-      <parent link="${prefix}outer_pitch_back_link"/>
-      <child link="${prefix}outer_pitch_bottom_link"/>
+      <parent link="${prefix}pitch_back_link"/>
+      <child link="${prefix}pitch_bottom_link"/>
       <axis xyz="0 0 1"/>
       <origin rpy="0 0 0" xyz="0.04178 0.15007 -0.0137"/>
       <mimic joint="pitch" multiplier="-1"/>
     </joint>
-    <!-- link 2-3: outer_pitch_bottom -->
-    <link name="${prefix}outer_pitch_bottom_link">
+    <!-- link 2-3: pitch_bottom -->
+    <link name="${prefix}pitch_bottom_link">
       <visual>
         <origin rpy="0 -1.5708 0" xyz="0.009 0 0"/>
         <geometry>
-          <mesh filename="package://dvrk_model/meshes/Classic/PSM/outer_pitch_bottom.dae"/>
+          <mesh filename="package://dvrk_model/meshes/Classic/PSM/pitch_bottom.dae"/>
         </geometry>
       </visual>
     </link>
-    <!-- joint 2-4: outer_pitch_4 -->
+    <!-- joint 2-4: pitch_4 -->
     <joint name="pitch_4" type="continuous">
-      <parent link="${prefix}outer_pitch_back_link"/>
-      <child link="${prefix}outer_pitch_top_link"/>
+      <parent link="${prefix}pitch_back_link"/>
+      <child link="${prefix}pitch_top_link"/>
       <axis xyz="0 0 1"/>
       <origin rpy="0 0 0" xyz="0.04209 0.18695 -0.02412"/>
       <mimic joint="pitch" multiplier="-1"/>
     </joint>
-    <!-- link 2-4: outer_pitch_top -->
-    <link name="${prefix}outer_pitch_top_link">
+    <!-- link 2-4: pitch_top -->
+    <link name="${prefix}pitch_top_link">
       <visual>
         <origin rpy="0 -1.5708 0" xyz="0.009 0 0"/>
         <geometry>
-          <mesh filename="package://dvrk_model/meshes/Classic/PSM/outer_pitch_top.dae"/>
+          <mesh filename="package://dvrk_model/meshes/Classic/PSM/pitch_top.dae"/>
         </geometry>
       </visual>
     </link>
-    <!-- joint 2-5: outer_pitch_5 -->
+    <!-- joint 2-5: pitch_5 -->
     <joint name="pitch_5" type="continuous">
-      <parent link="${prefix}outer_pitch_bottom_link"/>
-      <child link="${prefix}outer_insertion_link"/>
+      <parent link="${prefix}pitch_bottom_link"/>
+      <child link="${prefix}insertion_link"/>
       <axis xyz="0 0 1"/>
       <origin rpy="0 0 0" xyz="-0.520 0 -0.0155"/>
       <mimic joint="pitch" multiplier="1"/>
     </joint>
-    <!-- link 2-5: outer_insertion -->
-    <link name="${prefix}outer_insertion_link">
+    <!-- link 2-5: insertion -->
+    <link name="${prefix}insertion_link">
       <visual>
         <origin rpy="0 -1.5708 1.5708" xyz="0.02528 0.429 0"/>
         <geometry>
-          <mesh filename="package://dvrk_model/meshes/Classic/PSM/outer_insertion.dae"/>
+          <mesh filename="package://dvrk_model/meshes/Classic/PSM/insertion.dae"/>
         </geometry>
       </visual>
@@ -136,7 +136,7 @@
     <!-- joint 3: insertion -->
     <joint name="insertion" type="prismatic">
-      <!-- <parent link="${prefix}outer_insertion_link"/> -->
+      <!-- <parent link="${prefix}insertion_link"/> -->
       <!-- <parent link="${prefix}psm_base_link"/> -->
-      <parent link="${prefix}outer_pitch_link"/>
+      <parent link="${prefix}pitch_link"/>
       <child link="${prefix}tool_main_link"/>
       <axis xyz="0 0 1"/>

File: urdf/Si/PSM_base.urdf.xacro (robot description, xacro)
@@ -44,6 +44,6 @@
       <origin rpy="${rpy}" xyz="${xyz}"/>
     </joint>
-    <!-- link 1: outer_yaw body -->
-    <link name="${prefix}PSM_ECM_outer_yaw_link">
+    <!-- link 1: yaw body -->
+    <link name="${prefix}PSM_ECM_yaw_link">
       <inertial>
         <origin xyz="0.1461 0.090363 -0.024957" rpy="0 0 0"/>
@@ -56,5 +56,5 @@
         <origin xyz="0 0 0" rpy="0 0 0"/>
         <geometry>
-          <mesh filename="package://dvrk_model/meshes/Si/PSM_ECM/PSM_ECM_outer_yaw.stl"/>
+          <mesh filename="package://dvrk_model/meshes/Si/PSM_ECM/PSM_ECM_yaw.stl"/>
         </geometry>
         <material name=""><color rgba="0.79216 0.81961 0.93333 1"/></material>
@@ -63,18 +63,18 @@
         <origin xyz="0 0 0" rpy="0 0 0"/>
         <geometry>
-          <mesh filename="package://dvrk_model/meshes/Si/PSM_ECM/PSM_ECM_outer_yaw.stl"/>
+          <mesh filename="package://dvrk_model/meshes/Si/PSM_ECM/PSM_ECM_yaw.stl"/>
         </geometry>
       </collision>
     </link>
     <!-- joint 1: yaw (outer yaw) -->
-    <joint name="yaw" type="revolute"> <!--outer_yaw-->
+    <joint name="yaw" type="revolute"> <!--yaw-->
       <origin xyz="0.158 0 0" rpy="0.0 0.0 0.0"/>
       <parent link="${prefix}PSM_ECM_base_link"/>
-      <child  link="${prefix}PSM_ECM_outer_yaw_link"/>
+      <child  link="${prefix}PSM_ECM_yaw_link"/>
       <axis xyz="-1.0 0.0 0.0"/>
       <limit lower="-3.14" upper="3.14" effort="0.0" velocity="0.0"/> <!--flagged placeholder and limits of ±π-->
     </joint>
     <!-- link 2: outer pitch arm -->
-    <link name="${prefix}PSM_ECM_outer_pitch_link">
+    <link name="${prefix}PSM_ECM_pitch_link">
       <inertial>
         <origin xyz="0.083895 -0.00073113 -0.028998" rpy="0.0 0.0 0.0"/>
@@ -87,5 +87,5 @@
         <origin xyz="0 0 0" rpy="0 0 0"/>
         <geometry>
-          <mesh filename="package://dvrk_model/meshes/Si/PSM_ECM/PSM_ECM_outer_pitch.stl"/>
+          <mesh filename="package://dvrk_model/meshes/Si/PSM_ECM/PSM_ECM_pitch.stl"/>
         </geometry>
         <material name=""><color rgba="0.79216 0.81961 0.93333 1"/></material>
@@ -94,18 +94,18 @@
         <origin xyz="0 0 0" rpy="0 0 0"/>
         <geometry>
-          <mesh filename="package://dvrk_model/meshes/Si/PSM_ECM/PSM_ECM_outer_pitch.stl"/>
+          <mesh filename="package://dvrk_model/meshes/Si/PSM_ECM/PSM_ECM_pitch.stl"/>
         </geometry>
       </collision>
     </link>
     <!-- joint 2: pitch (outer pitch) -->
-    <joint name="pitch" type="revolute"> <!--outer_pitch-->
+    <joint name="pitch" type="revolute"> <!--pitch-->
       <origin xyz="0.2987 0 -0.071222" rpy="0 -1.1345 -3.1416"/>
-      <parent link="${prefix}PSM_ECM_outer_yaw_link"/>
-      <child  link="${prefix}PSM_ECM_outer_pitch_link"/>
+      <parent link="${prefix}PSM_ECM_yaw_link"/>
+      <child  link="${prefix}PSM_ECM_pitch_link"/>
       <axis xyz="0 -1 0"/>
       <limit lower="-3.14" upper="3.14" effort="0" velocity="0"/> <!--flagged placeholder and limits of ±π-->
     </joint>
     <!-- link 3: pitch parallelogram arm (mimic pitch) -->
-    <link name="${prefix}PSM_ECM_outer_pitch_bottom_link">
+    <link name="${prefix}PSM_ECM_pitch_bottom_link">
       <inertial>
         <origin xyz="0.11824 1.9336E-19 0.12932" rpy="0 0 0"/>
@@ -118,5 +118,5 @@
         <origin xyz="0 0 0" rpy="0 0 0"/>
         <geometry>
-          <mesh filename="package://dvrk_model/meshes/Si/PSM_ECM/PSM_ECM_outer_pitch_bottom.stl"/>
+          <mesh filename="package://dvrk_model/meshes/Si/PSM_ECM/PSM_ECM_pitch_bottom.stl"/>
         </geometry>
         <material name=""><color rgba="0.79216 0.81961 0.93333 1"/></material>
@@ -125,5 +125,5 @@
         <origin xyz="0 0 0" rpy="0 0 0"/>
         <geometry>
-          <mesh filename="package://dvrk_model/meshes/Si/PSM_ECM/PSM_ECM_outer_pitch_bottom.stl"/>
+          <mesh filename="package://dvrk_model/meshes/Si/PSM_ECM/PSM_ECM_pitch_bottom.stl"/>
         </geometry>
       </collision>
@@ -131,6 +131,6 @@
     <joint name="pitch_2" type="revolute">
       <origin xyz="0.2032 0 0" rpy="0 -0.90761 -3.1416"/>
-      <parent link="${prefix}PSM_ECM_outer_pitch_link"/>
-      <child  link="${prefix}PSM_ECM_outer_pitch_bottom_link"/>
+      <parent link="${prefix}PSM_ECM_pitch_link"/>
+      <child  link="${prefix}PSM_ECM_pitch_bottom_link"/>
       <axis xyz="0 1 0"/>
       <limit lower="-3.14" upper="3.14" effort="0" velocity="0"/> <!--flagged placeholder and limits of ±π-->
@@ -138,5 +138,5 @@
     </joint>
     <!-- link 4: pitch parallelogram distal (mimic pitch) -->
-    <link name="${prefix}PSM_ECM_outer_pitch_top_link">
+    <link name="${prefix}PSM_ECM_pitch_top_link">
       <inertial>
         <origin xyz="0.041219 -9.0734E-08 0.13651" rpy="0 0 0"/>
@@ -149,5 +149,5 @@
         <origin xyz="0 0 0" rpy="0 0 0"/>
         <geometry>
-          <mesh filename="package://dvrk_model/meshes/Si/PSM_ECM/PSM_ECM_outer_pitch_top.stl"/>
+          <mesh filename="package://dvrk_model/meshes/Si/PSM_ECM/PSM_ECM_pitch_top.stl"/>
         </geometry>
         <material name=""><color rgba="0.79216 0.81961 0.93333 1"/></material>
@@ -156,5 +156,5 @@
         <origin xyz="0 0 0" rpy="0 0 0"/>
         <geometry>
-          <mesh filename="package://dvrk_model/meshes/Si/PSM_ECM/PSM_ECM_outer_pitch_top.stl"/>
+          <mesh filename="package://dvrk_model/meshes/Si/PSM_ECM/PSM_ECM_pitch_top.stl"/>
         </geometry>
       </collision>
@@ -162,6 +162,6 @@
     <joint name="pitch_3" type="revolute">
       <origin xyz="0.35966 0 0.16013" rpy="0 -0.063963 0"/>
-      <parent link="${prefix}PSM_ECM_outer_pitch_bottom_link"/>
-      <child  link="${prefix}PSM_ECM_outer_pitch_top_link"/>
+      <parent link="${prefix}PSM_ECM_pitch_bottom_link"/>
+      <child  link="${prefix}PSM_ECM_pitch_top_link"/>
       <axis xyz="0 1 0"/>
       <limit lower="-3.14" upper="3.14" effort="0" velocity="0"/> <!--flagged placeholder and limits of ±π-->
@@ -170,10 +170,10 @@
     <!--
       joint 3: insertion (prismatic) — moved here from psm_tool.
-      Origin from original outer_insertion_ref fixed joint (xyz 0.05061 0 0.41911)
+      Origin from original insertion_ref fixed joint (xyz 0.05061 0 0.41911)
       combined with the insertion joint offset.
     -->
     <joint name="insertion" type="prismatic">
       <origin xyz="0.05061 0 0.41911" rpy="${PI} 0 0"/>
-      <parent link="${prefix}PSM_ECM_outer_pitch_top_link"/>
+      <parent link="${prefix}PSM_ECM_pitch_top_link"/>
       <child  link="${prefix}PSM_tool_parent_link"/>
       <axis xyz="0 0 1"/>
@@ -190,5 +190,5 @@
     <joint name="${prefix}jrcm" type="fixed">
       <origin xyz="0.10643 0 -0.1731" rpy="3.1416 0 -1.5708"/>
-      <parent link="${prefix}PSM_ECM_outer_pitch_top_link"/>
+      <parent link="${prefix}PSM_ECM_pitch_top_link"/>
       <child  link="${prefix}PSM_RCM_link"/>
       <axis xyz="0 0 0"/>

File: urdf/Si/psm_base.urdf.xacro (robot description, xacro)
@@ -288,5 +288,5 @@
     <link name="${prefix}tool_parent"/>
     <joint
-        name="${prefix}outer_insertion_ref"
+        name="${prefix}insertion_ref"
         type="fixed">
       <origin

File: urdf/Virtual/PSM_base_virtual.urdf.xacro (robot description, xacro)
@@ -7,6 +7,6 @@
     This is sufficient for simulation when only the instrument matters.
     DOF layout (same joint names as full model — ROS-compatible):
-      Joint 1: outer_yaw   (revolute  z, ±π/2)
-      Joint 2: outer_pitch (revolute  y, ±π/4)
+      Joint 1: yaw   (revolute  z, ±π/2)
+      Joint 2: pitch (revolute  y, ±π/4)
       Joint 3: insertion   (prismatic z,  0–0.240 m)
     All three links share a small but non-zero inertia so physics
@@ -34,7 +34,7 @@
     <!-- RCM frame link — not a DOF, just a named coordinate frame -->
     <link name="${prefix}PSM_RCM_link"/>
-    <!-- ── Joint 1: outer_yaw ───────────────────────────────────────────── -->
+    <!-- ── Joint 1: yaw ───────────────────────────────────────────── -->
     <!--   Revolute about z at the RCM. Models the yaw of the PSM arm.      -->
-    <joint name="outer_yaw" type="revolute">
+    <joint name="yaw" type="revolute">
       <parent link="${prefix}PSM_RCM_link"/>
       <child  link="${prefix}PSM_RCM_yaw_link"/>
@@ -52,7 +52,7 @@
       </inertial>
     </link>
-    <!-- ── Joint 2: outer_pitch ─────────────────────────────────────────── -->
+    <!-- ── Joint 2: pitch ─────────────────────────────────────────── -->
     <!--   Revolute about y at the RCM. Models the pitch of the PSM arm.    -->
-    <joint name="outer_pitch" type="revolute">
+    <joint name="pitch" type="revolute">
       <parent link="${prefix}PSM_RCM_yaw_link"/>
       <child  link="${prefix}PSM_RCM_pitch_link"/>
