Commit message: Rename ECM_outer_yaw mesh to ECM_yaw to match sawIntuitiveResearchKit naming

File: urdf/Classic/ecm_base.urdf.xacro (robot description, xacro)
@@ -40,14 +40,14 @@
         <geometry>
           <mesh
-            filename="package://dvrk_model/meshes/Classic/ECM/ECM_outer_yaw.stl" />
-        </geometry>
-      </visual>
-      <collision>
-        <origin
-          xyz="0 0 0"
-          rpy="0 0 0" />
-        <geometry>
-          <mesh
-            filename="package://dvrk_model/meshes/Classic/ECM/ECM_outer_yaw.stl" />
+            filename="package://dvrk_model/meshes/Classic/ECM/ECM_yaw.stl" />
+        </geometry>
+      </visual>
+      <collision>
+        <origin
+          xyz="0 0 0"
+          rpy="0 0 0" />
+        <geometry>
+          <mesh
+            filename="package://dvrk_model/meshes/Classic/ECM/ECM_yaw.stl" />
         </geometry>
       </collision>
