Commit message: renaming instruments

File: urdf/Classic/PSM1.urdf.xacro (robot description, xacro)
@@ -3,8 +3,8 @@
   <!--
     Classic PSM1 entry point.
-    arg tool_model: last 6 digits of instrument model number (default: 400006)
+    arg instrument: last 6 digits of instrument model number (default: 400006)
     arm placed at a typical setup position; adjust xyz/rpy for your rig.
   -->
-  <xacro:arg name="tool_model" default="400006"/>
+  <xacro:arg name="instrument" default="400006"/>
   <xacro:include filename="$(find dvrk_model)/urdf/Classic/PSM_base.urdf.xacro"/>
   <xacro:include filename="$(find dvrk_model)/urdf/common/PSM_instrument.urdf.xacro"/>
@@ -12,7 +12,7 @@
   <xacro:PSM_base prefix="PSM1_"
                   parent_link="world"
-                  xyz="-0.25 0.0 0.5" rpy="0.0 0.0 ${pi}"/>
+                  xyz="-0.25 0.0 0.5" rpy="0.0 0.0 ${PI}"/>
   <xacro:PSM_instrument prefix="PSM1_"
                         parent_link="PSM1_PSM_tool_parent_link"
-                        tool_model="$(arg tool_model)"/>
+                        instrument="$(arg instrument)"/>
 </robot>

File: urdf/Classic/PSM2.urdf.xacro (robot description, xacro)
@@ -1,5 +1,5 @@
 <?xml version="1.0" ?>
 <robot name="PSM2" xmlns:xacro="http://www.ros.org/wiki/xacro">
-  <xacro:arg name="tool_model" default="400049"/>
+  <xacro:arg name="instrument" default="400049"/>
   <xacro:include filename="$(find dvrk_model)/urdf/Classic/PSM_base.urdf.xacro"/>
   <xacro:include filename="$(find dvrk_model)/urdf/common/PSM_instrument.urdf.xacro"/>
@@ -7,7 +7,7 @@
   <xacro:PSM_base prefix="PSM2_"
                   parent_link="world"
-                  xyz="-0.25 0.0 0.5" rpy="0.0 0.0 ${pi}"/>
+                  xyz="-0.25 0.0 0.5" rpy="0.0 0.0 ${PI}"/>
   <xacro:PSM_instrument prefix="PSM2_"
                         parent_link="PSM2_PSM_tool_parent_link"
-                        tool_model="$(arg tool_model)"/>
+                        instrument="$(arg instrument)"/>
 </robot>

File: urdf/Classic/PSM3.urdf.xacro (robot description, xacro)
@@ -1,5 +1,5 @@
 <?xml version="1.0" ?>
 <robot name="PSM3" xmlns:xacro="http://www.ros.org/wiki/xacro">
-  <xacro:arg name="tool_model" default="400049"/>
+  <xacro:arg name="instrument" default="400049"/>
   <xacro:include filename="$(find dvrk_model)/urdf/Classic/PSM_base.urdf.xacro"/>
   <xacro:include filename="$(find dvrk_model)/urdf/common/PSM_instrument.urdf.xacro"/>
@@ -7,7 +7,7 @@
   <xacro:PSM_base prefix="PSM3_"
                   parent_link="world"
-                  xyz="0.50 0.0 0.5" rpy="0.0 0.0 ${-pi}"/>
+                  xyz="0.50 0.0 0.5" rpy="0.0 0.0 ${-PI}"/>
   <xacro:PSM_instrument prefix="PSM3_"
                         parent_link="PSM3_PSM_tool_parent_link"
-                        tool_model="$(arg tool_model)"/>
+                        instrument="$(arg instrument)"/>
 </robot>

File: urdf/Si/PSM1.urdf.xacro (robot description, xacro)
@@ -3,7 +3,7 @@
   <!--
     Si PSM1 entry point.
-    arg tool_model: last 6 digits of instrument model number (default: 420006)
+    arg instrument: last 6 digits of instrument model number (default: 420006)
   -->
-  <xacro:arg name="tool_model" default="420006"/>
+  <xacro:arg name="instrument" default="420006"/>
   <xacro:include filename="$(find dvrk_model)/urdf/Si/PSM_base.urdf.xacro"/>
   <xacro:include filename="$(find dvrk_model)/urdf/common/PSM_instrument.urdf.xacro"/>
@@ -13,4 +13,4 @@
   <xacro:PSM_instrument prefix="PSM1_"
                         parent_link="PSM1_PSM_tool_parent_link"
-                        tool_model="$(arg tool_model)"/>
+                        instrument="$(arg instrument)"/>
 </robot>

File: urdf/Si/PSM2.urdf.xacro (robot description, xacro)
@@ -1,5 +1,5 @@
 <?xml version="1.0" ?>
 <robot name="PSM2" xmlns:xacro="http://www.ros.org/wiki/xacro">
-  <xacro:arg name="tool_model" default="420006"/>
+  <xacro:arg name="instrument" default="420006"/>
   <xacro:include filename="$(find dvrk_model)/urdf/Si/PSM_base.urdf.xacro"/>
   <xacro:include filename="$(find dvrk_model)/urdf/common/PSM_instrument.urdf.xacro"/>
@@ -9,4 +9,4 @@
   <xacro:PSM_instrument prefix="PSM2_"
                         parent_link="PSM2_PSM_tool_parent_link"
-                        tool_model="$(arg tool_model)"/>
+                        instrument="$(arg instrument)"/>
 </robot>

File: urdf/Si/PSM3.urdf.xacro (robot description, xacro)
@@ -1,5 +1,5 @@
 <?xml version="1.0" ?>
 <robot name="PSM3" xmlns:xacro="http://www.ros.org/wiki/xacro">
-  <xacro:arg name="tool_model" default="420006"/>
+  <xacro:arg name="instrument" default="420006"/>
   <xacro:include filename="$(find dvrk_model)/urdf/Si/PSM_base.urdf.xacro"/>
   <xacro:include filename="$(find dvrk_model)/urdf/common/PSM_instrument.urdf.xacro"/>
@@ -9,4 +9,4 @@
   <xacro:PSM_instrument prefix="PSM3_"
                         parent_link="PSM3_PSM_tool_parent_link"
-                        tool_model="$(arg tool_model)"/>
+                        instrument="$(arg instrument)"/>
 </robot>

File: urdf/Virtual/PSM1.urdf.xacro (robot description, xacro)
@@ -4,10 +4,10 @@
     Virtual PSM1 entry point — simulator variant.
     args:
-      tool_model   — instrument model number (default: 420006 = Si large needle driver)
+      instrument   — instrument model number (default: 420006 = Si large needle driver)
       shaft_length — shaft length in metres  (0.4162 Classic, 0.4670 Si)
       rcm_xyz      — trocar position in world frame
       rcm_rpy      — trocar orientation in world frame
   -->
-  <xacro:arg name="tool_model"   default="420006"/>
+  <xacro:arg name="instrument"   default="420006"/>
   <xacro:arg name="rcm_xyz"      default="0 0 0"/>
   <xacro:arg name="rcm_rpy"      default="0 0 0"/>
@@ -22,4 +22,4 @@
   <xacro:PSM_instrument prefix="PSM1_"
                         parent_link="PSM1_PSM_tool_parent_link"
-                        tool_model="$(arg tool_model)"/>
+                        instrument="$(arg instrument)"/>
 </robot>

File: urdf/Virtual/PSM2.urdf.xacro (robot description, xacro)
@@ -1,5 +1,5 @@
 <?xml version="1.0" ?>
 <robot name="PSM2" xmlns:xacro="http://www.ros.org/wiki/xacro">
-  <xacro:arg name="tool_model"   default="420006"/>
+  <xacro:arg name="instrument"   default="420006"/>
   <xacro:arg name="rcm_xyz"      default="0 0 0"/>
   <xacro:arg name="rcm_rpy"      default="0 0 0"/>
@@ -12,4 +12,4 @@
   <xacro:PSM_instrument prefix="PSM2_"
                         parent_link="PSM2_PSM_tool_parent_link"
-                        tool_model="$(arg tool_model)"/>
+                        instrument="$(arg instrument)"/>
 </robot>

File: urdf/Virtual/PSM3.urdf.xacro (robot description, xacro)
@@ -1,5 +1,5 @@
 <?xml version="1.0" ?>
 <robot name="PSM3" xmlns:xacro="http://www.ros.org/wiki/xacro">
-  <xacro:arg name="tool_model"   default="420006"/>
+  <xacro:arg name="instrument"   default="420006"/>
   <xacro:arg name="rcm_xyz"      default="0 0 0"/>
   <xacro:arg name="rcm_rpy"      default="0 0 0"/>
@@ -12,4 +12,4 @@
   <xacro:PSM_instrument prefix="PSM3_"
                         parent_link="PSM3_PSM_tool_parent_link"
-                        tool_model="$(arg tool_model)"/>
+                        instrument="$(arg instrument)"/>
 </robot>

File: urdf/common/PSM_instrument.urdf.xacro (robot description, xacro)
@@ -14,5 +14,5 @@
       parent_link   — must be ${prefix}PSM_tool_parent_link
       shaft_length  — D parameter of roll joint (Classic: 0.4162, Si: 0.4670)
-      tool_model    — last 6 digits of instrument model number (e.g. "420006")
+      instrument    — last 6 digits of instrument model number (e.g. "420006")
                       used to select the correct PSM_tip_XXX macro
   -->
@@ -20,7 +20,7 @@
   <xacro:include filename="$(find dvrk_model)/urdf/common/PSM_tips.urdf.xacro"/>
   <xacro:macro name="PSM_instrument"
-               params="prefix parent_link tool_model">
+               params="prefix parent_link instrument">
     <!-- Detect if this is an Si generation instrument (42xxxx) -->
-    <xacro:property name="is_si" value="${str(tool_model).startswith('42')}"/>
+    <xacro:property name="is_si" value="${str(instrument).startswith('42')}"/>
     <!-- Dynamically select the correct shaft length based on generation -->
     <xacro:property name="shaft_length" value="${0.53559 if is_si else 0.4162}"/>
@@ -145,5 +145,5 @@
     </link>
     <!--
-      Tip dispatch: select the correct wrist+jaw macro by tool_model.
+      Tip dispatch: select the correct wrist+jaw macro by instrument.
       Convention: last 3 digits of the model number identify the tip family.
         006 → standard SCA wrist (most instruments, A=0.0091)
@@ -153,24 +153,24 @@
         183 → cautery / no-jaw tools
     -->
-    <xacro:if value="${str(tool_model) == '420006' or str(tool_model) == '400006' or
-                      str(tool_model) == '420036' or str(tool_model) == '400036' or
-                      str(tool_model) == '420093' or str(tool_model) == '400093' or
-                      str(tool_model) == '420168' or str(tool_model) == '400168'}">
+    <xacro:if value="${str(instrument) == '420006' or str(instrument) == '400006' or
+                      str(instrument) == '420036' or str(instrument) == '400036' or
+                      str(instrument) == '420093' or str(instrument) == '400093' or
+                      str(instrument) == '420168' or str(instrument) == '400168'}">
       <xacro:PSM_tip_006 prefix="${prefix}"
                          parent_link="${prefix}PSM_wrist_shaft_link"/>
     </xacro:if>
-    <xacro:if value="${str(tool_model) == '420049' or str(tool_model) == '400049'}">
+    <xacro:if value="${str(instrument) == '420049' or str(instrument) == '400049'}">
       <xacro:PSM_tip_049 prefix="${prefix}"
                          parent_link="${prefix}PSM_wrist_shaft_link"/>
     </xacro:if>
-    <xacro:if value="${str(tool_model) == '420172' or str(tool_model) == '400172'}">
+    <xacro:if value="${str(instrument) == '420172' or str(instrument) == '400172'}">
       <xacro:PSM_tip_172 prefix="${prefix}"
                          parent_link="${prefix}PSM_wrist_shaft_link"/>
     </xacro:if>
-    <xacro:if value="${str(tool_model) == '400117'}">
+    <xacro:if value="${str(instrument) == '400117'}">
       <xacro:PSM_tip_117 prefix="${prefix}"
                          parent_link="${prefix}PSM_wrist_shaft_link"/>
     </xacro:if>
-    <xacro:if value="${str(tool_model) == 'SF0826001'}">
+    <xacro:if value="${str(instrument) == 'SF0826001'}">
       <xacro:PSM_tip_ECM prefix="${prefix}"
                          parent_link="${prefix}PSM_wrist_shaft_link"/>

File: urdf/common/PSM_tips.urdf.xacro (robot description, xacro)
@@ -102,5 +102,5 @@
       <parent link="${prefix}PSM_tip_006_shaft_link"/>
       <child  link="${prefix}PSM_tool_tip_link"/>
-      <origin rpy="0 ${pi/2} ${pi/2}" xyz="0 0.0102 0"/>
+      <origin rpy="0 ${PI/2} ${PI/2}" xyz="0 0.0102 0"/>
     </joint>
     <link name="${prefix}PSM_tool_tip_link"/>
@@ -280,5 +280,5 @@
       <parent link="${prefix}PSM_tip_172_shaft_link"/>
       <child  link="${prefix}PSM_tool_tip_link"/>
-      <origin rpy="0 ${pi/2} ${pi/2}" xyz="0 0.0107 0"/>
+      <origin rpy="0 ${PI/2} ${PI/2}" xyz="0 0.0107 0"/>
     </joint>
     <link name="${prefix}PSM_tool_tip_link"/>

Commit message: Drop PSM_ prefix from base macros (base, base_virtual); keep filenames and meshes

File: urdf/Classic/PSM1.urdf.xacro (robot description, xacro)
@@ -10,5 +10,5 @@
   <xacro:include filename="$(find dvrk_model)/urdf/common/PSM_instrument.urdf.xacro"/>
   <link name="world"/>
-  <xacro:PSM_base prefix="PSM1_"
+  <xacro:base prefix="PSM1_"
                   parent_link="world"
                   xyz="-0.25 0.0 0.5" rpy="0.0 0.0 ${PI}"/>

File: urdf/Classic/PSM2.urdf.xacro (robot description, xacro)
@@ -5,5 +5,5 @@
   <xacro:include filename="$(find dvrk_model)/urdf/common/PSM_instrument.urdf.xacro"/>
   <link name="world"/>
-  <xacro:PSM_base prefix="PSM2_"
+  <xacro:base prefix="PSM2_"
                   parent_link="world"
                   xyz="-0.25 0.0 0.5" rpy="0.0 0.0 ${PI}"/>

File: urdf/Classic/PSM3.urdf.xacro (robot description, xacro)
@@ -5,5 +5,5 @@
   <xacro:include filename="$(find dvrk_model)/urdf/common/PSM_instrument.urdf.xacro"/>
   <link name="world"/>
-  <xacro:PSM_base prefix="PSM3_"
+  <xacro:base prefix="PSM3_"
                   parent_link="world"
                   xyz="0.50 0.0 0.5" rpy="0.0 0.0 ${-PI}"/>

File: urdf/Si/ECM.urdf.xacro (robot description, xacro)
@@ -4,5 +4,5 @@
   <xacro:include filename="$(find dvrk_model)/urdf/common/PSM_instrument.urdf.xacro"/>
   <link name="world"/>
-  <xacro:PSM_base prefix="ECM_"
+  <xacro:base prefix="ECM_"
                   parent_link="world"/>
   <xacro:PSM_instrument prefix="ECM_"

File: urdf/Si/PSM1.urdf.xacro (robot description, xacro)
@@ -9,5 +9,5 @@
   <xacro:include filename="$(find dvrk_model)/urdf/common/PSM_instrument.urdf.xacro"/>
   <link name="world"/>
-  <xacro:PSM_base prefix="PSM1_"
+  <xacro:base prefix="PSM1_"
                   parent_link="world"/>
   <xacro:PSM_instrument prefix="PSM1_"

File: urdf/Si/PSM2.urdf.xacro (robot description, xacro)
@@ -5,5 +5,5 @@
   <xacro:include filename="$(find dvrk_model)/urdf/common/PSM_instrument.urdf.xacro"/>
   <link name="world"/>
-  <xacro:PSM_base prefix="PSM2_"
+  <xacro:base prefix="PSM2_"
                   parent_link="world"/>
   <xacro:PSM_instrument prefix="PSM2_"

File: urdf/Si/PSM3.urdf.xacro (robot description, xacro)
@@ -5,5 +5,5 @@
   <xacro:include filename="$(find dvrk_model)/urdf/common/PSM_instrument.urdf.xacro"/>
   <link name="world"/>
-  <xacro:PSM_base prefix="PSM3_"
+  <xacro:base prefix="PSM3_"
                   parent_link="world"/>
   <xacro:PSM_instrument prefix="PSM3_"

File: urdf/Virtual/PSM1.urdf.xacro (robot description, xacro)
@@ -16,5 +16,5 @@
   <link name="world"/>
   <!-- 3 virtual DOFs at the trocar — no arm geometry -->
-  <xacro:PSM_base_virtual prefix="PSM1_"
+  <xacro:base_virtual prefix="PSM1_"
                           rcm_xyz="$(arg rcm_xyz)"
                           rcm_rpy="$(arg rcm_rpy)"/>

File: urdf/Virtual/PSM2.urdf.xacro (robot description, xacro)
@@ -7,5 +7,5 @@
   <xacro:include filename="$(find dvrk_model)/urdf/common/PSM_instrument.urdf.xacro"/>
   <link name="world"/>
-  <xacro:PSM_base_virtual prefix="PSM2_"
+  <xacro:base_virtual prefix="PSM2_"
                           rcm_xyz="$(arg rcm_xyz)"
                           rcm_rpy="$(arg rcm_rpy)"/>

File: urdf/Virtual/PSM3.urdf.xacro (robot description, xacro)
@@ -7,5 +7,5 @@
   <xacro:include filename="$(find dvrk_model)/urdf/common/PSM_instrument.urdf.xacro"/>
   <link name="world"/>
-  <xacro:PSM_base_virtual prefix="PSM3_"
+  <xacro:base_virtual prefix="PSM3_"
                           rcm_xyz="$(arg rcm_xyz)"
                           rcm_rpy="$(arg rcm_rpy)"/>

File: urdf/Virtual/PSM_base_virtual.urdf.xacro (robot description, xacro)
@@ -22,5 +22,5 @@
   <xacro:property name="virtual_mass"  value="0.001"/>  <!-- 1 gram -->
   <xacro:property name="virtual_inertia" value="1e-6"/>  <!-- 1e-6 kg·m² -->
-  <xacro:macro name="PSM_base_virtual"
+  <xacro:macro name="base_virtual"
                params="prefix
                        rcm_xyz:='0 0 0'
