Commit message: fix mesh file references

File: urdf/Classic/PSM1.urdf.xacro (robot description, xacro)
@@ -8,7 +8,7 @@
   <xacro:arg name="instrument" default="400006"/>
   <xacro:arg name="parent_link_" default="world"/>
-  <xacro:property name="parent_link" default="$(arg parent_link_)"/>
+  <xacro:property name="parent_link" value="$(arg parent_link_)"/>
   <xacro:include filename="$(find dvrk_model)/urdf/Classic/PSM_base_macros.urdf.xacro"/>
-  <xacro:include filename="$(find dvrk_model)/urdf/common/PSM_instrument_macros.urdf.xacro"/>
+  <xacro:include filename="$(find dvrk_model)/urdf/common/PSM_instrument.urdf.xacro"/>
   <link name="${parent_link}"/>
   <xacro:base prefix="PSM1_"

File: urdf/Classic/PSM2.urdf.xacro (robot description, xacro)
@@ -3,7 +3,7 @@
   <xacro:arg name="instrument" default="400049"/>
   <xacro:arg name="parent_link_" default="world"/>
-  <xacro:property name="parent_link" default="$(arg parent_link_)"/>
+  <xacro:property name="parent_link" value="$(arg parent_link_)"/>
   <xacro:include filename="$(find dvrk_model)/urdf/Classic/PSM_base_macros.urdf.xacro"/>
-  <xacro:include filename="$(find dvrk_model)/urdf/common/PSM_instrument_macros.urdf.xacro"/>
+  <xacro:include filename="$(find dvrk_model)/urdf/common/PSM_instrument.urdf.xacro"/>
   <link name="${parent_link}"/>
   <xacro:base prefix="PSM2_"

File: urdf/Classic/PSM3.urdf.xacro (robot description, xacro)
@@ -3,7 +3,7 @@
   <xacro:arg name="instrument" default="400049"/>
   <xacro:arg name="parent_link_" default="world"/>
-  <xacro:property name="parent_link" default="$(arg parent_link_)"/>
+  <xacro:property name="parent_link" value="$(arg parent_link_)"/>
   <xacro:include filename="$(find dvrk_model)/urdf/Classic/PSM_base_macros.urdf.xacro"/>
-  <xacro:include filename="$(find dvrk_model)/urdf/common/PSM_instrument_macros.urdf.xacro"/>
+  <xacro:include filename="$(find dvrk_model)/urdf/common/PSM_instrument.urdf.xacro"/>
   <link name="${parent_link}"/>
   <xacro:base prefix="PSM3_"

File: urdf/Si/ECM.urdf.xacro (robot description, xacro)
@@ -4,5 +4,5 @@
   <xacro:property name="parent_link" default="$(arg parent_link_)"/>
   <xacro:include filename="$(find dvrk_model)/urdf/Si/PSM_base_macros.urdf.xacro"/>
-  <xacro:include filename="$(find dvrk_model)/urdf/common/PSM_instrument_macros.urdf.xacro"/>
+  <xacro:include filename="$(find dvrk_model)/urdf/common/PSM_instrument.urdf.xacro"/>
   <link name="${parent_link}"/>
   <xacro:base prefix="ECM_"

File: urdf/Si/PSM1.urdf.xacro (robot description, xacro)
@@ -7,7 +7,7 @@
   <xacro:arg name="instrument" default="420006"/>
   <xacro:arg name="parent_link_" default="world"/>
-  <xacro:property name="parent_link" default="$(arg parent_link_)"/>
+  <xacro:property name="parent_link" value="$(arg parent_link_)"/>
   <xacro:include filename="$(find dvrk_model)/urdf/Si/PSM_base_macros.urdf.xacro"/>
-  <xacro:include filename="$(find dvrk_model)/urdf/common/PSM_instrument_macros.urdf.xacro"/>
+  <xacro:include filename="$(find dvrk_model)/urdf/common/PSM_instrument.urdf.xacro"/>
   <link name="${parent_link}"/>
   <xacro:base prefix="PSM1_"

File: urdf/Si/PSM2.urdf.xacro (robot description, xacro)
@@ -3,7 +3,7 @@
   <xacro:arg name="instrument" default="420006"/>
   <xacro:arg name="parent_link_" default="world"/>
-  <xacro:property name="parent_link" default="$(arg parent_link_)"/>
+  <xacro:property name="parent_link" value="$(arg parent_link_)"/>
   <xacro:include filename="$(find dvrk_model)/urdf/Si/PSM_base_macros.urdf.xacro"/>
-  <xacro:include filename="$(find dvrk_model)/urdf/common/PSM_instrument_macros.urdf.xacro"/>
+  <xacro:include filename="$(find dvrk_model)/urdf/common/PSM_instrument.urdf.xacro"/>
   <link name="${parent_link}"/>
   <xacro:base prefix="PSM2_"

File: urdf/Si/PSM3.urdf.xacro (robot description, xacro)
@@ -3,7 +3,7 @@
   <xacro:arg name="instrument" default="420006"/>
   <xacro:arg name="parent_link_" default="world"/>
-  <xacro:property name="parent_link" default="$(arg parent_link_)"/>
+  <xacro:property name="parent_link" value="$(arg parent_link_)"/>
   <xacro:include filename="$(find dvrk_model)/urdf/Si/PSM_base_macros.urdf.xacro"/>
-  <xacro:include filename="$(find dvrk_model)/urdf/common/PSM_instrument_macros.urdf.xacro"/>
+  <xacro:include filename="$(find dvrk_model)/urdf/common/PSM_instrument.urdf.xacro"/>
   <link name="${parent_link}"/>
   <xacro:base prefix="PSM3_"

File: urdf/Si/PSM_base_macros.urdf.xacro (robot description, xacro)
@@ -27,5 +27,5 @@
         <origin xyz="0 0 0" rpy="0 0 0"/>
         <geometry>
-          <mesh filename="package://dvrk_model/meshes/Si/USM/USM_base.stl"/>
+          <mesh filename="package://dvrk_model/meshes/arms/Si/USM/USM_base.stl"/>
         </geometry>
         <material name=""><color rgba="0.79216 0.81961 0.93333 1"/></material>
@@ -34,5 +34,5 @@
         <origin xyz="0 0 0" rpy="0 0 0"/>
         <geometry>
-          <mesh filename="package://dvrk_model/meshes/Si/USM/USM_base.stl"/>
+          <mesh filename="package://dvrk_model/meshes/arms/Si/USM/USM_base.stl"/>
         </geometry>
       </collision>
@@ -56,5 +56,5 @@
         <origin xyz="0 0 0" rpy="0 0 0"/>
         <geometry>
-          <mesh filename="package://dvrk_model/meshes/Si/USM/USM_yaw.stl"/>
+          <mesh filename="package://dvrk_model/meshes/arms/Si/USM/USM_yaw.stl"/>
         </geometry>
         <material name=""><color rgba="0.79216 0.81961 0.93333 1"/></material>
@@ -63,5 +63,5 @@
         <origin xyz="0 0 0" rpy="0 0 0"/>
         <geometry>
-          <mesh filename="package://dvrk_model/meshes/Si/USM/USM_yaw.stl"/>
+          <mesh filename="package://dvrk_model/meshes/arms/Si/USM/USM_yaw.stl"/>
         </geometry>
       </collision>
@@ -87,5 +87,5 @@
         <origin xyz="0 0 0" rpy="0 0 0"/>
         <geometry>
-          <mesh filename="package://dvrk_model/meshes/Si/USM/USM_pitch.stl"/>
+          <mesh filename="package://dvrk_model/meshes/arms/Si/USM/USM_pitch.stl"/>
         </geometry>
         <material name=""><color rgba="0.79216 0.81961 0.93333 1"/></material>
@@ -94,5 +94,5 @@
         <origin xyz="0 0 0" rpy="0 0 0"/>
         <geometry>
-          <mesh filename="package://dvrk_model/meshes/Si/USM/USM_pitch.stl"/>
+          <mesh filename="package://dvrk_model/meshes/arms/Si/USM/USM_pitch.stl"/>
         </geometry>
       </collision>
@@ -118,5 +118,5 @@
         <origin xyz="0 0 0" rpy="0 0 0"/>
         <geometry>
-          <mesh filename="package://dvrk_model/meshes/Si/USM/USM_pitch_3.stl"/>
+          <mesh filename="package://dvrk_model/meshes/arms/Si/USM/USM_pitch_3.stl"/>
         </geometry>
         <material name=""><color rgba="0.79216 0.81961 0.93333 1"/></material>
@@ -125,5 +125,5 @@
         <origin xyz="0 0 0" rpy="0 0 0"/>
         <geometry>
-          <mesh filename="package://dvrk_model/meshes/Si/USM/USM_pitch_3.stl"/>
+          <mesh filename="package://dvrk_model/meshes/arms/Si/USM/USM_pitch_3.stl"/>
         </geometry>
       </collision>
@@ -149,5 +149,5 @@
         <origin xyz="0 0 0" rpy="0 0 0"/>
         <geometry>
-          <mesh filename="package://dvrk_model/meshes/Si/USM/USM_pitch_4.stl"/>
+          <mesh filename="package://dvrk_model/meshes/arms/Si/USM/USM_pitch_4.stl"/>
         </geometry>
         <material name=""><color rgba="0.79216 0.81961 0.93333 1"/></material>
@@ -156,5 +156,5 @@
         <origin xyz="0 0 0" rpy="0 0 0"/>
         <geometry>
-          <mesh filename="package://dvrk_model/meshes/Si/USM/USM_pitch_4.stl"/>
+          <mesh filename="package://dvrk_model/meshes/arms/Si/USM/USM_pitch_4.stl"/>
         </geometry>
       </collision>

File: urdf/Virtual/PSM1.urdf.xacro (robot description, xacro)
@@ -13,5 +13,5 @@
   <xacro:arg name="rcm_rpy"      default="0 0 0"/>
   <xacro:include filename="$(find dvrk_model)/urdf/Virtual/PSM_base_virtual_macros.urdf.xacro"/>
-  <xacro:include filename="$(find dvrk_model)/urdf/common/PSM_instrument_macros.urdf.xacro"/>
+  <xacro:include filename="$(find dvrk_model)/urdf/common/PSM_instrument.urdf.xacro"/>
   <link name="world"/>
   <!-- 3 virtual DOFs at the trocar — no arm geometry -->

File: urdf/Virtual/PSM2.urdf.xacro (robot description, xacro)
@@ -5,5 +5,5 @@
   <xacro:arg name="rcm_rpy"      default="0 0 0"/>
   <xacro:include filename="$(find dvrk_model)/urdf/Virtual/PSM_base_virtual_macros.urdf.xacro"/>
-  <xacro:include filename="$(find dvrk_model)/urdf/common/PSM_instrument_macros.urdf.xacro"/>
+  <xacro:include filename="$(find dvrk_model)/urdf/common/PSM_instrument.urdf.xacro"/>
   <link name="world"/>
   <xacro:base_virtual prefix="PSM2_"

File: urdf/Virtual/PSM3.urdf.xacro (robot description, xacro)
@@ -5,5 +5,5 @@
   <xacro:arg name="rcm_rpy"      default="0 0 0"/>
   <xacro:include filename="$(find dvrk_model)/urdf/Virtual/PSM_base_virtual_macros.urdf.xacro"/>
-  <xacro:include filename="$(find dvrk_model)/urdf/common/PSM_instrument_macros.urdf.xacro"/>
+  <xacro:include filename="$(find dvrk_model)/urdf/common/PSM_instrument.urdf.xacro"/>
   <link name="world"/>
   <xacro:base_virtual prefix="PSM3_"

File: urdf/common/PSM_instrument.urdf.xacro (robot description, xacro)
@@ -18,5 +18,5 @@
   -->
   <xacro:include filename="$(find dvrk_model)/urdf/common.urdf.xacro"/>
-  <xacro:include filename="$(find dvrk_model)/urdf/common/PSM_tips_macros.urdf.xacro"/>
+  <xacro:include filename="$(find dvrk_model)/urdf/common/PSM_tips.urdf.xacro"/>
   <xacro:macro name="PSM_instrument"
                params="prefix parent_link instrument">
