Commit message: Refactor URDF structure and update instrument macros, renamed and refactored the instrument macro from `PSM_instrument` to `instrument` for consistency across the codebase.

File: urdf/Classic/PSM1.urdf.xacro (robot description, xacro)
@@ -10,10 +10,10 @@
   <xacro:property name="parent_link" value="$(arg parent_link_)"/>
   <xacro:include filename="$(find dvrk_model)/urdf/Classic/PSM_base.urdf.xacro"/>
-  <xacro:include filename="$(find dvrk_model)/urdf/common/PSM_instrument.urdf.xacro"/>
+  <xacro:include filename="$(find dvrk_model)/urdf/common/instrument.urdf.xacro"/>
   <link name="${parent_link}"/>
   <xacro:base prefix="PSM1_"
                   parent_link="${parent_link}"
                   xyz="0.0 0.0 0.0" rpy="0.0 0.0 0.0"/>
-  <xacro:PSM_instrument prefix="PSM1_"
+  <xacro:instrument prefix="PSM1_"
                         parent_link="PSM1_adaptor_link"
                         instrument="$(arg instrument)"/>

File: urdf/Classic/PSM2.urdf.xacro (robot description, xacro)
@@ -5,10 +5,10 @@
   <xacro:property name="parent_link" value="$(arg parent_link_)"/>
   <xacro:include filename="$(find dvrk_model)/urdf/Classic/PSM_base.urdf.xacro"/>
-  <xacro:include filename="$(find dvrk_model)/urdf/common/PSM_instrument.urdf.xacro"/>
+  <xacro:include filename="$(find dvrk_model)/urdf/common/instrument.urdf.xacro"/>
   <link name="${parent_link}"/>
   <xacro:base prefix="PSM2_"
                   parent_link="${parent_link}"
                   xyz="0.0 0.0 0.0" rpy="0.0 0.0 0.0"/>
-  <xacro:PSM_instrument prefix="PSM2_"
+  <xacro:instrument prefix="PSM2_"
                         parent_link="PSM2_adaptor_link"
                         instrument="$(arg instrument)"/>

File: urdf/Classic/PSM3.urdf.xacro (robot description, xacro)
@@ -5,10 +5,10 @@
   <xacro:property name="parent_link" value="$(arg parent_link_)"/>
   <xacro:include filename="$(find dvrk_model)/urdf/Classic/PSM_base.urdf.xacro"/>
-  <xacro:include filename="$(find dvrk_model)/urdf/common/PSM_instrument.urdf.xacro"/>
+  <xacro:include filename="$(find dvrk_model)/urdf/common/instrument.urdf.xacro"/>
   <link name="${parent_link}"/>
   <xacro:base prefix="PSM3_"
                   parent_link="${parent_link}"
                   xyz="0.0 0.0 0.0" rpy="0.0 0.0 0.0"/>
-  <xacro:PSM_instrument prefix="PSM3_"
+  <xacro:instrument prefix="PSM3_"
                         parent_link="PSM3_adaptor_link"
                         instrument="$(arg instrument)"/>

File: urdf/Classic/PSM_base.urdf.xacro (robot description, xacro)
@@ -9,5 +9,5 @@
       Joint 3: insertion    (prismatic)
     Macro output: ends at ${prefix}adaptor_link.
-    The instrument macro (PSM_instrument) attaches here and owns roll onward.
+    The instrument macro (instrument) attaches here and owns roll onward.
     Parameters:
       prefix      — arm instance prefix, e.g. "PSM1_"
@@ -163,5 +163,5 @@
     <!--
       link 3: adaptor_link
-      Massless boundary link — handoff point to PSM_instrument.
+      Massless boundary link — handoff point to instrument.
       This is the instrument_base frame from the kinematic JSON: aligned
       with the insertion/roll axis and offset 0.4318 m from the RCM.

File: urdf/Si/PSM1.urdf.xacro (robot description, xacro)
@@ -9,9 +9,9 @@
   <xacro:property name="parent_link" value="$(arg parent_link_)"/>
   <xacro:include filename="$(find dvrk_model)/urdf/Si/PSM_base.urdf.xacro"/>
-  <xacro:include filename="$(find dvrk_model)/urdf/common/PSM_instrument.urdf.xacro"/>
+  <xacro:include filename="$(find dvrk_model)/urdf/common/instrument.urdf.xacro"/>
   <link name="${parent_link}"/>
   <xacro:base prefix="PSM1_"
                   parent_link="${parent_link}"/>
-  <xacro:PSM_instrument prefix="PSM1_"
+  <xacro:instrument prefix="PSM1_"
                         parent_link="PSM1_adaptor_link"
                         instrument="$(arg instrument)"/>

File: urdf/Si/PSM2.urdf.xacro (robot description, xacro)
@@ -5,9 +5,9 @@
   <xacro:property name="parent_link" value="$(arg parent_link_)"/>
   <xacro:include filename="$(find dvrk_model)/urdf/Si/PSM_base.urdf.xacro"/>
-  <xacro:include filename="$(find dvrk_model)/urdf/common/PSM_instrument.urdf.xacro"/>
+  <xacro:include filename="$(find dvrk_model)/urdf/common/instrument.urdf.xacro"/>
   <link name="${parent_link}"/>
   <xacro:base prefix="PSM2_"
                   parent_link="${parent_link}"/>
-  <xacro:PSM_instrument prefix="PSM2_"
+  <xacro:instrument prefix="PSM2_"
                         parent_link="PSM2_adaptor_link"
                         instrument="$(arg instrument)"/>

File: urdf/Si/PSM3.urdf.xacro (robot description, xacro)
@@ -5,9 +5,9 @@
   <xacro:property name="parent_link" value="$(arg parent_link_)"/>
   <xacro:include filename="$(find dvrk_model)/urdf/Si/PSM_base.urdf.xacro"/>
-  <xacro:include filename="$(find dvrk_model)/urdf/common/PSM_instrument.urdf.xacro"/>
+  <xacro:include filename="$(find dvrk_model)/urdf/common/instrument.urdf.xacro"/>
   <link name="${parent_link}"/>
   <xacro:base prefix="PSM3_"
                   parent_link="${parent_link}"/>
-  <xacro:PSM_instrument prefix="PSM3_"
+  <xacro:instrument prefix="PSM3_"
                         parent_link="PSM3_adaptor_link"
                         instrument="$(arg instrument)"/>

File: urdf/Si/PSM_base.urdf.xacro (robot description, xacro)
@@ -9,5 +9,5 @@
       Joint 3: insertion (prismatic)
     Macro output: ends at ${prefix}adaptor_link.
-    PSM_instrument attaches here and owns roll onward.
+    instrument attaches here and owns roll onward.
     Inertial data retained from original Si CAD export.
   -->
@@ -192,6 +192,6 @@
     </joint>
     <!--
-      adaptor_link — boundary link; PSM_instrument attaches here.
-      No geometry; same name as Classic so PSM_instrument is
+      adaptor_link — boundary link; instrument attaches here.
+      No geometry; same name as Classic so instrument is
       generation-agnostic.
     -->

File: urdf/Virtual/PSM1.urdf.xacro (robot description, xacro)
@@ -5,5 +5,5 @@
     args:
       instrument   — instrument model number (default: 420006 = Si large needle driver)
-                     shaft/roll geometry is selected in common/PSM_instrument
+                     shaft/roll geometry is selected in common/instrument
                      using the instrument code (Classic 40xxxx, Si 42xxxx)
       rcm_xyz      — trocar position in world frame
@@ -16,5 +16,5 @@
   <xacro:arg name="rcm_rpy"      default="0 0 0"/>
   <xacro:include filename="$(find dvrk_model)/urdf/Virtual/PSM_base_virtual.urdf.xacro"/>
-  <xacro:include filename="$(find dvrk_model)/urdf/common/PSM_instrument.urdf.xacro"/>
+  <xacro:include filename="$(find dvrk_model)/urdf/common/instrument.urdf.xacro"/>
   <link name="world"/>
   <!-- 3 virtual DOFs at the trocar — no arm geometry -->
@@ -24,5 +24,5 @@
                           rcm_rpy="$(arg rcm_rpy)"/>
   <!-- Instrument: identical to Classic/Si — attaches at PSM_adaptor_link -->
-  <xacro:PSM_instrument prefix="PSM1_"
+  <xacro:instrument prefix="PSM1_"
                         parent_link="PSM1_adaptor_link"
                         instrument="$(arg instrument)"/>

File: urdf/Virtual/PSM2.urdf.xacro (robot description, xacro)
@@ -6,5 +6,5 @@
   <xacro:arg name="rcm_rpy"      default="0 0 0"/>
   <xacro:include filename="$(find dvrk_model)/urdf/Virtual/PSM_base_virtual.urdf.xacro"/>
-  <xacro:include filename="$(find dvrk_model)/urdf/common/PSM_instrument.urdf.xacro"/>
+  <xacro:include filename="$(find dvrk_model)/urdf/common/instrument.urdf.xacro"/>
   <link name="world"/>
   <xacro:base_virtual prefix="PSM2_"
@@ -12,5 +12,5 @@
                           rcm_xyz="$(arg rcm_xyz)"
                           rcm_rpy="$(arg rcm_rpy)"/>
-  <xacro:PSM_instrument prefix="PSM2_"
+  <xacro:instrument prefix="PSM2_"
                         parent_link="PSM2_adaptor_link"
                         instrument="$(arg instrument)"/>

File: urdf/Virtual/PSM3.urdf.xacro (robot description, xacro)
@@ -6,5 +6,5 @@
   <xacro:arg name="rcm_rpy"      default="0 0 0"/>
   <xacro:include filename="$(find dvrk_model)/urdf/Virtual/PSM_base_virtual.urdf.xacro"/>
-  <xacro:include filename="$(find dvrk_model)/urdf/common/PSM_instrument.urdf.xacro"/>
+  <xacro:include filename="$(find dvrk_model)/urdf/common/instrument.urdf.xacro"/>
   <link name="world"/>
   <xacro:base_virtual prefix="PSM3_"
@@ -12,5 +12,5 @@
                           rcm_xyz="$(arg rcm_xyz)"
                           rcm_rpy="$(arg rcm_rpy)"/>
-  <xacro:PSM_instrument prefix="PSM3_"
+  <xacro:instrument prefix="PSM3_"
                         parent_link="PSM3_adaptor_link"
                         instrument="$(arg instrument)"/>

File: urdf/Virtual/PSM_base_virtual.urdf.xacro (robot description, xacro)
@@ -14,5 +14,5 @@
     simulators (Gazebo, Isaac) can integrate without singularities.
     Output: ends at ${prefix}adaptor_link — identical to the
-    full Classic/Si base so PSM_instrument attaches without modification.
+    full Classic/Si base so instrument attaches without modification.
     Parameters:
       prefix    — arm instance prefix, e.g. "PSM1_"
@@ -77,5 +77,5 @@
     <!--   Prismatic along the PSM DH insertion axis. Models insertion depth. -->
     <!--   adaptor_link serves as the insertion child AND the handoff link -->
-    <!--   to PSM_instrument (same name as in Classic/Si base).            -->
+    <!--   to instrument (same name as in Classic/Si base).            -->
     <joint name="insertion" type="prismatic">
       <parent link="${prefix}RCM_pitch_link"/>
@@ -88,5 +88,5 @@
     <!--
       adaptor_link — identical name to Classic/Si boundary link.
-      PSM_instrument attaches here; no change needed for any generation.
+      instrument attaches here; no change needed for any generation.
     -->
     <link name="${prefix}adaptor_link">

File: urdf/common/instrument.urdf.xacro (robot description, xacro)
@@ -1,6 +1,6 @@
 <?xml version="1.0" encoding="utf-8"?>
-<robot name="dvrk_psm_instrument" xmlns:xacro="http://www.ros.org/wiki/xacro">
+<robot name="dvrk_instrument" xmlns:xacro="http://www.ros.org/wiki/xacro">
   <!--
-    PSM instrument macro — generation-agnostic.
+    Instrument macro — generation-agnostic.
     Attaches to ${parent_link} (= ${prefix}adaptor_link from the PSM base).
     DOF layout:
@@ -17,43 +17,43 @@
   -->
   <xacro:include filename="$(find dvrk_model)/urdf/common.urdf.xacro"/>
-  <xacro:include filename="$(find dvrk_model)/urdf/common/psm_tools/PSM_housing.urdf.xacro"/>
-  <xacro:include filename="$(find dvrk_model)/urdf/common/psm_tools/PSM_roll.urdf.xacro"/>
-  <xacro:include filename="$(find dvrk_model)/urdf/common/psm_tools/wrist/PSM_0091m_wrist.urdf.xacro"/>
-  <xacro:include filename="$(find dvrk_model)/urdf/common/psm_tools/tip/PSM_006_tip.urdf.xacro"/>
-  <xacro:include filename="$(find dvrk_model)/urdf/common/psm_tools/tip/PSM_049_tip.urdf.xacro"/>
-  <xacro:macro name="PSM_instrument_variant"
+  <xacro:include filename="$(find dvrk_model)/urdf/common/instruments/housing.urdf.xacro"/>
+  <xacro:include filename="$(find dvrk_model)/urdf/common/instruments/roll.urdf.xacro"/>
+  <xacro:include filename="$(find dvrk_model)/urdf/common/instruments/wrist/0091m_wrist.urdf.xacro"/>
+  <xacro:include filename="$(find dvrk_model)/urdf/common/instruments/tip/006_tip.urdf.xacro"/>
+  <xacro:include filename="$(find dvrk_model)/urdf/common/instruments/tip/049_tip.urdf.xacro"/>
+  <xacro:macro name="instrument_variant"
                params="prefix parent_link generation roll_origin wrist_parent_link wrist_0091m_variant tip_style is_si:=false">
-    <xacro:PSM_instrument_housing prefix="${prefix}"
+    <xacro:instrument_housing prefix="${prefix}"
                                   parent_link="${parent_link}"
                                   housing_family="${generation}"/>
     <xacro:if value="${generation == 'Si'}">
-      <xacro:PSM_instrument_si_roll_shaft prefix="${prefix}"
+      <xacro:instrument_si_roll_shaft prefix="${prefix}"
                                           parent_link="${parent_link}"
                                           roll_origin="${roll_origin}"/>
     </xacro:if>
     <xacro:if value="${generation == 'Classic'}">
-      <xacro:PSM_instrument_classic_roll_shaft prefix="${prefix}"
+      <xacro:instrument_classic_roll_shaft prefix="${prefix}"
                                                parent_link="${parent_link}"
                                                roll_origin="${roll_origin}"/>
     </xacro:if>
-    <xacro:PSM_wrist_0091m prefix="${prefix}"
+    <xacro:wrist_0091m prefix="${prefix}"
                            parent_link="${wrist_parent_link}"
                            wrist_0091m_variant="${wrist_0091m_variant}"
                            is_si="${is_si}"/>
     <xacro:if value="${tip_style == '006'}">
-      <xacro:PSM_tool_tip_006 prefix="${prefix}"
+      <xacro:tool_tip_006 prefix="${prefix}"
                               parent_link="${prefix}wrist_yaw_0091m_link"
                               is_si="${is_si}"/>
     </xacro:if>
     <xacro:if value="${tip_style == '049'}">
-      <xacro:PSM_tool_tip_049 prefix="${prefix}"
+      <xacro:tool_tip_049 prefix="${prefix}"
                               parent_link="${prefix}wrist_yaw_0091m_link"/>
     </xacro:if>
   </xacro:macro>
-  <xacro:macro name="PSM_instrument"
+  <xacro:macro name="instrument"
                params="prefix parent_link instrument">
     <!-- 420006: Si 006 -->
     <xacro:if value="${str(instrument) == '420006'}">
-      <xacro:PSM_instrument_variant prefix="${prefix}"
+      <xacro:instrument_variant prefix="${prefix}"
                                     parent_link="${parent_link}"
                                     generation="Si"
@@ -66,5 +66,5 @@
     <!-- 400006: Classic 006 -->
     <xacro:if value="${str(instrument) == '400006'}">
-      <xacro:PSM_instrument_variant prefix="${prefix}"
+      <xacro:instrument_variant prefix="${prefix}"
                                     parent_link="${parent_link}"
                                     generation="Classic"
@@ -77,5 +77,5 @@
     <!-- 400049: Classic 049 -->
     <xacro:if value="${str(instrument) == '400049'}">
-      <xacro:PSM_instrument_variant prefix="${prefix}"
+      <xacro:instrument_variant prefix="${prefix}"
                                     parent_link="${parent_link}"
                                     generation="Classic"

File: urdf/common/instruments/housing.urdf.xacro (robot description, xacro)
@@ -1,6 +1,6 @@
 <?xml version="1.0" encoding="utf-8"?>
-<robot name="dvrk_psm_housing" xmlns:xacro="http://www.ros.org/wiki/xacro">
+<robot name="dvrk_instrument_housing" xmlns:xacro="http://www.ros.org/wiki/xacro">
   <xacro:include filename="$(find dvrk_model)/urdf/common.urdf.xacro"/>
-  <xacro:macro name="PSM_instrument_housing"
+  <xacro:macro name="instrument_housing"
                params="prefix parent_link housing_family:=Classic">
     <xacro:property name="is_si_housing" value="${housing_family == 'Si'}"/>

File: urdf/common/instruments/roll.urdf.xacro (robot description, xacro)
@@ -1,5 +1,5 @@
 <?xml version="1.0" encoding="utf-8"?>
-<robot name="dvrk_psm_roll" xmlns:xacro="http://www.ros.org/wiki/xacro">
-  <xacro:macro name="PSM_instrument_si_roll_shaft"
+<robot name="dvrk_instrument_roll" xmlns:xacro="http://www.ros.org/wiki/xacro">
+  <xacro:macro name="instrument_si_roll_shaft"
                params="prefix parent_link roll_origin">
     <joint name="roll" type="revolute">
@@ -50,5 +50,5 @@
     </link>
   </xacro:macro>
-  <xacro:macro name="PSM_instrument_classic_roll_shaft"
+  <xacro:macro name="instrument_classic_roll_shaft"
                params="prefix parent_link roll_origin">
     <joint name="roll" type="revolute">

File: urdf/common/instruments/tip/006_tip.urdf.xacro (robot description, xacro)
@@ -1,5 +1,5 @@
 <?xml version="1.0" encoding="utf-8"?>
-<robot name="dvrk_psm_006_tip" xmlns:xacro="http://www.ros.org/wiki/xacro">
-  <xacro:macro name="PSM_tool_tip_006" params="prefix parent_link is_si:=false">
+<robot name="dvrk_instrument_006_tip" xmlns:xacro="http://www.ros.org/wiki/xacro">
+  <xacro:macro name="tool_tip_006" params="prefix parent_link is_si:=false">
     <joint name="jaw" type="revolute">
       <parent link="${parent_link}"/>

File: urdf/common/instruments/tip/049_tip.urdf.xacro (robot description, xacro)
@@ -1,5 +1,5 @@
 <?xml version="1.0" encoding="utf-8"?>
-<robot name="dvrk_psm_049_tip" xmlns:xacro="http://www.ros.org/wiki/xacro">
-  <xacro:macro name="PSM_tool_tip_049" params="prefix parent_link">
+<robot name="dvrk_instrument_049_tip" xmlns:xacro="http://www.ros.org/wiki/xacro">
+  <xacro:macro name="tool_tip_049" params="prefix parent_link">
     <joint name="jaw" type="revolute">
       <parent link="${parent_link}"/>

File: urdf/common/instruments/wrist/0091m_wrist.urdf.xacro (robot description, xacro)
@@ -1,5 +1,5 @@
 <?xml version="1.0" encoding="utf-8"?>
-<robot name="dvrk_psm_0091m_wrist" xmlns:xacro="http://www.ros.org/wiki/xacro">
-  <xacro:macro name="PSM_wrist_0091m"
+<robot name="dvrk_instrument_0091m_wrist" xmlns:xacro="http://www.ros.org/wiki/xacro">
+  <xacro:macro name="wrist_0091m"
                params="prefix parent_link wrist_0091m_variant:=sca is_si:=false">
     <!-- 0091m fixes the wrist spacing; the variant stays because SCA and Cadiere use different meshes. -->
