Commit message: Refactor instrument housing and roll URDF files
- Removed the generic housing.urdf.xacro and created specific files for Classic and Si housing: housing_Classic.urdf.xacro and housing_Si.urdf.xacro.
- Deleted the roll.urdf.xacro file and added two new roll definitions: roll_4162.urdf.xacro and roll_4670.urdf.xacro.
- Removed the 006_tip.urdf.xacro file and created a new tip_006.urdf.xacro with updated definitions.
- Added a new tip_049.urdf.xacro for the 049 tip.
- Deleted the 0091m_wrist.urdf.xacro and created wrist_pitch_0091.urdf.xacro and wrist_yaw_0091.urdf.xacro for the wrist components.

File: urdf/Classic/PSM1.urdf.xacro (robot description, xacro)
@@ -16,5 +16,4 @@
                   xyz="0.0 0.0 0.0" rpy="0.0 0.0 0.0"/>
   <xacro:instrument prefix="PSM1_"
-                        parent_link="PSM1_adaptor_link"
                         instrument="$(arg instrument)"/>
 </robot>

File: urdf/Classic/PSM2.urdf.xacro (robot description, xacro)
@@ -11,5 +11,4 @@
                   xyz="0.0 0.0 0.0" rpy="0.0 0.0 0.0"/>
   <xacro:instrument prefix="PSM2_"
-                        parent_link="PSM2_adaptor_link"
                         instrument="$(arg instrument)"/>
 </robot>

File: urdf/Classic/PSM3.urdf.xacro (robot description, xacro)
@@ -11,5 +11,4 @@
                   xyz="0.0 0.0 0.0" rpy="0.0 0.0 0.0"/>
   <xacro:instrument prefix="PSM3_"
-                        parent_link="PSM3_adaptor_link"
                         instrument="$(arg instrument)"/>
 </robot>

File: urdf/Si/PSM1.urdf.xacro (robot description, xacro)
@@ -14,5 +14,4 @@
                   parent_link="${parent_link}"/>
   <xacro:instrument prefix="PSM1_"
-                        parent_link="PSM1_adaptor_link"
                         instrument="$(arg instrument)"/>
 </robot>

File: urdf/Si/PSM2.urdf.xacro (robot description, xacro)
@@ -10,5 +10,4 @@
                   parent_link="${parent_link}"/>
   <xacro:instrument prefix="PSM2_"
-                        parent_link="PSM2_adaptor_link"
                         instrument="$(arg instrument)"/>
 </robot>

File: urdf/Si/PSM3.urdf.xacro (robot description, xacro)
@@ -10,5 +10,4 @@
                   parent_link="${parent_link}"/>
   <xacro:instrument prefix="PSM3_"
-                        parent_link="PSM3_adaptor_link"
                         instrument="$(arg instrument)"/>
 </robot>

File: urdf/Si/PSM_420006_zero_check.urdf.xacro (robot description, xacro)
@@ -18,5 +18,5 @@
       <origin xyz="0.0 0.0 0.0" rpy="0.0 0.0 0.0"/>
       <geometry>
-        <mesh filename="package://dvrk_model/meshes/instruments/Si/roll/PSM_roll_8mm.OBJ"/>
+        <mesh filename="package://dvrk_model/meshes/instruments/roll/4670/roll_4670.obj"/>
       </geometry>
     </visual>
@@ -24,5 +24,5 @@
       <origin xyz="0.0 0.0 0.0" rpy="0.0 0.0 0.0"/>
       <geometry>
-        <mesh filename="package://dvrk_model/meshes/instruments/Si/pitch/PSM_006_pitch.OBJ"/>
+        <mesh filename="package://dvrk_model/meshes/instruments/wrist_pitch/0091/wrist_pitch_0091.obj"/>
       </geometry>
     </visual>
@@ -30,5 +30,5 @@
       <origin xyz="0.0 0.0 0.0" rpy="0.0 0.0 0.0"/>
       <geometry>
-        <mesh filename="package://dvrk_model/meshes/instruments/Si/yaw/PSM_006_yaw.OBJ"/>
+        <mesh filename="package://dvrk_model/meshes/instruments/wrist_yaw/0091/wrist_yaw_0091.obj"/>
       </geometry>
     </visual>
@@ -36,5 +36,5 @@
       <origin xyz="0.0 0.0 0.0" rpy="0.0 0.0 0.0"/>
       <geometry>
-        <mesh filename="package://dvrk_model/meshes/instruments/Si/tip/PSM_006_jaw_1.OBJ"/>
+        <mesh filename="package://dvrk_model/meshes/instruments/tip/006/tip_006_1.obj"/>
       </geometry>
     </visual>
@@ -42,5 +42,5 @@
       <origin xyz="0.0 0.0 0.0" rpy="0.0 0.0 0.0"/>
       <geometry>
-        <mesh filename="package://dvrk_model/meshes/instruments/Si/tip/PSM_006_jaw_2.OBJ"/>
+        <mesh filename="package://dvrk_model/meshes/instruments/tip/006/tip_006_2.obj"/>
       </geometry>
     </visual>

File: urdf/Virtual/PSM1.urdf.xacro (robot description, xacro)
@@ -25,5 +25,4 @@
   <!-- Instrument: identical to Classic/Si — attaches at PSM_adaptor_link -->
   <xacro:instrument prefix="PSM1_"
-                        parent_link="PSM1_adaptor_link"
                         instrument="$(arg instrument)"/>
 </robot>

File: urdf/Virtual/PSM2.urdf.xacro (robot description, xacro)
@@ -13,5 +13,4 @@
                           rcm_rpy="$(arg rcm_rpy)"/>
   <xacro:instrument prefix="PSM2_"
-                        parent_link="PSM2_adaptor_link"
                         instrument="$(arg instrument)"/>
 </robot>

File: urdf/Virtual/PSM3.urdf.xacro (robot description, xacro)
@@ -13,5 +13,4 @@
                           rcm_rpy="$(arg rcm_rpy)"/>
   <xacro:instrument prefix="PSM3_"
-                        parent_link="PSM3_adaptor_link"
                         instrument="$(arg instrument)"/>
 </robot>

File: urdf/common/instrument.urdf.xacro (robot description, xacro)
@@ -3,85 +3,78 @@
   <!--
     Instrument macro — generation-agnostic.
-    Attaches to ${parent_link} (= ${prefix}adaptor_link from the PSM base).
-    DOF layout:
-      Joint 4: roll         (revolute, D = shaft_length along z)
-      Joint 5: wrist_pitch  (revolute)
-      Joint 6: wrist_yaw    (revolute)
-      Joint 7: jaw + mimics (revolute)
+    Attaches to ${prefix}adaptor_link from the PSM base.
+    Instruments are assembled from four physical stages:
+      1. housing
+      2. roll
+      3. wrist_pitch + wrist_yaw
+      4. tip
     Parameters:
       prefix        — arm instance prefix, e.g. "PSM1_"
-      parent_link   — must be ${prefix}adaptor_link
-      shaft_length  — D parameter of roll joint (Classic: 0.4162, Si: 0.4670)
       instrument    — last 6 digits of instrument model number (e.g. "420006")
-                      used to select the correct full instrument assembly
   -->
   <xacro:include filename="$(find dvrk_model)/urdf/common.urdf.xacro"/>
-  <xacro:include filename="$(find dvrk_model)/urdf/common/instruments/housing.urdf.xacro"/>
-  <xacro:include filename="$(find dvrk_model)/urdf/common/instruments/roll.urdf.xacro"/>
-  <xacro:include filename="$(find dvrk_model)/urdf/common/instruments/wrist/0091m_wrist.urdf.xacro"/>
-  <xacro:include filename="$(find dvrk_model)/urdf/common/instruments/tip/006_tip.urdf.xacro"/>
-  <xacro:include filename="$(find dvrk_model)/urdf/common/instruments/tip/049_tip.urdf.xacro"/>
-  <xacro:macro name="instrument_variant"
-               params="prefix parent_link generation roll_origin wrist_parent_link wrist_0091m_variant tip_style is_si:=false">
-    <xacro:instrument_housing prefix="${prefix}"
-                                  parent_link="${parent_link}"
-                                  housing_family="${generation}"/>
-    <xacro:if value="${generation == 'Si'}">
-      <xacro:instrument_si_roll_shaft prefix="${prefix}"
-                                          parent_link="${parent_link}"
-                                          roll_origin="${roll_origin}"/>
+  <xacro:include filename="$(find dvrk_model)/urdf/common/instruments/housing/housing_Classic.urdf.xacro"/>
+  <xacro:include filename="$(find dvrk_model)/urdf/common/instruments/housing/housing_Si.urdf.xacro"/>
+  <xacro:include filename="$(find dvrk_model)/urdf/common/instruments/roll/roll_4162.urdf.xacro"/>
+  <xacro:include filename="$(find dvrk_model)/urdf/common/instruments/roll/roll_4670.urdf.xacro"/>
+  <xacro:include filename="$(find dvrk_model)/urdf/common/instruments/wrist_pitch/wrist_pitch_0091.urdf.xacro"/>
+  <xacro:include filename="$(find dvrk_model)/urdf/common/instruments/wrist_yaw/wrist_yaw_0091.urdf.xacro"/>
+  <xacro:include filename="$(find dvrk_model)/urdf/common/instruments/tip/tip_006.urdf.xacro"/>
+  <xacro:include filename="$(find dvrk_model)/urdf/common/instruments/tip/tip_049.urdf.xacro"/>
+  <xacro:macro name="instrument_model"
+               params="prefix housing roll wrist_pitch wrist_yaw tip">
+    <xacro:if value="${str(housing) == 'Classic'}">
+      <xacro:housing_Classic prefix="${prefix}"/>
     </xacro:if>
-    <xacro:if value="${generation == 'Classic'}">
-      <xacro:instrument_classic_roll_shaft prefix="${prefix}"
-                                               parent_link="${parent_link}"
-                                               roll_origin="${roll_origin}"/>
+    <xacro:if value="${str(housing) == 'Si'}">
+      <xacro:housing_Si prefix="${prefix}"/>
     </xacro:if>
-    <xacro:wrist_0091m prefix="${prefix}"
-                           parent_link="${wrist_parent_link}"
-                           wrist_0091m_variant="${wrist_0091m_variant}"
-                           is_si="${is_si}"/>
-    <xacro:if value="${tip_style == '006'}">
-      <xacro:tool_tip_006 prefix="${prefix}"
-                              parent_link="${prefix}wrist_yaw_0091m_link"
-                              is_si="${is_si}"/>
+    <xacro:if value="${str(roll) == '4162'}">
+      <xacro:roll_4162 prefix="${prefix}"/>
     </xacro:if>
-    <xacro:if value="${tip_style == '049'}">
-      <xacro:tool_tip_049 prefix="${prefix}"
-                              parent_link="${prefix}wrist_yaw_0091m_link"/>
+    <xacro:if value="${str(roll) == '4670'}">
+      <xacro:roll_4670 prefix="${prefix}"/>
+    </xacro:if>
+    <xacro:if value="${str(wrist_pitch) == '0091' or str(wrist_pitch) == '91'}">
+      <xacro:wrist_pitch_0091 prefix="${prefix}"/>
+    </xacro:if>
+    <xacro:if value="${str(wrist_yaw) == '0091' or str(wrist_yaw) == '91'}">
+      <xacro:wrist_yaw_0091 prefix="${prefix}"/>
+    </xacro:if>
+    <xacro:if value="${str(tip) == '006' or str(tip) == '6'}">
+      <xacro:tip_006 prefix="${prefix}"/>
+    </xacro:if>
+    <xacro:if value="${str(tip) == '049' or str(tip) == '49'}">
+      <xacro:tip_049 prefix="${prefix}"/>
     </xacro:if>
   </xacro:macro>
   <xacro:macro name="instrument"
-               params="prefix parent_link instrument">
+               params="prefix instrument">
     <!-- 420006: Si 006 -->
     <xacro:if value="${str(instrument) == '420006'}">
-      <xacro:instrument_variant prefix="${prefix}"
-                                    parent_link="${parent_link}"
-                                    generation="Si"
-                                    roll_origin="${0.4670}"
-                                    wrist_parent_link="${prefix}roll_link"
-                                    wrist_0091m_variant="sca"
-                                    tip_style="006"
-                                    is_si="true"/>
+      <xacro:instrument_model prefix="${prefix}"
+                              housing="Si"
+                              roll="4670"
+                              wrist_pitch="0091"
+                              wrist_yaw="0091"
+                              tip="006"/>
     </xacro:if>
     <!-- 400006: Classic 006 -->
     <xacro:if value="${str(instrument) == '400006'}">
-      <xacro:instrument_variant prefix="${prefix}"
-                                    parent_link="${parent_link}"
-                                    generation="Classic"
-                                    roll_origin="${0.4572}"
-                                    wrist_parent_link="${prefix}roll_link"
-                                    wrist_0091m_variant="sca"
-                                    tip_style="006"
-                                    is_si="false"/>
+      <xacro:instrument_model prefix="${prefix}"
+                              housing="Classic"
+                              roll="4162"
+                              wrist_pitch="0091"
+                              wrist_yaw="0091"
+                              tip="006"/>
     </xacro:if>
     <!-- 400049: Classic 049 -->
     <xacro:if value="${str(instrument) == '400049'}">
-      <xacro:instrument_variant prefix="${prefix}"
-                                    parent_link="${parent_link}"
-                                    generation="Classic"
-                                    roll_origin="${0.4572}"
-                                    wrist_parent_link="${prefix}roll_link"
-                                    wrist_0091m_variant="cadiere"
-                                    tip_style="049"/>
+      <xacro:instrument_model prefix="${prefix}"
+                              housing="Classic"
+                              roll="4162"
+                              wrist_pitch="0091"
+                              wrist_yaw="0091"
+                              tip="049"/>
     </xacro:if>
   </xacro:macro>
