Commit message: * renamed `suj_tf` to `suj` * removed parameters from PSM{1,2,3}/ECM Si launch files since these are intended as top launch files * added ECM to Si cart using a PSM

File: urdf/Classic/ECM.urdf.xacro (robot description, xacro)
@@ -5,5 +5,5 @@
   <link name="world"/>
   <xacro:ecm
-      prefix="ecm"
+      prefix="ECM_"
       parent_link="world"
       xyz="0 0.0 0.0" rpy="0.0 0.0 0.0"/>

File: urdf/Si/ECM.urdf.xacro (robot description, xacro)
@@ -2,13 +2,10 @@
 <robot name="ECM" xmlns:xacro="http://www.ros.org/wiki/xacro">
     <xacro:property name="ECM" value="ECM_"/>
-    <xacro:property name="ECM_tool" value="SF826001"/>
-    <xacro:arg name="parent_link_" default="world"/>
-    <xacro:property name="parent_link" default="$(arg parent_link_)"/>
     <xacro:include filename="$(find dvrk_model)/urdf/Si/psm_base.urdf.xacro"/>
     <xacro:include filename="$(find dvrk_model)/urdf/Si/tools.urdf.xacro"/>
-    <link name="${parent_link}"/>
+    <link name="world"/>
     <xacro:psm_arm_active
-        prefix="${ECM}"
-        parent_link="${parent_link}"/>
-    <xacro:tool tool_name="SF826001" prefix="${ECM}" parent_link="${ECM}tool_parent"/>
+        prefix="ECM_"
+        parent_link="world"/>
+    <xacro:tool tool_name="SF826001" prefix="ECM_" parent_link="ECM_tool_parent"/>
 </robot>

File: urdf/Si/PSM1.urdf.xacro (robot description, xacro)
@@ -2,13 +2,10 @@
 <robot name="PSM1" xmlns:xacro="http://www.ros.org/wiki/xacro">
   <xacro:property name="tool_name" value="P420006"/>
-  <xacro:property name="PSM1" value="PSM1_"/>
-  <xacro:arg name="parent_link_" default="world"/>
-  <xacro:property name="parent_link" default="$(arg parent_link_)"/>
   <xacro:include filename="$(find dvrk_model)/urdf/Si/psm_base.urdf.xacro"/>
   <xacro:include filename="$(find dvrk_model)/urdf/Si/tools.urdf.xacro"/>
-  <link name="${parent_link}"/>
+  <link name="world"/>
   <xacro:psm_arm_active
-      prefix="${PSM1}"
-      parent_link="${parent_link}"/>
-  <xacro:tool tool_name="${tool_name}" prefix="${PSM1}_" parent_link="${PSM1}tool_parent"/>
+      prefix="PSM1_"
+      parent_link="world"/>
+  <xacro:tool tool_name="${tool_name}" prefix="PSM1_" parent_link="PSM1_tool_parent"/>
 </robot>

File: urdf/Si/PSM2.urdf.xacro (robot description, xacro)
@@ -2,13 +2,10 @@
 <robot name="PSM2" xmlns:xacro="http://www.ros.org/wiki/xacro">
   <xacro:property name="tool_name" value="P420006"/>
-  <xacro:property name="PSM2" value="PSM2_"/>
-  <xacro:arg name="parent_link_" default="world"/>
-  <xacro:property name="parent_link" default="$(arg parent_link_)"/>
   <xacro:include filename="$(find dvrk_model)/urdf/Si/psm_base.urdf.xacro"/>
   <xacro:include filename="$(find dvrk_model)/urdf/Si/tools.urdf.xacro"/>
-  <link name="${parent_link}"/>
+  <link name="world"/>
   <xacro:psm_arm_active
-      prefix="${PSM2}"
-      parent_link="${parent_link}"/>
-  <xacro:tool tool_name="${tool_name}" prefix="${PSM2}" parent_link="${PSM2}tool_parent"/>
+      prefix="PSM2_"
+      parent_link="world"/>
+  <xacro:tool tool_name="${tool_name}" prefix="PSM2_" parent_link="PSM2_tool_parent"/>
 </robot>

File: urdf/Si/PSM3.urdf.xacro (robot description, xacro)
@@ -2,13 +2,10 @@
 <robot name="PSM3" xmlns:xacro="http://www.ros.org/wiki/xacro">
   <xacro:property name="tool_name" value="P420006"/>
-  <xacro:property name="PSM3" value="PSM3_">
-  <xacro:arg name="parent_link_" default="world"/>
-  <xacro:property name="parent_link" default="$(arg parent_link_)"/>
   <xacro:include filename="$(find dvrk_model)/urdf/Si/psm_base.urdf.xacro"/>
   <xacro:include filename="$(find dvrk_model)/urdf/Si/tools.urdf.xacro"/>
-  <link name="${parent_link}"/>
+  <link name="world"/>
   <xacro:psm_arm_active
-      prefix="${PSM3}"
-      parent_link="${parent_link}"/>
-  <xacro:tool tool_name="${tool_name}" prefix="${PSM3}" parent_link="${PSM3}tool_parent"/>
+      prefix="PSM3_"
+      parent_link="world"/>
+  <xacro:tool tool_name="${tool_name}" prefix="PSM3_" parent_link="PSM3_tool_parent"/>
 </robot>
