Commit message: * move dVRK cube to top level for meshes * renamed mesh directories using upper case for Classic and Si * renamed some .STL to .stl * removed duplicate STL files for ECM Classic * added meshes for SUJ Classic (from WPI AIM) * initial standardization of URDF xacros for Si/Classic using {psm,ecm}_{base,tool}.  Tools still need to be factorized across Si/Classic and need to add `ecm_tool` for different endoscopes

File: urdf/Classic/ECM.urdf.xacro (robot description, xacro)
@@ -1,8 +1,7 @@
 <?xml version="1.0" ?>
 <robot name="ecm" xmlns:xacro="http://www.ros.org/wiki/xacro">
-  <!-- Macros -->
-  <xacro:include filename="$(find dvrk_model)/urdf/Classic/ecm.urdf.xacro"/>
+  <xacro:include filename="$(find dvrk_model)/urdf/Classic/ecm_base.urdf.xacro"/>
   <link name="world"/>
-  <xacro:ecm
+  <xacro:ecm_base
       prefix="ECM_"
       parent_link="world"

File: urdf/Classic/PSM1.urdf.xacro (robot description, xacro)
@@ -1,10 +1,11 @@
 <?xml version="1.0" ?>
 <robot name="dvrk_psm" xmlns:xacro="http://www.ros.org/wiki/xacro">
-  <!-- Macros -->
-  <xacro:include filename="$(find dvrk_model)/urdf/Classic/psm.urdf.xacro"/>
+  <xacro:include filename="$(find dvrk_model)/urdf/Classic/psm_base.urdf.xacro"/>
+  <xacro:include filename="$(find dvrk_model)/urdf/Classic/psm_tool.urdf.xacro"/>
   <link name="world"/>
-  <xacro:psm_sca
+  <xacro:psm_base
       prefix="PSM1_"
       parent_link="world"
-      xyz="-0.25 0.0 0.5" rpy="0.0 0.0 3.1415926"/>
+      xyz="-0.25 0.0 0.5" rpy="0.0 0.0 ${PI}"/>
+  <xacro:psm_tool tool_name="sca" prefix="PSM1_"/>
 </robot>

File: urdf/Classic/PSM2.urdf.xacro (robot description, xacro)
@@ -1,10 +1,11 @@
 <?xml version="1.0" ?>
 <robot name="dvrk_psm" xmlns:xacro="http://www.ros.org/wiki/xacro">
-  <!-- Macros -->
-  <xacro:include filename="$(find dvrk_model)/urdf/Classic/psm.urdf.xacro"/>
+  <xacro:include filename="$(find dvrk_model)/urdf/Classic/psm_base.urdf.xacro"/>
+  <xacro:include filename="$(find dvrk_model)/urdf/Classic/psm_tool.urdf.xacro"/>
   <link name="world"/>
-  <xacro:psm_caudier
+  <xacro:psm_base
       prefix="PSM2_"
       parent_link="world"
-      xyz="0.25 0.0 0.5" rpy="0.0 0.0 -3.1415926"/>
+      xyz="-0.25 0.0 0.5" rpy="0.0 0.0 ${PI}"/>
+  <xacro:psm_tool tool_name="caudier" prefix="PSM2_"/>
 </robot>

File: urdf/Classic/PSM3.urdf.xacro (robot description, xacro)
@@ -1,10 +1,11 @@
 <?xml version="1.0" ?>
 <robot name="dvrk_psm" xmlns:xacro="http://www.ros.org/wiki/xacro">
-  <!-- Macros -->
-  <xacro:include filename="$(find dvrk_model)/urdf/Classic/psm.urdf.xacro"/>
+  <xacro:include filename="$(find dvrk_model)/urdf/Classic/psm_base.urdf.xacro"/>
+  <xacro:include filename="$(find dvrk_model)/urdf/Classic/psm_tool.urdf.xacro"/>
   <link name="world"/>
-  <xacro:psm_caudier
+  <xacro:psm_base
       prefix="PSM3_"
       parent_link="world"
-      xyz="0.50 0.0 0.5" rpy="0.0 0.0 -3.1415926"/>
+      xyz="0.50 0.0 0.5" rpy="0.0 0.0 ${-PI}"/>
+  <xacro:psm_tool tool_name="caudier" prefix="PSM3_"/>
 </robot>

File: urdf/Classic/ecm.urdf.xacro (robot description, xacro)
@@ -1,180 +1,11 @@
 <?xml version="1.0" ?>
-<robot name="ecm" xmlns:xacro="http://www.ros.org/wiki/xacro">
-  <!-- Colors -->
-  <xacro:include filename="$(find dvrk_model)/urdf/Classic/common.urdf.xacro"/>
-  <!-- Macro for da Vinci Endoscope Camera Manipulator (ECM) -->
-  <xacro:macro name="ecm" params="prefix parent_link xyz rpy">
-    <!-- Joint 0: Fixed to World-->
-    <joint name="fixed" type="fixed">
-      <parent link="${parent_link}"/>
-      <child link="${prefix}_base_link"/>
-      <origin rpy="${rpy}" xyz="${xyz}"/>
-    </joint>
-    <link name="${prefix}_base_link"/>
-    <!-- Joint 1: Outer Yaw -->
-    <joint name="yaw" type="revolute">
-      <parent link="${prefix}_base_link"/>
-      <child link="${prefix}_yaw_link"/>
-      <origin rpy="0 -${PI/2} ${PI/2}" xyz="0 0 0"/>
-      <axis xyz="0 0 1"/>
-      <!--rotates about z axis-->
-      <!--limit effort and velocity picked arbitrarily check-->
-      <limit effort="50.0" lower="${-75/180*PI}" upper="${PI/4}" velocity="2"/>
-      <joint_properties damping="1.0" friction="0.0"/>
-    </joint>
-    <link name="${prefix}_yaw_link">
-      <visual>
-        <origin rpy="0 0 -${PI/2}" xyz="0.0 0 0.603"/>
-        <geometry>
-          <mesh filename="package://dvrk_model/meshes/Classic/ecm/Endo_Link_5.STL"/>
-        </geometry>
-	<material name="DaVinciGreen"/>
-      </visual>
-      <collision>
-        <origin rpy="0 0 -${PI/2}" xyz="0.0 0 0.603"/>
-        <geometry>
-          <mesh filename="package://dvrk_model/meshes/Classic/ecm/Endo_Link_5.STL"/>
-        </geometry>
-      </collision>
-    </link>
-    <!-- Joint 2: Pitch -->
-    <joint name="pitch" type="revolute">
-      <parent link="${prefix}_yaw_link"/>
-      <child link="${prefix}_pitch_link"/>
-      <origin rpy="-${PI/2} -${PI/2} 0" xyz="0 0 0"/>
-      <axis xyz="0 0 1"/>
-      <limit effort="100.0" lower="${-PI/4}" upper="${PI*65/180}" velocity="10"/>
-      <joint_properties damping="1.0" friction="0.0"/>
-    </joint>
-    <link name="${prefix}_pitch_link"/>
-    <joint name="pitch_0" type="continuous">
-      <parent link="${prefix}_yaw_link"/>
-      <child link="${prefix}_pitch_link_1"/>
-      <origin rpy="-${PI/2} -${PI/2} 0" xyz="0 0 0.378"/>
-      <axis xyz="0 0 1"/>
-      <joint_properties damping="1.0" friction="0.0"/>
-      <mimic joint="pitch" multiplier="1"/>
-    </joint>
-    <link name="${prefix}_pitch_link_1">
-      <visual>
-        <origin rpy="${PI} 0 ${PI*78.5/180}" xyz="0.0 0 0.0"/>
-        <geometry>
-          <mesh filename="package://dvrk_model/meshes/Classic/ecm/Endo_Link_5_2.STL"/>
-        </geometry>
-	<material name="DaVinciMedGray"/>
-      </visual>
-      <collision>
-        <origin rpy="${PI} 0 ${PI*78.5/180}" xyz="0.0 0 0.0"/>
-        <geometry>
-          <mesh filename="package://dvrk_model/meshes/Classic/ecm/Endo_Link_5_2.STL"/>
-        </geometry>
-      </collision>
-      <inertial>
-        <mass value=".9"/>
-        <inertia ixx="9.0" ixy="0.0" ixz="0.0" iyy="9.0" iyz="0.0" izz="9.0"/>
-      </inertial>
-    </link>
-    <joint name="pitch_1" type="continuous">
-      <parent link="${prefix}_pitch_link_1"/>
-      <child link="${prefix}_pitch_link_2"/>
-      <origin rpy="0 0 0" xyz="0.0558629 0.274575 0"/>
-      <axis xyz="0 0 1"/>
-      <joint_properties damping="1.0" friction="0.0"/>
-      <mimic joint="pitch" multiplier="-1"/>
-    </joint>
-    <link name="${prefix}_pitch_link_2">
-      <visual>
-        <origin rpy="0 0 0" xyz="0.0 0 -0.0225"/>
-        <geometry>
-          <mesh filename="package://dvrk_model/meshes/Classic/ecm/Endo_Link_6_2.STL"/>
-        </geometry>
-	<material name="DaVinciMedGray"/>
-      </visual>
-      <collision>
-        <origin rpy="0 0 0" xyz="0.0 0 -0.0225"/>
-        <geometry>
-          <mesh filename="package://dvrk_model/meshes/Classic/ecm/Endo_Link_6_2.STL"/>
-        </geometry>
-      </collision>
-      <inertial>
-        <mass value=".9"/>
-        <inertia ixx="9.0" ixy="0.0" ixz="0.0" iyy="9.0" iyz="0.0" izz="9.0"/>
-      </inertial>
-    </link>
-    <joint name="pitch_2" type="continuous">
-      <parent link="${prefix}_pitch_link_2"/>
-      <child link="${prefix}_pitch_link_3"/>
-      <origin rpy="0 0 0" xyz="-0.340 0 0"/>
-      <axis xyz="0 0 1"/>
-      <joint_properties damping="1.0" friction="0.0"/>
-      <mimic joint="pitch" multiplier="1"/>
-    </joint>
-    <link name="${prefix}_pitch_link_3">
-      <visual>
-        <origin rpy="0 0 -${PI/2}" xyz="0.0 0 0.025"/>
-        <geometry>
-          <mesh filename="package://dvrk_model/meshes/Classic/ecm/Endo_Link_7.STL"/>
-        </geometry>
-	<material name="DaVinciMedGray"/>
-      </visual>
-      <collision>
-        <origin rpy="0 0 -${PI/2}" xyz="0.0 0 0.025"/>
-        <geometry>
-          <mesh filename="package://dvrk_model/meshes/Classic/ecm/Endo_Link_7.STL"/>
-        </geometry>
-      </collision>
-      <inertial>
-        <mass value=".9"/>
-        <inertia ixx="9.0" ixy="0.0" ixz="0.0" iyy="9.0" iyz="0.0" izz="9.0"/>
-      </inertial>
-    </link>
-    <!-- Joint 3: Insertion -->
-    <joint name="insertion" type="prismatic">
-      <parent link="${prefix}_pitch_link"/>
-      <child link="${prefix}_insertion_link"/>
-      <origin rpy="${PI/2} 0 0" xyz="0 0.3822 0"/>
-      <axis xyz="0 0 1"/>
-      <joint_properties damping="1.0" friction="0.0"/>
-      <limit effort="100.0" lower="0" upper="0.235" velocity="10"/>
-    </joint>
-    <link name="${prefix}_insertion_link">
-      <visual>
-        <origin rpy="0 0 -${PI/2}" xyz="0.0 0 -0.015"/>
-        <geometry>
-          <mesh filename="package://dvrk_model/meshes/Classic/ecm/Endo_Link_8.STL"/>
-        </geometry>
-	<material name="DaVinciBlue"/>
-      </visual>
-      <collision>
-        <origin rpy="0 0 -${PI/2}" xyz="0.0 0 -0.015"/>
-        <geometry>
-          <mesh filename="package://dvrk_model/meshes/Classic/ecm/Endo_Link_8.STL"/>
-        </geometry>
-      </collision>
-    </link>
-    <!-- Joint 4: Roll -->
-    <joint name="roll" type="revolute">
-      <parent link="${prefix}_insertion_link"/>
-      <child link="${prefix}_roll_link"/>
-      <origin rpy="0 0 0" xyz="0 0 0.3829"/>
-      <axis xyz="0 0 1"/>
-      <joint_properties damping="1.0" friction="0.0"/>
-      <limit effort="100.0" lower="-${PI/2}" upper="${PI/2}" velocity="10"/>
-    </joint>
-    <link name="${prefix}_roll_link">
-      <visual>
-        <origin rpy="0 0 ${PI/2}" xyz="0.0 0 -0.3979"/>
-        <geometry>
-          <mesh filename="package://dvrk_model/meshes/Classic/ecm/EndoScope.STL"/>
-        </geometry>
-	<material name="DaVinciBlue"/>
-      </visual>
-      <collision>
-        <origin rpy="0 0 ${PI/2}" xyz="0.0 0 -0.3979"/>
-        <geometry>
-          <mesh filename="package://dvrk_model/meshes/Classic/ecm/EndoScope.STL"/>
-        </geometry>
-      </collision>
-    </link>
-  </xacro:macro>
+<robot name="dvrk_psm" xmlns:xacro="http://www.ros.org/wiki/xacro">
+  <xacro:property name="arm" default="$(arg arm)"/>
+  <xacro:arg name="parent_link_" default="world"/>
+  <xacro:property name="parent_link" default="$(arg parent_link_)"/>
+  <xacro:include filename="$(find dvrk_model)/urdf/Classic/ecm_base.urdf.xacro"/>
+  <link name="${parent_link}"/>
+  <xacro:ecm_base
+      prefix="${arm}_"
+      parent_link="${parent_link}"/>
 </robot>

File: urdf/Classic/mtm.urdf.xacro (robot description, xacro)
@@ -2,5 +2,5 @@
 <robot name="mtm" xmlns:xacro="http://www.ros.org/wiki/xacro">
   <!-- Colors -->
-  <xacro:include filename="$(find dvrk_model)/urdf/Classic/common.urdf.xacro"/>
+  <xacro:include filename="$(find dvrk_model)/urdf/common.urdf.xacro"/>
   <!-- Macro for the da Vinci Master Console -->
   <xacro:macro name="master_console" params="prefix parent_link xyz:='0.0 0.0 0.0' rpy:='0.0 0.0 0.0'">
@@ -41,5 +41,5 @@
         <origin rpy="0 0 0" xyz="0 0 0.19037"/>
         <geometry>
-          <mesh filename="package://dvrk_model/meshes/Classic/mtm/Top_Panel.dae"/>
+          <mesh filename="package://dvrk_model/meshes/Classic/MTM/Top_Panel.dae"/>
         </geometry>
       </visual>
@@ -47,5 +47,5 @@
         <origin rpy="0 0 0" xyz="0 0 0.19037"/>
         <geometry>
-          <mesh filename="package://dvrk_model/meshes/Classic/mtm/Top_Panel.STL"/>
+          <mesh filename="package://dvrk_model/meshes/Classic/MTM/Top_Panel.stl"/>
         </geometry>
       </collision>
@@ -73,5 +73,5 @@
         <origin rpy="0 0 0" xyz="0.025 0 0.19037"/>
         <geometry>
-          <mesh filename="package://dvrk_model/meshes/Classic/mtm/OutPitch_Shoulder.dae"/>
+          <mesh filename="package://dvrk_model/meshes/Classic/MTM/OutPitch_Shoulder.dae"/>
         </geometry>
       </visual>
@@ -79,5 +79,5 @@
         <origin rpy="0 0 0" xyz="0.025 0 0.19037"/>
         <geometry>
-          <mesh filename="package://dvrk_model/meshes/Classic/mtm/OutPitch_Shoulder.STL"/>
+          <mesh filename="package://dvrk_model/meshes/Classic/MTM/OutPitch_Shoulder.stl"/>
         </geometry>
       </collision>
@@ -100,10 +100,10 @@
       <visual>
         <geometry>
-          <mesh filename="package://dvrk_model/meshes/Classic/mtm/ArmParallel.dae"/>
-        </geometry>
-      </visual>
-      <collision>
-        <geometry>
-          <mesh filename="package://dvrk_model/meshes/Classic/mtm/ArmParallel.STL"/>
+          <mesh filename="package://dvrk_model/meshes/Classic/MTM/ArmParallel.dae"/>
+        </geometry>
+      </visual>
+      <collision>
+        <geometry>
+          <mesh filename="package://dvrk_model/meshes/Classic/MTM/ArmParallel.stl"/>
         </geometry>
       </collision>
@@ -128,5 +128,5 @@
         <origin rpy="0 0 ${-PI/2}" xyz="0 0 0.065"/>
         <geometry>
-          <mesh filename="package://dvrk_model/meshes/Classic/mtm/ArmParallel1.dae"/>
+          <mesh filename="package://dvrk_model/meshes/Classic/MTM/ArmParallel1.dae"/>
         </geometry>
       </visual>
@@ -134,5 +134,5 @@
         <origin rpy="0 0 0" xyz="0 0 0"/>
         <geometry>
-          <mesh filename="package://dvrk_model/meshes/Classic/mtm/ArmParallel1.STL"/>
+          <mesh filename="package://dvrk_model/meshes/Classic/MTM/ArmParallel1.stl"/>
         </geometry>
       </collision>
@@ -155,10 +155,10 @@
       <visual>
         <geometry>
-          <mesh filename="package://dvrk_model/meshes/Classic/mtm/BottomArm.dae"/>
-        </geometry>
-      </visual>
-      <collision>
-        <geometry>
-          <mesh filename="package://dvrk_model/meshes/Classic/mtm/BottomArm.STL"/>
+          <mesh filename="package://dvrk_model/meshes/Classic/MTM/BottomArm.dae"/>
+        </geometry>
+      </visual>
+      <collision>
+        <geometry>
+          <mesh filename="package://dvrk_model/meshes/Classic/MTM/BottomArm.stl"/>
         </geometry>
       </collision>
@@ -225,10 +225,10 @@
       <visual>
         <geometry>
-          <mesh filename="package://dvrk_model/meshes/Classic/mtm/WristPlatform.dae"/>
-        </geometry>
-      </visual>
-      <collision>
-        <geometry>
-          <mesh filename="package://dvrk_model/meshes/Classic/mtm/WristPlatform.STL"/>
+          <mesh filename="package://dvrk_model/meshes/Classic/MTM/WristPlatform.dae"/>
+        </geometry>
+      </visual>
+      <collision>
+        <geometry>
+          <mesh filename="package://dvrk_model/meshes/Classic/MTM/WristPlatform.stl"/>
         </geometry>
       </collision>
@@ -253,10 +253,10 @@
       <visual>        <!-- defined from CAD file (increased in the y dir by .005-->
         <geometry>
-          <mesh filename="package://dvrk_model/meshes/Classic/mtm/WristPitch.dae"/>
+          <mesh filename="package://dvrk_model/meshes/Classic/MTM/WristPitch.dae"/>
         </geometry>
       </visual>
       <collision>        <!-- defined from CAD file (increased in the y dir by .005-->
         <geometry>
-          <mesh filename="package://dvrk_model/meshes/Classic/mtm/WristPitch.STL"/>
+          <mesh filename="package://dvrk_model/meshes/Classic/MTM/WristPitch.stl"/>
         </geometry>
       </collision>
@@ -282,10 +282,10 @@
       <visual>
         <geometry>
-          <mesh filename="package://dvrk_model/meshes/Classic/mtm/WristYaw.dae"/>
-        </geometry>
-      </visual>
-      <collision>
-        <geometry>
-          <mesh filename="package://dvrk_model/meshes/Classic/mtm/WristYaw.STL"/>
+          <mesh filename="package://dvrk_model/meshes/Classic/MTM/WristYaw.dae"/>
+        </geometry>
+      </visual>
+      <collision>
+        <geometry>
+          <mesh filename="package://dvrk_model/meshes/Classic/MTM/WristYaw.stl"/>
         </geometry>
       </collision>
@@ -312,5 +312,5 @@
         <origin rpy="${PI} 0 0" xyz="0 0 0.039"/>
         <geometry>
-          <mesh filename="package://dvrk_model/meshes/Classic/mtm/WristRoll.dae"/>
+          <mesh filename="package://dvrk_model/meshes/Classic/MTM/WristRoll.dae"/>
         </geometry>
       </visual>
@@ -318,5 +318,5 @@
         <origin rpy="${PI} 0 0" xyz="0 0 0.039"/>
         <geometry>
-          <mesh filename="package://dvrk_model/meshes/Classic/mtm/WristRoll.STL"/>
+          <mesh filename="package://dvrk_model/meshes/Classic/MTM/WristRoll.stl"/>
         </geometry>
       </collision>
@@ -378,5 +378,5 @@
         <origin rpy="0 0 ${PI}" xyz="0.0 0.0 0.0"/>
         <geometry>
-          <mesh filename="package://dvrk_model/meshes/Classic/mtm/WristPlatform.dae"/>
+          <mesh filename="package://dvrk_model/meshes/Classic/MTM/WristPlatform.dae"/>
         </geometry>
       </visual>
@@ -384,5 +384,5 @@
         <origin rpy="0 0 ${PI}" xyz="0.0 0.0 0.0"/>
         <geometry>
-          <mesh filename="package://dvrk_model/meshes/Classic/mtm/WristPlatform.STL"/>
+          <mesh filename="package://dvrk_model/meshes/Classic/MTM/WristPlatform.stl"/>
         </geometry>
       </collision>
@@ -408,5 +408,5 @@
         <origin rpy="0 ${PI} 0" xyz="0.0 0.0 0.0"/>
         <geometry>
-          <mesh filename="package://dvrk_model/meshes/Classic/mtm/WristPitch.dae"/>
+          <mesh filename="package://dvrk_model/meshes/Classic/MTM/WristPitch.dae"/>
         </geometry>
       </visual>
@@ -414,5 +414,5 @@
         <origin rpy="0 ${PI} 0" xyz="0.0 0.0 0.0"/>
         <geometry>
-          <mesh filename="package://dvrk_model/meshes/Classic/mtm/WristPitch.STL"/>
+          <mesh filename="package://dvrk_model/meshes/Classic/MTM/WristPitch.stl"/>
         </geometry>
       </collision>
@@ -438,10 +438,10 @@
       <visual>
         <geometry>
-          <mesh filename="package://dvrk_model/meshes/Classic/mtm/WristYaw.dae"/>
-        </geometry>
-      </visual>
-      <collision>
-        <geometry>
-          <mesh filename="package://dvrk_model/meshes/Classic/mtm/WristYaw.STL"/>
+          <mesh filename="package://dvrk_model/meshes/Classic/MTM/WristYaw.dae"/>
+        </geometry>
+      </visual>
+      <collision>
+        <geometry>
+          <mesh filename="package://dvrk_model/meshes/Classic/MTM/WristYaw.stl"/>
         </geometry>
       </collision>
@@ -468,5 +468,5 @@
         <origin rpy="${PI} 0 0" xyz="0 0 0.039"/>
         <geometry>
-          <mesh filename="package://dvrk_model/meshes/Classic/mtm/WristRoll.dae"/>
+          <mesh filename="package://dvrk_model/meshes/Classic/MTM/WristRoll.dae"/>
         </geometry>
       </visual>
@@ -474,5 +474,5 @@
         <origin rpy="${PI} 0 0" xyz="0 0 0.039"/>
         <geometry>
-          <mesh filename="package://dvrk_model/meshes/Classic/mtm/WristRoll.STL"/>
+          <mesh filename="package://dvrk_model/meshes/Classic/MTM/WristRoll.stl"/>
         </geometry>
       </collision>

File: urdf/Classic/psm.urdf.xacro (robot description, xacro)
@@ -1,35 +1,14 @@
 <?xml version="1.0" ?>
 <robot name="dvrk_psm" xmlns:xacro="http://www.ros.org/wiki/xacro">
-  <!-- Macros -->
-  <xacro:include filename="$(find dvrk_model)/urdf/Classic/psm.base.urdf.xacro"/>
-  <xacro:include filename="$(find dvrk_model)/urdf/Classic/psm.tool.sca.urdf.xacro"/>
-  <xacro:include filename="$(find dvrk_model)/urdf/Classic/psm.tool.caudier.urdf.xacro"/>
-  <xacro:include filename="$(find dvrk_model)/urdf/Classic/psm.tool.snake.urdf.xacro"/>
-  <!-- Macro for psm with snake -->
-  <xacro:macro name="psm_snake" params="prefix parent_link xyz rpy">
-    <xacro:psm
-        prefix="${prefix}"
-        parent_link="${parent_link}"
-        xyz="${xyz}" rpy="${rpy}"/>
-    <xacro:psm_tool_snake
-        prefix="${prefix}"/>
-  </xacro:macro>
-  <!-- Macro for psm with sca -->
-  <xacro:macro name="psm_sca" params="prefix parent_link xyz rpy">
-    <xacro:psm
-        prefix="${prefix}"
-        parent_link="${parent_link}"
-        xyz="${xyz}" rpy="${rpy}"/>
-    <xacro:psm_tool_sca
-        prefix="${prefix}"/>
-  </xacro:macro>
-  <!-- Macro for psm with caudier -->
-  <xacro:macro name="psm_caudier" params="prefix parent_link xyz rpy">
-    <xacro:psm
-        prefix="${prefix}"
-        parent_link="${parent_link}"
-        xyz="${xyz}" rpy="${rpy}"/>
-    <xacro:psm_tool_caudier
-        prefix="${prefix}"/>
-  </xacro:macro>
+  <xacro:property name="tool_name" default="sca"/>
+  <xacro:property name="arm" default="$(arg arm)"/>
+  <xacro:arg name="parent_link_" default="world"/>
+  <xacro:property name="parent_link" default="$(arg parent_link_)"/>
+  <xacro:include filename="$(find dvrk_model)/urdf/Classic/psm_base.urdf.xacro"/>
+  <xacro:include filename="$(find dvrk_model)/urdf/Classic/psm_tool.urdf.xacro"/>
+  <link name="${parent_link}"/>
+  <xacro:psm_base
+      prefix="${arm}_"
+      parent_link="${parent_link}"/>
+  <xacro:psm_tool tool_name="${tool_name}" prefix="${arm}_"/>
 </robot>
