Commit message: * move dVRK cube to top level for meshes * renamed mesh directories using upper case for Classic and Si * renamed some .STL to .stl * removed duplicate STL files for ECM Classic * added meshes for SUJ Classic (from WPI AIM) * initial standardization of URDF xacros for Si/Classic using {psm,ecm}_{base,tool}.  Tools still need to be factorized across Si/Classic and need to add `ecm_tool` for different endoscopes

File: urdf/Classic/psm_base.urdf.xacro (robot description, xacro)
@@ -1,5 +1,5 @@
 <?xml version="1.0" encoding="utf-8"?>
 <robot name="dvrk_psm" xmlns:xacro="http://www.ros.org/wiki/xacro">
-  <xacro:macro name="psm" params="prefix parent_link xyz rpy">
+  <xacro:macro name="psm_base" params="prefix parent_link xyz:='0.0 0.0 0.0' rpy:='0.0 0.0 0.0'">
     <!-- fixed joint -->
     <joint name="fixed" type="fixed">
@@ -13,5 +13,5 @@
         <origin rpy="1.5708 0 3.1416" xyz="0.039 -0.40788 -0.07879"/>
         <geometry>
-          <mesh filename="package://dvrk_model/meshes/Classic/psm/psm_base.dae"/>
+          <mesh filename="package://dvrk_model/meshes/Classic/PSM/psm_base.dae"/>
         </geometry>
       </visual>
@@ -31,5 +31,5 @@
         <origin rpy="3.1416 0 1.5708" xyz="0.0125 0 0.5265"/>
         <geometry>
-          <mesh filename="package://dvrk_model/meshes/Classic/psm/outer_yaw.dae"/>
+          <mesh filename="package://dvrk_model/meshes/Classic/PSM/outer_yaw.dae"/>
         </geometry>
       </visual>
@@ -62,5 +62,5 @@
         <origin rpy="0 0 -0.27129" xyz="0 0 0"/>
         <geometry>
-          <mesh filename="package://dvrk_model/meshes/Classic/psm/outer_pitch_back.dae"/>
+          <mesh filename="package://dvrk_model/meshes/Classic/PSM/outer_pitch_back.dae"/>
         </geometry>
       </visual>
@@ -79,5 +79,5 @@
         <origin rpy="0 0 -0.27129" xyz="0 0 0"/>
         <geometry>
-          <mesh filename="package://dvrk_model/meshes/Classic/psm/outer_pitch_front.dae"/>
+          <mesh filename="package://dvrk_model/meshes/Classic/PSM/outer_pitch_front.dae"/>
         </geometry>
       </visual>
@@ -96,5 +96,5 @@
         <origin rpy="0 -1.5708 0" xyz="0.009 0 0"/>
         <geometry>
-          <mesh filename="package://dvrk_model/meshes/Classic/psm/outer_pitch_bottom.dae"/>
+          <mesh filename="package://dvrk_model/meshes/Classic/PSM/outer_pitch_bottom.dae"/>
         </geometry>
       </visual>
@@ -113,5 +113,5 @@
         <origin rpy="0 -1.5708 0" xyz="0.009 0 0"/>
         <geometry>
-          <mesh filename="package://dvrk_model/meshes/Classic/psm/outer_pitch_top.dae"/>
+          <mesh filename="package://dvrk_model/meshes/Classic/PSM/outer_pitch_top.dae"/>
         </geometry>
       </visual>
@@ -130,5 +130,5 @@
         <origin rpy="0 -1.5708 1.5708" xyz="0.02528 0.429 0"/>
         <geometry>
-          <mesh filename="package://dvrk_model/meshes/Classic/psm/outer_insertion.dae"/>
+          <mesh filename="package://dvrk_model/meshes/Classic/PSM/outer_insertion.dae"/>
         </geometry>
       </visual>
@@ -149,5 +149,5 @@
         <origin rpy="0 0 1.5708" xyz="0 0 0.041"/>
         <geometry>
-          <mesh filename="package://dvrk_model/meshes/Classic/psm/tool_main.dae"/>
+          <mesh filename="package://dvrk_model/meshes/Classic/PSM/tool_main.dae"/>
         </geometry>
       </visual>
@@ -166,5 +166,5 @@
         <origin rpy="0 0 1.5708" xyz="0 0 -0.0091"/>
         <geometry>
-          <mesh filename="package://dvrk_model/meshes/Classic/psm/tool_wrist_link.dae"/>
+          <mesh filename="package://dvrk_model/meshes/Classic/PSM/tool_wrist_link.dae"/>
         </geometry>
       </visual>
@@ -182,5 +182,5 @@
         <origin rpy="1.5708 0 0" xyz="0 0.00401 0"/>
         <geometry>
-          <mesh filename="package://dvrk_model/meshes/Classic/psm/tool_wrist_shaft_link.dae"/>
+          <mesh filename="package://dvrk_model/meshes/Classic/PSM/tool_wrist_shaft_link.dae"/>
         </geometry>
       </visual>

File: urdf/Classic/psm_tool_caudier.urdf.xacro (robot description, xacro)
@@ -15,5 +15,5 @@
         <origin rpy="0.00 -1.5708 0.0" xyz="-0.0024 0.00 0.000"/>
         <geometry>
-          <mesh filename="package://dvrk_model/meshes/Classic/psm/tool_wrist_caudier_link_1.stl"/>
+          <mesh filename="package://dvrk_model/meshes/Classic/PSM/tool_wrist_caudier_link_1.stl"/>
         </geometry>
         <material name="gray"><color rgba="0.5 0.5 0.9 1.0"/></material>
@@ -22,5 +22,5 @@
         <origin rpy="0.00 -1.5708 0.0" xyz="-0.0024 0.00 0.000"/>
         <geometry>
-          <mesh filename="package://dvrk_model/meshes/Classic/psm/tool_wrist_caudier_link_1.stl"/>
+          <mesh filename="package://dvrk_model/meshes/Classic/PSM/tool_wrist_caudier_link_1.stl"/>
         </geometry>
       </collision>
@@ -39,5 +39,5 @@
         <origin rpy="0.00 1.5708 0.0" xyz="0.0 -0.0002 0.000"/>
         <geometry>
-          <mesh filename="package://dvrk_model/meshes/Classic/psm/tool_wrist_caudier_link_1_shaft.stl"/>
+          <mesh filename="package://dvrk_model/meshes/Classic/PSM/tool_wrist_caudier_link_1_shaft.stl"/>
         </geometry>
         <material name="gray"><color rgba="0.5 0.5 0.9 1.0"/></material>
@@ -46,5 +46,5 @@
         <origin rpy="0.00 1.5708 0.0" xyz="0.0 0.00 0.000"/>
         <geometry>
-          <mesh filename="package://dvrk_model/meshes/Classic/psm/tool_wrist_caudier_link_1_shaft.stl"/>
+          <mesh filename="package://dvrk_model/meshes/Classic/PSM/tool_wrist_caudier_link_1_shaft.stl"/>
         </geometry>
       </collision>
@@ -81,5 +81,5 @@
         <origin rpy="0.0 0 0.0" xyz="0 0 0.00195"/>
         <geometry>
-          <mesh filename="package://dvrk_model/meshes/Classic/psm/tool_wrist_caudier_link_2.stl"/>
+          <mesh filename="package://dvrk_model/meshes/Classic/PSM/tool_wrist_caudier_link_2.stl"/>
         </geometry>
       </visual>
@@ -99,5 +99,5 @@
         <origin rpy="0 0 -3.1415926" xyz="0 0 0.00195"/>
         <geometry>
-          <mesh filename="package://dvrk_model/meshes/Classic/psm/tool_wrist_caudier_link_2.stl"/>
+          <mesh filename="package://dvrk_model/meshes/Classic/PSM/tool_wrist_caudier_link_2.stl"/>
         </geometry>
       </visual>

File: urdf/Classic/psm_tool_sca.urdf.xacro (robot description, xacro)
@@ -2,5 +2,5 @@
 <robot name="dvrk_psm" xmlns:xacro="http://www.ros.org/wiki/xacro">
   <!-- This file contains different tool urdf -->
-  <xacro:include filename="$(find dvrk_model)/urdf/Classic/common.urdf.xacro"/>
+  <xacro:include filename="$(find dvrk_model)/urdf/common.urdf.xacro"/>
   <!-- sca  -->
   <xacro:macro name="psm_tool_sca" params="prefix">
@@ -19,5 +19,5 @@
         <origin rpy="1.5708 3.1416 0" xyz="0.0051 0.0032 0"/>
         <geometry>
-          <mesh filename="package://dvrk_model/meshes/Classic/psm/tool_wrist_sca_link.dae"/>
+          <mesh filename="package://dvrk_model/meshes/Classic/PSM/tool_wrist_sca_link.dae"/>
         </geometry>
       </visual>
@@ -37,5 +37,5 @@
         <origin rpy="0 0 0" xyz="0 -0.0002 -0.0025"/>
         <geometry>
-          <mesh filename="package://dvrk_model/meshes/Classic/psm/tool_wrist_sca_shaft_link.dae"/>
+          <mesh filename="package://dvrk_model/meshes/Classic/PSM/tool_wrist_sca_shaft_link.dae"/>
         </geometry>
       </visual>
@@ -72,5 +72,5 @@
         <origin rpy="0 0 0" xyz="0 0 0"/>
         <geometry>
-          <mesh filename="package://dvrk_model/meshes/Classic/psm/tool_wrist_sca_link_2.dae"/>
+          <mesh filename="package://dvrk_model/meshes/Classic/PSM/tool_wrist_sca_link_2.dae"/>
         </geometry>
       </visual>
@@ -90,5 +90,5 @@
         <origin rpy="0 3.1516 0" xyz="0 0 0"/>
         <geometry>
-          <mesh filename="package://dvrk_model/meshes/Classic/psm/tool_wrist_sca_link_2.dae"/>
+          <mesh filename="package://dvrk_model/meshes/Classic/PSM/tool_wrist_sca_link_2.dae"/>
         </geometry>
       </visual>

File: urdf/Classic/psm_tool_snake.urdf.xacro (robot description, xacro)
@@ -16,5 +16,5 @@
         <origin rpy="1.5708 0 0" xyz="0.0027 0 0"/>
         <geometry>
-          <mesh filename="package://dvrk_model/meshes/Classic/psm/snake_tool/link_1.STL"/>
+          <mesh filename="package://dvrk_model/meshes/Classic/PSM/snake_tool/link_1.STL"/>
         </geometry>
       </visual>
@@ -33,5 +33,5 @@
         <origin rpy="1.5708 0 0" xyz="0.0027 0 0"/>
         <geometry>
-          <mesh filename="package://dvrk_model/meshes/Classic/psm/snake_tool/link_2.STL"/>
+          <mesh filename="package://dvrk_model/meshes/Classic/PSM/snake_tool/link_2.STL"/>
         </geometry>
       </visual>
@@ -50,5 +50,5 @@
         <origin rpy="1.5708 0 0" xyz="0.0027 0 0"/>
         <geometry>
-          <mesh filename="package://dvrk_model/meshes/Classic/psm/snake_tool/link_3.STL"/>
+          <mesh filename="package://dvrk_model/meshes/Classic/PSM/snake_tool/link_3.STL"/>
         </geometry>
       </visual>
@@ -67,5 +67,5 @@
         <origin rpy="0 1.5708 0" xyz="0 -0.0027 0"/>
         <geometry>
-          <mesh filename="package://dvrk_model/meshes/Classic/psm/snake_tool/link_4.STL"/>
+          <mesh filename="package://dvrk_model/meshes/Classic/PSM/snake_tool/link_4.STL"/>
         </geometry>
       </visual>
@@ -103,5 +103,5 @@
         <origin rpy="-1.5708 -0.7854 0" xyz="0 0 0"/>
         <geometry>
-          <mesh filename="package://dvrk_model/meshes/Classic/psm/snake_tool/gripper_2.STL"/>
+          <mesh filename="package://dvrk_model/meshes/Classic/PSM/snake_tool/gripper_2.STL"/>
         </geometry>
       </visual>
@@ -121,5 +121,5 @@
         <origin rpy="-1.5708 2.3561 0" xyz="0 0 0"/>
         <geometry>
-          <mesh filename="package://dvrk_model/meshes/Classic/psm/snake_tool/gripper_3.STL"/>
+          <mesh filename="package://dvrk_model/meshes/Classic/PSM/snake_tool/gripper_3.STL"/>
         </geometry>
       </visual>

File: urdf/Si/ECM.urdf.xacro (robot description, xacro)
@@ -1,11 +1,10 @@
 <?xml version="1.0" ?>
 <robot name="ECM" xmlns:xacro="http://www.ros.org/wiki/xacro">
-    <xacro:property name="ECM" value="ECM_"/>
     <xacro:include filename="$(find dvrk_model)/urdf/Si/psm_base.urdf.xacro"/>
-    <xacro:include filename="$(find dvrk_model)/urdf/Si/tools.urdf.xacro"/>
+    <xacro:include filename="$(find dvrk_model)/urdf/Si/psm_tool.urdf.xacro"/>
     <link name="world"/>
-    <xacro:psm_arm_active
+    <xacro:psm_base
         prefix="ECM_"
         parent_link="world"/>
-    <xacro:tool tool_name="SF826001" prefix="ECM_" parent_link="ECM_tool_parent"/>
+    <xacro:psm_tool tool_name="SF826001" prefix="ECM_" parent_link="ECM_tool_parent"/>
 </robot>

File: urdf/Si/PSM1.urdf.xacro (robot description, xacro)
@@ -3,9 +3,9 @@
   <xacro:property name="tool_name" value="P420006"/>
   <xacro:include filename="$(find dvrk_model)/urdf/Si/psm_base.urdf.xacro"/>
-  <xacro:include filename="$(find dvrk_model)/urdf/Si/tools.urdf.xacro"/>
+  <xacro:include filename="$(find dvrk_model)/urdf/Si/psm_tool.urdf.xacro"/>
   <link name="world"/>
-  <xacro:psm_arm_active
+  <xacro:psm_base
       prefix="PSM1_"
       parent_link="world"/>
-  <xacro:tool tool_name="${tool_name}" prefix="PSM1_" parent_link="PSM1_tool_parent"/>
+  <xacro:psm_tool tool_name="${tool_name}" prefix="PSM1_" parent_link="PSM1_tool_parent"/>
 </robot>

File: urdf/Si/PSM2.urdf.xacro (robot description, xacro)
@@ -3,9 +3,9 @@
   <xacro:property name="tool_name" value="P420006"/>
   <xacro:include filename="$(find dvrk_model)/urdf/Si/psm_base.urdf.xacro"/>
-  <xacro:include filename="$(find dvrk_model)/urdf/Si/tools.urdf.xacro"/>
+  <xacro:include filename="$(find dvrk_model)/urdf/Si/psm_tool.urdf.xacro"/>
   <link name="world"/>
-  <xacro:psm_arm_active
+  <xacro:psm_base
       prefix="PSM2_"
       parent_link="world"/>
-  <xacro:tool tool_name="${tool_name}" prefix="PSM2_" parent_link="PSM2_tool_parent"/>
+  <xacro:psm_tool tool_name="${tool_name}" prefix="PSM2_" parent_link="PSM2_tool_parent"/>
 </robot>

File: urdf/Si/PSM3.urdf.xacro (robot description, xacro)
@@ -3,9 +3,9 @@
   <xacro:property name="tool_name" value="P420006"/>
   <xacro:include filename="$(find dvrk_model)/urdf/Si/psm_base.urdf.xacro"/>
-  <xacro:include filename="$(find dvrk_model)/urdf/Si/tools.urdf.xacro"/>
+  <xacro:include filename="$(find dvrk_model)/urdf/Si/psm_tool.urdf.xacro"/>
   <link name="world"/>
-  <xacro:psm_arm_active
+  <xacro:psm_base
       prefix="PSM3_"
       parent_link="world"/>
-  <xacro:tool tool_name="${tool_name}" prefix="PSM3_" parent_link="PSM3_tool_parent"/>
+  <xacro:psm_tool tool_name="${tool_name}" prefix="PSM3_" parent_link="PSM3_tool_parent"/>
 </robot>

File: urdf/Si/ecm.urdf.xacro (robot description, xacro)
@@ -1,5 +1,5 @@
 <?xml version="1.0" ?>
-<robot name="PSM" xmlns:xacro="http://www.ros.org/wiki/xacro">
-  <xacro:property name="tool_name" default="P420006"/>
+<robot name="ECM" xmlns:xacro="http://www.ros.org/wiki/xacro">
+  <xacro:property name="tool_name" default="SF826001"/>
   <xacro:property name="arm" default="$(arg arm)"/>
   <xacro:arg name="parent_link_" default="world"/>

File: urdf/Si/patient_cart.urdf.xacro (robot description, xacro)
@@ -9,8 +9,8 @@
     <xacro:property name="PSM3_tool" value="420006"/>
     <xacro:property name="ECM_tool" value="SF826001"/>
-    <xacro:include filename="$(find dvrk_model)/urdf/Si/psm.base.urdf.xacro"/>
+    <xacro:include filename="$(find dvrk_model)/urdf/Si/psm_base.urdf.xacro"/>
     <xacro:include filename="$(find dvrk_model)/urdf/Si/SUJ.urdf.xacro"/>
     <xacro:include filename="$(find dvrk_model)/urdf/Si/SUJ_tower.urdf.xacro"/>
-    <xacro:include filename="$(find dvrk_model)/urdf/Si/tools.urdf.xacro"/>
+    <xacro:include filename="$(find dvrk_model)/urdf/Si/psm_tools.urdf.xacro"/>
     <xacro:suj_tower/>
     <xacro:suj

File: urdf/Si/psm_base.urdf.xacro (robot description, xacro)
@@ -1,5 +1,5 @@
 <?xml version="1.0"?>
 <robot name="dvrk_si" xmlns:xacro="http://www.ros.org/wiki/xacro">
-  <xacro:macro name="psm_arm_active" params="prefix parent_link xyz:='0.0 0.0 0.0' rpy:='0.0 0.0 0.0'">
+  <xacro:macro name="psm_base" params="prefix parent_link xyz:='0.0 0.0 0.0' rpy:='0.0 0.0 0.0'">
     <link
         name="${prefix}link_0">

File: urdf/Si/psm_tool.urdf.xacro (robot description, xacro)
@@ -1,5 +1,5 @@
 <?xml version="1.0"?>
 <robot name="dvrk_si" xmlns:xacro="http://www.ros.org/wiki/xacro">
-  <xacro:macro name="tool" params="tool_name prefix parent_link">
+  <xacro:macro name="psm_tool" params="tool_name prefix parent_link">
     <xacro:if value="${tool_name == 'P420006'}">
       <link
@@ -479,6 +479,6 @@
       </link>
       <joint
-          name="wrist_pitch"
-          type="revolute">
+          name="insertion"
+          type="prismatic">
         <origin
             xyz="0 0 0"
@@ -489,5 +489,5 @@
             link="${prefix}tool_main_link" />
         <axis
-            xyz="0 0 1" />
+            xyz="0 0 -1" />
         <limit
             lower="0"
@@ -537,5 +537,5 @@
       </link>
       <joint
-          name="wrist_yaw"
+          name="roll"
           type="revolute">
         <origin
