Commit message: work in progress: SUJ Classic, imported ECM meshes from WPI

File: urdf/Classic/ECM.urdf.xacro (robot description, xacro)
@@ -5,5 +5,4 @@
   <xacro:ecm_base
       prefix="ECM_"
-      parent_link="world"
-      xyz="0 0.0 0.0" rpy="0.0 0.0 0.0"/>
+      parent_link="world"/>
 </robot>

File: urdf/Classic/SUJ.urdf.xacro (robot description, xacro)
@@ -67,5 +67,5 @@
     <origin
         xyz="0.1912 -0.101599999999999 0.761099999999999"
-        rpy="-3.14159265358979 0 3.14159265358979" />
+        rpy="-${PI} 0.0 ${PI}" />
     <parent
         link="base_link" />
@@ -111,5 +111,5 @@
     <origin
         xyz="0 0 0"
-        rpy="0 0 1.5707963267949" />
+        rpy="0 0 ${PI/2}" />
     <parent
         link="suj_psm2_L0" />
@@ -150,5 +150,5 @@
     <origin
         xyz="0 0.4318 -0.17125"
-        rpy="3.14159265358979 0 1.5707963267949" />
+        rpy="${PI} 0.0 ${PI/2}" />
     <parent
         link="suj_psm2_L1" />
@@ -189,5 +189,5 @@
     <origin
         xyz="0.4318 0 0"
-        rpy="-1.5707963267949 0 -1.5707963267949" />
+        rpy="-${PI/2} 0 -${PI/2}" />
     <parent
         link="suj_psm2_L2" />
@@ -228,5 +228,5 @@
     <origin
         xyz="0 0.0730499999999998 0.0609999999999997"
-        rpy="1.5707963267949 0 3.14159265358979" />
+        rpy="${PI/2} 0.0 ${PI}" />
     <parent
         link="suj_psm2_L3" />
@@ -240,7 +240,6 @@
       name="PSM2_RCM"
       type="fixed">
-    <!-- from DH (??) and (-0.1524 - -0.1029 = -0.0495) -->
-    <origin
-        xyz="0.0 0.83 -0.0495"
+    <origin
+        xyz="0.0 0.8343 -0.04984"
         rpy="0.0 ${PI} 0.0" />
     <parent
@@ -280,5 +279,5 @@
     <origin
         xyz="0 0.0896 0.7611"
-        rpy="3.14159265358979 0 -1.5707963267949" />
+        rpy="${PI} 0 -${PI/2}" />
     <parent
         link="base_link" />
@@ -324,5 +323,5 @@
     <origin
         xyz="0 0 0"
-        rpy="3.14159265358979 0 1.5707963267949" />
+        rpy="${PI} 0 ${PI/2}" />
     <parent
         link="suj_ecm_L0" />
@@ -363,5 +362,5 @@
     <origin
         xyz="0 -0.4318 0.17125"
-        rpy="3.14159265358979 0 -1.5707963267949" />
+        rpy="${PI} 0 -${PI/2}" />
     <parent
         link="suj_ecm_L1" />
@@ -401,6 +400,6 @@
       type="continuous">
     <origin
-        xyz="0.4318 0 0.052"
-        rpy="1.5707963267949 0 3.14159265358979" />
+        xyz="0.4318 0.0 0.052"
+        rpy="${PI/2} 0.0 0.0" />
     <parent
         link="suj_ecm_L2" />
@@ -415,6 +414,6 @@
       type="fixed">
     <origin
-        xyz="0.0 0.0 0.0"
-        rpy="0.0 0.0 0.0" />
+        xyz="-0.45788 0.55053 0.0"
+        rpy="${PI/2} ${PI} -${PI/4}" />
     <parent
         link="suj_ecm_L3" />
@@ -453,5 +452,5 @@
     <origin
         xyz="-0.191199999999999 -0.1016 0.761099999999999"
-        rpy="3.14159265358979 0 0" />
+        rpy="${PI} 0 0" />
     <parent
         link="base_link" />
@@ -497,5 +496,5 @@
     <origin
         xyz="0 0 0"
-        rpy="0 0 1.5707963267949" />
+        rpy="0 0 ${PI/2}" />
     <parent
         link="suj_psm1_L0" />
@@ -536,5 +535,5 @@
     <origin
         xyz="0 0.4318 -0.171250000000001"
-        rpy="3.14159265358979 0 1.5707963267949" />
+        rpy="${PI} 0 ${PI/2}" />
     <parent
         link="suj_psm1_L1" />
@@ -575,5 +574,5 @@
     <origin
         xyz="0.4318 0 0"
-        rpy="1.5707963267949 0 -1.5707963267949" />
+        rpy="${PI/2} 0 -${PI/2}" />
     <parent
         link="suj_psm1_L2" />
@@ -614,5 +613,5 @@
     <origin
         xyz="0 -0.0730499999999998 -0.0609999999999999"
-        rpy="-1.5707963267949 0 3.14159265358979" />
+        rpy="-${PI/2} 0 ${PI}" />
     <parent
         link="suj_psm1_L3" />
@@ -627,5 +626,5 @@
       type="fixed">
     <origin
-        xyz="0.0 0.83 -0.0495"
+        xyz="0.0 0.8343 -0.04984"
         rpy="0.0 ${PI} 0.0" />
     <parent
@@ -665,5 +664,5 @@
     <origin
         xyz="0 0.0895999999999999 0.3813"
-        rpy="3.14159265358979 0 -1.5707963267949" />
+        rpy="${PI} 0 -${PI/2}" />
     <parent
         link="base_link" />
@@ -709,5 +708,5 @@
     <origin
         xyz="0 0 0"
-        rpy="3.14159265358979 0 1.5707963267949" />
+        rpy="${PI} 0 ${PI/2}" />
     <parent
         link="suj_psm3_L0" />
@@ -748,5 +747,5 @@
     <origin
         xyz="0 -0.5842 -0.000249999999999639"
-        rpy="3.14159265358979 0 -1.5707963267949" />
+        rpy="${PI} 0 -${PI/2}" />
     <parent
         link="suj_psm3_L1" />
@@ -787,5 +786,5 @@
     <origin
         xyz="0.431800000000001 0 0"
-        rpy="1.5707963267949 0 -1.5707963267949" />
+        rpy="${PI/2} 0 -${PI/2}" />
     <parent
         link="suj_psm3_L2" />
@@ -826,5 +825,5 @@
     <origin
         xyz="0 -0.199949999999999 -0.061"
-        rpy="-1.5707963267949 0 0" />
+        rpy="-${PI/2} 0 0" />
     <parent
         link="suj_psm3_L3" />
@@ -839,5 +838,5 @@
       type="fixed">
     <origin
-        xyz="0.0 0.83 -0.0495"
+        xyz="0.0 0.8343 -0.04984"
         rpy="0.0 ${PI} 0.0" />
     <parent

File: urdf/Classic/ecm_base.urdf.xacro (robot description, xacro)
@@ -4,177 +4,446 @@
   <xacro:include filename="$(find dvrk_model)/urdf/common.urdf.xacro"/>
   <!-- Macro for da Vinci Endoscope Camera Manipulator (ECM) -->
-  <xacro:macro name="ecm_base" params="prefix parent_link xyz:='0.0 0.0 0.0' rpy:='0.0 0.0 0.0'">
-    <!-- Joint 0: Fixed to World-->
-    <joint name="fixed" type="fixed">
+  <xacro:macro name="ecm_base" params="prefix parent_link xyz:='-0.612599 0.0 -0.101595' rpy:='0.0 0.0 0.0'">
+    <!-- Joint 0: Fixed to Setup Joint-->
+    <joint name="fixed_joint" type="fixed">
       <parent link="${parent_link}"/>
-      <child link="${prefix}_base_link"/>
+      <child link="${prefix}base_link"/>
       <origin rpy="${rpy}" xyz="${xyz}"/>
     </joint>
-    <link name="${prefix}_base_link"/>
-    <!-- Joint 1: Outer Yaw -->
-    <joint name="yaw" type="revolute">
-      <parent link="${prefix}_base_link"/>
-      <child link="${prefix}_yaw_link"/>
-      <origin rpy="0 -${PI/2} ${PI/2}" xyz="0 0 0"/>
-      <axis xyz="0 0 1"/>
-      <!--rotates about z axis-->
-      <!--limit effort and velocity picked arbitrarily check-->
-      <limit effort="50.0" lower="${-75/180*PI}" upper="${PI/4}" velocity="2"/>
-      <joint_properties damping="1.0" friction="0.0"/>
-    </joint>
-    <link name="${prefix}_yaw_link">
-      <visual>
-        <origin rpy="0 0 -${PI/2}" xyz="0 0 0.603"/>
-        <geometry>
-          <mesh filename="package://dvrk_model/meshes/Classic/ECM/ecm_yaw_link.stl"/>
-        </geometry>
-	<material name="DaVinciGreen"/>
-      </visual>
-      <collision>
-        <origin rpy="0 0 -${PI/2}" xyz="0 0 0.603"/>
-        <geometry>
-          <mesh filename="package://dvrk_model/meshes/Classic/ECM/ecm_yaw_link.stl"/>
-        </geometry>
-      </collision>
-    </link>
-    <!-- Joint 2: Pitch -->
-    <joint name="pitch" type="revolute">
-      <parent link="${prefix}_yaw_link"/>
-      <child link="${prefix}_pitch_link"/>
-      <origin rpy="-${PI/2} -${PI/2} 0" xyz="0 0 0"/>
-      <axis xyz="0 0 1"/>
-      <limit effort="100.0" lower="${-PI/4}" upper="${PI*65/180}" velocity="10"/>
-      <joint_properties damping="1.0" friction="0.0"/>
-    </joint>
-    <link name="${prefix}_pitch_link"/>
-    <joint name="pitch_0" type="continuous">
-      <parent link="${prefix}_yaw_link"/>
-      <child link="${prefix}_pitch_link_1"/>
-      <origin rpy="-${PI/2} -${PI/2} 0" xyz="0 0 0.378"/>
-      <axis xyz="0 0 1"/>
-      <joint_properties damping="1.0" friction="0.0"/>
+    <link
+      name="${prefix}base_link">
+      <visual>
+        <origin
+          xyz="0 0 0"
+          rpy="0 0 0" />
+        <geometry>
+          <mesh
+            filename="package://dvrk_model/meshes/Classic/ECM/ecm_base_link.stl" />
+        </geometry>
+        <material
+          name="">
+          <color
+            rgba="0.64706 0.61961 0.58824 1" />
+        </material>
+      </visual>
+      <collision>
+        <origin
+          xyz="0 0 0"
+          rpy="0 0 0" />
+        <geometry>
+          <mesh
+            filename="package://dvrk_model/meshes/Classic/ECM/ecm_base_link.stl" />
+        </geometry>
+      </collision>
+    </link>
+    <link
+      name="${prefix}yaw_link">
+      <visual>
+        <origin
+          xyz="0 0 0"
+          rpy="0 0 0" />
+        <geometry>
+          <mesh
+            filename="package://dvrk_model/meshes/Classic/ECM/ecm_yaw_link.stl" />
+        </geometry>
+        <material
+          name="">
+          <color
+            rgba="0.64706 0.61961 0.58824 1" />
+        </material>
+      </visual>
+      <collision>
+        <origin
+          xyz="0 0 0"
+          rpy="0 0 0" />
+        <geometry>
+          <mesh
+            filename="package://dvrk_model/meshes/Classic/ECM/ecm_yaw_link.stl" />
+        </geometry>
+      </collision>
+    </link>
+    <joint
+      name="yaw"
+      type="revolute">
+      <origin
+        xyz="0.0731999999999783 0 0.101460000000185"
+        rpy="1.57079632679615 0 1.5707963267949" />
+      <parent
+        link="${prefix}base_link" />
+      <child
+        link="${prefix}yaw_link" />
+      <axis
+        xyz="0 0 1" />
+      <limit
+        lower="-1.595183"
+        upper="1.581733"
+        effort="1000"
+        velocity="10" />
+    </joint>
+    <link
+      name="${prefix}pitch_front_link">
+      <visual>
+        <origin
+          xyz="0 0 0"
+          rpy="0 0 0" />
+        <geometry>
+          <mesh
+            filename="package://dvrk_model/meshes/Classic/ECM/ecm_pitch_front_link.stl" />
+        </geometry>
+        <material
+          name="">
+          <color
+            rgba="0.64706 0.61961 0.58824 1" />
+        </material>
+      </visual>
+      <collision>
+        <origin
+          xyz="0 0 0"
+          rpy="0 0 0" />
+        <geometry>
+          <mesh
+            filename="package://dvrk_model/meshes/Classic/ECM/ecm_pitch_front_link.stl" />
+        </geometry>
+      </collision>
+    </link>
+    <joint
+      name="pitch"
+      type="revolute">
+      <origin
+        xyz="0 0 0.199000000000014"
+        rpy="3.14 -1.5707963267949 0" />
+      <parent
+        link="${prefix}yaw_link" />
+      <child
+        link="${prefix}pitch_front_link" />
+      <axis
+        xyz="0 0 1" />
+      <limit
+        lower="-0.783710"
+        upper="1.157657"
+        effort="1000"
+        velocity="10" />
+    </joint>
+    <link
+      name="${prefix}pitch_bottom_link">
+      <visual>
+        <origin
+          xyz="0 0 0"
+          rpy="0 0 0" />
+        <geometry>
+          <mesh
+            filename="package://dvrk_model/meshes/Classic/ECM/ecm_pitch_bottom_link.stl" />
+        </geometry>
+        <material
+          name="">
+          <color
+            rgba="0.25098 0.25098 0.25098 1" />
+        </material>
+      </visual>
+      <collision>
+        <origin
+          xyz="0 0 0"
+          rpy="0 0 0" />
+        <geometry>
+          <mesh
+            filename="package://dvrk_model/meshes/Classic/ECM/ecm_pitch_bottom_link.stl" />
+        </geometry>
+      </collision>
+    </link>
+    <joint
+      name="pitch_bottom"
+      type="revolute">
+      <origin
+        xyz="-0.103000865501078 -0.286804989831434 0"
+        rpy="0 0 0" />
+      <parent
+        link="${prefix}pitch_front_link" />
+      <child
+        link="${prefix}pitch_bottom_link" />
+      <axis
+        xyz="0 0 1" />
+      <limit
+        lower="-1.157657"
+        upper="0.783710"
+        effort="1000"
+        velocity="10" />
+      <mimic joint="pitch" multiplier="-1"/>
+    </joint>
+    <link
+      name="${prefix}pitch_end_link">
+      <visual>
+        <origin
+          xyz="0 0 0"
+          rpy="0 0 0" />
+        <geometry>
+          <mesh
+            filename="package://dvrk_model/meshes/Classic/ECM/ecm_pitch_end_link.stl" />
+        </geometry>
+        <material
+          name="">
+          <color
+            rgba="0.89804 0.91765 0.92941 1" />
+        </material>
+      </visual>
+      <collision>
+        <origin
+          xyz="0 0 0"
+          rpy="0 0 0" />
+        <geometry>
+          <mesh
+            filename="package://dvrk_model/meshes/Classic/ECM/ecm_pitch_end_link.stl" />
+        </geometry>
+      </collision>
+    </link>
+    <joint
+      name="pitch_end"
+      type="revolute">
+      <origin
+        xyz="0.340400072983362 -0.000135620545844151 0"
+        rpy="0 0 0" />
+      <parent
+        link="${prefix}pitch_bottom_link" />
+      <child
+        link="${prefix}pitch_end_link" />
+      <axis
+        xyz="0 0 1" />
+      <limit
+        lower="-0.783710"
+        upper="1.157657"
+        effort="1000"
+        velocity="10" />
       <mimic joint="pitch" multiplier="1"/>
     </joint>
-    <link name="${prefix}_pitch_link_1">
-      <visual>
-        <origin rpy="0 0 0" xyz="0 0 0"/>
-        <geometry>
-          <mesh filename="package://dvrk_model/meshes/Classic/ECM/ecm_pitch_link_1.stl"/>
-        </geometry>
-	<material name="DaVinciMedGray"/>
-      </visual>
-      <collision>
-        <origin rpy="0 0 0" xyz="0 0 0"/>
-        <geometry>
-          <mesh filename="package://dvrk_model/meshes/Classic/ECM/ecm_pitch_link_1.stl"/>
-        </geometry>
-      </collision>
-      <inertial>
-        <mass value=".9"/>
-        <inertia ixx="9.0" ixy="0.0" ixz="0.0" iyy="9.0" iyz="0.0" izz="9.0"/>
-      </inertial>
-    </link>
-    <joint name="pitch_1" type="continuous">
-      <parent link="${prefix}_pitch_link_1"/>
-      <child link="${prefix}_pitch_link_2"/>
-      <origin rpy="0 0 0" xyz="0.0558629 0.274575 0"/>
-      <axis xyz="0 0 1"/>
-      <joint_properties damping="1.0" friction="0.0"/>
+    <link
+      name="${prefix}main_insertion_link">
+      <visual>
+        <origin
+          xyz="0 0 0"
+          rpy="0 0 0" />
+        <geometry>
+          <mesh
+            filename="package://dvrk_model/meshes/Classic/ECM/ecm_main_insertion_link.stl" />
+        </geometry>
+        <material
+          name="">
+          <color
+            rgba="0.25 0.25 0.25 1" />
+        </material>
+      </visual>
+      <collision>
+        <origin
+          xyz="0 0 0"
+          rpy="0 0 0" />
+        <geometry>
+          <mesh
+            filename="package://dvrk_model/meshes/Classic/ECM/ecm_main_insertion_link.stl" />
+        </geometry>
+      </collision>
+    </link>
+    <joint
+      name="insertion"
+      type="prismatic">
+      <origin
+        xyz="0.042 -0.086143 0"
+        rpy="-1.5708 0 0" />
+      <parent
+        link="${prefix}pitch_end_link" />
+      <child
+        link="${prefix}main_insertion_link" />
+      <axis
+        xyz="0 0 1" />
+      <limit
+        lower="0"
+        upper="0.254193"
+        effort="50"
+        velocity="100" />
+    </joint>
+    <link
+      name="${prefix}tool_link">
+      <visual>
+        <origin
+          xyz="0 0 0"
+          rpy="0 0 0" />
+        <geometry>
+          <mesh
+            filename="package://dvrk_model/meshes/Classic/ECM/ecm_tool_link.stl" />
+        </geometry>
+        <material
+          name="">
+          <color
+            rgba="0.7 0.7 0.7 1" />
+        </material>
+      </visual>
+      <collision>
+        <origin
+          xyz="0 0 0"
+          rpy="0 0 0" />
+        <geometry>
+          <mesh
+            filename="package://dvrk_model/meshes/Classic/ECM/ecm_tool_link.stl" />
+        </geometry>
+      </collision>
+    </link>
+    <joint
+      name="roll"
+      type="revolute">
+      <origin
+        xyz="0.0609999999999996 0 0"
+        rpy="0 0 0" />
+      <parent
+        link="${prefix}main_insertion_link" />
+      <child
+        link="${prefix}tool_link" />
+      <axis
+        xyz="0 0 -1" />
+      <limit
+        lower="-1.552676"
+        upper="1.566741"
+        effort="1000"
+        velocity="10" />
+    </joint>
+    <link
+      name="${prefix}pitch_top_link">
+      <visual>
+        <origin
+          xyz="0 0 0"
+          rpy="0 0 0" />
+        <geometry>
+          <mesh
+            filename="package://dvrk_model/meshes/Classic/ECM/ecm_pitch_top_link.stl" />
+        </geometry>
+        <material
+          name="">
+          <color
+            rgba="0.64706 0.51765 0 1" />
+        </material>
+      </visual>
+      <collision>
+        <origin
+          xyz="0 0 0"
+          rpy="0 0 0" />
+        <geometry>
+          <mesh
+            filename="package://dvrk_model/meshes/Classic/ECM/ecm_pitch_top_link.stl" />
+        </geometry>
+      </collision>
+    </link>
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