Commit message: fix uppercase urdf and link naming

File: urdf/Classic/ECM.urdf.xacro (robot description, xacro)
@@ -1,8 +1,10 @@
 <?xml version="1.0" ?>
 <robot name="ECM" xmlns:xacro="http://www.ros.org/wiki/xacro">
+  <xacro:arg name="parent_link_" default="world"/>
+  <xacro:property name="parent_link" default="$(arg parent_link_)"/>
   <xacro:include filename="$(find dvrk_model)/urdf/Classic/ecm_base.urdf.xacro"/>
-  <link name="world"/>
+  <link name="${parent_link}"/>
   <xacro:ecm_base
       prefix="ECM_"
-      parent_link="world"/>
+      parent_link="${parent_link}"/>
 </robot>

File: urdf/Classic/PSM1.urdf.xacro (robot description, xacro)
@@ -7,12 +7,14 @@
   -->
   <xacro:arg name="instrument" default="400006"/>
+  <xacro:arg name="parent_link_" default="world"/>
+  <xacro:property name="parent_link" default="$(arg parent_link_)"/>
   <xacro:include filename="$(find dvrk_model)/urdf/Classic/PSM_base.urdf.xacro"/>
   <xacro:include filename="$(find dvrk_model)/urdf/common/PSM_instrument.urdf.xacro"/>
-  <link name="world"/>
+  <link name="${parent_link}"/>
   <xacro:base prefix="PSM1_"
-                  parent_link="world"
+                  parent_link="${parent_link}"
                   xyz="-0.25 0.0 0.5" rpy="0.0 0.0 ${PI}"/>
   <xacro:PSM_instrument prefix="PSM1_"
-                        parent_link="PSM1_PSM_tool_parent_link"
+                        parent_link="PSM1_tool_parent_link"
                         instrument="$(arg instrument)"/>
 </robot>

File: urdf/Classic/PSM2.urdf.xacro (robot description, xacro)
@@ -2,12 +2,14 @@
 <robot name="PSM2" xmlns:xacro="http://www.ros.org/wiki/xacro">
   <xacro:arg name="instrument" default="400049"/>
+  <xacro:arg name="parent_link_" default="world"/>
+  <xacro:property name="parent_link" default="$(arg parent_link_)"/>
   <xacro:include filename="$(find dvrk_model)/urdf/Classic/PSM_base.urdf.xacro"/>
   <xacro:include filename="$(find dvrk_model)/urdf/common/PSM_instrument.urdf.xacro"/>
-  <link name="world"/>
+  <link name="${parent_link}"/>
   <xacro:base prefix="PSM2_"
-                  parent_link="world"
+                  parent_link="${parent_link}"
                   xyz="-0.25 0.0 0.5" rpy="0.0 0.0 ${PI}"/>
   <xacro:PSM_instrument prefix="PSM2_"
-                        parent_link="PSM2_PSM_tool_parent_link"
+                        parent_link="PSM2_tool_parent_link"
                         instrument="$(arg instrument)"/>
 </robot>

File: urdf/Classic/PSM3.urdf.xacro (robot description, xacro)
@@ -2,12 +2,14 @@
 <robot name="PSM3" xmlns:xacro="http://www.ros.org/wiki/xacro">
   <xacro:arg name="instrument" default="400049"/>
+  <xacro:arg name="parent_link_" default="world"/>
+  <xacro:property name="parent_link" default="$(arg parent_link_)"/>
   <xacro:include filename="$(find dvrk_model)/urdf/Classic/PSM_base.urdf.xacro"/>
   <xacro:include filename="$(find dvrk_model)/urdf/common/PSM_instrument.urdf.xacro"/>
-  <link name="world"/>
+  <link name="${parent_link}"/>
   <xacro:base prefix="PSM3_"
-                  parent_link="world"
+                  parent_link="${parent_link}"
                   xyz="0.50 0.0 0.5" rpy="0.0 0.0 ${-PI}"/>
   <xacro:PSM_instrument prefix="PSM3_"
-                        parent_link="PSM3_PSM_tool_parent_link"
+                        parent_link="PSM3_tool_parent_link"
                         instrument="$(arg instrument)"/>
 </robot>

File: urdf/Classic/PSM_base.urdf.xacro (robot description, xacro)
@@ -153,5 +153,5 @@
       link 3: tool_parent_link
       Massless boundary link — handoff point to PSM_instrument.
-      No mesh; both Classic and Virtual use this exact link name
+      No mesh; both Si and Classic use this exact link name
       so PSM_instrument is generation-agnostic.
     -->

File: urdf/Si/ECM.urdf.xacro (robot description, xacro)
@@ -1,12 +1,13 @@
 <?xml version="1.0" ?>
 <robot name="ECM" xmlns:xacro="http://www.ros.org/wiki/xacro">
+  <xacro:arg name="parent_link_" default="world"/>
+  <xacro:property name="parent_link" default="$(arg parent_link_)"/>
   <xacro:include filename="$(find dvrk_model)/urdf/Si/PSM_base.urdf.xacro"/>
   <xacro:include filename="$(find dvrk_model)/urdf/common/PSM_instrument.urdf.xacro"/>
-  <link name="world"/>
+  <link name="${parent_link}"/>
   <xacro:base prefix="ECM_"
-                  parent_link="world"/>
+                  parent_link="${parent_link}"/>
   <xacro:PSM_instrument prefix="ECM_"
-                        parent_link="ECM_PSM_tool_parent_link"
-                        shaft_length="0.4670"
+                        parent_link="ECM_tool_parent_link"
                         instrument="SF0826001"/>
 </robot>

File: urdf/Si/PSM1.urdf.xacro (robot description, xacro)
@@ -6,11 +6,13 @@
   -->
   <xacro:arg name="instrument" default="420006"/>
+  <xacro:arg name="parent_link_" default="world"/>
+  <xacro:property name="parent_link" default="$(arg parent_link_)"/>
   <xacro:include filename="$(find dvrk_model)/urdf/Si/PSM_base.urdf.xacro"/>
   <xacro:include filename="$(find dvrk_model)/urdf/common/PSM_instrument.urdf.xacro"/>
-  <link name="world"/>
+  <link name="${parent_link}"/>
   <xacro:base prefix="PSM1_"
-                  parent_link="world"/>
+                  parent_link="${parent_link}"/>
   <xacro:PSM_instrument prefix="PSM1_"
-                        parent_link="PSM1_PSM_tool_parent_link"
+                        parent_link="PSM1_tool_parent_link"
                         instrument="$(arg instrument)"/>
 </robot>

File: urdf/Si/PSM2.urdf.xacro (robot description, xacro)
@@ -2,11 +2,13 @@
 <robot name="PSM2" xmlns:xacro="http://www.ros.org/wiki/xacro">
   <xacro:arg name="instrument" default="420006"/>
+  <xacro:arg name="parent_link_" default="world"/>
+  <xacro:property name="parent_link" default="$(arg parent_link_)"/>
   <xacro:include filename="$(find dvrk_model)/urdf/Si/PSM_base.urdf.xacro"/>
   <xacro:include filename="$(find dvrk_model)/urdf/common/PSM_instrument.urdf.xacro"/>
-  <link name="world"/>
+  <link name="${parent_link}"/>
   <xacro:base prefix="PSM2_"
-                  parent_link="world"/>
+                  parent_link="${parent_link}"/>
   <xacro:PSM_instrument prefix="PSM2_"
-                        parent_link="PSM2_PSM_tool_parent_link"
+                        parent_link="PSM2_tool_parent_link"
                         instrument="$(arg instrument)"/>
 </robot>

File: urdf/Si/PSM3.urdf.xacro (robot description, xacro)
@@ -2,11 +2,13 @@
 <robot name="PSM3" xmlns:xacro="http://www.ros.org/wiki/xacro">
   <xacro:arg name="instrument" default="420006"/>
+  <xacro:arg name="parent_link_" default="world"/>
+  <xacro:property name="parent_link" default="$(arg parent_link_)"/>
   <xacro:include filename="$(find dvrk_model)/urdf/Si/PSM_base.urdf.xacro"/>
   <xacro:include filename="$(find dvrk_model)/urdf/common/PSM_instrument.urdf.xacro"/>
-  <link name="world"/>
+  <link name="${parent_link}"/>
   <xacro:base prefix="PSM3_"
-                  parent_link="world"/>
+                  parent_link="${parent_link}"/>
   <xacro:PSM_instrument prefix="PSM3_"
-                        parent_link="PSM3_PSM_tool_parent_link"
+                        parent_link="PSM3_tool_parent_link"
                         instrument="$(arg instrument)"/>
 </robot>

File: urdf/Si/PSM_base.urdf.xacro (robot description, xacro)
@@ -7,5 +7,5 @@
       Joint 2: pitch  (revolute, pitch, parallelogram linkage ×3)
       Joint 3: insertion (prismatic)
-    Macro output: ends at ${prefix}PSM_tool_parent_link.
+    Macro output: ends at ${prefix}tool_parent_link.
     PSM_instrument attaches here and owns roll onward.
     Inertial data retained from original Si CAD export.
@@ -16,5 +16,5 @@
                        rpy:='0.0 0.0 0.0'">
     <!-- link 0: arm base -->
-    <link name="${prefix}USM_base_link">
+    <link name="${prefix}base_link">
       <inertial>
         <origin xyz="-0.080771 2.1131E-08 1.8613E-07" rpy="0 0 0"/>
@@ -41,9 +41,9 @@
     <joint name="${prefix}base_fixed" type="fixed">
       <parent link="${parent_link}"/>
-      <child  link="${prefix}USM_base_link"/>
+      <child  link="${prefix}base_link"/>
       <origin rpy="${rpy}" xyz="${xyz}"/>
     </joint>
     <!-- link 1: yaw body -->
-    <link name="${prefix}USM_yaw_link">
+    <link name="${prefix}yaw_link">
       <inertial>
         <origin xyz="0.1461 0.090363 -0.024957" rpy="0 0 0"/>
@@ -70,11 +70,11 @@
     <joint name="yaw" type="revolute">
       <origin xyz="0.158 0 0" rpy="0.0 0.0 0.0"/>
-      <parent link="${prefix}USM_base_link"/>
-      <child  link="${prefix}USM_yaw_link"/>
+      <parent link="${prefix}base_link"/>
+      <child  link="${prefix}yaw_link"/>
       <axis xyz="-1.0 0.0 0.0"/>
       <limit lower="-3.14" upper="3.14" effort="0.0" velocity="0.0"/>
     </joint>
     <!-- link 2: pitch arm -->
-    <link name="${prefix}USM_pitch_link">
+    <link name="${prefix}pitch_link">
       <inertial>
         <origin xyz="0.083895 -0.00073113 -0.028998" rpy="0.0 0.0 0.0"/>
@@ -101,11 +101,11 @@
     <joint name="pitch" type="revolute">
       <origin xyz="0.2987 0 -0.071222" rpy="0 -1.1345 -3.1416"/>
-      <parent link="${prefix}USM_yaw_link"/>
-      <child  link="${prefix}USM_pitch_link"/>
+      <parent link="${prefix}yaw_link"/>
+      <child  link="${prefix}pitch_link"/>
       <axis xyz="0 -1 0"/>
       <limit lower="-3.14" upper="3.14" effort="0" velocity="0"/>
     </joint>
     <!-- link 3: pitch parallelogram arm (mimic pitch) -->
-    <link name="${prefix}USM_pitch_3_link">
+    <link name="${prefix}pitch_3_link">
       <inertial>
         <origin xyz="0.11824 1.9336E-19 0.12932" rpy="0 0 0"/>
@@ -131,6 +131,6 @@
     <joint name="pitch_2" type="revolute">
       <origin xyz="0.2032 0 0" rpy="0 -0.90761 -3.1416"/>
-      <parent link="${prefix}USM_pitch_link"/>
-      <child  link="${prefix}USM_pitch_3_link"/>
+      <parent link="${prefix}pitch_link"/>
+      <child  link="${prefix}pitch_3_link"/>
       <axis xyz="0 1 0"/>
       <limit lower="-3.14" upper="3.14" effort="0" velocity="0"/>
@@ -138,5 +138,5 @@
     </joint>
     <!-- link 4: pitch parallelogram distal (mimic pitch) -->
-    <link name="${prefix}USM_pitch_4_link">
+    <link name="${prefix}pitch_4_link">
       <inertial>
         <origin xyz="0.041219 -9.0734E-08 0.13651" rpy="0 0 0"/>
@@ -162,6 +162,6 @@
     <joint name="pitch_3" type="revolute">
       <origin xyz="0.35966 0 0.16013" rpy="0 -0.063963 0"/>
-      <parent link="${prefix}USM_pitch_3_link"/>
-      <child  link="${prefix}USM_pitch_4_link"/>
+      <parent link="${prefix}pitch_3_link"/>
+      <child  link="${prefix}pitch_4_link"/>
       <axis xyz="0 1 0"/>
       <limit lower="-3.14" upper="3.14" effort="0" velocity="0"/>
@@ -175,21 +175,21 @@
     <joint name="insertion" type="prismatic">
       <origin xyz="0.05061 0 0.41911" rpy="${PI} 0 0"/>
-      <parent link="${prefix}USM_pitch_4_link"/>
-      <child  link="${prefix}PSM_tool_parent_link"/>
+      <parent link="${prefix}pitch_4_link"/>
+      <child  link="${prefix}tool_parent_link"/>
       <axis xyz="0 0 1"/>
       <limit lower="0.0" upper="0.299" velocity="0.4" effort="1000"/>
     </joint>
     <!--
-      PSM_tool_parent_link — boundary link; PSM_instrument attaches here.
+      tool_parent_link — boundary link; PSM_instrument attaches here.
       No geometry; same name as Classic and Virtual so PSM_instrument
       macro is generation-agnostic.
     -->
-    <link name="${prefix}PSM_tool_parent_link"/>
+    <link name="${prefix}tool_parent_link"/>
     <!-- RCM reference frame (kept for any downstream code that uses it) -->
-    <link name="${prefix}PSM_RCM_link"/>
+    <link name="${prefix}RCM_link"/>
     <joint name="${prefix}jrcm" type="fixed">
       <origin xyz="0.10643 0 -0.1731" rpy="3.1416 0 -1.5708"/>
-      <parent link="${prefix}USM_pitch_4_link"/>
-      <child  link="${prefix}PSM_RCM_link"/>
+      <parent link="${prefix}pitch_4_link"/>
+      <child  link="${prefix}RCM_link"/>
       <axis xyz="0 0 0"/>
     </joint>

File: urdf/Virtual/PSM1.urdf.xacro (robot description, xacro)
@@ -21,5 +21,5 @@
   <!-- Instrument: identical to Classic/Si — attaches at PSM_tool_parent_link -->
   <xacro:PSM_instrument prefix="PSM1_"
-                        parent_link="PSM1_PSM_tool_parent_link"
+                        parent_link="PSM1_tool_parent_link"
                         instrument="$(arg instrument)"/>
 </robot>

File: urdf/Virtual/PSM2.urdf.xacro (robot description, xacro)
@@ -11,5 +11,5 @@
                           rcm_rpy="$(arg rcm_rpy)"/>
   <xacro:PSM_instrument prefix="PSM2_"
-                        parent_link="PSM2_PSM_tool_parent_link"
+                        parent_link="PSM2_tool_parent_link"
                         instrument="$(arg instrument)"/>
 </robot>

File: urdf/Virtual/PSM3.urdf.xacro (robot description, xacro)
@@ -11,5 +11,5 @@
                           rcm_rpy="$(arg rcm_rpy)"/>
   <xacro:PSM_instrument prefix="PSM3_"
-                        parent_link="PSM3_PSM_tool_parent_link"
+                        parent_link="PSM3_tool_parent_link"
                         instrument="$(arg instrument)"/>
 </robot>

File: urdf/Virtual/PSM_base_virtual.urdf.xacro (robot description, xacro)
@@ -12,5 +12,5 @@
     All three links share a small but non-zero inertia so physics
     simulators (Gazebo, Isaac) can integrate without singularities.
-    Output: ends at ${prefix}PSM_tool_parent_link — identical to the
+    Output: ends at ${prefix}tool_parent_link — identical to the
     full Classic/Si base so PSM_instrument attaches without modification.
     Parameters:
@@ -29,14 +29,14 @@
     <joint name="${prefix}RCM_fixed" type="fixed">
       <parent link="world"/>
-      <child  link="${prefix}PSM_RCM_link"/>
+      <child  link="${prefix}RCM_link"/>
       <origin xyz="${rcm_xyz}" rpy="${rcm_rpy}"/>
     </joint>
     <!-- RCM frame link — not a DOF, just a named coordinate frame -->
-    <link name="${prefix}PSM_RCM_link"/>
+    <link name="${prefix}RCM_link"/>
     <!-- ── Joint 1: yaw ───────────────────────────────────────────── -->
     <!--   Revolute about z at the RCM. Models the yaw of the PSM arm.      -->
     <joint name="yaw" type="revolute">
-      <parent link="${prefix}PSM_RCM_link"/>
-      <child  link="${prefix}PSM_RCM_yaw_link"/>
+      <parent link="${prefix}RCM_link"/>
+      <child  link="${prefix}RCM_yaw_link"/>
       <axis xyz="0 0 1"/>
       <origin xyz="0 0 0" rpy="0 0 0"/>
@@ -44,5 +44,5 @@
              effort="50" velocity="1.0"/>
     </joint>
-    <link name="${prefix}PSM_RCM_yaw_link">
+    <link name="${prefix}RCM_yaw_link">
       <inertial>
         <mass value="${virtual_mass}"/>
@@ -55,6 +55,6 @@
     <!--   Revolute about y at the RCM. Models the pitch of the PSM arm.    -->
     <joint name="pitch" type="revolute">
-      <parent link="${prefix}PSM_RCM_yaw_link"/>
-      <child  link="${prefix}PSM_RCM_pitch_link"/>
+      <parent link="${prefix}RCM_yaw_link"/>
+      <child  link="${prefix}RCM_pitch_link"/>
       <axis xyz="0 1 0"/>
       <origin xyz="0 0 0" rpy="0 0 0"/>
@@ -62,5 +62,5 @@
              effort="50" velocity="1.0"/>
     </joint>
-    <link name="${prefix}PSM_RCM_pitch_link">
+    <link name="${prefix}RCM_pitch_link">
       <inertial>
         <mass value="${virtual_mass}"/>
@@ -72,9 +72,9 @@
     <!-- ── Joint 3: insertion ───────────────────────────────────────────── -->
     <!--   Prismatic along z at the RCM. Models insertion depth.            -->
-    <!--   PSM_tool_parent_link serves as the insertion child AND the        -->
+    <!--   tool_parent_link serves as the insertion child AND the        -->
     <!--   handoff link to PSM_instrument (same name as in Classic/Si base). -->
     <joint name="insertion" type="prismatic">
-      <parent link="${prefix}PSM_RCM_pitch_link"/>
-      <child  link="${prefix}PSM_tool_parent_link"/>
+      <parent link="${prefix}RCM_pitch_link"/>
+      <child  link="${prefix}tool_parent_link"/>
       <axis xyz="0 0 1"/>
       <origin xyz="0 0 0" rpy="0 0 0"/>
@@ -83,8 +83,8 @@
     </joint>
     <!--
-      PSM_tool_parent_link — identical name to Classic/Si boundary link.
+      tool_parent_link — identical name to Classic/Si boundary link.
       PSM_instrument attaches here; no change needed for any generation.
     -->
-    <link name="${prefix}PSM_tool_parent_link">
+    <link name="${prefix}tool_parent_link">
       <inertial>
         <mass value="${virtual_mass}"/>
