Commit message: fix uppercase urdf and link naming

File: urdf/common/PSM_instrument.urdf.xacro (robot description, xacro)
@@ -3,5 +3,5 @@
   <!--
     PSM instrument macro — generation-agnostic.
-    Attaches to ${parent_link} (= ${prefix}PSM_tool_parent_link from any
+    Attaches to ${parent_link} (= ${prefix}tool_parent_link from any
     PSM_base variant: Classic, Si, or Virtual).
     DOF layout:
@@ -12,5 +12,5 @@
     Parameters:
       prefix        — arm instance prefix, e.g. "PSM1_"
-      parent_link   — must be ${prefix}PSM_tool_parent_link
+      parent_link   — must be ${prefix}tool_parent_link
       shaft_length  — D parameter of roll joint (Classic: 0.4162, Si: 0.4670)
       instrument    — last 6 digits of instrument model number (e.g. "420006")
@@ -21,23 +21,29 @@
   <xacro:macro name="PSM_instrument"
                params="prefix parent_link instrument">
-    <!-- Detect if this is an Si generation instrument (42xxxx) -->
-    <xacro:property name="is_si" value="${str(instrument).startswith('42')}"/>
-    <!-- Dynamically select the correct shaft length based on generation -->
-    <xacro:property name="shaft_length" value="${0.53559 if is_si else 0.4162}"/> <!--0.4670 for Si as also in strucuture.md-->
+    <!-- Detect generation. ECM (SF0826001) uses Si-style mesh format. -->
+    <xacro:property name="is_ecm" value="${str(instrument) == 'SF0826001'}"/>
+    <xacro:property name="is_si"  value="${str(instrument).startswith('42') or is_ecm}"/>
+    <!--
+      Shaft length (D parameter of the roll joint):
+        Classic PSM instruments → 0.4162
+        Si PSM instruments      → 0.53559
+        Si ECM (SF0826001)      → 0.4670   (camera tube is shorter than PSM shafts)
+    -->
+    <xacro:property name="shaft_length" value="${0.4670 if is_ecm else (0.53559 if is_si else 0.4162)}"/>
     <!-- fixed joint to hold the shaft visual BEFORE the roll joint -->
     <joint name="instrument_base_fixed" type="fixed">
       <parent link="${parent_link}"/>
-      <child  link="${prefix}PSM_instrument_base_link"/>
+      <child  link="${prefix}instrument_base_link"/>
       <origin rpy="0 0 0" xyz="0 0 0"/>
     </joint>
-    <link name="${prefix}PSM_instrument_base_link">
+    <link name="${prefix}instrument_base_link">
       <visual>
         <origin rpy="0 0 0" xyz="0 0 0"/>
         <geometry>
           <xacro:if value="${is_si}">
-            <mesh filename="package://dvrk_model/meshes/instruments/420006/tool_main_link.STL"/>
+            <mesh filename="package://dvrk_model/meshes/instruments/420006/PSM_shaft.stl"/>
           </xacro:if>
           <xacro:unless value="${is_si}">
-            <mesh filename="package://dvrk_model/meshes/Classic/PSM/PSM_tool_main.dae"/>
+            <mesh filename="package://dvrk_model/meshes/Classic/PSM/PSM_shaft.dae"/>
           </xacro:unless>
         </geometry>
@@ -47,8 +53,8 @@
         <geometry>
           <xacro:if value="${is_si}">
-            <mesh filename="package://dvrk_model/meshes/instruments/420006/tool_main_link.STL"/>
+            <mesh filename="package://dvrk_model/meshes/instruments/420006/PSM_shaft.stl"/>
           </xacro:if>
           <xacro:unless value="${is_si}">
-            <mesh filename="package://dvrk_model/meshes/Classic/PSM/PSM_tool_main.dae"/>
+            <mesh filename="package://dvrk_model/meshes/Classic/PSM/PSM_shaft.dae"/>
           </xacro:unless>
         </geometry>
@@ -58,5 +64,5 @@
     <joint name="roll" type="revolute">
       <parent link="${parent_link}"/>
-      <child  link="${prefix}PSM_roll_link"/>
+      <child  link="${prefix}roll_link"/>
       <axis xyz="0 0 1"/>
       <origin rpy="0 0 0" xyz="0 0 ${shaft_length}"/>
@@ -67,12 +73,12 @@
       The outer shaft mesh (above) does not roll or shift.
     -->
-    <link name="${prefix}PSM_roll_link"/>
+    <link name="${prefix}roll_link"/>
     <!-- fixed joint to wrist body -->
     <joint name="roll_fixed" type="fixed">
-      <parent link="${prefix}PSM_roll_link"/>
-      <child  link="${prefix}PSM_wrist_link"/>
+      <parent link="${prefix}roll_link"/>
+      <child  link="${prefix}wrist_link"/>
       <origin rpy="0 0 0" xyz="0 0 0"/>
     </joint>
-    <link name="${prefix}PSM_wrist_link">
+    <link name="${prefix}wrist_link">
       <visual>
         <xacro:if value="${is_si}">
@@ -80,5 +86,5 @@
           <origin rpy="-${PI} 0 0" xyz="0.05591 0 0"/>
           <geometry>
-            <mesh filename="package://dvrk_model/meshes/instruments/420006/tool_wrist_link.STL"/>
+            <mesh filename="package://dvrk_model/meshes/instruments/420006/PSM_wrist.stl"/>
           </geometry>
           <material name=""><color rgba="0.79216 0.81961 0.93333 1"/></material>
@@ -96,5 +102,5 @@
           <origin rpy="-${PI} 0 0" xyz="0.05591 0 0"/>
           <geometry>
-            <mesh filename="package://dvrk_model/meshes/instruments/420006/tool_wrist_link.STL"/>
+            <mesh filename="package://dvrk_model/meshes/instruments/420006/PSM_wrist.stl"/>
           </geometry>
         </xacro:if>
@@ -109,14 +115,14 @@
     <!-- fixed joint to wrist shaft -->
     <joint name="wrist_shaft_fixed" type="fixed">
-      <parent link="${prefix}PSM_wrist_link"/>
-      <child  link="${prefix}PSM_wrist_shaft_link"/>
+      <parent link="${prefix}wrist_link"/>
+      <child  link="${prefix}wrist_shaft_link"/>
       <origin rpy="0 0 0" xyz="0 0 0"/>
     </joint>
-    <link name="${prefix}PSM_wrist_shaft_link">
+    <link name="${prefix}wrist_shaft_link">
       <visual>
         <xacro:if value="${is_si}">
           <origin rpy="0 0 0" xyz="0 0 0"/>
           <geometry>
-            <mesh filename="package://dvrk_model/meshes/instruments/420006/tool_wrist_shaft_link.STL"/>
+            <mesh filename="package://dvrk_model/meshes/instruments/420006/PSM_wrist_shaft.stl"/>
           </geometry>
           <material name=""><color rgba="0.79216 0.81961 0.93333 1"/></material>
@@ -133,5 +139,5 @@
           <origin rpy="0 0 0" xyz="0 0 0"/>
           <geometry>
-            <mesh filename="package://dvrk_model/meshes/instruments/420006/tool_wrist_shaft_link.STL"/>
+            <mesh filename="package://dvrk_model/meshes/instruments/420006/PSM_wrist_shaft.stl"/>
           </geometry>
         </xacro:if>
@@ -158,21 +164,21 @@
                       str(instrument) == '420168' or str(instrument) == '400168'}">
       <xacro:PSM_tip_006 prefix="${prefix}"
-                         parent_link="${prefix}PSM_wrist_shaft_link"/>
+                         parent_link="${prefix}wrist_shaft_link"/>
     </xacro:if>
     <xacro:if value="${str(instrument) == '420049' or str(instrument) == '400049'}">
       <xacro:PSM_tip_049 prefix="${prefix}"
-                         parent_link="${prefix}PSM_wrist_shaft_link"/>
+                         parent_link="${prefix}wrist_shaft_link"/>
     </xacro:if>
     <xacro:if value="${str(instrument) == '420172' or str(instrument) == '400172'}">
       <xacro:PSM_tip_172 prefix="${prefix}"
-                         parent_link="${prefix}PSM_wrist_shaft_link"/>
+                         parent_link="${prefix}wrist_shaft_link"/>
     </xacro:if>
     <xacro:if value="${str(instrument) == '400117'}">
       <xacro:PSM_tip_117 prefix="${prefix}"
-                         parent_link="${prefix}PSM_wrist_shaft_link"/>
+                         parent_link="${prefix}wrist_shaft_link"/>
     </xacro:if>
     <xacro:if value="${str(instrument) == 'SF0826001'}">
       <xacro:PSM_tip_ECM prefix="${prefix}"
-                         parent_link="${prefix}PSM_wrist_shaft_link"/>
+                         parent_link="${prefix}wrist_shaft_link"/>
     </xacro:if>
   </xacro:macro>

File: urdf/common/PSM_tips.urdf.xacro (robot description, xacro)
@@ -3,5 +3,5 @@
   <!--
     PSM tip family macros — generation-agnostic.
-    All macros attach to ${parent_link} (= ${prefix}PSM_wrist_shaft_link).
+    All macros attach to ${parent_link} (= ${prefix}wrist_shaft_link).
     Tip families are identified by the last 3 digits of the instrument model:
       PSM_tip_006  — standard SCA wrist  (A=0.0091 m, most instruments)
@@ -20,10 +20,10 @@
     <joint name="wrist_pitch" type="revolute">
       <parent link="${parent_link}"/>
-      <child  link="${prefix}PSM_tip_006_wrist_link"/>
+      <child  link="${prefix}tip_006_wrist_link"/>
       <axis xyz="0 0 1"/>
       <origin rpy="-${PI_2} -${PI_2} 0" xyz="0 0 0"/>
       <limit lower="-${PI_2}" upper="${PI_2}" velocity=".4" effort="1000"/>
     </joint>
-    <link name="${prefix}PSM_tip_006_wrist_link">
+    <link name="${prefix}tip_006_wrist_link">
       <visual>
         <origin rpy="${PI_2} ${PI} 0" xyz="0.0051 0.0032 0"/>
@@ -35,11 +35,11 @@
     <!-- joint 6: wrist_yaw -->
     <joint name="wrist_yaw" type="revolute">
-      <parent link="${prefix}PSM_tip_006_wrist_link"/>
-      <child  link="${prefix}PSM_tip_006_shaft_link"/>
+      <parent link="${prefix}tip_006_wrist_link"/>
+      <child  link="${prefix}tip_006_shaft_link"/>
       <axis xyz="0 0 1"/>
       <origin rpy="-${PI_2} -${PI_2} 0" xyz="0.0091 0 0"/>
       <limit lower="-1.3963" upper="1.3963" velocity=".4" effort="1000"/>
     </joint>
-    <link name="${prefix}PSM_tip_006_shaft_link">
+    <link name="${prefix}tip_006_shaft_link">
       <visual>
         <origin rpy="0 0 0" xyz="0 -0.0002 -0.0025"/>
@@ -51,6 +51,6 @@
     <!-- joint 7-0: jaw (virtual centre — drives the mimics) -->
     <joint name="jaw" type="revolute">
-      <parent link="${prefix}PSM_tip_006_shaft_link"/>
-      <child  link="${prefix}PSM_jaw_link"/>
+      <parent link="${prefix}tip_006_shaft_link"/>
+      <child  link="${prefix}jaw_link"/>
       <axis xyz="0 0 1"/>
       <origin rpy="0 0 0" xyz="0 0 0"/>
@@ -58,5 +58,5 @@
     </joint>
     <!-- virtual jaw link (zero-size, drives mimics) -->
-    <link name="${prefix}PSM_jaw_link">
+    <link name="${prefix}jaw_link">
       <visual>
         <origin rpy="0 0 0" xyz="0 0 0"/>
@@ -66,6 +66,6 @@
     <!-- jaw mimic 1 — opens +0.5× -->
     <joint name="jaw_1" type="revolute">
-      <parent link="${prefix}PSM_tip_006_shaft_link"/>
-      <child  link="${prefix}PSM_jaw_1_link"/>
+      <parent link="${prefix}tip_006_shaft_link"/>
+      <child  link="${prefix}jaw_1_link"/>
       <axis xyz="0 0 1"/>
       <origin rpy="0 0 0" xyz="0 0 0"/>
@@ -73,5 +73,5 @@
       <mimic joint="jaw" multiplier="0.5"/>
     </joint>
-    <link name="${prefix}PSM_jaw_1_link">
+    <link name="${prefix}jaw_1_link">
       <visual>
         <origin rpy="0 0 0" xyz="0 0 0"/>
@@ -83,6 +83,6 @@
     <!-- jaw mimic 2 — opens −0.5× (symmetric) -->
     <joint name="jaw_2" type="revolute">
-      <parent link="${prefix}PSM_tip_006_shaft_link"/>
-      <child  link="${prefix}PSM_jaw_2_link"/>
+      <parent link="${prefix}tip_006_shaft_link"/>
+      <child  link="${prefix}jaw_2_link"/>
       <axis xyz="0 0 1"/>
       <origin rpy="0 0 0" xyz="0 0 0"/>
@@ -90,5 +90,5 @@
       <mimic joint="jaw" multiplier="-0.5"/>
     </joint>
-    <link name="${prefix}PSM_jaw_2_link">
+    <link name="${prefix}jaw_2_link">
       <visual>
         <origin rpy="0 ${PI} 0" xyz="0 0 0"/>
@@ -100,9 +100,9 @@
     <!-- tool tip reference frame -->
     <joint name="tool_tip" type="fixed">
-      <parent link="${prefix}PSM_tip_006_shaft_link"/>
-      <child  link="${prefix}PSM_tool_tip_link"/>
+      <parent link="${prefix}tip_006_shaft_link"/>
+      <child  link="${prefix}tool_tip_link"/>
       <origin rpy="0 ${PI/2} ${PI/2}" xyz="0 0.0102 0"/>
     </joint>
-    <link name="${prefix}PSM_tool_tip_link"/>
+    <link name="${prefix}tool_tip_link"/>
   </xacro:macro>
   <!-- ════════════════════════════════════════════════════════════════════ -->
@@ -112,10 +112,10 @@
     <joint name="wrist_pitch" type="revolute">
       <parent link="${parent_link}"/>
-      <child  link="${prefix}PSM_tip_049_wrist_link"/>
+      <child  link="${prefix}tip_049_wrist_link"/>
       <axis xyz="0 0 1"/>
       <origin rpy="-${PI_2} -${PI_2} 0" xyz="0 0 0"/>
       <limit lower="-${PI_2}" upper="${PI_2}" velocity=".4" effort="1000"/>
     </joint>
-    <link name="${prefix}PSM_tip_049_wrist_link">
+    <link name="${prefix}tip_049_wrist_link">
       <visual>
         <origin rpy="0 -${PI_2} 0" xyz="-0.0024 0 0"/>
@@ -126,11 +126,11 @@
     </link>
     <joint name="wrist_yaw" type="revolute">
-      <parent link="${prefix}PSM_tip_049_wrist_link"/>
-      <child  link="${prefix}PSM_tip_049_shaft_link"/>
+      <parent link="${prefix}tip_049_wrist_link"/>
+      <child  link="${prefix}tip_049_shaft_link"/>
       <axis xyz="0 0 1"/>
       <origin rpy="0 -${PI_2} -${PI_2}" xyz="0.0091 0 0"/>
       <limit lower="-1.3963" upper="1.3963" velocity=".4" effort="1000"/>
     </joint>
-    <link name="${prefix}PSM_tip_049_shaft_link">
+    <link name="${prefix}tip_049_shaft_link">
       <visual>
         <origin rpy="0 ${PI_2} 0" xyz="0 -0.0002 0"/>
@@ -141,11 +141,11 @@
     </link>
     <joint name="jaw" type="revolute">
-      <parent link="${prefix}PSM_tip_049_shaft_link"/>
-      <child link="${prefix}PSM_jaw_link"/>
+      <parent link="${prefix}tip_049_shaft_link"/>
+      <child link="${prefix}jaw_link"/>
       <axis xyz="0 0 1"/>
       <origin rpy="0 0 0" xyz="0 0 0"/>
       <limit lower="-0.349066" upper="1.5708" velocity=".4" effort="1000"/>
     </joint>
-    <link name="${prefix}PSM_jaw_link">
+    <link name="${prefix}jaw_link">
       <visual>
         <origin rpy="0 0 0" xyz="0 0 0"/>
@@ -154,6 +154,6 @@
     </link>
     <joint name="jaw_1" type="revolute">
-      <parent link="${prefix}PSM_tip_049_shaft_link"/>
-      <child link="${prefix}PSM_jaw_1_link"/>
+      <parent link="${prefix}tip_049_shaft_link"/>
+      <child link="${prefix}jaw_1_link"/>
       <axis xyz="0 0 1"/>
       <origin rpy="0 0 0" xyz="0 0 0"/>
@@ -161,5 +161,5 @@
       <mimic joint="jaw" multiplier="0.5"/>
     </joint>
-    <link name="${prefix}PSM_jaw_1_link">
+    <link name="${prefix}jaw_1_link">
       <visual>
         <origin rpy="0 0 0" xyz="0 0 0.00195"/>
@@ -170,6 +170,6 @@
     </link>
     <joint name="jaw_2" type="revolute">
-      <parent link="${prefix}PSM_tip_049_shaft_link"/>
-      <child link="${prefix}PSM_jaw_2_link"/>
+      <parent link="${prefix}tip_049_shaft_link"/>
+      <child link="${prefix}jaw_2_link"/>
       <axis xyz="0 0 1"/>
       <origin rpy="${PI} 0 0" xyz="0 0 0"/>
@@ -177,5 +177,5 @@
       <mimic joint="jaw" multiplier="0.5"/>
     </joint>
-    <link name="${prefix}PSM_jaw_2_link">
+    <link name="${prefix}jaw_2_link">
       <visual>
         <origin rpy="0 0 -${PI}" xyz="0 0 0.00195"/>
@@ -186,9 +186,9 @@
     </link>
     <joint name="tool_tip" type="fixed">
-      <parent link="${prefix}PSM_tip_049_shaft_link"/>
-      <child link="${prefix}PSM_tool_tip_link"/>
+      <parent link="${prefix}tip_049_shaft_link"/>
+      <child link="${prefix}tool_tip_link"/>
       <origin rpy="0 ${PI_2} ${PI_2}" xyz="0 0 0"/>
     </joint>
-    <link name="${prefix}PSM_tool_tip_link"/>
+    <link name="${prefix}tool_tip_link"/>
   </xacro:macro>
   <!-- ════════════════════════════════════════════════════════════════════ -->
@@ -199,5 +199,5 @@
     <joint name="wrist_pitch" type="revolute">
       <parent link="${parent_link}"/>
-      <child  link="${prefix}PSM_tip_172_wrist_link"/>
+      <child  link="${prefix}tip_172_wrist_link"/>
       <axis xyz="0 0 1"/>
       <origin rpy="-${PI_2} -${PI_2} 0" xyz="0 0 0"/>
@@ -208,5 +208,5 @@
       until a dedicated Maryland wrist mesh is added to the repo.
     -->
-    <link name="${prefix}PSM_tip_172_wrist_link">
+    <link name="${prefix}tip_172_wrist_link">
       <visual>
         <origin rpy="${PI_2} ${PI} 0" xyz="0.0051 0.0032 0"/>
@@ -218,11 +218,11 @@
     <!-- joint 6: wrist_yaw (A=0.0107 — Maryland specific) -->
     <joint name="wrist_yaw" type="revolute">
-      <parent link="${prefix}PSM_tip_172_wrist_link"/>
-      <child  link="${prefix}PSM_tip_172_shaft_link"/>
+      <parent link="${prefix}tip_172_wrist_link"/>
+      <child  link="${prefix}tip_172_shaft_link"/>
       <axis xyz="0 0 1"/>
       <origin rpy="-${PI_2} -${PI_2} 0" xyz="0.0107 0 0"/>
       <limit lower="-1.3963" upper="1.3963" velocity=".4" effort="1000"/>
     </joint>
-    <link name="${prefix}PSM_tip_172_shaft_link">
+    <link name="${prefix}tip_172_shaft_link">
       <visual>
         <origin rpy="0 0 0" xyz="0 -0.0002 -0.0025"/>
@@ -234,11 +234,11 @@
     <!-- jaw + symmetric mimics (same as tip_006) -->
     <joint name="jaw" type="revolute">
-      <parent link="${prefix}PSM_tip_172_shaft_link"/>
-      <child  link="${prefix}PSM_jaw_link"/>
+      <parent link="${prefix}tip_172_shaft_link"/>
+      <child  link="${prefix}jaw_link"/>
       <axis xyz="0 0 1"/>
       <origin rpy="0 0 0" xyz="0 0 0"/>
       <limit lower="0" upper="${PI_2}" velocity=".4" effort="1000"/>
     </joint>
-    <link name="${prefix}PSM_jaw_link">
+    <link name="${prefix}jaw_link">
       <visual><origin rpy="0 0 0" xyz="0 0 0"/>
         <geometry><box size="0 0 0"/></geometry>
@@ -246,6 +246,6 @@
     </link>
     <joint name="jaw_1" type="revolute">
-      <parent link="${prefix}PSM_tip_172_shaft_link"/>
-      <child  link="${prefix}PSM_jaw_1_link"/>
+      <parent link="${prefix}tip_172_shaft_link"/>
+      <child  link="${prefix}jaw_1_link"/>
       <axis xyz="0 0 1"/>
       <origin rpy="0 0 0" xyz="0 0 0"/>
@@ -253,5 +253,5 @@
       <mimic joint="jaw" multiplier="0.5"/>
     </joint>
-    <link name="${prefix}PSM_jaw_1_link">
+    <link name="${prefix}jaw_1_link">
       <visual>
         <origin rpy="0 0 0" xyz="0 0 0"/>
@@ -262,6 +262,6 @@
     </link>
     <joint name="jaw_2" type="revolute">
-      <parent link="${prefix}PSM_tip_172_shaft_link"/>
-      <child  link="${prefix}PSM_jaw_2_link"/>
+      <parent link="${prefix}tip_172_shaft_link"/>
+      <child  link="${prefix}jaw_2_link"/>
       <axis xyz="0 0 1"/>
       <origin rpy="0 0 0" xyz="0 0 0"/>
@@ -269,5 +269,5 @@
       <mimic joint="jaw" multiplier="-0.5"/>
     </joint>
-    <link name="${prefix}PSM_jaw_2_link">
+    <link name="${prefix}jaw_2_link">
       <visual>
         <origin rpy="0 ${PI} 0" xyz="0 0 0"/>
@@ -278,9 +278,9 @@
     </link>
     <joint name="tool_tip" type="fixed">
-      <parent link="${prefix}PSM_tip_172_shaft_link"/>
-      <child  link="${prefix}PSM_tool_tip_link"/>
+      <parent link="${prefix}tip_172_shaft_link"/>
+      <child  link="${prefix}tool_tip_link"/>
       <origin rpy="0 ${PI/2} ${PI/2}" xyz="0 0.0107 0"/>
     </joint>
-    <link name="${prefix}PSM_tool_tip_link"/>
+    <link name="${prefix}tool_tip_link"/>
   </xacro:macro>
   <!-- ════════════════════════════════════════════════════════════════════ -->
@@ -297,24 +297,24 @@
     <joint name="wrist_pitch" type="revolute">
       <parent link="${parent_link}"/>
-      <child  link="${prefix}PSM_tip_117_wrist_link"/>
+      <child  link="${prefix}tip_117_wrist_link"/>
       <axis xyz="0 0 1"/>
       <origin rpy="-${PI_2} -${PI_2} 0" xyz="0 0 0"/>
       <limit lower="-${PI_2}" upper="${PI_2}" velocity=".4" effort="1000"/>
     </joint>
-    <link name="${prefix}PSM_tip_117_wrist_link"/>
+    <link name="${prefix}tip_117_wrist_link"/>
     <joint name="jaw" type="revolute">
-      <parent link="${prefix}PSM_tip_117_wrist_link"/>
-      <child  link="${prefix}PSM_jaw_link"/>
+      <parent link="${prefix}tip_117_wrist_link"/>
+      <child  link="${prefix}jaw_link"/>
       <axis xyz="0 0 1"/>
       <origin rpy="0 0 0" xyz="0 0 0"/>
       <limit lower="0" upper="${PI_2}" velocity=".4" effort="1000"/>
     </joint>
-    <link name="${prefix}PSM_jaw_link"/>
-    <joint name="tool_tip" type="fixed">
-      <parent link="${prefix}PSM_tip_117_wrist_link"/>
-      <child  link="${prefix}PSM_tool_tip_link"/>
-      <origin rpy="0 0 0" xyz="0 0 0"/>
-    </joint>
-    <link name="${prefix}PSM_tool_tip_link"/>
+    <link name="${prefix}jaw_link"/>
+    <joint name="tool_tip" type="fixed">
+      <parent link="${prefix}tip_117_wrist_link"/>
+      <child  link="${prefix}tool_tip_link"/>
+      <origin rpy="0 0 0" xyz="0 0 0"/>
+    </joint>
+    <link name="${prefix}tool_tip_link"/>
   </xacro:macro>
   <!-- ════════════════════════════════════════════════════════════════════ -->
@@ -325,8 +325,8 @@
     <joint name="tool_tip" type="fixed">
       <parent link="${parent_link}"/>
-      <child  link="${prefix}PSM_tool_tip_link"/>
-      <origin rpy="0 0 0" xyz="0 0 0"/>
-    </joint>
-    <link name="${prefix}PSM_tool_tip_link"/>
+      <child  link="${prefix}tool_tip_link"/>
+      <origin rpy="0 0 0" xyz="0 0 0"/>
+    </joint>
+    <link name="${prefix}tool_tip_link"/>
   </xacro:macro>
   <!-- ════════════════════════════════════════════════════════════════════ -->
@@ -336,10 +336,10 @@
     <joint name="wrist_pitch" type="revolute">
       <parent link="${parent_link}"/>
-      <child  link="${prefix}ECM_tip_roll_link"/>
+      <child  link="${prefix}tip_roll_link"/>
       <axis xyz="0 0 1"/>
       <origin rpy="-1.5708 -1.5708 0" xyz="0 0 0"/>
       <limit lower="-1.5707" upper="1.5707" velocity=".4" effort="1000"/>
     </joint>
-    <link name="${prefix}ECM_tip_roll_link">
+    <link name="${prefix}tip_roll_link">
       <visual>
         <origin rpy="0 -${PI_2} 0" xyz="0.0051 0.0032 0"/>
@@ -350,9 +350,9 @@
     </link>
     <joint name="tool_tip" type="fixed">
-      <parent link="${prefix}ECM_tip_roll_link"/>
-      <child  link="${prefix}PSM_tool_tip_link"/>
+      <parent link="${prefix}tip_roll_link"/>
+      <child  link="${prefix}tool_tip_link"/>
       <origin rpy="0 0 0" xyz="0 0.0102 0"/>
     </joint>
-    <link name="${prefix}PSM_tool_tip_link"/>
+    <link name="${prefix}tool_tip_link"/>
   </xacro:macro>
 </robot>
