Commit message: roll in instrument only

File: urdf/Classic/ECM.urdf.xacro (robot description, xacro)
@@ -4,7 +4,11 @@
   <xacro:property name="parent_link" default="$(arg parent_link_)"/>
   <xacro:include filename="$(find dvrk_model)/urdf/Classic/ECM_base.urdf.xacro"/>
+  <xacro:include filename="$(find dvrk_model)/urdf/Classic/ECM_instrument.urdf.xacro"/>
   <link name="${parent_link}"/>
   <xacro:ecm_base
       prefix="ECM_"
       parent_link="${parent_link}"/>
+  <xacro:ECM_instrument
+      prefix="ECM_"
+      parent_link="ECM_tool_parent_link"/>
 </robot>

File: urdf/Classic/ECM_base.urdf.xacro (robot description, xacro)
@@ -190,6 +190,7 @@
       <mimic joint="pitch" multiplier="1"/>
     </joint>
-    <link
-      name="${prefix}main_insertion_link">
+    <!-- tool_parent_link — boundary link; ECM_instrument attaches here. -->
+    <link
+      name="${prefix}tool_parent_link">
       <visual>
         <origin
@@ -220,5 +221,5 @@
         link="${prefix}pitch_end_link" />
       <child
-        link="${prefix}main_insertion_link" />
+        link="${prefix}tool_parent_link" />
       <axis
         xyz="0 0 1" />
@@ -230,43 +231,4 @@
     </joint>
     <link
-      name="${prefix}tool_link">
-      <visual>
-        <origin
-          xyz="0 0 0"
-          rpy="0 0 0" />
-        <geometry>
-          <mesh
-            filename="package://dvrk_model/meshes/arms/Classic/ECM/ECM_tool.stl" />
-        </geometry>
-      </visual>
-      <collision>
-        <origin
-          xyz="0 0 0"
-          rpy="0 0 0" />
-        <geometry>
-          <mesh
-            filename="package://dvrk_model/meshes/arms/Classic/ECM/ECM_tool.stl" />
-        </geometry>
-      </collision>
-    </link>
-    <joint
-      name="roll"
-      type="revolute">
-      <origin
-        xyz="0.0609999999999996 0 0"
-        rpy="0 0 0" />
-      <parent
-        link="${prefix}main_insertion_link" />
-      <child
-        link="${prefix}tool_link" />
-      <axis
-        xyz="0 0 -1" />
-      <limit
-        lower="-1.552676"
-        upper="1.566741"
-        effort="1000"
-        velocity="10" />
-    </joint>
-    <link
       name="${prefix}pitch_top_link">
       <visual>
@@ -382,18 +344,4 @@
         xyz="0 0 0" />
     </joint>
-    <link name="${prefix}end_link"/>
-    <joint
-      name="end_joint"
-      type="fixed">
-      <origin
-        xyz="0 0 0.37364"
-        rpy="0 0 0" />
-      <parent
-        link="${prefix}tool_link" />
-      <child
-        link="${prefix}end_link" />
-      <axis
-        xyz="0 0 0" />
-    </joint>
   </xacro:macro>
 </robot>

File: urdf/Si/ECM.urdf.xacro (robot description, xacro)
@@ -3,5 +3,5 @@
   <xacro:arg name="parent_link_" default="world"/>
   <xacro:property name="parent_link" default="$(arg parent_link_)"/>
-  <xacro:include filename="$(find dvrk_model)/urdf/Si/PSM_base_macros.urdf.xacro"/>
+  <xacro:include filename="$(find dvrk_model)/urdf/Si/PSM_base.urdf.xacro"/>
   <xacro:include filename="$(find dvrk_model)/urdf/common/PSM_instrument.urdf.xacro"/>
   <link name="${parent_link}"/>

File: urdf/Si/PSM1.urdf.xacro (robot description, xacro)
@@ -8,5 +8,5 @@
   <xacro:arg name="parent_link_" default="world"/>
   <xacro:property name="parent_link" value="$(arg parent_link_)"/>
-  <xacro:include filename="$(find dvrk_model)/urdf/Si/PSM_base_macros.urdf.xacro"/>
+  <xacro:include filename="$(find dvrk_model)/urdf/Si/PSM_base.urdf.xacro"/>
   <xacro:include filename="$(find dvrk_model)/urdf/common/PSM_instrument.urdf.xacro"/>
   <link name="${parent_link}"/>

File: urdf/Si/PSM2.urdf.xacro (robot description, xacro)
@@ -4,5 +4,5 @@
   <xacro:arg name="parent_link_" default="world"/>
   <xacro:property name="parent_link" value="$(arg parent_link_)"/>
-  <xacro:include filename="$(find dvrk_model)/urdf/Si/PSM_base_macros.urdf.xacro"/>
+  <xacro:include filename="$(find dvrk_model)/urdf/Si/PSM_base.urdf.xacro"/>
   <xacro:include filename="$(find dvrk_model)/urdf/common/PSM_instrument.urdf.xacro"/>
   <link name="${parent_link}"/>

File: urdf/Si/PSM3.urdf.xacro (robot description, xacro)
@@ -4,5 +4,5 @@
   <xacro:arg name="parent_link_" default="world"/>
   <xacro:property name="parent_link" value="$(arg parent_link_)"/>
-  <xacro:include filename="$(find dvrk_model)/urdf/Si/PSM_base_macros.urdf.xacro"/>
+  <xacro:include filename="$(find dvrk_model)/urdf/Si/PSM_base.urdf.xacro"/>
   <xacro:include filename="$(find dvrk_model)/urdf/common/PSM_instrument.urdf.xacro"/>
   <link name="${parent_link}"/>

File: urdf/Si/SUJ.urdf.xacro (robot description, xacro)
@@ -2,6 +2,6 @@
 <robot name="patient_cart" xmlns:xacro="http://www.ros.org/wiki/xacro">
   <xacro:include filename="$(find dvrk_model)/urdf/common.urdf.xacro"/>
-  <xacro:include filename="$(find dvrk_model)/urdf/Si/SUJ_base_macros.urdf.xacro"/>
-  <xacro:include filename="$(find dvrk_model)/urdf/Si/SUJ_column_macros.urdf.xacro"/>
+  <xacro:include filename="$(find dvrk_model)/urdf/Si/SUJ_base.urdf.xacro"/>
+  <xacro:include filename="$(find dvrk_model)/urdf/Si/SUJ_column.urdf.xacro"/>
   <xacro:suj_column/>
   <xacro:suj
