Commit message: Initial re-organization for ECM

File: urdf/Classic/ECM.urdf.xacro (robot description, xacro)
@@ -1,13 +1,15 @@
 <?xml version="1.0" ?>
 <robot name="ECM" xmlns:xacro="http://www.ros.org/wiki/xacro">
+  <xacro:arg name="endoscope" default="Classic_SD_straight"/>
   <xacro:arg name="parent_link_" default="world"/>
   <xacro:property name="parent_link" default="$(arg parent_link_)"/>
   <xacro:include filename="$(find dvrk_model)/urdf/Classic/ECM_base.urdf.xacro"/>
-  <xacro:include filename="$(find dvrk_model)/urdf/Classic/ECM_instrument.urdf.xacro"/>
+    <xacro:include filename="$(find dvrk_model)/urdf/common/endoscope.urdf.xacro"/>
   <link name="${parent_link}"/>
+  <xacro:dvrk_materials/>
   <xacro:ecm_base
       prefix="ECM_"
       parent_link="${parent_link}"/>
-  <xacro:ECM_instrument
+  <xacro:endoscope
       prefix="ECM_"
       parent_link="ECM_tool_parent_link"/>

File: urdf/Classic/ECM_base.urdf.xacro (robot description, xacro)
@@ -21,4 +21,5 @@
             filename="package://dvrk_model/meshes/arms/Classic/ECM/ECM_base.stl" />
         </geometry>
+        <material name="DaVinciLightGray"><color rgba="0.64706 0.61961 0.58824 1"/></material>
       </visual>
       <collision>
@@ -42,4 +43,5 @@
             filename="package://dvrk_model/meshes/arms/Classic/ECM/ECM_yaw.stl" />
         </geometry>
+        <material name="DaVinciLightGray"><color rgba="0.64706 0.61961 0.58824 1"/></material>
       </visual>
       <collision>
@@ -81,4 +83,5 @@
             filename="package://dvrk_model/meshes/arms/Classic/ECM/ECM_pitch_front.stl" />
         </geometry>
+        <material name="DaVinciLightGray"><color rgba="0.64706 0.61961 0.58824 1"/></material>
       </visual>
       <collision>
@@ -120,4 +123,5 @@
             filename="package://dvrk_model/meshes/arms/Classic/ECM/ECM_pitch_bottom.stl" />
         </geometry>
+        <material name="DaVinciDarkGray"><color rgba="0.25098 0.25098 0.25098 1"/></material>
       </visual>
       <collision>
@@ -160,4 +164,5 @@
             filename="package://dvrk_model/meshes/arms/Classic/ECM/ECM_pitch_end.stl" />
         </geometry>
+        <material name="DaVinciWhite"><color rgba="0.89804 0.91765 0.92941 1"/></material>
       </visual>
       <collision>
@@ -201,4 +206,5 @@
             filename="package://dvrk_model/meshes/arms/Classic/ECM/ECM_main_insertion.stl" />
         </geometry>
+        <material name="DaVinciDarkGray"><color rgba="0.25 0.25 0.25 1"/></material>
       </visual>
       <collision>
@@ -240,4 +246,5 @@
             filename="package://dvrk_model/meshes/arms/Classic/ECM/ECM_pitch_top.stl" />
         </geometry>
+        <material name="DaVinciRed"><color rgba="0.64706 0.51765 0 1"/></material>
       </visual>
       <collision>
@@ -280,4 +287,5 @@
             filename="package://dvrk_model/meshes/arms/Classic/ECM/ECM_pitch_back.stl" />
         </geometry>
+        <material name="DaVinciRed"><color rgba="0.64706 0.51765 0 1"/></material>
       </visual>
       <collision>
@@ -320,4 +328,5 @@
             filename="package://dvrk_model/meshes/arms/Classic/ECM/ECM_RCM.stl" />
         </geometry>
+        <material name="DaVinciRed"><color rgba="1.0 0.7 0.7 1"/></material>
       </visual>
       <collision>

File: urdf/Classic/MTM.urdf.xacro (robot description, xacro)
@@ -47,5 +47,5 @@
         <origin rpy="0 0 0" xyz="0 0 0.19037"/>
         <geometry>
-          <mesh filename="package://dvrk_model/meshes/arms/Classic/MTM/MTM_top_panel.stl"/>
+          <mesh filename="package://dvrk_model/meshes/arms/Classic/MTM/MTM_top_panel.dae"/>
         </geometry>
       </collision>
@@ -79,5 +79,5 @@
         <origin rpy="0 0 0" xyz="0.025 0 0.19037"/>
         <geometry>
-          <mesh filename="package://dvrk_model/meshes/arms/Classic/MTM/MTM_outer_yaw.stl"/>
+          <mesh filename="package://dvrk_model/meshes/arms/Classic/MTM/MTM_outer_yaw.dae"/>
         </geometry>
       </collision>
@@ -105,5 +105,5 @@
       <collision>
         <geometry>
-          <mesh filename="package://dvrk_model/meshes/arms/Classic/MTM/MTM_shoulder_pitch.stl"/>
+          <mesh filename="package://dvrk_model/meshes/arms/Classic/MTM/MTM_shoulder_pitch.dae"/>
         </geometry>
       </collision>
@@ -134,5 +134,5 @@
         <origin rpy="0 0 0" xyz="0 0 0"/>
         <geometry>
-          <mesh filename="package://dvrk_model/meshes/arms/Classic/MTM/MTM_shoulder_pitch_parallel.stl"/>
+          <mesh filename="package://dvrk_model/meshes/arms/Classic/MTM/MTM_shoulder_pitch_parallel.dae"/>
         </geometry>
       </collision>
@@ -160,5 +160,5 @@
       <collision>
         <geometry>
-          <mesh filename="package://dvrk_model/meshes/arms/Classic/MTM/MTM_elbow_pitch.stl"/>
+          <mesh filename="package://dvrk_model/meshes/arms/Classic/MTM/MTM_elbow_pitch.dae"/>
         </geometry>
       </collision>
@@ -229,6 +229,6 @@
       </visual>
       <collision>
-        <geometry>
-          <mesh filename="package://dvrk_model/meshes/arms/Classic/MTM/MTM_wrist_platform.stl"/>
+          <geometry>
+            <mesh filename="package://dvrk_model/meshes/arms/Classic/MTM/MTM_wrist_platform.dae"/>
         </geometry>
       </collision>
@@ -257,6 +257,6 @@
       </visual>
       <collision>        <!-- defined from CAD file (increased in the y dir by .005-->
-        <geometry>
-          <mesh filename="package://dvrk_model/meshes/arms/Classic/MTM/MTM_wrist_pitch.stl"/>
+          <geometry>
+            <mesh filename="package://dvrk_model/meshes/arms/Classic/MTM/MTM_wrist_pitch.dae"/>
         </geometry>
       </collision>
@@ -286,6 +286,6 @@
       </visual>
       <collision>
-        <geometry>
-          <mesh filename="package://dvrk_model/meshes/arms/Classic/MTM/MTM_wrist_yaw.stl"/>
+          <geometry>
+            <mesh filename="package://dvrk_model/meshes/arms/Classic/MTM/MTM_wrist_yaw.dae"/>
         </geometry>
       </collision>
@@ -317,6 +317,6 @@
       <collision>
         <origin rpy="${PI} 0 0" xyz="0 0 0.039"/>
-        <geometry>
-          <mesh filename="package://dvrk_model/meshes/arms/Classic/MTM/MTM_wrist_roll.stl"/>
+          <geometry>
+            <mesh filename="package://dvrk_model/meshes/arms/Classic/MTM/MTM_wrist_roll.dae"/>
         </geometry>
       </collision>
@@ -378,5 +378,5 @@
         <origin rpy="0 0 ${PI}" xyz="0.0 0.0 0.0"/>
         <geometry>
-          <mesh filename="package://dvrk_model/meshes/arms/Classic/MTM/MTM_wrist_platform.dae"/>
+            <mesh filename="package://dvrk_model/meshes/arms/Classic/MTM/MTM_wrist_platform.dae"/>
         </geometry>
       </visual>
@@ -384,5 +384,5 @@
         <origin rpy="0 0 ${PI}" xyz="0.0 0.0 0.0"/>
         <geometry>
-          <mesh filename="package://dvrk_model/meshes/arms/Classic/MTM/MTM_wrist_platform.stl"/>
+            <mesh filename="package://dvrk_model/meshes/arms/Classic/MTM/MTM_wrist_platform.dae"/>
         </geometry>
       </collision>
@@ -408,5 +408,5 @@
         <origin rpy="0 ${PI} 0" xyz="0.0 0.0 0.0"/>
         <geometry>
-          <mesh filename="package://dvrk_model/meshes/arms/Classic/MTM/MTM_wrist_pitch.dae"/>
+            <mesh filename="package://dvrk_model/meshes/arms/Classic/MTM/MTM_wrist_pitch.dae"/>
         </geometry>
       </visual>
@@ -414,5 +414,5 @@
         <origin rpy="0 ${PI} 0" xyz="0.0 0.0 0.0"/>
         <geometry>
-          <mesh filename="package://dvrk_model/meshes/arms/Classic/MTM/MTM_wrist_pitch.stl"/>
+            <mesh filename="package://dvrk_model/meshes/arms/Classic/MTM/MTM_wrist_pitch.dae"/>
         </geometry>
       </collision>
@@ -438,10 +438,10 @@
       <visual>
         <geometry>
-          <mesh filename="package://dvrk_model/meshes/arms/Classic/MTM/MTM_wrist_yaw.dae"/>
-        </geometry>
-      </visual>
-      <collision>
-        <geometry>
-          <mesh filename="package://dvrk_model/meshes/arms/Classic/MTM/MTM_wrist_yaw.stl"/>
+            <mesh filename="package://dvrk_model/meshes/arms/Classic/MTM/MTM_wrist_yaw.dae"/>
+        </geometry>
+      </visual>
+      <collision>
+        <geometry>
+            <mesh filename="package://dvrk_model/meshes/arms/Classic/MTM/MTM_wrist_yaw.dae"/>
         </geometry>
       </collision>
@@ -468,5 +468,5 @@
         <origin rpy="${PI} 0 0" xyz="0 0 0.039"/>
         <geometry>
-          <mesh filename="package://dvrk_model/meshes/arms/Classic/MTM/MTM_wrist_roll.dae"/>
+            <mesh filename="package://dvrk_model/meshes/arms/Classic/MTM/MTM_wrist_roll.dae"/>
         </geometry>
       </visual>
@@ -474,5 +474,5 @@
         <origin rpy="${PI} 0 0" xyz="0 0 0.039"/>
         <geometry>
-          <mesh filename="package://dvrk_model/meshes/arms/Classic/MTM/MTM_wrist_roll.stl"/>
+            <mesh filename="package://dvrk_model/meshes/arms/Classic/MTM/MTM_wrist_roll.dae"/>
         </geometry>
       </collision>

File: urdf/Si/ECM.urdf.xacro (robot description, xacro)
@@ -1,13 +1,14 @@
 <?xml version="1.0" ?>
 <robot name="ECM" xmlns:xacro="http://www.ros.org/wiki/xacro">
+  <xacro:arg name="endoscope" default="Si_straight"/>
   <xacro:arg name="parent_link_" default="world"/>
   <xacro:property name="parent_link" default="$(arg parent_link_)"/>
-  <xacro:include filename="$(find dvrk_model)/urdf/Si/PSM_base.urdf.xacro"/>
-  <xacro:include filename="$(find dvrk_model)/urdf/common/PSM_instrument.urdf.xacro"/>
+  <xacro:include filename="$(find dvrk_model)/urdf/Si/ECM_base.urdf.xacro"/>
+  <xacro:include filename="$(find dvrk_model)/urdf/common/endoscope.urdf.xacro"/>
   <link name="${parent_link}"/>
-  <xacro:base prefix="ECM_"
+  <xacro:dvrk_materials/>
+  <xacro:ecm_base prefix="ECM_"
                   parent_link="${parent_link}"/>
-  <xacro:PSM_instrument prefix="ECM_"
-                        parent_link="ECM_tool_parent_link"
-                        instrument="SF0826001"/>
+  <xacro:endoscope prefix="ECM_"
+                   parent_link="ECM_tool_parent_link"/>
 </robot>

File: urdf/common/PSM_instrument.urdf.xacro (robot description, xacro)
@@ -21,7 +21,6 @@
   <xacro:macro name="PSM_instrument"
                params="prefix parent_link instrument">
-    <!-- Detect generation. ECM (SF0826001) uses Si-style mesh format. -->
-    <xacro:property name="is_ecm" value="${str(instrument) == 'SF0826001'}"/>
-    <xacro:property name="is_si"  value="${str(instrument).startswith('42') or is_ecm}"/>
+    <!-- Detect generation. Si instruments use Si-style mesh format. -->
+    <xacro:property name="is_si"  value="${str(instrument).startswith('42')}"/>
     <!--
       Shaft length (D parameter of the roll joint):
@@ -185,9 +184,4 @@
                          parent_link="${tip_parent_link}"/>
     </xacro:if>
-    <!-- ECM: Si camera tip -->
-    <xacro:if value="${str(instrument) == 'SF0826001'}">
-      <xacro:PSM_tip_ECM prefix="${prefix}"
-                         parent_link="${tip_parent_link}"/>
-    </xacro:if>
     <!-- 183: cautery / no-jaw tools — PSM_tip_183 macro exists in PSM_tips.urdf.xacro but is not yet wired into this dispatch -->
   </xacro:macro>

File: urdf/common/endoscopes/Classic_SD_straight.urdf.xacro (robot description, xacro)
@@ -1,13 +1,7 @@
 <?xml version="1.0" encoding="utf-8"?>
-<robot name="dvrk_ecm_classic_instrument" xmlns:xacro="http://www.ros.org/wiki/xacro">
-  <!--
-    Classic ECM instrument macro.
-    Attaches to ${parent_link} (= ${prefix}tool_parent_link from ECM_base).
-    DOF layout:
-      Joint 4: roll  (revolute, axis 0 0 -1)
-      end_joint: fixed tip frame offset
-  -->
-  <xacro:macro name="ECM_instrument" params="prefix parent_link">
-    <!-- joint 4: roll -->
+<robot name="dvrk_endoscope_classic_sd_straight" xmlns:xacro="http://www.ros.org/wiki/xacro">
+  <xacro:include filename="$(find dvrk_model)/urdf/common.urdf.xacro"/>
+  <xacro:macro name="endoscope"
+               params="prefix:='ECM_' parent_link:='ECM_tool_parent_link'">
     <joint name="roll" type="revolute">
       <origin xyz="0.0609999999999996 0 0" rpy="0 0 0"/>
@@ -21,11 +15,12 @@
         <origin xyz="0 0 0" rpy="0 0 0"/>
         <geometry>
-          <mesh filename="package://dvrk_model/meshes/arms/Classic/ECM/ECM_tool.stl"/>
+          <mesh filename="package://dvrk_model/meshes/endoscopes/Classic_SD_straight/ECM_tool.stl"/>
         </geometry>
+        <material name="DaVinciLightGray"><color rgba="0.7 0.7 0.7 1"/></material>
       </visual>
       <collision>
         <origin xyz="0 0 0" rpy="0 0 0"/>
         <geometry>
-          <mesh filename="package://dvrk_model/meshes/arms/Classic/ECM/ECM_tool.stl"/>
+          <mesh filename="package://dvrk_model/meshes/endoscopes/Classic_SD_straight/ECM_tool.stl"/>
         </geometry>
       </collision>
