Commit message: Update dVRK instrument models and visuals (#6)
* Migrate README commands from ROS to ROS 2

Updated ROS commands to ROS 2 format in examples and xacro usage.

* Refactoring: work in progress

* check git branch commit

* Update README.md

* update connection

* renaming instruments

* update bugs in urdf/psm files

* new instrument file directory

* Remove 'outer' from PSM joint/link/mesh names (Classic + Si)

* Update .gitignore

* Update .gitignore

* Rename outer_roll -> roll in Si PSM tool

* Clean build artifacts and update PSM base files

* update Classic PSM_base_urdf.xacro file with respective mesh naming updates

* update base naming

* Drop PSM_ prefix from base macros (base, base_virtual); keep filenames and meshes

* Rename ECM_outer_yaw mesh to ECM_yaw to match sawIntuitiveResearchKit naming

* Si: rename shared meshes to USM/USM_*

* Si remove all outer

* update mesh file names for USM, change PSM_ECM to USM

* fix uppercase urdf and link naming

* delete lowercase Si chain, Classic ECM, update launch

* uppercase all macro files with _macros suffix

* reorganize instrument meshes by type and DH joint names

* reorganize meshes directories

* update structure and readme

* fix mesh file references

* remove cisst logs

* removed macros

* change Snake and remove macros from base_virtual

* update PSM reference to virtual

* Mapping of all renamed and rellocated mesh files

* update covers to housing for psm

* update mesh map

* rename classic psm files after mesh review

* update mesh mapping

* update folder names by removing plural s

* update mesh mapping

* reorganize mesh locations wrt kinematics

* update mesh mapping wrt kinematics

* update Si folder instrument name and housing instead of cover

* update mesh map for Si housing

* rename classic folder to Classic under instruments

* update instruments/Classic in mesh map

* remove excess Si folder

* update mesh map

* update si mesh file names and locations

* update si mesh mapping

* update ecm mesh names and locations

* update ecm mesh map

* import high res cad

* rename and move high res si 006 meshes

* copy/paste code to switch between branches

* copy/paste code to switch to main

* fix rotated housing

* update housing origin

* organize urdf classic with archived files

* remove macros

* roll only in instrument

* roll in instrument only

* swap si roll connector and housing

* update comments for each instrument

* remove wrist variables in psm instruments and tool common files

* swap high res meshes with stl and rename stl to archive

* swap high res meshes with archived stl

* remove redundant mesh for 006

* Si instrument loaded to Classic - still need to resolve incorrect mesh placements

* Si instrument load in Classic arm - resolved mesh appearance/positioning

* Initial re-organization for ECM

* ECM renaming, also making sure arms are defined with respect to RCM and EE matches DH from json files in dvrk

* update naming scheme: wrist instead of tip

* Reorganize PSM_tips.urdf by tools

* update virtual urdf to use the same logic as classic and si arms

* fix launch parsing error for si instrument on classic arm

* fix 006 gripper positioning not facing each other

* First draft - reorganize urdf instrument

* Cleanup for SUJ, active arms mounting on RCM needs fix.

* Refactor URDF files for classic and si arms to use RCM frame as reference frame, arm only or arm + SUJ.  instrument frame still broken.

* Renamed link between PSM active arm and instrument adaptor_link.  Fixed for PSM Classic and Si.

* Some simplification in instrument URDF

* Some simplification in instrument URDF

* Refactor ECM URDF and endoscope definitions to use adaptor_link; update joint and link references for compatibility. Added check for launch file parameters

* Reverted change in directory names under urdf so the generation parameter can be used directly to define directories.

* Refactor URDF structure and update instrument macros, renamed and refactored the instrument macro from `PSM_instrument` to `instrument` for consistency across the codebase.

* Refactor instrument housing and roll URDF files

- Removed the generic housing.urdf.xacro and created specific files for Classic and Si housing: housing_Classic.urdf.xacro and housing_Si.urdf.xacro.
- Deleted the roll.urdf.xacro file and added two new roll definitions: roll_4162.urdf.xacro and roll_4670.urdf.xacro.
- Removed the 006_tip.urdf.xacro file and created a new tip_006.urdf.xacro with updated definitions.
- Added a new tip_049.urdf.xacro for the 049 tip.
- Deleted the 0091m_wrist.urdf.xacro and created wrist_pitch_0091.urdf.xacro and wrist_yaw_0091.urdf.xacro for the wrist components.

* Add support for additional PSM instruments and update URDF files

- Introduced new wrist pitch and yaw models (0107) for PSM instruments.
- Added placeholder tips for instruments lacking complete meshes.
- Updated README and structure documentation to reflect new instrument configurations.
- Enhanced launch files to include new instrument options and descriptions.

* Add instrument model-to-part mappings and refactor URDF integration

* Created an ugly Si endoscope :-)

* upload 179 and 093 tips mesh files

* First attempt to add 179 and 093 to urdf

* feat: add Virtual generation support with configurable parent links, RCM parameters, and updated ROS2 launch configurations.

* Enforce dVRK generation launch arguments

* feat: shift Si endoscope tip alignment

* Complete tip 179 mesh placement

* Fix change in 006 from editing the 179

* SWap to updated 049 obj files

* Implement tool 309 to urdf

* Fix 0167 wrist pitch texture error and tips rotation direction

* Fixed wrist pitch orientation and yaw placement

* Fix 0167 wrist pitch orientation and import roll housing with pulleys

* Reposition wrist pitch wrt roll

* Fix wrist yaw rotation and jaw placement/hinge rotation direction

* Upload 172 tip files

* Implement 172 tips

* Fixed 172 tips rotation

* fix 0167 wrist pitch and yaw rotation and placement, and 093 tool complete

* Fix 0167 related 093 and 172 tool tip location and rotation

* tf verify instrument links

* updated arm.launch.py to use single PSM virtual + error messages

* Refactor tip_093 URDF: update jaw joint configuration and mesh references

* Update 0167 error to 0107 and corrected 093 and 172 dh parameters - both use 0107 but with different angle specification

* Implemented 327 with 0107_73 yaw

* UPdate 327 tip texture

* Import 0107 wrist pulleys

* Import wrist 0100

* Import 194 tip and wrist

* Renamed 194 tool tip

* Import 183 and 184 tips and 0093 wrist

* Update 0100 pitch position and wrists textures

* Removed varying 0107 pitch and yaw constraints - unified as +/- 80

* Modify wrist textures

* Removed blue and green from 0091 wrist

* Updated 309 wrist texture and position

* Created wrist pitch and yaw frames for visualization. wrist 0112 position is fixed

* Update 194 tips texture

* Update yaw and tip position for 183

* Constrain 183 and 184 jaw motion to yaw link

* remove mesh files in wrong location

* remove unnecessary components in roll

* removed reference to roll connector

* Updatred  meshes restructure

* Add verification script for instrument DH and asset validation; update CMakeLists and package.xml

* Add 'is_virtual' argument to URDF files and update jaw_zero_publisher logging format

* Add visual validation script and update testing documentation;

* Fixed glitching due to jaw_zero_publisher.py and publisher error

* Updated Si roll 4670 position to match dh parameters

* Updated 0107 yaw position

* Fix error message regarding mixing instrus

* Updated 0091 yaw location

* Differentiate rope and wrist pitch textures

* Differentiate wrist yaw and wire

* Differentiate wrist yaw 0112 and rope

* Updated 194 instrument tool tip position

* Updated metallic Si arms

* Remove jaw zero publisher and frame display

* Update URDF models for housing and roll instruments

- Changed the mesh file for the housing_Classic instrument from housing_Classic.dae to housing_Classic_body.dae in both visual and collision elements.
- Updated the roll_4162 instrument to use roll_4670.obj instead of roll_4162.dae, adjusted the origin parameters, and modified the material name accordingly.

* F2 - Updated naming scheme for materials (6 instruments fixed)

* Updated yaw and tip 183 and 184 with pin and separated gears/tip

* Updated same silver texture for all meshes

---------

Co-authored-by: Anton Deguet <anton.deguet@jhu.edu>

File: urdf/Classic/ECM.urdf.xacro (robot description, xacro)
@@ -1,8 +1,16 @@
 <?xml version="1.0" ?>
-<robot name="ecm" xmlns:xacro="http://www.ros.org/wiki/xacro">
-  <xacro:include filename="$(find dvrk_model)/urdf/Classic/ecm_base.urdf.xacro"/>
-  <link name="world"/>
+<robot name="ECM" xmlns:xacro="http://www.ros.org/wiki/xacro">
+  <xacro:arg name="endoscope" default="Classic_SD_straight"/>
+  <xacro:arg name="parent_link_" default="world"/>
+  <xacro:property name="parent_link" default="$(arg parent_link_)"/>
+  <xacro:include filename="$(find dvrk_model)/urdf/Classic/ECM_base.urdf.xacro"/>
+    <xacro:include filename="$(find dvrk_model)/urdf/common/endoscope.urdf.xacro"/>
+  <link name="${parent_link}"/>
+  <xacro:dvrk_materials/>
   <xacro:ecm_base
       prefix="ECM_"
-      parent_link="world"/>
+      parent_link="${parent_link}"/>
+  <xacro:endoscope
+      prefix="ECM_"
+      parent_link="ECM_adaptor_link"/>
 </robot>

File: urdf/Classic/MTML.urdf.xacro (robot description, xacro)
@@ -1,6 +1,6 @@
 <?xml version="1.0" ?>
-<robot name="master" xmlns:xacro="http://www.ros.org/wiki/xacro">
+<robot name="MTML" xmlns:xacro="http://www.ros.org/wiki/xacro">
   <!-- Macros -->
-  <xacro:include filename="$(find dvrk_model)/urdf/Classic/mtm.urdf.xacro"/>
+  <xacro:include filename="$(find dvrk_model)/urdf/Classic/MTM.urdf.xacro"/>
   <link name="world"/>
   <xacro:mtm_left

File: urdf/Classic/MTMR.urdf.xacro (robot description, xacro)
@@ -1,6 +1,6 @@
 <?xml version="1.0" ?>
-<robot name="master" xmlns:xacro="http://www.ros.org/wiki/xacro">
+<robot name="MTMR" xmlns:xacro="http://www.ros.org/wiki/xacro">
   <!-- Macros -->
-  <xacro:include filename="$(find dvrk_model)/urdf/Classic/mtm.urdf.xacro"/>
+  <xacro:include filename="$(find dvrk_model)/urdf/Classic/MTM.urdf.xacro"/>
   <link name="world"/>
   <xacro:mtm_right

File: urdf/Classic/PSM1.urdf.xacro (robot description, xacro)
@@ -1,11 +1,21 @@
 <?xml version="1.0" ?>
-<robot name="dvrk_psm" xmlns:xacro="http://www.ros.org/wiki/xacro">
-  <xacro:include filename="$(find dvrk_model)/urdf/Classic/psm_base.urdf.xacro"/>
-  <xacro:include filename="$(find dvrk_model)/urdf/Classic/psm_tool.urdf.xacro"/>
-  <link name="world"/>
-  <xacro:psm_base
-      prefix="PSM1_"
-      parent_link="world"
-      xyz="-0.25 0.0 0.5" rpy="0.0 0.0 ${PI}"/>
-  <xacro:psm_tool tool_name="sca" prefix="PSM1_"/>
+<robot name="PSM1" xmlns:xacro="http://www.ros.org/wiki/xacro">
+  <!--
+    Classic PSM1 entry point.
+    arg instrument: last 6 digits of instrument model number (default: 400006)
+    arm placed at a typical setup position; adjust xyz/rpy for your rig.
+  -->
+  <xacro:arg name="instrument" default="400006"/>
+  <xacro:arg name="is_virtual" default="false"/>
+  <xacro:arg name="parent_link_" default="world"/>
+  <xacro:property name="parent_link" value="$(arg parent_link_)"/>
+  <xacro:include filename="$(find dvrk_model)/urdf/Classic/PSM_base.urdf.xacro"/>
+  <xacro:include filename="$(find dvrk_model)/urdf/common/instrument.urdf.xacro"/>
+  <link name="${parent_link}"/>
+  <xacro:base prefix="PSM1_"
+                  parent_link="${parent_link}"
+                  xyz="0.0 0.0 0.0" rpy="0.0 0.0 0.0"/>
+  <xacro:instrument prefix="PSM1_"
+                        instrument="$(arg instrument)"
+                        is_virtual="$(arg is_virtual)"/>
 </robot>

File: urdf/Classic/PSM2.urdf.xacro (robot description, xacro)
@@ -1,11 +1,16 @@
 <?xml version="1.0" ?>
-<robot name="dvrk_psm" xmlns:xacro="http://www.ros.org/wiki/xacro">
-  <xacro:include filename="$(find dvrk_model)/urdf/Classic/psm_base.urdf.xacro"/>
-  <xacro:include filename="$(find dvrk_model)/urdf/Classic/psm_tool.urdf.xacro"/>
-  <link name="world"/>
-  <xacro:psm_base
-      prefix="PSM2_"
-      parent_link="world"
-      xyz="-0.25 0.0 0.5" rpy="0.0 0.0 ${PI}"/>
-  <xacro:psm_tool tool_name="caudier" prefix="PSM2_"/>
+<robot name="PSM2" xmlns:xacro="http://www.ros.org/wiki/xacro">
+  <xacro:arg name="instrument" default="400049"/>
+  <xacro:arg name="is_virtual" default="false"/>
+  <xacro:arg name="parent_link_" default="world"/>
+  <xacro:property name="parent_link" value="$(arg parent_link_)"/>
+  <xacro:include filename="$(find dvrk_model)/urdf/Classic/PSM_base.urdf.xacro"/>
+  <xacro:include filename="$(find dvrk_model)/urdf/common/instrument.urdf.xacro"/>
+  <link name="${parent_link}"/>
+  <xacro:base prefix="PSM2_"
+                  parent_link="${parent_link}"
+                  xyz="0.0 0.0 0.0" rpy="0.0 0.0 0.0"/>
+  <xacro:instrument prefix="PSM2_"
+                        instrument="$(arg instrument)"
+                        is_virtual="$(arg is_virtual)"/>
 </robot>

File: urdf/Classic/PSM3.urdf.xacro (robot description, xacro)
@@ -1,11 +1,16 @@
 <?xml version="1.0" ?>
-<robot name="dvrk_psm" xmlns:xacro="http://www.ros.org/wiki/xacro">
-  <xacro:include filename="$(find dvrk_model)/urdf/Classic/psm_base.urdf.xacro"/>
-  <xacro:include filename="$(find dvrk_model)/urdf/Classic/psm_tool.urdf.xacro"/>
-  <link name="world"/>
-  <xacro:psm_base
-      prefix="PSM3_"
-      parent_link="world"
-      xyz="0.50 0.0 0.5" rpy="0.0 0.0 ${-PI}"/>
-  <xacro:psm_tool tool_name="caudier" prefix="PSM3_"/>
+<robot name="PSM3" xmlns:xacro="http://www.ros.org/wiki/xacro">
+  <xacro:arg name="instrument" default="400049"/>
+  <xacro:arg name="is_virtual" default="false"/>
+  <xacro:arg name="parent_link_" default="world"/>
+  <xacro:property name="parent_link" value="$(arg parent_link_)"/>
+  <xacro:include filename="$(find dvrk_model)/urdf/Classic/PSM_base.urdf.xacro"/>
+  <xacro:include filename="$(find dvrk_model)/urdf/common/instrument.urdf.xacro"/>
+  <link name="${parent_link}"/>
+  <xacro:base prefix="PSM3_"
+                  parent_link="${parent_link}"
+                  xyz="0.0 0.0 0.0" rpy="0.0 0.0 0.0"/>
+  <xacro:instrument prefix="PSM3_"
+                        instrument="$(arg instrument)"
+                        is_virtual="$(arg is_virtual)"/>
 </robot>
