Commit message: update ecm mesh map

File: urdf/common/PSM_tips.urdf.xacro (robot description, xacro)
@@ -345,5 +345,5 @@
         <origin rpy="0 -${PI_2} 0" xyz="0.0051 0.0032 0"/>
         <geometry>
-          <mesh filename="package://dvrk_model/meshes/instruments/Si/tip/ECM_tip_roll.stl"/>
+          <mesh filename="package://dvrk_model/meshes/instruments/Si/roll/ECM_roll.stl"/>
         </geometry>
       </visual>
