Commit message: update naming scheme: wrist instead of tip

File: urdf/common/PSM_tips.urdf.xacro (robot description, xacro)
@@ -20,10 +20,10 @@
     <joint name="wrist_pitch" type="revolute">
       <parent link="${parent_link}"/>
-      <child  link="${prefix}wrist_pitch_link"/>
+      <child  link="${prefix}wrist_006_pitch_link"/>
       <axis xyz="0 0 1"/>
       <origin rpy="-${PI_2} -${PI_2} 0" xyz="0 0 0"/>
       <limit lower="-${PI_2}" upper="${PI_2}" velocity=".4" effort="1000"/>
     </joint>
-    <link name="${prefix}wrist_pitch_link">
+    <link name="${prefix}wrist_006_pitch_link">
       <visual>
         <xacro:if value="${is_si}">
@@ -43,11 +43,11 @@
     <!-- joint 6: wrist_yaw -->
     <joint name="wrist_yaw" type="revolute">
-      <parent link="${prefix}wrist_pitch_link"/>
-      <child  link="${prefix}wrist_yaw_link"/>
+      <parent link="${prefix}wrist_006_pitch_link"/>
+      <child  link="${prefix}wrist_006_yaw_link"/>
       <axis xyz="0 0 1"/>
       <origin rpy="-${PI_2} -${PI_2} 0" xyz="0.0091 0 0"/>
       <limit lower="-1.3963" upper="1.3963" velocity=".4" effort="1000"/>
     </joint>
-    <link name="${prefix}wrist_yaw_link">
+    <link name="${prefix}wrist_006_yaw_link">
       <visual>
         <xacro:if value="${is_si}">
@@ -67,5 +67,5 @@
     <!-- joint 7-0: jaw (virtual centre — drives the mimics) -->
     <joint name="jaw" type="revolute">
-      <parent link="${prefix}wrist_yaw_link"/>
+      <parent link="${prefix}wrist_006_yaw_link"/>
       <child  link="${prefix}jaw_link"/>
       <axis xyz="0 0 1"/>
@@ -82,5 +82,5 @@
     <!-- jaw mimic 1 — opens +0.5× -->
     <joint name="jaw_1" type="revolute">
-      <parent link="${prefix}wrist_yaw_link"/>
+      <parent link="${prefix}wrist_006_yaw_link"/>
       <child  link="${prefix}jaw_1_link"/>
       <axis xyz="0 0 1"/>
@@ -107,5 +107,5 @@
     <!-- jaw mimic 2 — opens −0.5× (symmetric) -->
     <joint name="jaw_2" type="revolute">
-      <parent link="${prefix}wrist_yaw_link"/>
+      <parent link="${prefix}wrist_006_yaw_link"/>
       <child  link="${prefix}jaw_2_link"/>
       <axis xyz="0 0 1"/>
@@ -132,5 +132,5 @@
     <!-- tool tip reference frame -->
     <joint name="tool_tip" type="fixed">
-      <parent link="${prefix}wrist_yaw_link"/>
+      <parent link="${prefix}wrist_006_yaw_link"/>
       <child  link="${prefix}tool_tip_link"/>
       <origin rpy="0 ${PI/2} ${PI/2}" xyz="0 0.0102 0"/>
@@ -144,10 +144,10 @@
     <joint name="wrist_pitch" type="revolute">
       <parent link="${parent_link}"/>
-      <child  link="${prefix}wrist_pitch_link"/>
+      <child  link="${prefix}wrist_049_pitch_link"/>
       <axis xyz="0 0 1"/>
       <origin rpy="-${PI_2} -${PI_2} 0" xyz="0 0 0"/>
       <limit lower="-${PI_2}" upper="${PI_2}" velocity=".4" effort="1000"/>
     </joint>
-    <link name="${prefix}wrist_pitch_link">
+    <link name="${prefix}wrist_049_pitch_link">
       <visual>
         <origin rpy="0 -${PI_2} 0" xyz="-0.0024 0 0"/>
@@ -158,11 +158,11 @@
     </link>
     <joint name="wrist_yaw" type="revolute">
-      <parent link="${prefix}wrist_pitch_link"/>
-      <child  link="${prefix}wrist_yaw_link"/>
+      <parent link="${prefix}wrist_049_pitch_link"/>
+      <child  link="${prefix}wrist_049_yaw_link"/>
       <axis xyz="0 0 1"/>
       <origin rpy="0 -${PI_2} -${PI_2}" xyz="0.0091 0 0"/>
       <limit lower="-1.3963" upper="1.3963" velocity=".4" effort="1000"/>
     </joint>
-    <link name="${prefix}wrist_yaw_link">
+    <link name="${prefix}wrist_049_yaw_link">
       <visual>
         <origin rpy="0 ${PI_2} 0" xyz="0 -0.0002 0"/>
@@ -173,5 +173,5 @@
     </link>
     <joint name="jaw" type="revolute">
-      <parent link="${prefix}wrist_yaw_link"/>
+      <parent link="${prefix}wrist_049_yaw_link"/>
       <child link="${prefix}jaw_link"/>
       <axis xyz="0 0 1"/>
@@ -186,5 +186,5 @@
     </link>
     <joint name="jaw_1" type="revolute">
-      <parent link="${prefix}wrist_yaw_link"/>
+      <parent link="${prefix}wrist_049_yaw_link"/>
       <child link="${prefix}jaw_1_link"/>
       <axis xyz="0 0 1"/>
@@ -202,5 +202,5 @@
     </link>
     <joint name="jaw_2" type="revolute">
-      <parent link="${prefix}wrist_yaw_link"/>
+      <parent link="${prefix}wrist_049_yaw_link"/>
       <child link="${prefix}jaw_2_link"/>
       <axis xyz="0 0 1"/>
@@ -218,5 +218,5 @@
     </link>
     <joint name="tool_tip" type="fixed">
-      <parent link="${prefix}wrist_yaw_link"/>
+      <parent link="${prefix}wrist_049_yaw_link"/>
       <child link="${prefix}tool_tip_link"/>
       <origin rpy="0 ${PI_2} ${PI_2}" xyz="0 0 0"/>
@@ -231,5 +231,5 @@
     <joint name="wrist_pitch" type="revolute">
       <parent link="${parent_link}"/>
-      <child  link="${prefix}wrist_pitch_link"/>
+      <child  link="${prefix}wrist_172_pitch_link"/>
       <axis xyz="0 0 1"/>
       <origin rpy="-${PI_2} -${PI_2} 0" xyz="0 0 0"/>
@@ -240,5 +240,5 @@
       until a dedicated Maryland wrist mesh is added to the repo.
     -->
-    <link name="${prefix}wrist_pitch_link">
+    <link name="${prefix}wrist_172_pitch_link">
       <visual>
         <origin rpy="${PI_2} ${PI} 0" xyz="0.0051 0.0032 0"/>
@@ -250,11 +250,11 @@
     <!-- joint 6: wrist_yaw (A=0.0107 — Maryland specific) -->
     <joint name="wrist_yaw" type="revolute">
-      <parent link="${prefix}wrist_pitch_link"/>
-      <child  link="${prefix}wrist_yaw_link"/>
+      <parent link="${prefix}wrist_172_pitch_link"/>
+      <child  link="${prefix}wrist_172_yaw_link"/>
       <axis xyz="0 0 1"/>
       <origin rpy="-${PI_2} -${PI_2} 0" xyz="0.0107 0 0"/>
       <limit lower="-1.3963" upper="1.3963" velocity=".4" effort="1000"/>
     </joint>
-    <link name="${prefix}wrist_yaw_link">
+    <link name="${prefix}wrist_172_yaw_link">
       <visual>
         <origin rpy="0 0 0" xyz="0 -0.0002 -0.0025"/>
@@ -266,5 +266,5 @@
     <!-- jaw + symmetric mimics (same as tip_006) -->
     <joint name="jaw" type="revolute">
-      <parent link="${prefix}wrist_yaw_link"/>
+      <parent link="${prefix}wrist_172_yaw_link"/>
       <child  link="${prefix}jaw_link"/>
       <axis xyz="0 0 1"/>
@@ -278,5 +278,5 @@
     </link>
     <joint name="jaw_1" type="revolute">
-      <parent link="${prefix}wrist_yaw_link"/>
+      <parent link="${prefix}wrist_172_yaw_link"/>
       <child  link="${prefix}jaw_1_link"/>
       <axis xyz="0 0 1"/>
@@ -294,5 +294,5 @@
     </link>
     <joint name="jaw_2" type="revolute">
-      <parent link="${prefix}wrist_yaw_link"/>
+      <parent link="${prefix}wrist_172_yaw_link"/>
       <child  link="${prefix}jaw_2_link"/>
       <axis xyz="0 0 1"/>
@@ -310,5 +310,5 @@
     </link>
     <joint name="tool_tip" type="fixed">
-      <parent link="${prefix}wrist_yaw_link"/>
+      <parent link="${prefix}wrist_172_yaw_link"/>
       <child  link="${prefix}tool_tip_link"/>
       <origin rpy="0 ${PI/2} ${PI/2}" xyz="0 0.0107 0"/>
@@ -329,12 +329,12 @@
     <joint name="wrist_pitch" type="revolute">
       <parent link="${parent_link}"/>
-      <child  link="${prefix}wrist_pitch_link"/>
+      <child  link="${prefix}wrist_117_pitch_link"/>
       <axis xyz="0 0 1"/>
       <origin rpy="-${PI_2} -${PI_2} 0" xyz="0 0 0"/>
       <limit lower="-${PI_2}" upper="${PI_2}" velocity=".4" effort="1000"/>
     </joint>
-    <link name="${prefix}wrist_pitch_link"/>
+    <link name="${prefix}wrist_117_pitch_link"/>
     <joint name="jaw" type="revolute">
-      <parent link="${prefix}wrist_pitch_link"/>
+      <parent link="${prefix}wrist_117_pitch_link"/>
       <child  link="${prefix}jaw_link"/>
       <axis xyz="0 0 1"/>
@@ -344,5 +344,5 @@
     <link name="${prefix}jaw_link"/>
     <joint name="tool_tip" type="fixed">
-      <parent link="${prefix}wrist_pitch_link"/>
+      <parent link="${prefix}wrist_117_pitch_link"/>
       <child  link="${prefix}tool_tip_link"/>
       <origin rpy="0 0 0" xyz="0 0 0"/>
