Commit message: update mesh map

File: urdf/common/PSM_instrument.urdf.xacro (robot description, xacro)
@@ -45,5 +45,5 @@
           </xacro:if>
           <xacro:unless value="${is_si}">
-            <mesh filename="package://dvrk_model/meshes/instruments/rolls/Classic/PSM_roll.dae"/>
+            <mesh filename="package://dvrk_model/meshes/instruments/housing/Classic/PSM_housing.dae"/>
           </xacro:unless>
         </geometry>
@@ -56,5 +56,5 @@
           </xacro:if>
           <xacro:unless value="${is_si}">
-            <mesh filename="package://dvrk_model/meshes/instruments/rolls/Classic/PSM_roll.dae"/>
+            <mesh filename="package://dvrk_model/meshes/instruments/housing/Classic/PSM_housing.dae"/>
           </xacro:unless>
         </geometry>
@@ -94,5 +94,5 @@
           <origin rpy="0 0 0" xyz="0 0 -${shaft_length}"/>
           <geometry>
-            <mesh filename="package://dvrk_model/meshes/instruments/rolls/Classic/PSM_roll.dae"/>
+            <mesh filename="package://dvrk_model/meshes/instruments/housing/Classic/PSM_housing.dae"/>
           </geometry>
         </xacro:unless>
@@ -108,5 +108,5 @@
           <origin rpy="0 0 0" xyz="0 0 -${shaft_length}"/>
           <geometry>
-            <mesh filename="package://dvrk_model/meshes/instruments/rolls/Classic/PSM_roll.dae"/>
+            <mesh filename="package://dvrk_model/meshes/instruments/housing/Classic/PSM_housing.dae"/>
           </geometry>
         </xacro:unless>

Commit message: update mesh mapping

File: urdf/common/PSM_instrument.urdf.xacro (robot description, xacro)
@@ -131,5 +131,5 @@
           <origin rpy="${PI_2} 0 0" xyz="0 0.00401 0"/>
           <geometry>
-            <mesh filename="package://dvrk_model/meshes/instruments/rolls/Classic/PSM_roll_connector.dae"/>
+            <mesh filename="package://dvrk_model/meshes/instruments/rolls/Classic/PSM_yaw.dae"/>
           </geometry>
         </xacro:unless>
@@ -145,5 +145,5 @@
           <origin rpy="${PI_2} 0 0" xyz="0 0.00401 0"/>
           <geometry>
-            <mesh filename="package://dvrk_model/meshes/instruments/rolls/Classic/PSM_roll_connector.dae"/>
+            <mesh filename="package://dvrk_model/meshes/instruments/rolls/Classic/PSM_yaw.dae"/>
           </geometry>
         </xacro:unless>

File: urdf/common/PSM_tips.urdf.xacro (robot description, xacro)
@@ -29,5 +29,5 @@
         <origin rpy="${PI_2} ${PI} 0" xyz="0.0051 0.0032 0"/>
         <geometry>
-          <mesh filename="package://dvrk_model/meshes/instruments/tips/Classic/400006/PSM_tip_006_pitch.dae"/>
+          <mesh filename="package://dvrk_model/meshes/instruments/tips/Classic/400006/PSM_006_pitch.dae"/>
         </geometry>
       </visual>
@@ -45,5 +45,5 @@
         <origin rpy="0 0 0" xyz="0 -0.0002 -0.0025"/>
         <geometry>
-          <mesh filename="package://dvrk_model/meshes/instruments/tips/Classic/400006/PSM_tip_006_yaw.dae"/>
+          <mesh filename="package://dvrk_model/meshes/instruments/tips/Classic/400006/PSM_006_yaw.dae"/>
         </geometry>
       </visual>
@@ -77,5 +77,5 @@
         <origin rpy="0 0 0" xyz="0 0 0"/>
         <geometry>
-          <mesh filename="package://dvrk_model/meshes/instruments/tips/Classic/400006/PSM_tip_006_jaw.dae"/>
+          <mesh filename="package://dvrk_model/meshes/instruments/tips/Classic/400006/PSM_006_jaw.dae"/>
         </geometry>
       </visual>
@@ -94,5 +94,5 @@
         <origin rpy="0 ${PI} 0" xyz="0 0 0"/>
         <geometry>
-          <mesh filename="package://dvrk_model/meshes/instruments/tips/Classic/400006/PSM_tip_006_jaw.dae"/>
+          <mesh filename="package://dvrk_model/meshes/instruments/tips/Classic/400006/PSM_006_jaw.dae"/>
         </geometry>
       </visual>
@@ -121,5 +121,5 @@
         <origin rpy="0 -${PI_2} 0" xyz="-0.0024 0 0"/>
         <geometry>
-          <mesh filename="package://dvrk_model/meshes/instruments/tips/Classic/400049/PSM_tip_049_pitch.stl"/>
+          <mesh filename="package://dvrk_model/meshes/instruments/tips/Classic/400049/PSM_049_pitch.stl"/>
         </geometry>
       </visual>
@@ -136,5 +136,5 @@
         <origin rpy="0 ${PI_2} 0" xyz="0 -0.0002 0"/>
         <geometry>
-          <mesh filename="package://dvrk_model/meshes/instruments/tips/Classic/400049/PSM_tip_049_yaw.stl"/>
+          <mesh filename="package://dvrk_model/meshes/instruments/tips/Classic/400049/PSM_049_yaw.stl"/>
         </geometry>
       </visual>
@@ -165,5 +165,5 @@
         <origin rpy="0 0 0" xyz="0 0 0.00195"/>
         <geometry>
-          <mesh filename="package://dvrk_model/meshes/instruments/tips/Classic/400049/PSM_tip_049_jaw.stl"/>
+          <mesh filename="package://dvrk_model/meshes/instruments/tips/Classic/400049/PSM_049_jaw.stl"/>
         </geometry>
       </visual>
@@ -181,5 +181,5 @@
         <origin rpy="0 0 -${PI}" xyz="0 0 0.00195"/>
         <geometry>
-          <mesh filename="package://dvrk_model/meshes/instruments/tips/Classic/400049/PSM_tip_049_jaw.stl"/>
+          <mesh filename="package://dvrk_model/meshes/instruments/tips/Classic/400049/PSM_049_jaw.stl"/>
         </geometry>
       </visual>
@@ -212,5 +212,5 @@
         <origin rpy="${PI_2} ${PI} 0" xyz="0.0051 0.0032 0"/>
         <geometry>
-          <mesh filename="package://dvrk_model/meshes/instruments/tips/Classic/400006/PSM_tip_006_pitch.dae"/>
+          <mesh filename="package://dvrk_model/meshes/instruments/tips/Classic/400006/PSM_006_pitch.dae"/>
         </geometry>
       </visual>
@@ -228,5 +228,5 @@
         <origin rpy="0 0 0" xyz="0 -0.0002 -0.0025"/>
         <geometry>
-          <mesh filename="package://dvrk_model/meshes/instruments/tips/Classic/400006/PSM_tip_006_yaw.dae"/>
+          <mesh filename="package://dvrk_model/meshes/instruments/tips/Classic/400006/PSM_006_yaw.dae"/>
         </geometry>
       </visual>
@@ -257,5 +257,5 @@
         <origin rpy="0 0 0" xyz="0 0 0"/>
         <geometry>
-          <mesh filename="package://dvrk_model/meshes/instruments/tips/Classic/400006/PSM_tip_006_jaw.dae"/>
+          <mesh filename="package://dvrk_model/meshes/instruments/tips/Classic/400006/PSM_006_jaw.dae"/>
         </geometry>
       </visual>
@@ -273,5 +273,5 @@
         <origin rpy="0 ${PI} 0" xyz="0 0 0"/>
         <geometry>
-          <mesh filename="package://dvrk_model/meshes/instruments/tips/Classic/400006/PSM_tip_006_jaw.dae"/>
+          <mesh filename="package://dvrk_model/meshes/instruments/tips/Classic/400006/PSM_006_jaw.dae"/>
         </geometry>
       </visual>

Commit message: update mesh mapping

File: urdf/common/PSM_instrument.urdf.xacro (robot description, xacro)
@@ -42,5 +42,5 @@
         <geometry>
           <xacro:if value="${is_si}">
-            <mesh filename="package://dvrk_model/meshes/instruments/rolls/Si/PSM_roll_8mm.stl"/>
+            <mesh filename="package://dvrk_model/meshes/instruments/roll/Si/PSM_roll_8mm.stl"/>
           </xacro:if>
           <xacro:unless value="${is_si}">
@@ -53,5 +53,5 @@
         <geometry>
           <xacro:if value="${is_si}">
-            <mesh filename="package://dvrk_model/meshes/instruments/rolls/Si/PSM_roll_8mm.stl"/>
+            <mesh filename="package://dvrk_model/meshes/instruments/roll/Si/PSM_roll_8mm.stl"/>
           </xacro:if>
           <xacro:unless value="${is_si}">
@@ -86,5 +86,5 @@
           <origin rpy="-${PI} 0 0" xyz="0.05591 0 0"/>
           <geometry>
-            <mesh filename="package://dvrk_model/meshes/instruments/rolls/Si/PSM_roll_housing_8mm.stl"/>
+            <mesh filename="package://dvrk_model/meshes/instruments/roll/Si/PSM_roll_housing_8mm.stl"/>
           </geometry>
           <material name=""><color rgba="0.79216 0.81961 0.93333 1"/></material>
@@ -102,5 +102,5 @@
           <origin rpy="-${PI} 0 0" xyz="0.05591 0 0"/>
           <geometry>
-            <mesh filename="package://dvrk_model/meshes/instruments/rolls/Si/PSM_roll_housing_8mm.stl"/>
+            <mesh filename="package://dvrk_model/meshes/instruments/roll/Si/PSM_roll_housing_8mm.stl"/>
           </geometry>
         </xacro:if>
@@ -124,5 +124,5 @@
           <origin rpy="0 0 0" xyz="0 0 0"/>
           <geometry>
-            <mesh filename="package://dvrk_model/meshes/instruments/rolls/Si/PSM_roll_connector_8mm.stl"/>
+            <mesh filename="package://dvrk_model/meshes/instruments/roll/Si/PSM_roll_connector_8mm.stl"/>
           </geometry>
           <material name=""><color rgba="0.79216 0.81961 0.93333 1"/></material>
@@ -131,5 +131,5 @@
           <origin rpy="${PI_2} 0 0" xyz="0 0.00401 0"/>
           <geometry>
-            <mesh filename="package://dvrk_model/meshes/instruments/rolls/Classic/PSM_yaw.dae"/>
+            <mesh filename="package://dvrk_model/meshes/instruments/roll/Classic/PSM_yaw.dae"/>
           </geometry>
         </xacro:unless>
@@ -139,5 +139,5 @@
           <origin rpy="0 0 0" xyz="0 0 0"/>
           <geometry>
-            <mesh filename="package://dvrk_model/meshes/instruments/rolls/Si/PSM_roll_connector_8mm.stl"/>
+            <mesh filename="package://dvrk_model/meshes/instruments/roll/Si/PSM_roll_connector_8mm.stl"/>
           </geometry>
         </xacro:if>
@@ -145,5 +145,5 @@
           <origin rpy="${PI_2} 0 0" xyz="0 0.00401 0"/>
           <geometry>
-            <mesh filename="package://dvrk_model/meshes/instruments/rolls/Classic/PSM_yaw.dae"/>
+            <mesh filename="package://dvrk_model/meshes/instruments/roll/Classic/PSM_yaw.dae"/>
           </geometry>
         </xacro:unless>

File: urdf/common/PSM_tips.urdf.xacro (robot description, xacro)
@@ -29,5 +29,5 @@
         <origin rpy="${PI_2} ${PI} 0" xyz="0.0051 0.0032 0"/>
         <geometry>
-          <mesh filename="package://dvrk_model/meshes/instruments/tips/Classic/400006/PSM_006_pitch.dae"/>
+          <mesh filename="package://dvrk_model/meshes/instruments/tip/Classic/400006/PSM_006_pitch.dae"/>
         </geometry>
       </visual>
@@ -45,5 +45,5 @@
         <origin rpy="0 0 0" xyz="0 -0.0002 -0.0025"/>
         <geometry>
-          <mesh filename="package://dvrk_model/meshes/instruments/tips/Classic/400006/PSM_006_yaw.dae"/>
+          <mesh filename="package://dvrk_model/meshes/instruments/tip/Classic/400006/PSM_006_yaw.dae"/>
         </geometry>
       </visual>
@@ -77,5 +77,5 @@
         <origin rpy="0 0 0" xyz="0 0 0"/>
         <geometry>
-          <mesh filename="package://dvrk_model/meshes/instruments/tips/Classic/400006/PSM_006_jaw.dae"/>
+          <mesh filename="package://dvrk_model/meshes/instruments/tip/Classic/400006/PSM_006_jaw.dae"/>
         </geometry>
       </visual>
@@ -94,5 +94,5 @@
         <origin rpy="0 ${PI} 0" xyz="0 0 0"/>
         <geometry>
-          <mesh filename="package://dvrk_model/meshes/instruments/tips/Classic/400006/PSM_006_jaw.dae"/>
+          <mesh filename="package://dvrk_model/meshes/instruments/tip/Classic/400006/PSM_006_jaw.dae"/>
         </geometry>
       </visual>
@@ -121,5 +121,5 @@
         <origin rpy="0 -${PI_2} 0" xyz="-0.0024 0 0"/>
         <geometry>
-          <mesh filename="package://dvrk_model/meshes/instruments/tips/Classic/400049/PSM_049_pitch.stl"/>
+          <mesh filename="package://dvrk_model/meshes/instruments/tip/Classic/400049/PSM_049_pitch.stl"/>
         </geometry>
       </visual>
@@ -136,5 +136,5 @@
         <origin rpy="0 ${PI_2} 0" xyz="0 -0.0002 0"/>
         <geometry>
-          <mesh filename="package://dvrk_model/meshes/instruments/tips/Classic/400049/PSM_049_yaw.stl"/>
+          <mesh filename="package://dvrk_model/meshes/instruments/tip/Classic/400049/PSM_049_yaw.stl"/>
         </geometry>
       </visual>
@@ -165,5 +165,5 @@
         <origin rpy="0 0 0" xyz="0 0 0.00195"/>
         <geometry>
-          <mesh filename="package://dvrk_model/meshes/instruments/tips/Classic/400049/PSM_049_jaw.stl"/>
+          <mesh filename="package://dvrk_model/meshes/instruments/tip/Classic/400049/PSM_049_jaw.stl"/>
         </geometry>
       </visual>
@@ -181,5 +181,5 @@
         <origin rpy="0 0 -${PI}" xyz="0 0 0.00195"/>
         <geometry>
-          <mesh filename="package://dvrk_model/meshes/instruments/tips/Classic/400049/PSM_049_jaw.stl"/>
+          <mesh filename="package://dvrk_model/meshes/instruments/tip/Classic/400049/PSM_049_jaw.stl"/>
         </geometry>
       </visual>
@@ -212,5 +212,5 @@
         <origin rpy="${PI_2} ${PI} 0" xyz="0.0051 0.0032 0"/>
         <geometry>
-          <mesh filename="package://dvrk_model/meshes/instruments/tips/Classic/400006/PSM_006_pitch.dae"/>
+          <mesh filename="package://dvrk_model/meshes/instruments/tip/Classic/400006/PSM_006_pitch.dae"/>
         </geometry>
       </visual>
@@ -228,5 +228,5 @@
         <origin rpy="0 0 0" xyz="0 -0.0002 -0.0025"/>
         <geometry>
-          <mesh filename="package://dvrk_model/meshes/instruments/tips/Classic/400006/PSM_006_yaw.dae"/>
+          <mesh filename="package://dvrk_model/meshes/instruments/tip/Classic/400006/PSM_006_yaw.dae"/>
         </geometry>
       </visual>
@@ -257,5 +257,5 @@
         <origin rpy="0 0 0" xyz="0 0 0"/>
         <geometry>
-          <mesh filename="package://dvrk_model/meshes/instruments/tips/Classic/400006/PSM_006_jaw.dae"/>
+          <mesh filename="package://dvrk_model/meshes/instruments/tip/Classic/400006/PSM_006_jaw.dae"/>
         </geometry>
       </visual>
@@ -273,5 +273,5 @@
         <origin rpy="0 ${PI} 0" xyz="0 0 0"/>
         <geometry>
-          <mesh filename="package://dvrk_model/meshes/instruments/tips/Classic/400006/PSM_006_jaw.dae"/>
+          <mesh filename="package://dvrk_model/meshes/instruments/tip/Classic/400006/PSM_006_jaw.dae"/>
         </geometry>
       </visual>
@@ -345,5 +345,5 @@
         <origin rpy="0 -${PI_2} 0" xyz="0.0051 0.0032 0"/>
         <geometry>
-          <mesh filename="package://dvrk_model/meshes/instruments/tips/Si/SF0826001/ECM_tip_roll.stl"/>
+          <mesh filename="package://dvrk_model/meshes/instruments/tip/Si/SF0826001/ECM_tip_roll.stl"/>
         </geometry>
       </visual>

Commit message: update mesh mapping wrt kinematics

File: urdf/common/PSM_instrument.urdf.xacro (robot description, xacro)
@@ -42,8 +42,8 @@
         <geometry>
           <xacro:if value="${is_si}">
-            <mesh filename="package://dvrk_model/meshes/instruments/roll/Si/PSM_roll_8mm.stl"/>
+            <mesh filename="package://dvrk_model/meshes/instruments/si/roll/PSM_roll_8mm.stl"/>
           </xacro:if>
           <xacro:unless value="${is_si}">
-            <mesh filename="package://dvrk_model/meshes/instruments/housing/Classic/PSM_housing.dae"/>
+            <mesh filename="package://dvrk_model/meshes/instruments/classic/housing/PSM_housing.dae"/>
           </xacro:unless>
         </geometry>
@@ -53,8 +53,8 @@
         <geometry>
           <xacro:if value="${is_si}">
-            <mesh filename="package://dvrk_model/meshes/instruments/roll/Si/PSM_roll_8mm.stl"/>
+            <mesh filename="package://dvrk_model/meshes/instruments/si/roll/PSM_roll_8mm.stl"/>
           </xacro:if>
           <xacro:unless value="${is_si}">
-            <mesh filename="package://dvrk_model/meshes/instruments/housing/Classic/PSM_housing.dae"/>
+            <mesh filename="package://dvrk_model/meshes/instruments/classic/housing/PSM_housing.dae"/>
           </xacro:unless>
         </geometry>
@@ -86,5 +86,5 @@
           <origin rpy="-${PI} 0 0" xyz="0.05591 0 0"/>
           <geometry>
-            <mesh filename="package://dvrk_model/meshes/instruments/roll/Si/PSM_roll_housing_8mm.stl"/>
+            <mesh filename="package://dvrk_model/meshes/instruments/si/roll/PSM_roll_housing_8mm.stl"/>
           </geometry>
           <material name=""><color rgba="0.79216 0.81961 0.93333 1"/></material>
@@ -94,5 +94,5 @@
           <origin rpy="0 0 0" xyz="0 0 -${shaft_length}"/>
           <geometry>
-            <mesh filename="package://dvrk_model/meshes/instruments/housing/Classic/PSM_housing.dae"/>
+            <mesh filename="package://dvrk_model/meshes/instruments/classic/housing/PSM_housing.dae"/>
           </geometry>
         </xacro:unless>
@@ -102,5 +102,5 @@
           <origin rpy="-${PI} 0 0" xyz="0.05591 0 0"/>
           <geometry>
-            <mesh filename="package://dvrk_model/meshes/instruments/roll/Si/PSM_roll_housing_8mm.stl"/>
+            <mesh filename="package://dvrk_model/meshes/instruments/si/roll/PSM_roll_housing_8mm.stl"/>
           </geometry>
         </xacro:if>
@@ -108,5 +108,5 @@
           <origin rpy="0 0 0" xyz="0 0 -${shaft_length}"/>
           <geometry>
-            <mesh filename="package://dvrk_model/meshes/instruments/housing/Classic/PSM_housing.dae"/>
+            <mesh filename="package://dvrk_model/meshes/instruments/classic/housing/PSM_housing.dae"/>
           </geometry>
         </xacro:unless>
@@ -124,5 +124,5 @@
           <origin rpy="0 0 0" xyz="0 0 0"/>
           <geometry>
-            <mesh filename="package://dvrk_model/meshes/instruments/roll/Si/PSM_roll_connector_8mm.stl"/>
+            <mesh filename="package://dvrk_model/meshes/instruments/si/roll/PSM_roll_connector_8mm.stl"/>
           </geometry>
           <material name=""><color rgba="0.79216 0.81961 0.93333 1"/></material>
@@ -131,5 +131,5 @@
           <origin rpy="${PI_2} 0 0" xyz="0 0.00401 0"/>
           <geometry>
-            <mesh filename="package://dvrk_model/meshes/instruments/roll/Classic/PSM_yaw.dae"/>
+            <mesh filename="package://dvrk_model/meshes/instruments/classic/yaw/PSM_yaw.dae"/>
           </geometry>
         </xacro:unless>
@@ -139,5 +139,5 @@
           <origin rpy="0 0 0" xyz="0 0 0"/>
           <geometry>
-            <mesh filename="package://dvrk_model/meshes/instruments/roll/Si/PSM_roll_connector_8mm.stl"/>
+            <mesh filename="package://dvrk_model/meshes/instruments/si/roll/PSM_roll_connector_8mm.stl"/>
           </geometry>
         </xacro:if>
@@ -145,5 +145,5 @@
           <origin rpy="${PI_2} 0 0" xyz="0 0.00401 0"/>
           <geometry>
-            <mesh filename="package://dvrk_model/meshes/instruments/roll/Classic/PSM_yaw.dae"/>
+            <mesh filename="package://dvrk_model/meshes/instruments/classic/yaw/PSM_yaw.dae"/>
           </geometry>
         </xacro:unless>

File: urdf/common/PSM_tips.urdf.xacro (robot description, xacro)
@@ -29,5 +29,5 @@
         <origin rpy="${PI_2} ${PI} 0" xyz="0.0051 0.0032 0"/>
         <geometry>
-          <mesh filename="package://dvrk_model/meshes/instruments/tip/Classic/400006/PSM_006_pitch.dae"/>
+          <mesh filename="package://dvrk_model/meshes/instruments/classic/pitch/PSM_006_pitch.dae"/>
         </geometry>
       </visual>
@@ -45,5 +45,5 @@
         <origin rpy="0 0 0" xyz="0 -0.0002 -0.0025"/>
         <geometry>
-          <mesh filename="package://dvrk_model/meshes/instruments/tip/Classic/400006/PSM_006_yaw.dae"/>
+          <mesh filename="package://dvrk_model/meshes/instruments/classic/yaw/PSM_006_yaw.dae"/>
         </geometry>
       </visual>
@@ -77,5 +77,5 @@
         <origin rpy="0 0 0" xyz="0 0 0"/>
         <geometry>
-          <mesh filename="package://dvrk_model/meshes/instruments/tip/Classic/400006/PSM_006_jaw.dae"/>
+          <mesh filename="package://dvrk_model/meshes/instruments/classic/tip/PSM_006_jaw.dae"/>
         </geometry>
       </visual>
@@ -94,5 +94,5 @@
         <origin rpy="0 ${PI} 0" xyz="0 0 0"/>
         <geometry>
-          <mesh filename="package://dvrk_model/meshes/instruments/tip/Classic/400006/PSM_006_jaw.dae"/>
+          <mesh filename="package://dvrk_model/meshes/instruments/classic/tip/PSM_006_jaw.dae"/>
         </geometry>
       </visual>
@@ -121,5 +121,5 @@
         <origin rpy="0 -${PI_2} 0" xyz="-0.0024 0 0"/>
         <geometry>
-          <mesh filename="package://dvrk_model/meshes/instruments/tip/Classic/400049/PSM_049_pitch.stl"/>
+          <mesh filename="package://dvrk_model/meshes/instruments/classic/pitch/PSM_049_pitch.stl"/>
         </geometry>
       </visual>
@@ -136,5 +136,5 @@
         <origin rpy="0 ${PI_2} 0" xyz="0 -0.0002 0"/>
         <geometry>
-          <mesh filename="package://dvrk_model/meshes/instruments/tip/Classic/400049/PSM_049_yaw.stl"/>
+          <mesh filename="package://dvrk_model/meshes/instruments/classic/yaw/PSM_049_yaw.stl"/>
         </geometry>
       </visual>
@@ -165,5 +165,5 @@
         <origin rpy="0 0 0" xyz="0 0 0.00195"/>
         <geometry>
-          <mesh filename="package://dvrk_model/meshes/instruments/tip/Classic/400049/PSM_049_jaw.stl"/>
+          <mesh filename="package://dvrk_model/meshes/instruments/classic/tip/PSM_049_jaw.stl"/>
         </geometry>
       </visual>
@@ -181,5 +181,5 @@
         <origin rpy="0 0 -${PI}" xyz="0 0 0.00195"/>
         <geometry>
-          <mesh filename="package://dvrk_model/meshes/instruments/tip/Classic/400049/PSM_049_jaw.stl"/>
+          <mesh filename="package://dvrk_model/meshes/instruments/classic/tip/PSM_049_jaw.stl"/>
         </geometry>
       </visual>
@@ -212,5 +212,5 @@
         <origin rpy="${PI_2} ${PI} 0" xyz="0.0051 0.0032 0"/>
         <geometry>
-          <mesh filename="package://dvrk_model/meshes/instruments/tip/Classic/400006/PSM_006_pitch.dae"/>
+          <mesh filename="package://dvrk_model/meshes/instruments/classic/pitch/PSM_006_pitch.dae"/>
         </geometry>
       </visual>
@@ -228,5 +228,5 @@
         <origin rpy="0 0 0" xyz="0 -0.0002 -0.0025"/>
         <geometry>
-          <mesh filename="package://dvrk_model/meshes/instruments/tip/Classic/400006/PSM_006_yaw.dae"/>
+          <mesh filename="package://dvrk_model/meshes/instruments/classic/yaw/PSM_006_yaw.dae"/>
         </geometry>
       </visual>
@@ -257,5 +257,5 @@
         <origin rpy="0 0 0" xyz="0 0 0"/>
         <geometry>
-          <mesh filename="package://dvrk_model/meshes/instruments/tip/Classic/400006/PSM_006_jaw.dae"/>
+          <mesh filename="package://dvrk_model/meshes/instruments/classic/tip/PSM_006_jaw.dae"/>
         </geometry>
       </visual>
@@ -273,5 +273,5 @@
         <origin rpy="0 ${PI} 0" xyz="0 0 0"/>
         <geometry>
-          <mesh filename="package://dvrk_model/meshes/instruments/tip/Classic/400006/PSM_006_jaw.dae"/>
+          <mesh filename="package://dvrk_model/meshes/instruments/classic/tip/PSM_006_jaw.dae"/>
         </geometry>
       </visual>
@@ -345,5 +345,5 @@
         <origin rpy="0 -${PI_2} 0" xyz="0.0051 0.0032 0"/>
         <geometry>
-          <mesh filename="package://dvrk_model/meshes/instruments/tip/Si/SF0826001/ECM_tip_roll.stl"/>
+          <mesh filename="package://dvrk_model/meshes/instruments/si/tip/ECM_tip_roll.stl"/>
         </geometry>
       </visual>
