Commit message: update mesh map for Si housing

File: urdf/common/PSM_instrument.urdf.xacro (robot description, xacro)
@@ -42,5 +42,5 @@
         <geometry>
           <xacro:if value="${is_si}">
-            <mesh filename="package://dvrk_model/meshes/instruments/si/roll/PSM_roll_8mm.stl"/>
+            <mesh filename="package://dvrk_model/meshes/instruments/Si/roll/PSM_roll_8mm.stl"/>
           </xacro:if>
           <xacro:unless value="${is_si}">
@@ -53,5 +53,5 @@
         <geometry>
           <xacro:if value="${is_si}">
-            <mesh filename="package://dvrk_model/meshes/instruments/si/roll/PSM_roll_8mm.stl"/>
+            <mesh filename="package://dvrk_model/meshes/instruments/Si/roll/PSM_roll_8mm.stl"/>
           </xacro:if>
           <xacro:unless value="${is_si}">
@@ -86,5 +86,5 @@
           <origin rpy="-${PI} 0 0" xyz="0.05591 0 0"/>
           <geometry>
-            <mesh filename="package://dvrk_model/meshes/instruments/si/roll/PSM_roll_housing_8mm.stl"/>
+            <mesh filename="package://dvrk_model/meshes/instruments/Si/roll/PSM_roll_housing_8mm.stl"/>
           </geometry>
           <material name=""><color rgba="0.79216 0.81961 0.93333 1"/></material>
@@ -102,5 +102,5 @@
           <origin rpy="-${PI} 0 0" xyz="0.05591 0 0"/>
           <geometry>
-            <mesh filename="package://dvrk_model/meshes/instruments/si/roll/PSM_roll_housing_8mm.stl"/>
+            <mesh filename="package://dvrk_model/meshes/instruments/Si/roll/PSM_roll_housing_8mm.stl"/>
           </geometry>
         </xacro:if>
@@ -124,5 +124,5 @@
           <origin rpy="0 0 0" xyz="0 0 0"/>
           <geometry>
-            <mesh filename="package://dvrk_model/meshes/instruments/si/roll/PSM_roll_connector_8mm.stl"/>
+            <mesh filename="package://dvrk_model/meshes/instruments/Si/roll/PSM_roll_connector_8mm.stl"/>
           </geometry>
           <material name=""><color rgba="0.79216 0.81961 0.93333 1"/></material>
@@ -139,5 +139,5 @@
           <origin rpy="0 0 0" xyz="0 0 0"/>
           <geometry>
-            <mesh filename="package://dvrk_model/meshes/instruments/si/roll/PSM_roll_connector_8mm.stl"/>
+            <mesh filename="package://dvrk_model/meshes/instruments/Si/roll/PSM_roll_connector_8mm.stl"/>
           </geometry>
         </xacro:if>

File: urdf/common/PSM_tips.urdf.xacro (robot description, xacro)
@@ -345,5 +345,5 @@
         <origin rpy="0 -${PI_2} 0" xyz="0.0051 0.0032 0"/>
         <geometry>
-          <mesh filename="package://dvrk_model/meshes/instruments/si/tip/ECM_tip_roll.stl"/>
+          <mesh filename="package://dvrk_model/meshes/instruments/Si/tip/ECM_tip_roll.stl"/>
         </geometry>
       </visual>

Commit message: update instruments/Classic in mesh map

File: urdf/common/PSM_instrument.urdf.xacro (robot description, xacro)
@@ -45,5 +45,5 @@
           </xacro:if>
           <xacro:unless value="${is_si}">
-            <mesh filename="package://dvrk_model/meshes/instruments/classic/housing/PSM_housing.dae"/>
+            <mesh filename="package://dvrk_model/meshes/instruments/Classic/housing/PSM_housing.dae"/>
           </xacro:unless>
         </geometry>
@@ -56,5 +56,5 @@
           </xacro:if>
           <xacro:unless value="${is_si}">
-            <mesh filename="package://dvrk_model/meshes/instruments/classic/housing/PSM_housing.dae"/>
+            <mesh filename="package://dvrk_model/meshes/instruments/Classic/housing/PSM_housing.dae"/>
           </xacro:unless>
         </geometry>
@@ -94,5 +94,5 @@
           <origin rpy="0 0 0" xyz="0 0 -${shaft_length}"/>
           <geometry>
-            <mesh filename="package://dvrk_model/meshes/instruments/classic/housing/PSM_housing.dae"/>
+            <mesh filename="package://dvrk_model/meshes/instruments/Classic/housing/PSM_housing.dae"/>
           </geometry>
         </xacro:unless>
@@ -108,5 +108,5 @@
           <origin rpy="0 0 0" xyz="0 0 -${shaft_length}"/>
           <geometry>
-            <mesh filename="package://dvrk_model/meshes/instruments/classic/housing/PSM_housing.dae"/>
+            <mesh filename="package://dvrk_model/meshes/instruments/Classic/housing/PSM_housing.dae"/>
           </geometry>
         </xacro:unless>
@@ -131,5 +131,5 @@
           <origin rpy="${PI_2} 0 0" xyz="0 0.00401 0"/>
           <geometry>
-            <mesh filename="package://dvrk_model/meshes/instruments/classic/yaw/PSM_yaw.dae"/>
+            <mesh filename="package://dvrk_model/meshes/instruments/Classic/yaw/PSM_yaw.dae"/>
           </geometry>
         </xacro:unless>
@@ -145,5 +145,5 @@
           <origin rpy="${PI_2} 0 0" xyz="0 0.00401 0"/>
           <geometry>
-            <mesh filename="package://dvrk_model/meshes/instruments/classic/yaw/PSM_yaw.dae"/>
+            <mesh filename="package://dvrk_model/meshes/instruments/Classic/yaw/PSM_yaw.dae"/>
           </geometry>
         </xacro:unless>

File: urdf/common/PSM_tips.urdf.xacro (robot description, xacro)
@@ -29,5 +29,5 @@
         <origin rpy="${PI_2} ${PI} 0" xyz="0.0051 0.0032 0"/>
         <geometry>
-          <mesh filename="package://dvrk_model/meshes/instruments/classic/pitch/PSM_006_pitch.dae"/>
+          <mesh filename="package://dvrk_model/meshes/instruments/Classic/pitch/PSM_006_pitch.dae"/>
         </geometry>
       </visual>
@@ -45,5 +45,5 @@
         <origin rpy="0 0 0" xyz="0 -0.0002 -0.0025"/>
         <geometry>
-          <mesh filename="package://dvrk_model/meshes/instruments/classic/yaw/PSM_006_yaw.dae"/>
+          <mesh filename="package://dvrk_model/meshes/instruments/Classic/yaw/PSM_006_yaw.dae"/>
         </geometry>
       </visual>
@@ -77,5 +77,5 @@
         <origin rpy="0 0 0" xyz="0 0 0"/>
         <geometry>
-          <mesh filename="package://dvrk_model/meshes/instruments/classic/tip/PSM_006_jaw.dae"/>
+          <mesh filename="package://dvrk_model/meshes/instruments/Classic/tip/PSM_006_jaw.dae"/>
         </geometry>
       </visual>
@@ -94,5 +94,5 @@
         <origin rpy="0 ${PI} 0" xyz="0 0 0"/>
         <geometry>
-          <mesh filename="package://dvrk_model/meshes/instruments/classic/tip/PSM_006_jaw.dae"/>
+          <mesh filename="package://dvrk_model/meshes/instruments/Classic/tip/PSM_006_jaw.dae"/>
         </geometry>
       </visual>
@@ -121,5 +121,5 @@
         <origin rpy="0 -${PI_2} 0" xyz="-0.0024 0 0"/>
         <geometry>
-          <mesh filename="package://dvrk_model/meshes/instruments/classic/pitch/PSM_049_pitch.stl"/>
+          <mesh filename="package://dvrk_model/meshes/instruments/Classic/pitch/PSM_049_pitch.stl"/>
         </geometry>
       </visual>
@@ -136,5 +136,5 @@
         <origin rpy="0 ${PI_2} 0" xyz="0 -0.0002 0"/>
         <geometry>
-          <mesh filename="package://dvrk_model/meshes/instruments/classic/yaw/PSM_049_yaw.stl"/>
+          <mesh filename="package://dvrk_model/meshes/instruments/Classic/yaw/PSM_049_yaw.stl"/>
         </geometry>
       </visual>
@@ -165,5 +165,5 @@
         <origin rpy="0 0 0" xyz="0 0 0.00195"/>
         <geometry>
-          <mesh filename="package://dvrk_model/meshes/instruments/classic/tip/PSM_049_jaw.stl"/>
+          <mesh filename="package://dvrk_model/meshes/instruments/Classic/tip/PSM_049_jaw.stl"/>
         </geometry>
       </visual>
@@ -181,5 +181,5 @@
         <origin rpy="0 0 -${PI}" xyz="0 0 0.00195"/>
         <geometry>
-          <mesh filename="package://dvrk_model/meshes/instruments/classic/tip/PSM_049_jaw.stl"/>
+          <mesh filename="package://dvrk_model/meshes/instruments/Classic/tip/PSM_049_jaw.stl"/>
         </geometry>
       </visual>
@@ -212,5 +212,5 @@
         <origin rpy="${PI_2} ${PI} 0" xyz="0.0051 0.0032 0"/>
         <geometry>
-          <mesh filename="package://dvrk_model/meshes/instruments/classic/pitch/PSM_006_pitch.dae"/>
+          <mesh filename="package://dvrk_model/meshes/instruments/Classic/pitch/PSM_006_pitch.dae"/>
         </geometry>
       </visual>
@@ -228,5 +228,5 @@
         <origin rpy="0 0 0" xyz="0 -0.0002 -0.0025"/>
         <geometry>
-          <mesh filename="package://dvrk_model/meshes/instruments/classic/yaw/PSM_006_yaw.dae"/>
+          <mesh filename="package://dvrk_model/meshes/instruments/Classic/yaw/PSM_006_yaw.dae"/>
         </geometry>
       </visual>
@@ -257,5 +257,5 @@
         <origin rpy="0 0 0" xyz="0 0 0"/>
         <geometry>
-          <mesh filename="package://dvrk_model/meshes/instruments/classic/tip/PSM_006_jaw.dae"/>
+          <mesh filename="package://dvrk_model/meshes/instruments/Classic/tip/PSM_006_jaw.dae"/>
         </geometry>
       </visual>
@@ -273,5 +273,5 @@
         <origin rpy="0 ${PI} 0" xyz="0 0 0"/>
         <geometry>
-          <mesh filename="package://dvrk_model/meshes/instruments/classic/tip/PSM_006_jaw.dae"/>
+          <mesh filename="package://dvrk_model/meshes/instruments/Classic/tip/PSM_006_jaw.dae"/>
         </geometry>
       </visual>

Commit message: update si mesh mapping

File: urdf/common/PSM_instrument.urdf.xacro (robot description, xacro)
@@ -42,5 +42,5 @@
         <geometry>
           <xacro:if value="${is_si}">
-            <mesh filename="package://dvrk_model/meshes/instruments/Si/roll/PSM_roll_8mm.stl"/>
+            <mesh filename="package://dvrk_model/meshes/instruments/Si/roll/PSM_roll_housing_8mm.stl"/>
           </xacro:if>
           <xacro:unless value="${is_si}">
@@ -53,5 +53,5 @@
         <geometry>
           <xacro:if value="${is_si}">
-            <mesh filename="package://dvrk_model/meshes/instruments/Si/roll/PSM_roll_8mm.stl"/>
+            <mesh filename="package://dvrk_model/meshes/instruments/Si/housing/PSM_housing.stl"/>
           </xacro:if>
           <xacro:unless value="${is_si}">

Commit message: fix rotated housing

File: urdf/common/PSM_instrument.urdf.xacro (robot description, xacro)
@@ -31,4 +31,6 @@
     -->
     <xacro:property name="shaft_length" value="${0.4670 if is_ecm else (0.53559 if is_si else 0.4162)}"/>
+    <xacro:property name="tool_main_offset" value="${0.0 if is_si else 0.041}"/>
+    <xacro:property name="roll_origin" value="${shaft_length + tool_main_offset}"/>
     <!-- fixed joint to hold the shaft visual BEFORE the roll joint -->
     <joint name="instrument_base_fixed" type="fixed">
@@ -39,24 +41,30 @@
     <link name="${prefix}instrument_base_link">
       <visual>
-        <origin rpy="0 0 0" xyz="0 0 0"/>
-        <geometry>
-          <xacro:if value="${is_si}">
+        <xacro:if value="${is_si}">
+          <origin rpy="0 0 0" xyz="0 0 0"/>
+          <geometry>
             <mesh filename="package://dvrk_model/meshes/instruments/Si/roll/PSM_roll_housing_8mm.stl"/>
-          </xacro:if>
-          <xacro:unless value="${is_si}">
+          </geometry>
+        </xacro:if>
+        <xacro:unless value="${is_si}">
+          <origin rpy="0 0 1.5708" xyz="0 0 0.041"/>
+          <geometry>
             <mesh filename="package://dvrk_model/meshes/instruments/Classic/housing/PSM_housing.dae"/>
-          </xacro:unless>
-        </geometry>
+          </geometry>
+        </xacro:unless>
       </visual>
       <collision>
-        <origin rpy="0 0 0" xyz="0 0 0"/>
-        <geometry>
-          <xacro:if value="${is_si}">
+        <xacro:if value="${is_si}">
+          <origin rpy="0 0 0" xyz="0 0 0"/>
+          <geometry>
             <mesh filename="package://dvrk_model/meshes/instruments/Si/housing/PSM_housing.stl"/>
-          </xacro:if>
-          <xacro:unless value="${is_si}">
+          </geometry>
+        </xacro:if>
+        <xacro:unless value="${is_si}">
+          <origin rpy="0 0 1.5708" xyz="0 0 0.041"/>
+          <geometry>
             <mesh filename="package://dvrk_model/meshes/instruments/Classic/housing/PSM_housing.dae"/>
-          </xacro:unless>
-        </geometry>
+          </geometry>
+        </xacro:unless>
       </collision>
     </link>
@@ -66,5 +74,5 @@
       <child  link="${prefix}roll_link"/>
       <axis xyz="0 0 1"/>
-      <origin rpy="0 0 0" xyz="0 0 ${shaft_length}"/>
+      <origin rpy="0 0 0" xyz="0 0 ${roll_origin}"/>
       <limit lower="-4.53786" upper="4.53786" velocity=".4" effort="1000"/>
     </joint>
@@ -91,8 +99,8 @@
         </xacro:if>
         <xacro:unless value="${is_si}">
-          <!-- Classic shaft spins with the wrist -->
-          <origin rpy="0 0 0" xyz="0 0 -${shaft_length}"/>
+          <!-- Classic wrist roll housing at the shaft end -->
+          <origin rpy="0 0 1.5708" xyz="0 0 -0.0091"/>
           <geometry>
-            <mesh filename="package://dvrk_model/meshes/instruments/Classic/housing/PSM_housing.dae"/>
+            <mesh filename="package://dvrk_model/meshes/instruments/Classic/roll/PSM_roll.dae"/>
           </geometry>
         </xacro:unless>
@@ -106,7 +114,7 @@
         </xacro:if>
         <xacro:unless value="${is_si}">
-          <origin rpy="0 0 0" xyz="0 0 -${shaft_length}"/>
+          <origin rpy="0 0 1.5708" xyz="0 0 -0.0091"/>
           <geometry>
-            <mesh filename="package://dvrk_model/meshes/instruments/Classic/housing/PSM_housing.dae"/>
+            <mesh filename="package://dvrk_model/meshes/instruments/Classic/roll/PSM_roll.dae"/>
           </geometry>
         </xacro:unless>

Commit message: update housing origin

File: urdf/common/PSM_instrument.urdf.xacro (robot description, xacro)
@@ -48,5 +48,5 @@
         </xacro:if>
         <xacro:unless value="${is_si}">
-          <origin rpy="0 0 1.5708" xyz="0 0 0.041"/>
+          <origin rpy="0 0 1.5708" xyz="0 0 0.0904"/>
           <geometry>
             <mesh filename="package://dvrk_model/meshes/instruments/Classic/housing/PSM_housing.dae"/>
@@ -62,5 +62,5 @@
         </xacro:if>
         <xacro:unless value="${is_si}">
-          <origin rpy="0 0 1.5708" xyz="0 0 0.041"/>
+          <origin rpy="0 0 1.5708" xyz="0 0 0.0904"/>
           <geometry>
             <mesh filename="package://dvrk_model/meshes/instruments/Classic/housing/PSM_housing.dae"/>

Commit message: organize urdf classic with archived files

File: urdf/common/PSM_instrument.urdf.xacro (robot description, xacro)
@@ -42,7 +42,7 @@
       <visual>
         <xacro:if value="${is_si}">
-          <origin rpy="0 0 0" xyz="0 0 0"/>
+          <origin rpy="0 0 0" xyz="-0.05591 0 ${roll_origin}"/>
           <geometry>
-            <mesh filename="package://dvrk_model/meshes/instruments/Si/roll/PSM_roll_housing_8mm.stl"/>
+            <mesh filename="package://dvrk_model/meshes/instruments/Si/housing/PSM_housing.stl"/>
           </geometry>
         </xacro:if>
@@ -56,5 +56,5 @@
       <collision>
         <xacro:if value="${is_si}">
-          <origin rpy="0 0 0" xyz="0 0 0"/>
+          <origin rpy="0 0 0" xyz="-0.05591 0 ${roll_origin}"/>
           <geometry>
             <mesh filename="package://dvrk_model/meshes/instruments/Si/housing/PSM_housing.stl"/>

Commit message: update comments for each instrument

File: urdf/common/PSM_instrument.urdf.xacro (robot description, xacro)
@@ -94,5 +94,5 @@
           <origin rpy="-${PI} 0 0" xyz="0.05591 0 0"/>
           <geometry>
-            <mesh filename="package://dvrk_model/meshes/instruments/Si/roll/PSM_roll_housing_8mm.stl"/>
+            <mesh filename="package://dvrk_model/meshes/instruments/Si/roll/PSM_roll_8mm.stl"/>
           </geometry>
           <material name=""><color rgba="0.79216 0.81961 0.93333 1"/></material>
@@ -110,5 +110,5 @@
           <origin rpy="-${PI} 0 0" xyz="0.05591 0 0"/>
           <geometry>
-            <mesh filename="package://dvrk_model/meshes/instruments/Si/roll/PSM_roll_housing_8mm.stl"/>
+            <mesh filename="package://dvrk_model/meshes/instruments/Si/roll/PSM_roll_8mm.stl"/>
           </geometry>
         </xacro:if>
@@ -132,5 +132,5 @@
           <origin rpy="0 0 0" xyz="0 0 0"/>
           <geometry>
-            <mesh filename="package://dvrk_model/meshes/instruments/Si/roll/PSM_roll_connector_8mm.stl"/>
+            <mesh filename="package://dvrk_model/meshes/instruments/Si/roll/PSM_roll_8mm.stl"/>
           </geometry>
           <material name=""><color rgba="0.79216 0.81961 0.93333 1"/></material>
@@ -147,5 +147,5 @@
           <origin rpy="0 0 0" xyz="0 0 0"/>
           <geometry>
-            <mesh filename="package://dvrk_model/meshes/instruments/Si/roll/PSM_roll_connector_8mm.stl"/>
+            <mesh filename="package://dvrk_model/meshes/instruments/Si/roll/PSM_roll_8mm.stl"/>
           </geometry>
         </xacro:if>
@@ -167,4 +167,5 @@
         183 → cautery / no-jaw tools
     -->
+    <!-- 006: standard SCA wrist -->
     <xacro:if value="${str(instrument) == '420006' or str(instrument) == '400006' or
                       str(instrument) == '420036' or str(instrument) == '400036' or
@@ -174,20 +175,25 @@
                          parent_link="${prefix}wrist_shaft_link"/>
     </xacro:if>
+    <!-- 049: Cadiere jaw -->
     <xacro:if value="${str(instrument) == '420049' or str(instrument) == '400049'}">
       <xacro:PSM_tip_049 prefix="${prefix}"
                          parent_link="${prefix}wrist_shaft_link"/>
     </xacro:if>
+    <!-- 172: Maryland wrist — currently reuses PSM_tip_006 placeholder meshes (see note in PSM_tips.urdf.xacro) -->
     <xacro:if value="${str(instrument) == '420172' or str(instrument) == '400172'}">
       <xacro:PSM_tip_172 prefix="${prefix}"
                          parent_link="${prefix}wrist_shaft_link"/>
     </xacro:if>
+    <!-- 117: snake tool — PSM_tip_117 is currently a kinematic stub only (no meshes, no jaw geometry, DOFs unconfirmed) -->
     <xacro:if value="${str(instrument) == '400117'}">
       <xacro:PSM_tip_117 prefix="${prefix}"
                          parent_link="${prefix}wrist_shaft_link"/>
     </xacro:if>
+    <!-- ECM: Si camera tip -->
     <xacro:if value="${str(instrument) == 'SF0826001'}">
       <xacro:PSM_tip_ECM prefix="${prefix}"
                          parent_link="${prefix}wrist_shaft_link"/>
     </xacro:if>
+    <!-- 183: cautery / no-jaw tools — PSM_tip_183 macro exists in PSM_tips.urdf.xacro but is not yet wired into this dispatch -->
   </xacro:macro>
 </robot>
