Commit message: swap high res meshes with archived stl

File: urdf/common/PSM_instrument.urdf.xacro (robot description, xacro)
@@ -44,5 +44,5 @@
           <origin rpy="0 0 0" xyz="-0.05591 0 ${roll_origin}"/>
           <geometry>
-            <mesh filename="package://dvrk_model/meshes/instruments/Si/housing/PSM_housing.stl"/>
+            <mesh filename="package://dvrk_model/meshes/instruments/Si/housing/PSM_housing.OBJ"/>
           </geometry>
         </xacro:if>
@@ -58,5 +58,5 @@
           <origin rpy="0 0 0" xyz="-0.05591 0 ${roll_origin}"/>
           <geometry>
-            <mesh filename="package://dvrk_model/meshes/instruments/Si/housing/PSM_housing.stl"/>
+            <mesh filename="package://dvrk_model/meshes/instruments/Si/housing/PSM_housing.OBJ"/>
           </geometry>
         </xacro:if>
@@ -94,5 +94,5 @@
           <origin rpy="-${PI} 0 0" xyz="0.05591 0 0"/>
           <geometry>
-            <mesh filename="package://dvrk_model/meshes/instruments/Si/roll/PSM_roll_8mm.stl"/>
+            <mesh filename="package://dvrk_model/meshes/instruments/Si/roll/PSM_roll_8mm.OBJ"/>
           </geometry>
           <material name=""><color rgba="0.79216 0.81961 0.93333 1"/></material>
@@ -110,5 +110,5 @@
           <origin rpy="-${PI} 0 0" xyz="0.05591 0 0"/>
           <geometry>
-            <mesh filename="package://dvrk_model/meshes/instruments/Si/roll/PSM_roll_8mm.stl"/>
+            <mesh filename="package://dvrk_model/meshes/instruments/Si/roll/PSM_roll_8mm.OBJ"/>
           </geometry>
         </xacro:if>
@@ -132,5 +132,5 @@
           <origin rpy="0 0 0" xyz="0 0 0"/>
           <geometry>
-            <mesh filename="package://dvrk_model/meshes/instruments/Si/roll/PSM_roll_8mm.stl"/>
+            <mesh filename="package://dvrk_model/meshes/instruments/Si/roll/PSM_roll_8mm.OBJ"/>
           </geometry>
           <material name=""><color rgba="0.79216 0.81961 0.93333 1"/></material>
@@ -147,5 +147,5 @@
           <origin rpy="0 0 0" xyz="0 0 0"/>
           <geometry>
-            <mesh filename="package://dvrk_model/meshes/instruments/Si/roll/PSM_roll_8mm.stl"/>
+            <mesh filename="package://dvrk_model/meshes/instruments/Si/roll/PSM_roll_8mm.OBJ"/>
           </geometry>
         </xacro:if>
@@ -173,5 +173,6 @@
                       str(instrument) == '420168' or str(instrument) == '400168'}">
       <xacro:PSM_tip_006 prefix="${prefix}"
-                         parent_link="${prefix}shaft_link"/>
+                         parent_link="${prefix}shaft_link"
+                         is_si="${is_si}"/>
     </xacro:if>
     <!-- 049: Cadiere jaw -->

File: urdf/common/PSM_tips.urdf.xacro (robot description, xacro)
@@ -16,5 +16,5 @@
   <!-- PSM_tip_006 — standard SCA wrist (most Classic and Si instruments)  -->
   <!-- ════════════════════════════════════════════════════════════════════ -->
-  <xacro:macro name="PSM_tip_006" params="prefix parent_link">
+  <xacro:macro name="PSM_tip_006" params="prefix parent_link is_si:=false">
     <!-- joint 5: tip_pitch -->
     <joint name="tip_pitch" type="revolute">
@@ -27,8 +27,16 @@
     <link name="${prefix}tip_006_pitch_link">
       <visual>
-        <origin rpy="${PI_2} ${PI} 0" xyz="0.0051 0.0032 0"/>
-        <geometry>
-          <mesh filename="package://dvrk_model/meshes/instruments/Classic/pitch/PSM_006_pitch.dae"/>
-        </geometry>
+        <xacro:if value="${is_si}">
+          <origin rpy="${PI_2} ${PI} 0" xyz="0.0051 0.0032 0"/>
+          <geometry>
+            <mesh filename="package://dvrk_model/meshes/instruments/Si/pitch/PSM_006_pitch.OBJ"/>
+          </geometry>
+        </xacro:if>
+        <xacro:unless value="${is_si}">
+          <origin rpy="${PI_2} ${PI} 0" xyz="0.0051 0.0032 0"/>
+          <geometry>
+            <mesh filename="package://dvrk_model/meshes/instruments/Classic/pitch/PSM_006_pitch.dae"/>
+          </geometry>
+        </xacro:unless>
       </visual>
     </link>
@@ -43,8 +51,16 @@
     <link name="${prefix}tip_006_yaw_link">
       <visual>
-        <origin rpy="0 0 0" xyz="0 -0.0002 -0.0025"/>
-        <geometry>
-          <mesh filename="package://dvrk_model/meshes/instruments/Classic/yaw/PSM_006_yaw.dae"/>
-        </geometry>
+        <xacro:if value="${is_si}">
+          <origin rpy="0 0 0" xyz="0 -0.0002 -0.0025"/>
+          <geometry>
+            <mesh filename="package://dvrk_model/meshes/instruments/Si/yaw/PSM_006_yaw.OBJ"/>
+          </geometry>
+        </xacro:if>
+        <xacro:unless value="${is_si}">
+          <origin rpy="0 0 0" xyz="0 -0.0002 -0.0025"/>
+          <geometry>
+            <mesh filename="package://dvrk_model/meshes/instruments/Classic/yaw/PSM_006_yaw.dae"/>
+          </geometry>
+        </xacro:unless>
       </visual>
     </link>
@@ -75,8 +91,16 @@
     <link name="${prefix}jaw_1_link">
       <visual>
-        <origin rpy="0 0 0" xyz="0 0 0"/>
-        <geometry>
-          <mesh filename="package://dvrk_model/meshes/instruments/Classic/tip/PSM_006_jaw.dae"/>
-        </geometry>
+        <xacro:if value="${is_si}">
+          <origin rpy="0 0 0" xyz="0 0 0"/>
+          <geometry>
+            <mesh filename="package://dvrk_model/meshes/instruments/Si/tip/PSM_006_jaw_1.OBJ"/>
+          </geometry>
+        </xacro:if>
+        <xacro:unless value="${is_si}">
+          <origin rpy="0 0 0" xyz="0 0 0"/>
+          <geometry>
+            <mesh filename="package://dvrk_model/meshes/instruments/Classic/tip/PSM_006_jaw.dae"/>
+          </geometry>
+        </xacro:unless>
       </visual>
     </link>
@@ -92,8 +116,16 @@
     <link name="${prefix}jaw_2_link">
       <visual>
-        <origin rpy="0 ${PI} 0" xyz="0 0 0"/>
-        <geometry>
-          <mesh filename="package://dvrk_model/meshes/instruments/Classic/tip/PSM_006_jaw.dae"/>
-        </geometry>
+        <xacro:if value="${is_si}">
+          <origin rpy="0 0 0" xyz="0 0 0"/>
+          <geometry>
+            <mesh filename="package://dvrk_model/meshes/instruments/Si/tip/PSM_006_jaw_2.OBJ"/>
+          </geometry>
+        </xacro:if>
+        <xacro:unless value="${is_si}">
+          <origin rpy="0 ${PI} 0" xyz="0 0 0"/>
+          <geometry>
+            <mesh filename="package://dvrk_model/meshes/instruments/Classic/tip/PSM_006_jaw.dae"/>
+          </geometry>
+        </xacro:unless>
       </visual>
     </link>

Commit message: Si instrument load in Classic arm - resolved mesh appearance/positioning

File: urdf/common/PSM_instrument.urdf.xacro (robot description, xacro)
@@ -27,20 +27,22 @@
       Shaft length (D parameter of the roll joint):
         Classic PSM instruments → 0.4162
-        Si PSM instruments      → 0.53559
-        Si ECM (SF0826001)      → 0.4670   (camera tube is shorter than PSM shafts)
+        Si instruments          → 0.4670
+        Classic instruments     → 0.4162
     -->
-    <xacro:property name="shaft_length" value="${0.4670 if is_ecm else (0.53559 if is_si else 0.4162)}"/>
+    <xacro:property name="shaft_length" value="${0.4670 if is_si else 0.4162}"/>
     <xacro:property name="tool_main_offset" value="${0.0 if is_si else 0.041}"/>
     <xacro:property name="roll_origin" value="${shaft_length + tool_main_offset}"/>
+    <xacro:property name="tip_parent_link" value="${prefix + ('roll_link' if is_si else 'shaft_link')}"/>
     <!-- fixed joint to hold the shaft visual BEFORE the roll joint -->
     <joint name="instrument_base_fixed" type="fixed">
       <parent link="${parent_link}"/>
       <child  link="${prefix}instrument_base_link"/>
-      <origin rpy="0 0 0" xyz="0 0 0"/>
+      <origin rpy="-1.5708 0 -1.5708" xyz="0 0 0"/>
     </joint>
     <link name="${prefix}instrument_base_link">
       <visual>
         <xacro:if value="${is_si}">
-          <origin rpy="0 0 0" xyz="-0.05591 0 ${roll_origin}"/>
+          <!-- Si housing lives at the proximal tool base (not along the shaft). -->
+          <origin rpy="-1.5708 0 -1.5708" xyz="0 0 0"/>
           <geometry>
             <mesh filename="package://dvrk_model/meshes/instruments/Si/housing/PSM_housing.OBJ"/>
@@ -56,5 +58,5 @@
       <collision>
         <xacro:if value="${is_si}">
-          <origin rpy="0 0 0" xyz="-0.05591 0 ${roll_origin}"/>
+          <origin rpy="0 0 0" xyz="0 0 0"/>
           <geometry>
             <mesh filename="package://dvrk_model/meshes/instruments/Si/housing/PSM_housing.OBJ"/>
@@ -81,5 +83,23 @@
       The outer shaft mesh (above) does not roll or shift.
     -->
-    <link name="${prefix}roll_link"/>
+    <link name="${prefix}roll_link">
+      <visual>
+        <xacro:if value="${is_si}">
+          <origin rpy="0 0 0" xyz="0 0 -0.216"/>
+          <geometry>
+            <mesh filename="package://dvrk_model/meshes/instruments/Si/roll/PSM_roll_8mm.OBJ"/>
+          </geometry>
+          <material name=""><color rgba="0.79216 0.81961 0.93333 1"/></material>
+        </xacro:if>
+      </visual>
+      <collision>
+        <xacro:if value="${is_si}">
+          <origin rpy="0 0 0" xyz="0 0 -0.216"/>
+          <geometry>
+            <mesh filename="package://dvrk_model/meshes/instruments/Si/roll/PSM_roll_8mm.OBJ"/>
+          </geometry>
+        </xacro:if>
+      </collision>
+    </link>
     <!-- fixed joint to roll housing -->
     <joint name="roll_fixed" type="fixed">
@@ -90,12 +110,5 @@
     <link name="${prefix}roll_housing_link">
       <visual>
-        <xacro:if value="${is_si}">
-          <!-- Si roll housing piece is centered at the roll joint -->
-          <origin rpy="-${PI} 0 0" xyz="0.05591 0 0"/>
-          <geometry>
-            <mesh filename="package://dvrk_model/meshes/instruments/Si/roll/PSM_roll_8mm.OBJ"/>
-          </geometry>
-          <material name=""><color rgba="0.79216 0.81961 0.93333 1"/></material>
-        </xacro:if>
+        <!-- Si: structural link only, no duplicate shaft visual here. -->
         <xacro:unless value="${is_si}">
           <!-- Classic roll housing at the shaft end -->
@@ -107,10 +120,4 @@
       </visual>
       <collision>
-        <xacro:if value="${is_si}">
-          <origin rpy="-${PI} 0 0" xyz="0.05591 0 0"/>
-          <geometry>
-            <mesh filename="package://dvrk_model/meshes/instruments/Si/roll/PSM_roll_8mm.OBJ"/>
-          </geometry>
-        </xacro:if>
         <xacro:unless value="${is_si}">
           <origin rpy="0 0 1.5708" xyz="0 0 -0.0091"/>
@@ -129,11 +136,4 @@
     <link name="${prefix}shaft_link">
       <visual>
-        <xacro:if value="${is_si}">
-          <origin rpy="0 0 0" xyz="0 0 0"/>
-          <geometry>
-            <mesh filename="package://dvrk_model/meshes/instruments/Si/roll/PSM_roll_8mm.OBJ"/>
-          </geometry>
-          <material name=""><color rgba="0.79216 0.81961 0.93333 1"/></material>
-        </xacro:if>
         <xacro:unless value="${is_si}">
           <origin rpy="${PI_2} 0 0" xyz="0 0.00401 0"/>
@@ -144,10 +144,4 @@
       </visual>
       <collision>
-        <xacro:if value="${is_si}">
-          <origin rpy="0 0 0" xyz="0 0 0"/>
-          <geometry>
-            <mesh filename="package://dvrk_model/meshes/instruments/Si/roll/PSM_roll_8mm.OBJ"/>
-          </geometry>
-        </xacro:if>
         <xacro:unless value="${is_si}">
           <origin rpy="${PI_2} 0 0" xyz="0 0.00401 0"/>
@@ -173,5 +167,5 @@
                       str(instrument) == '420168' or str(instrument) == '400168'}">
       <xacro:PSM_tip_006 prefix="${prefix}"
-                         parent_link="${prefix}shaft_link"
+                         parent_link="${tip_parent_link}"
                          is_si="${is_si}"/>
     </xacro:if>
@@ -179,20 +173,20 @@
     <xacro:if value="${str(instrument) == '420049' or str(instrument) == '400049'}">
       <xacro:PSM_tip_049 prefix="${prefix}"
-                         parent_link="${prefix}shaft_link"/>
+                         parent_link="${tip_parent_link}"/>
     </xacro:if>
     <!-- 172: Maryland wrist — currently reuses PSM_tip_006 placeholder meshes (see note in PSM_tips.urdf.xacro) -->
     <xacro:if value="${str(instrument) == '420172' or str(instrument) == '400172'}">
       <xacro:PSM_tip_172 prefix="${prefix}"
-                         parent_link="${prefix}shaft_link"/>
+                         parent_link="${tip_parent_link}"/>
     </xacro:if>
     <!-- 117: snake tool — PSM_tip_117 is currently a kinematic stub only (no meshes, no jaw geometry, DOFs unconfirmed) -->
     <xacro:if value="${str(instrument) == '400117'}">
       <xacro:PSM_tip_117 prefix="${prefix}"
-                         parent_link="${prefix}shaft_link"/>
+                         parent_link="${tip_parent_link}"/>
     </xacro:if>
     <!-- ECM: Si camera tip -->
     <xacro:if value="${str(instrument) == 'SF0826001'}">
       <xacro:PSM_tip_ECM prefix="${prefix}"
-                         parent_link="${prefix}shaft_link"/>
+                         parent_link="${tip_parent_link}"/>
     </xacro:if>
     <!-- 183: cautery / no-jaw tools — PSM_tip_183 macro exists in PSM_tips.urdf.xacro but is not yet wired into this dispatch -->

File: urdf/common/PSM_tips.urdf.xacro (robot description, xacro)
@@ -28,5 +28,5 @@
       <visual>
         <xacro:if value="${is_si}">
-          <origin rpy="${PI_2} ${PI} 0" xyz="0.0051 0.0032 0"/>
+          <origin rpy="0 0 0" xyz="0 0 0"/>
           <geometry>
             <mesh filename="package://dvrk_model/meshes/instruments/Si/pitch/PSM_006_pitch.OBJ"/>
@@ -52,5 +52,5 @@
       <visual>
         <xacro:if value="${is_si}">
-          <origin rpy="0 0 0" xyz="0 -0.0002 -0.0025"/>
+          <origin rpy="0 0 0" xyz="0 0 -0.000236"/>
           <geometry>
             <mesh filename="package://dvrk_model/meshes/instruments/Si/yaw/PSM_006_yaw.OBJ"/>
@@ -92,5 +92,5 @@
       <visual>
         <xacro:if value="${is_si}">
-          <origin rpy="0 0 0" xyz="0 0 0"/>
+          <origin rpy="0 0 0" xyz="0 0 -0.000936"/>
           <geometry>
             <mesh filename="package://dvrk_model/meshes/instruments/Si/tip/PSM_006_jaw_1.OBJ"/>
@@ -117,5 +117,5 @@
       <visual>
         <xacro:if value="${is_si}">
-          <origin rpy="0 0 0" xyz="0 0 0"/>
+          <origin rpy="0 0 0" xyz="0 0 0.000961"/>
           <geometry>
             <mesh filename="package://dvrk_model/meshes/instruments/Si/tip/PSM_006_jaw_2.OBJ"/>
