Commit message: Add instrument model-to-part mappings and refactor URDF integration

File: urdf/common/instrument.urdf.xacro (robot description, xacro)
@@ -25,4 +25,6 @@
   <xacro:include filename="$(find dvrk_model)/urdf/common/instruments/tip/tip_049.urdf.xacro"/>
   <xacro:include filename="$(find dvrk_model)/urdf/common/instruments/tip/tip_placeholder.urdf.xacro"/>
+  <xacro:property name="instrument_table"
+                  value="${xacro.load_yaml('$(find dvrk_model)/urdf/common/instruments/instruments.yaml')['instruments']}"/>
   <xacro:macro name="instrument_model"
                params="prefix housing roll wrist_pitch wrist_yaw tip">
@@ -63,337 +65,12 @@
   <xacro:macro name="instrument"
                params="prefix instrument">
-    <!-- 400001: Classic 001 -->
-    <xacro:if value="${str(instrument) == '400001'}">
-      <xacro:instrument_model prefix="${prefix}"
-                              housing="Classic"
-                              roll="4162"
-                              wrist_pitch="0091"
-                              wrist_yaw="0091"
-                              tip="001"/>
-    </xacro:if>
-    <!-- 400003: Classic 003 -->
-    <xacro:if value="${str(instrument) == '400003'}">
-      <xacro:instrument_model prefix="${prefix}"
-                              housing="Classic"
-                              roll="4162"
-                              wrist_pitch="0091"
-                              wrist_yaw="0091"
-                              tip="003"/>
-    </xacro:if>
-    <!-- 400006: Classic 006 -->
-    <xacro:if value="${str(instrument) == '400006'}">
-      <xacro:instrument_model prefix="${prefix}"
-                              housing="Classic"
-                              roll="4162"
-                              wrist_pitch="0091"
-                              wrist_yaw="0091"
-                              tip="006"/>
-    </xacro:if>
-    <!-- 400007: Classic 007 -->
-    <xacro:if value="${str(instrument) == '400007'}">
-      <xacro:instrument_model prefix="${prefix}"
-                              housing="Classic"
-                              roll="4162"
-                              wrist_pitch="0091"
-                              wrist_yaw="0091"
-                              tip="007"/>
-    </xacro:if>
-    <!-- 400033: Classic 033 -->
-    <xacro:if value="${str(instrument) == '400033'}">
-      <xacro:instrument_model prefix="${prefix}"
-                              housing="Classic"
-                              roll="4162"
-                              wrist_pitch="0091"
-                              wrist_yaw="0091"
-                              tip="033"/>
-    </xacro:if>
-    <!-- 400035: Classic 035 -->
-    <xacro:if value="${str(instrument) == '400035'}">
-      <xacro:instrument_model prefix="${prefix}"
-                              housing="Classic"
-                              roll="4162"
-                              wrist_pitch="0091"
-                              wrist_yaw="0091"
-                              tip="035"/>
-    </xacro:if>
-    <!-- 400036: Classic 036 -->
-    <xacro:if value="${str(instrument) == '400036'}">
-      <xacro:instrument_model prefix="${prefix}"
-                              housing="Classic"
-                              roll="4162"
-                              wrist_pitch="0091"
-                              wrist_yaw="0091"
-                              tip="036"/>
-    </xacro:if>
-    <!-- 400048: Classic 048 -->
-    <xacro:if value="${str(instrument) == '400048'}">
-      <xacro:instrument_model prefix="${prefix}"
-                              housing="Classic"
-                              roll="4162"
-                              wrist_pitch="0091"
-                              wrist_yaw="0091"
-                              tip="048"/>
-    </xacro:if>
-    <!-- 400049: Classic 049 -->
-    <xacro:if value="${str(instrument) == '400049'}">
-      <xacro:instrument_model prefix="${prefix}"
-                              housing="Classic"
-                              roll="4162"
-                              wrist_pitch="0091"
-                              wrist_yaw="0091"
-                              tip="049"/>
-    </xacro:if>
-    <!-- 400093: Classic 093 -->
-    <xacro:if value="${str(instrument) == '400093'}">
-      <xacro:instrument_model prefix="${prefix}"
-                              housing="Classic"
-                              roll="4162"
-                              wrist_pitch="0107"
-                              wrist_yaw="0107"
-                              tip="093"/>
-    </xacro:if>
-    <!-- 400127: Classic 127 -->
-    <xacro:if value="${str(instrument) == '400127'}">
-      <xacro:instrument_model prefix="${prefix}"
-                              housing="Classic"
-                              roll="4162"
-                              wrist_pitch="0107"
-                              wrist_yaw="0107"
-                              tip="127"/>
-    </xacro:if>
-    <!-- 400172: Classic 172 -->
-    <xacro:if value="${str(instrument) == '400172'}">
-      <xacro:instrument_model prefix="${prefix}"
-                              housing="Classic"
-                              roll="4162"
-                              wrist_pitch="0107"
-                              wrist_yaw="0107"
-                              tip="172"/>
-    </xacro:if>
-    <!-- 400178: Classic 178 -->
-    <xacro:if value="${str(instrument) == '400178'}">
-      <xacro:instrument_model prefix="${prefix}"
-                              housing="Classic"
-                              roll="4162"
-                              wrist_pitch="0091"
-                              wrist_yaw="0091"
-                              tip="178"/>
-    </xacro:if>
-    <!-- 400179: Classic 179 -->
-    <xacro:if value="${str(instrument) == '400179'}">
-      <xacro:instrument_model prefix="${prefix}"
-                              housing="Classic"
-                              roll="4162"
-                              wrist_pitch="0091"
-                              wrist_yaw="0091"
-                              tip="179"/>
-    </xacro:if>
-    <!-- 400181: Classic 181 -->
-    <xacro:if value="${str(instrument) == '400181'}">
-      <xacro:instrument_model prefix="${prefix}"
-                              housing="Classic"
-                              roll="4162"
-                              wrist_pitch="0091"
-                              wrist_yaw="0091"
-                              tip="181"/>
-    </xacro:if>
-    <!-- 400189: Classic 189 -->
-    <xacro:if value="${str(instrument) == '400189'}">
-      <xacro:instrument_model prefix="${prefix}"
-                              housing="Classic"
-                              roll="4162"
-                              wrist_pitch="0107"
-                              wrist_yaw="0107"
-                              tip="189"/>
-    </xacro:if>
-    <!-- 400205: Classic 205 -->
-    <xacro:if value="${str(instrument) == '400205'}">
-      <xacro:instrument_model prefix="${prefix}"
-                              housing="Classic"
-                              roll="4162"
-                              wrist_pitch="0107"
-                              wrist_yaw="0107"
-                              tip="205"/>
-    </xacro:if>
-    <!-- 400207: Classic 207 -->
-    <xacro:if value="${str(instrument) == '400207'}">
-      <xacro:instrument_model prefix="${prefix}"
-                              housing="Classic"
-                              roll="4162"
-                              wrist_pitch="0107"
-                              wrist_yaw="0107"
-                              tip="207"/>
-    </xacro:if>
-    <!-- 400208: Classic 208 -->
-    <xacro:if value="${str(instrument) == '400208'}">
-      <xacro:instrument_model prefix="${prefix}"
-                              housing="Classic"
-                              roll="4162"
-                              wrist_pitch="0107"
-                              wrist_yaw="0107"
-                              tip="208"/>
-    </xacro:if>
-    <!-- 400230: Classic 230 -->
-    <xacro:if value="${str(instrument) == '400230'}">
-      <xacro:instrument_model prefix="${prefix}"
-                              housing="Classic"
-                              roll="4162"
-                              wrist_pitch="0107"
-                              wrist_yaw="0107"
-                              tip="230"/>
-    </xacro:if>
-    <!-- 400296: Classic 296 -->
-    <xacro:if value="${str(instrument) == '400296'}">
-      <xacro:instrument_model prefix="${prefix}"
-                              housing="Classic"
-                              roll="4162"
-                              wrist_pitch="0091"
-                              wrist_yaw="0091"
-                              tip="296"/>
-    </xacro:if>
-    <!-- 420001: Si 001 -->
-    <xacro:if value="${str(instrument) == '420001'}">
-      <xacro:instrument_model prefix="${prefix}"
-                              housing="Si"
-                              roll="4670"
-                              wrist_pitch="0091"
-                              wrist_yaw="0091"
-                              tip="001"/>
-    </xacro:if>
-    <!-- 420006: Si 006 -->
-    <xacro:if value="${str(instrument) == '420006'}">
-      <xacro:instrument_model prefix="${prefix}"
-                              housing="Si"
-                              roll="4670"
-                              wrist_pitch="0091"
-                              wrist_yaw="0091"
-                              tip="006"/>
-    </xacro:if>
-    <!-- 420007: Si 007 -->
-    <xacro:if value="${str(instrument) == '420007'}">
-      <xacro:instrument_model prefix="${prefix}"
-                              housing="Si"
-                              roll="4670"
-                              wrist_pitch="0091"
-                              wrist_yaw="0091"
-                              tip="007"/>
-    </xacro:if>
-    <!-- 420033: Si 033 -->
-    <xacro:if value="${str(instrument) == '420033'}">
-      <xacro:instrument_model prefix="${prefix}"
-                              housing="Si"
-                              roll="4670"
-                              wrist_pitch="0091"
-                              wrist_yaw="0091"
-                              tip="033"/>
-    </xacro:if>
-    <!-- 420036: Si 036 -->
-    <xacro:if value="${str(instrument) == '420036'}">
-      <xacro:instrument_model prefix="${prefix}"
-                              housing="Si"
-                              roll="4670"
-                              wrist_pitch="0091"
-                              wrist_yaw="0091"
-                              tip="036"/>
-    </xacro:if>
-    <!-- 420048: Si 048 -->
-    <xacro:if value="${str(instrument) == '420048'}">
-      <xacro:instrument_model prefix="${prefix}"
-                              housing="Si"
-                              roll="4670"
-                              wrist_pitch="0091"
-                              wrist_yaw="0091"
-                              tip="048"/>
-    </xacro:if>
-    <!-- 420049: Si 049 -->
-    <xacro:if value="${str(instrument) == '420049'}">
-      <xacro:instrument_model prefix="${prefix}"
-                              housing="Si"
-                              roll="4670"
-                              wrist_pitch="0091"
-                              wrist_yaw="0091"
-                              tip="049"/>
-    </xacro:if>
-    <!-- 420093: Si 093 -->
-    <xacro:if value="${str(instrument) == '420093'}">
-      <xacro:instrument_model prefix="${prefix}"
-                              housing="Si"
-                              roll="4670"
-                              wrist_pitch="0107"
-                              wrist_yaw="0107"
-                              tip="093"/>
-    </xacro:if>
-    <!-- 420172: Si 172 -->
-    <xacro:if value="${str(instrument) == '420172'}">
-      <xacro:instrument_model prefix="${prefix}"
-                              housing="Si"
-                              roll="4670"
-                              wrist_pitch="0107"
-                              wrist_yaw="0107"
-                              tip="172"/>
-    </xacro:if>
-    <!-- 420178: Si 178 -->
-    <xacro:if value="${str(instrument) == '420178'}">
-      <xacro:instrument_model prefix="${prefix}"
-                              housing="Si"
-                              roll="4670"
-                              wrist_pitch="0091"
-                              wrist_yaw="0091"
-                              tip="178"/>
-    </xacro:if>
-    <!-- 420179: Si 179 -->
-    <xacro:if value="${str(instrument) == '420179'}">
-      <xacro:instrument_model prefix="${prefix}"
-                              housing="Si"
-                              roll="4670"
-                              wrist_pitch="0091"
-                              wrist_yaw="0091"
-                              tip="179"/>
-    </xacro:if>
-    <!-- 420181: Si 181 -->
-    <xacro:if value="${str(instrument) == '420181'}">
-      <xacro:instrument_model prefix="${prefix}"
-                              housing="Si"
-                              roll="4670"
-                              wrist_pitch="0091"
-                              wrist_yaw="0091"
-                              tip="181"/>
-    </xacro:if>
-    <!-- 420205: Si 205 -->
-    <xacro:if value="${str(instrument) == '420205'}">
-      <xacro:instrument_model prefix="${prefix}"
-                              housing="Si"
-                              roll="4670"
-                              wrist_pitch="0107"
-                              wrist_yaw="0107"
-                              tip="205"/>
-    </xacro:if>
-    <!-- 420230: Si 230 -->
-    <xacro:if value="${str(instrument) == '420230'}">
-      <xacro:instrument_model prefix="${prefix}"
-                              housing="Si"
-                              roll="4670"
-                              wrist_pitch="0107"
-                              wrist_yaw="0107"
-                              tip="230"/>
-    </xacro:if>
-    <!-- 420296: Si 296 -->
-    <xacro:if value="${str(instrument) == '420296'}">
-      <xacro:instrument_model prefix="${prefix}"
-                              housing="Si"
-                              roll="4670"
-                              wrist_pitch="0091"
-                              wrist_yaw="0091"
-                              tip="296"/>
-    </xacro:if>
-    <!-- 420327: Si 327 -->
-    <xacro:if value="${str(instrument) == '420327'}">
-      <xacro:instrument_model prefix="${prefix}"
-                              housing="Si"
-                              roll="4670"
-                              wrist_pitch="0107"
-                              wrist_yaw="0107"
-                              tip="327"/>
-    </xacro:if>
+    <xacro:property name="model" value="${instrument_table[str(instrument)]}"/>
+    <xacro:if value="${xacro.message('Using instrument ' + str(instrument) + ': ' + str(model['name'])) or False}"/>
+    <xacro:instrument_model prefix="${prefix}"
+                            housing="${model['housing']}"
+                            roll="${model['roll']}"
+                            wrist_pitch="${model['wrist_pitch']}"
+                            wrist_yaw="${model['wrist_yaw']}"
+                            tip="${model['tip']}"/>
   </xacro:macro>
 </robot>

Commit message: SWap to updated 049 obj files

File: urdf/common/instrument.urdf.xacro (robot description, xacro)
@@ -67,5 +67,8 @@
       <xacro:tip_179 prefix="${prefix}"/>
     </xacro:if>
-    <xacro:if value="${str(tip) not in ['006', '6', '049', '49', '093', '93', '179']}">
+    <xacro:if value="${str(tip) not in ['006', '6',
+                                        '049', '49',
+                                        '093', '93',
+                                        '179']}">
       <xacro:tip_placeholder prefix="${prefix}"/>
     </xacro:if>

File: urdf/common/instruments/tip/tip_049.urdf.xacro (robot description, xacro)
@@ -13,5 +13,7 @@
       <visual>
         <origin rpy="0.0 0.0 0.0" xyz="0.0 0.0 0.0"/>
-        <geometry><box size="0 0 0"/></geometry>
+        <geometry>
+          <box size="0 0 0"/>
+        </geometry>
       </visual>
     </link>
@@ -26,7 +28,11 @@
     <link name="${prefix}jaw_1_link">
       <visual>
-        <origin rpy="0.0 0.0 0.0" xyz="0.0 0.0 0.00195"/>
+        <origin
+          rpy="0.0 0.0 ${PI}"
+          xyz="0.0 0.021 0.0"/>
         <geometry>
-          <mesh filename="package://dvrk_model/meshes/instruments/tip/049/tip_049.stl"/>
+          <mesh
+            filename="package://dvrk_model/meshes/instruments/tip/049/tip_049_1.obj"
+            scale="0.1 0.1 0.1"/>
         </geometry>
       </visual>
@@ -36,13 +42,17 @@
       <child link="${prefix}jaw_2_link"/>
       <axis xyz="0.0 0.0 1"/>
-      <origin rpy="${PI} 0.0 0.0" xyz="0.0 0.0 0.0"/>
+      <origin rpy="0.0 0.0 0.0" xyz="0.0 0.0 0.0"/>
       <limit lower="-0.349066" upper="1.5708" velocity=".4" effort="1000"/>
-      <mimic joint="jaw" multiplier="0.5"/>
+      <mimic joint="jaw" multiplier="-0.5"/>
     </joint>
     <link name="${prefix}jaw_2_link">
       <visual>
-        <origin rpy="0.0 0.0 -${PI}" xyz="0.0 0.0 0.00195"/>
+        <origin
+          rpy="0.0 0.0 ${PI}"
+          xyz="0.0 0.021 0.0"/>
         <geometry>
-          <mesh filename="package://dvrk_model/meshes/instruments/tip/049/tip_049.stl"/>
+          <mesh
+            filename="package://dvrk_model/meshes/instruments/tip/049/tip_049_2.obj"
+            scale="0.1 0.1 0.1"/>
         </geometry>
       </visual>
@@ -51,5 +61,7 @@
       <parent link="${prefix}wrist_yaw_link"/>
       <child link="${prefix}tool_tip_link"/>
-      <origin rpy="0.0 ${PI_2} ${PI_2}" xyz="0.0 0.0 0.0"/>
+      <origin
+        rpy="0.0 ${PI_2} ${PI_2}"
+        xyz="0.0 0.0155 -0.0016"/>
     </joint>
     <link name="${prefix}tool_tip_link"/>

Commit message: Fix 0167 wrist pitch texture error and tips rotation direction

File: urdf/common/instrument.urdf.xacro (robot description, xacro)
@@ -20,6 +20,8 @@
   <xacro:include filename="$(find dvrk_model)/urdf/common/instruments/wrist_pitch/wrist_pitch_0091.urdf.xacro"/>
   <xacro:include filename="$(find dvrk_model)/urdf/common/instruments/wrist_pitch/wrist_pitch_0107.urdf.xacro"/>
+  <xacro:include filename="$(find dvrk_model)/urdf/common/instruments/wrist_pitch/wrist_pitch_0167.urdf.xacro"/>
   <xacro:include filename="$(find dvrk_model)/urdf/common/instruments/wrist_yaw/wrist_yaw_0091.urdf.xacro"/>
   <xacro:include filename="$(find dvrk_model)/urdf/common/instruments/wrist_yaw/wrist_yaw_0107.urdf.xacro"/>
+  <xacro:include filename="$(find dvrk_model)/urdf/common/instruments/wrist_yaw/wrist_yaw_0167.urdf.xacro"/>
   <xacro:include filename="$(find dvrk_model)/urdf/common/instruments/tip/tip_006.urdf.xacro"/>
   <xacro:include filename="$(find dvrk_model)/urdf/common/instruments/tip/tip_049.urdf.xacro"/>
@@ -50,4 +52,7 @@
       <xacro:wrist_pitch_0107 prefix="${prefix}"/>
     </xacro:if>
+    <xacro:if value="${str(wrist_pitch) == '0167' or str(wrist_pitch) == '167'}">
+      <xacro:wrist_pitch_0167 prefix="${prefix}"/>
+    </xacro:if>
     <xacro:if value="${str(wrist_yaw) == '0091' or str(wrist_yaw) == '91'}">
       <xacro:wrist_yaw_0091 prefix="${prefix}"/>
@@ -55,4 +60,7 @@
     <xacro:if value="${str(wrist_yaw) == '0107' or str(wrist_yaw) == '107'}">
       <xacro:wrist_yaw_0107 prefix="${prefix}"/>
+    </xacro:if>
+    <xacro:if value="${str(wrist_yaw) == '0167' or str(wrist_yaw) == '167'}">
+      <xacro:wrist_yaw_0167 prefix="${prefix}"/>
     </xacro:if>
     <xacro:if value="${str(tip) == '006' or str(tip) == '6'}">

File: urdf/common/instruments/tip/tip_093.urdf.xacro (robot description, xacro)
@@ -22,9 +22,9 @@
       <origin rpy="0.0 0.0 0.0" xyz="0.0 0.0 0.0"/>
       <limit lower="-1.5707" upper="1.5707" velocity=".4" effort="1000"/>
-      <mimic joint="jaw" multiplier="0.5"/>
+      <mimic joint="jaw" multiplier="-0.5"/>
     </joint>
     <link name="${prefix}jaw_1_link">
       <visual>
-        <origin rpy="0.0 0.0 0.0" xyz="0.0 0.0 0.0"/>
+        <origin rpy="0.0 0.0 ${PI}" xyz="0.0 0.0286 0.0"/>
         <geometry>
           <mesh filename="package://dvrk_model/meshes/instruments/tip/093/tip_093_1.obj" scale="0.001 0.001 0.001"/>
@@ -38,9 +38,9 @@
       <origin rpy="0.0 0.0 0.0" xyz="0.0 0.0 0.0"/>
       <limit lower="-1.5707" upper="1.5707" velocity=".4" effort="1000"/>
-      <mimic joint="jaw" multiplier="-0.5"/>
+      <mimic joint="jaw" multiplier="0.5"/>
     </joint>
     <link name="${prefix}jaw_2_link">
       <visual>
-        <origin rpy="0.0 0.0 0.0" xyz="0.0 0.0 0.0"/>
+        <origin rpy="0.0 0.0 ${PI}" xyz="0.0 0.0286 0.0"/>
         <geometry>
           <mesh filename="package://dvrk_model/meshes/instruments/tip/093/tip_093_2.obj" scale="0.001 0.001 0.001"/>
