Commit message: Update 0167 error to 0107 and corrected 093 and 172 dh parameters - both use 0107 but with different angle specification

File: urdf/common/instrument.urdf.xacro (robot description, xacro)
@@ -20,8 +20,8 @@
   <xacro:include filename="$(find dvrk_model)/urdf/common/instruments/wrist_pitch/wrist_pitch_0091.urdf.xacro"/>
   <xacro:include filename="$(find dvrk_model)/urdf/common/instruments/wrist_pitch/wrist_pitch_0107.urdf.xacro"/>
-  <xacro:include filename="$(find dvrk_model)/urdf/common/instruments/wrist_pitch/wrist_pitch_0167.urdf.xacro"/>
+  <xacro:include filename="$(find dvrk_model)/urdf/common/instruments/wrist_pitch/wrist_pitch_0107_80.urdf.xacro"/>
   <xacro:include filename="$(find dvrk_model)/urdf/common/instruments/wrist_yaw/wrist_yaw_0091.urdf.xacro"/>
   <xacro:include filename="$(find dvrk_model)/urdf/common/instruments/wrist_yaw/wrist_yaw_0107.urdf.xacro"/>
-  <xacro:include filename="$(find dvrk_model)/urdf/common/instruments/wrist_yaw/wrist_yaw_0167.urdf.xacro"/>
+  <xacro:include filename="$(find dvrk_model)/urdf/common/instruments/wrist_yaw/wrist_yaw_0107_90.urdf.xacro"/>
   <xacro:include filename="$(find dvrk_model)/urdf/common/instruments/tip/tip_006.urdf.xacro"/>
   <xacro:include filename="$(find dvrk_model)/urdf/common/instruments/tip/tip_049.urdf.xacro"/>
@@ -53,6 +53,6 @@
       <xacro:wrist_pitch_0107 prefix="${prefix}"/>
     </xacro:if>
-    <xacro:if value="${str(wrist_pitch) == '0167' or str(wrist_pitch) == '167'}">
-      <xacro:wrist_pitch_0167 prefix="${prefix}"/>
+    <xacro:if value="${str(wrist_pitch) == '0107_80'}">
+      <xacro:wrist_pitch_0107_80 prefix="${prefix}"/>
     </xacro:if>
     <xacro:if value="${str(wrist_yaw) == '0091' or str(wrist_yaw) == '91'}">
@@ -62,6 +62,6 @@
       <xacro:wrist_yaw_0107 prefix="${prefix}"/>
     </xacro:if>
-    <xacro:if value="${str(wrist_yaw) == '0167' or str(wrist_yaw) == '167'}">
-      <xacro:wrist_yaw_0167 prefix="${prefix}"/>
+    <xacro:if value="${str(wrist_yaw) == '0107_90'}">
+      <xacro:wrist_yaw_0107_90 prefix="${prefix}"/>
     </xacro:if>
     <xacro:if value="${str(tip) == '006' or str(tip) == '6'}">

File: urdf/common/instruments/wrist_pitch/wrist_pitch_0107.urdf.xacro (robot description, xacro)
@@ -12,7 +12,7 @@
     <link name="${prefix}wrist_pitch_link">
       <visual>
-        <origin rpy="0.0 0.0 0.0" xyz="0.0 0.0 0.0"/>
+        <origin rpy="0.0 ${PI_2} ${PI_2}" xyz="0.039 0.0 0.0"/>
         <geometry>
-          <mesh filename="package://dvrk_model/meshes/instruments/wrist_pitch/0091/wrist_pitch_0091.obj"/>
+          <mesh filename="package://dvrk_model/meshes/instruments/wrist_pitch/0107/wrist_pitch_0107.obj" scale="0.1 0.1 0.1"/>
         </geometry>
       </visual>

File: urdf/common/instruments/wrist_pitch/wrist_pitch_0107_80.urdf.xacro (robot description, xacro)
@@ -1,6 +1,6 @@
 <?xml version="1.0" encoding="utf-8"?>
-<robot name="dvrk_instrument_wrist_pitch_0167" xmlns:xacro="http://www.ros.org/wiki/xacro">
+<robot name="dvrk_instrument_wrist_pitch_0107_80" xmlns:xacro="http://www.ros.org/wiki/xacro">
   <xacro:include filename="$(find dvrk_model)/urdf/common.urdf.xacro"/>
-  <xacro:macro name="wrist_pitch_0167" params="prefix">
+  <xacro:macro name="wrist_pitch_0107_80" params="prefix">
     <joint name="wrist_pitch" type="revolute">
       <parent link="${prefix}roll_link"/>
@@ -8,5 +8,5 @@
       <axis xyz="0.0 0.0 1"/>
       <origin rpy="-${PI_2} -${PI_2} 0.0" xyz="0.0 0.0 0.0"/>
-      <limit lower="-1.2217" upper="1.2217" velocity=".4" effort="1000"/>
+      <limit lower="-1.39626" upper="1.39626" velocity=".4" effort="1000"/>
     </joint>
     <link name="${prefix}wrist_pitch_link">
@@ -14,5 +14,5 @@
         <origin rpy="0.0 ${PI_2} ${PI_2}" xyz="0.039 0.0 0.0"/>
         <geometry>
-          <mesh filename="package://dvrk_model/meshes/instruments/wrist_pitch/0167/wrist_pitch_0167.obj" scale="0.1 0.1 0.1"/>
+          <mesh filename="package://dvrk_model/meshes/instruments/wrist_pitch/0107/wrist_pitch_0107.obj" scale="0.1 0.1 0.1"/>
         </geometry>
       </visual>

File: urdf/common/instruments/wrist_yaw/wrist_yaw_0107.urdf.xacro (robot description, xacro)
@@ -12,7 +12,7 @@
     <link name="${prefix}wrist_yaw_link">
       <visual>
-        <origin rpy="0.0 0.0 0.0" xyz="0.0 0.0 -0.000236"/>
+        <origin rpy="${PI} 0.0 ${PI}" xyz="-0.000236 -0.02775 0.0"/>
         <geometry>
-          <mesh filename="package://dvrk_model/meshes/instruments/wrist_yaw/0091/wrist_yaw_0091.obj"/>
+          <mesh filename="package://dvrk_model/meshes/instruments/wrist_yaw/0107/wrist_yaw_0107.obj" scale="0.1 0.1 0.1"/>
         </geometry>
       </visual>

File: urdf/common/instruments/wrist_yaw/wrist_yaw_0107_90.urdf.xacro (robot description, xacro)
@@ -1,12 +1,12 @@
 <?xml version="1.0" encoding="utf-8"?>
-<robot name="dvrk_instrument_wrist_yaw_0167" xmlns:xacro="http://www.ros.org/wiki/xacro">
+<robot name="dvrk_instrument_wrist_yaw_0107_90" xmlns:xacro="http://www.ros.org/wiki/xacro">
   <xacro:include filename="$(find dvrk_model)/urdf/common.urdf.xacro"/>
-  <xacro:macro name="wrist_yaw_0167" params="prefix">
+  <xacro:macro name="wrist_yaw_0107_90" params="prefix">
     <joint name="wrist_yaw" type="revolute">
       <parent link="${prefix}wrist_pitch_link"/>
       <child link="${prefix}wrist_yaw_link"/>
       <axis xyz="0.0 0.0 1"/>
-      <origin rpy="-${PI_2} -${PI_2} 0.0" xyz="0.0110 0.0 0.0"/>
-      <limit lower="-1.39626" upper="1.39626" velocity=".4" effort="1000"/>
+      <origin rpy="-${PI_2} -${PI_2} 0.0" xyz="0.0107 0.0 0.0"/>
+      <limit lower="-1.5708" upper="1.5708" velocity=".4" effort="1000"/>
     </joint>
     <link name="${prefix}wrist_yaw_link">
@@ -14,5 +14,5 @@
         <origin rpy="${PI} 0.0 ${PI}" xyz="-0.000236 -0.02775 0.0"/>
         <geometry>
-          <mesh filename="package://dvrk_model/meshes/instruments/wrist_yaw/0167/wrist_yaw_0167.obj" scale="0.1 0.1 0.1"/>
+          <mesh filename="package://dvrk_model/meshes/instruments/wrist_yaw/0107/wrist_yaw_0107.obj" scale="0.1 0.1 0.1"/>
         </geometry>
       </visual>

Commit message: Removed varying 0107 pitch and yaw constraints - unified as +/- 80

File: urdf/common/instrument.urdf.xacro (robot description, xacro)
@@ -21,10 +21,7 @@
   <xacro:include filename="$(find dvrk_model)/urdf/common/instruments/wrist_pitch/wrist_pitch_0100.urdf.xacro"/>
   <xacro:include filename="$(find dvrk_model)/urdf/common/instruments/wrist_pitch/wrist_pitch_0107.urdf.xacro"/>
-  <xacro:include filename="$(find dvrk_model)/urdf/common/instruments/wrist_pitch/wrist_pitch_0107_80.urdf.xacro"/>
   <xacro:include filename="$(find dvrk_model)/urdf/common/instruments/wrist_yaw/wrist_yaw_0091.urdf.xacro"/>
   <xacro:include filename="$(find dvrk_model)/urdf/common/instruments/wrist_yaw/wrist_yaw_0100.urdf.xacro"/>
   <xacro:include filename="$(find dvrk_model)/urdf/common/instruments/wrist_yaw/wrist_yaw_0107.urdf.xacro"/>
-  <xacro:include filename="$(find dvrk_model)/urdf/common/instruments/wrist_yaw/wrist_yaw_0107_73.urdf.xacro"/>
-  <xacro:include filename="$(find dvrk_model)/urdf/common/instruments/wrist_yaw/wrist_yaw_0107_90.urdf.xacro"/>
   <xacro:include filename="$(find dvrk_model)/urdf/common/instruments/tip/tip_006.urdf.xacro"/>
   <xacro:include filename="$(find dvrk_model)/urdf/common/instruments/tip/tip_049.urdf.xacro"/>
@@ -60,7 +57,4 @@
       <xacro:wrist_pitch_0107 prefix="${prefix}"/>
     </xacro:if>
-    <xacro:if value="${str(wrist_pitch) == '0107_80'}">
-      <xacro:wrist_pitch_0107_80 prefix="${prefix}"/>
-    </xacro:if>
     <xacro:if value="${str(wrist_yaw) == '0091' or str(wrist_yaw) == '91'}">
       <xacro:wrist_yaw_0091 prefix="${prefix}"/>
@@ -71,10 +65,4 @@
     <xacro:if value="${str(wrist_yaw) == '0107' or str(wrist_yaw) == '107'}">
       <xacro:wrist_yaw_0107 prefix="${prefix}"/>
-    </xacro:if>
-    <xacro:if value="${str(wrist_yaw) == '0107_73'}">
-      <xacro:wrist_yaw_0107_73 prefix="${prefix}"/>
-    </xacro:if>
-    <xacro:if value="${str(wrist_yaw) == '0107_90'}">
-      <xacro:wrist_yaw_0107_90 prefix="${prefix}"/>
     </xacro:if>
     <xacro:if value="${str(tip) == '006' or str(tip) == '6'}">

File: urdf/common/instruments/wrist_pitch/wrist_pitch_0107.urdf.xacro (robot description, xacro)
@@ -8,5 +8,5 @@
       <axis xyz="0.0 0.0 1"/>
       <origin rpy="-${PI_2} -${PI_2} 0.0" xyz="0.0 0.0 0.0"/>
-      <limit lower="-1.2217" upper="1.2217" velocity=".4" effort="1000"/>
+      <limit lower="-1.39626" upper="1.39626" velocity=".4" effort="1000"/>
     </joint>
     <link name="${prefix}wrist_pitch_link">

Commit message: Updated 309 wrist texture and position

File: urdf/common/instrument.urdf.xacro (robot description, xacro)
@@ -19,9 +19,13 @@
   <xacro:include filename="$(find dvrk_model)/urdf/common/instruments/roll/roll_4670.urdf.xacro"/>
   <xacro:include filename="$(find dvrk_model)/urdf/common/instruments/wrist_pitch/wrist_pitch_0091.urdf.xacro"/>
+  <xacro:include filename="$(find dvrk_model)/urdf/common/instruments/wrist_pitch/wrist_pitch_0093.urdf.xacro"/>
   <xacro:include filename="$(find dvrk_model)/urdf/common/instruments/wrist_pitch/wrist_pitch_0100.urdf.xacro"/>
   <xacro:include filename="$(find dvrk_model)/urdf/common/instruments/wrist_pitch/wrist_pitch_0107.urdf.xacro"/>
+  <xacro:include filename="$(find dvrk_model)/urdf/common/instruments/wrist_pitch/wrist_pitch_0112.urdf.xacro"/>
   <xacro:include filename="$(find dvrk_model)/urdf/common/instruments/wrist_yaw/wrist_yaw_0091.urdf.xacro"/>
+  <xacro:include filename="$(find dvrk_model)/urdf/common/instruments/wrist_yaw/wrist_yaw_0093.urdf.xacro"/>
   <xacro:include filename="$(find dvrk_model)/urdf/common/instruments/wrist_yaw/wrist_yaw_0100.urdf.xacro"/>
   <xacro:include filename="$(find dvrk_model)/urdf/common/instruments/wrist_yaw/wrist_yaw_0107.urdf.xacro"/>
+  <xacro:include filename="$(find dvrk_model)/urdf/common/instruments/wrist_yaw/wrist_yaw_0112.urdf.xacro"/>
   <xacro:include filename="$(find dvrk_model)/urdf/common/instruments/tip/tip_006.urdf.xacro"/>
   <xacro:include filename="$(find dvrk_model)/urdf/common/instruments/tip/tip_049.urdf.xacro"/>
@@ -29,4 +33,7 @@
   <xacro:include filename="$(find dvrk_model)/urdf/common/instruments/tip/tip_172.urdf.xacro"/>
   <xacro:include filename="$(find dvrk_model)/urdf/common/instruments/tip/tip_179.urdf.xacro"/>
+  <xacro:include filename="$(find dvrk_model)/urdf/common/instruments/tip/tip_183.urdf.xacro"/>
+  <xacro:include filename="$(find dvrk_model)/urdf/common/instruments/tip/tip_184.urdf.xacro"/>
+  <xacro:include filename="$(find dvrk_model)/urdf/common/instruments/tip/tip_194.urdf.xacro"/>
   <xacro:include filename="$(find dvrk_model)/urdf/common/instruments/tip/tip_309.urdf.xacro"/>
   <xacro:include filename="$(find dvrk_model)/urdf/common/instruments/tip/tip_327.urdf.xacro"/>
@@ -51,4 +58,7 @@
       <xacro:wrist_pitch_0091 prefix="${prefix}"/>
     </xacro:if>
+    <xacro:if value="${str(wrist_pitch) == '0093' or str(wrist_pitch) == '93'}">
+      <xacro:wrist_pitch_0093 prefix="${prefix}"/>
+    </xacro:if>
     <xacro:if value="${str(wrist_pitch) == '0100' or str(wrist_pitch) == '100'}">
       <xacro:wrist_pitch_0100 prefix="${prefix}"/>
@@ -57,6 +67,12 @@
       <xacro:wrist_pitch_0107 prefix="${prefix}"/>
     </xacro:if>
+    <xacro:if value="${str(wrist_pitch) == '0112' or str(wrist_pitch) == '112'}">
+      <xacro:wrist_pitch_0112 prefix="${prefix}"/>
+    </xacro:if>
     <xacro:if value="${str(wrist_yaw) == '0091' or str(wrist_yaw) == '91'}">
       <xacro:wrist_yaw_0091 prefix="${prefix}"/>
+    </xacro:if>
+    <xacro:if value="${str(wrist_yaw) == '0093' or str(wrist_yaw) == '93'}">
+      <xacro:wrist_yaw_0093 prefix="${prefix}"/>
     </xacro:if>
     <xacro:if value="${str(wrist_yaw) == '0100' or str(wrist_yaw) == '100'}">
@@ -65,4 +81,7 @@
     <xacro:if value="${str(wrist_yaw) == '0107' or str(wrist_yaw) == '107'}">
       <xacro:wrist_yaw_0107 prefix="${prefix}"/>
+    </xacro:if>
+    <xacro:if value="${str(wrist_yaw) == '0112' or str(wrist_yaw) == '112'}">
+      <xacro:wrist_yaw_0112 prefix="${prefix}"/>
     </xacro:if>
     <xacro:if value="${str(tip) == '006' or str(tip) == '6'}">
@@ -81,4 +100,13 @@
       <xacro:tip_179 prefix="${prefix}"/>
     </xacro:if>
+    <xacro:if value="${str(tip) == '183'}">
+      <xacro:tip_183 prefix="${prefix}"/>
+    </xacro:if>
+    <xacro:if value="${str(tip) == '184'}">
+      <xacro:tip_184 prefix="${prefix}"/>
+    </xacro:if>
+    <xacro:if value="${str(tip) == '194'}">
+      <xacro:tip_194 prefix="${prefix}"/>
+    </xacro:if>
     <xacro:if value="${str(tip) == '309'}">
       <xacro:tip_309 prefix="${prefix}"/>
@@ -92,4 +120,7 @@
                                         '172',
                                         '179',
+                                        '183',
+                                        '184',
+                                        '194',
                                         '309',
                                         '327']}">

File: urdf/common/instruments/tip/tip_194.urdf.xacro (robot description, xacro)
@@ -1,12 +1,12 @@
 <?xml version="1.0" encoding="utf-8"?>
-<robot name="dvrk_instrument_tip_309" xmlns:xacro="http://www.ros.org/wiki/xacro">
+<robot name="dvrk_instrument_tip_194" xmlns:xacro="http://www.ros.org/wiki/xacro">
   <xacro:include filename="$(find dvrk_model)/urdf/common.urdf.xacro"/>
-  <xacro:macro name="tip_309" params="prefix">
+  <xacro:macro name="tip_194" params="prefix">
     <joint name="jaw" type="revolute">
       <parent link="${prefix}wrist_yaw_link"/>
       <child link="${prefix}jaw_link"/>
-      <axis xyz="0.0 0.0 1"/>
+      <axis xyz="0.0 0.0 1.0"/>
       <origin rpy="0.0 0.0 0.0" xyz="0.0 0.0 0.0"/>
-      <limit lower="-0.349066" upper="1.5708" velocity=".4" effort="1000"/>
+      <limit lower="-0.349066" upper="1.39626" velocity=".4" effort="1000"/>
     </joint>
     <link name="${prefix}jaw_link">
@@ -21,18 +21,14 @@
       <parent link="${prefix}wrist_yaw_link"/>
       <child link="${prefix}jaw_1_link"/>
-      <axis xyz="0.0 0.0 1"/>
+      <axis xyz="0.0 0.0 1.0"/>
       <origin rpy="0.0 0.0 0.0" xyz="0.0 0.0 0.0"/>
-      <limit lower="-0.349066" upper="1.5708" velocity=".4" effort="1000"/>
+      <limit lower="-1.5707" upper="1.5707" velocity=".4" effort="1000"/>
       <mimic joint="jaw" multiplier="-0.5"/>
     </joint>
     <link name="${prefix}jaw_1_link">
       <visual>
-        <origin
-          rpy="0.0 0.0 ${PI}"
-          xyz="0.0 0.0108 0.0"/>
+        <origin rpy="0.0 0.0 ${PI}" xyz="0.0 0.0108 0.0"/>
         <geometry>
-          <mesh
-            filename="package://dvrk_model/meshes/instruments/tip/309/tip_309_1.obj"
-            scale="0.1 0.1 0.1"/>
+          <mesh filename="package://dvrk_model/meshes/instruments/tip/194/tip_194_1.obj" scale="0.1 0.1 0.1"/>
         </geometry>
       </visual>
@@ -41,17 +37,14 @@
       <parent link="${prefix}wrist_yaw_link"/>
       <child link="${prefix}jaw_2_link"/>
-      <axis xyz="0.0 0.0 1"/>
+      <axis xyz="0.0 0.0 1.0"/>
       <origin rpy="0.0 0.0 0.0" xyz="0.0 0.0 0.0"/>
-      <limit lower="-0.349066" upper="1.5708" velocity=".4" effort="1000"/>
+      <limit lower="-1.5707" upper="1.5707" velocity=".4" effort="1000"/>
       <mimic joint="jaw" multiplier="0.5"/>
     </joint>
     <link name="${prefix}jaw_2_link">
       <visual>
-        <origin
-          rpy="0.0 0.0 ${PI}" xyz="0.0 0.0108 0.0"/>
+        <origin rpy="0.0 0.0 ${PI}" xyz="0.0 0.0108 0.0"/>
         <geometry>
-          <mesh
-            filename="package://dvrk_model/meshes/instruments/tip/309/tip_309_2.obj"
-            scale="0.1 0.1 0.1"/>
+          <mesh filename="package://dvrk_model/meshes/instruments/tip/194/tip_194_2.obj" scale="0.1 0.1 0.1"/>
         </geometry>
       </visual>
@@ -60,7 +53,5 @@
       <parent link="${prefix}wrist_yaw_link"/>
       <child link="${prefix}tool_tip_link"/>
-      <origin
-        rpy="0.0 ${PI_2} ${PI_2}"
-        xyz="0.0 0.0155 -0.0016"/>
+      <origin rpy="0.0 ${PI_2} ${PI_2}" xyz="0.0 0.0164 0.0"/>
     </joint>
     <link name="${prefix}tool_tip_link"/>
