Commit message: remove wrist variables in psm instruments and tool common files

File: ros2/ros2_control/psm_base.ros2_control.xacro (robot description, xacro)
@@ -38,5 +38,5 @@
                 <state_interface name="velocity"/>
             </joint>
-            <joint name="wrist_pitch">
+            <joint name="tip_pitch">
                 <command_interface name="position">
                 <param name="min">-1.5707</param>
@@ -46,5 +46,5 @@
                 <state_interface name="velocity"/>
             </joint>
-            <joint name="wrist_yaw">
+            <joint name="tip_yaw">
                 <command_interface name="position">
                 <param name="min">-1.5707</param>

File: urdf/common/PSM_instrument.urdf.xacro (robot description, xacro)
@@ -7,6 +7,6 @@
     DOF layout:
       Joint 4: roll         (revolute, D = shaft_length along z)
-      Joint 5: wrist_pitch  (revolute)  ┐
-      Joint 6: wrist_yaw    (revolute)  ├── dispatched via PSM_tip_XXX macro
+      Joint 5: tip_pitch    (revolute)  ┐
+      Joint 6: tip_yaw      (revolute)  ├── dispatched via PSM_tip_XXX macro
       Joint 7: jaw + mimics (revolute)  ┘
     Parameters:
@@ -82,14 +82,14 @@
     -->
     <link name="${prefix}roll_link"/>
-    <!-- fixed joint to wrist body -->
+    <!-- fixed joint to roll housing -->
     <joint name="roll_fixed" type="fixed">
       <parent link="${prefix}roll_link"/>
-      <child  link="${prefix}wrist_link"/>
+      <child  link="${prefix}roll_housing_link"/>
       <origin rpy="0 0 0" xyz="0 0 0"/>
     </joint>
-    <link name="${prefix}wrist_link">
+    <link name="${prefix}roll_housing_link">
       <visual>
         <xacro:if value="${is_si}">
-          <!-- Si roll wrist piece is centered at the roll joint -->
+          <!-- Si roll housing piece is centered at the roll joint -->
           <origin rpy="-${PI} 0 0" xyz="0.05591 0 0"/>
           <geometry>
@@ -99,5 +99,5 @@
         </xacro:if>
         <xacro:unless value="${is_si}">
-          <!-- Classic wrist roll housing at the shaft end -->
+          <!-- Classic roll housing at the shaft end -->
           <origin rpy="0 0 1.5708" xyz="0 0 -0.0091"/>
           <geometry>
@@ -121,11 +121,11 @@
       </collision>
     </link>
-    <!-- fixed joint to wrist shaft -->
-    <joint name="wrist_shaft_fixed" type="fixed">
-      <parent link="${prefix}wrist_link"/>
-      <child  link="${prefix}wrist_shaft_link"/>
+    <!-- fixed joint to shaft -->
+    <joint name="shaft_fixed" type="fixed">
+      <parent link="${prefix}roll_housing_link"/>
+      <child  link="${prefix}shaft_link"/>
       <origin rpy="0 0 0" xyz="0 0 0"/>
     </joint>
-    <link name="${prefix}wrist_shaft_link">
+    <link name="${prefix}shaft_link">
       <visual>
         <xacro:if value="${is_si}">
@@ -159,5 +159,5 @@
     </link>
     <!--
-      Tip dispatch: select the correct wrist+jaw macro by instrument.
+      Tip dispatch: select the correct tip+jaw macro by instrument.
       Convention: last 3 digits of the model number identify the tip family.
         006 → standard SCA wrist (most instruments, A=0.0091)
@@ -173,25 +173,25 @@
                       str(instrument) == '420168' or str(instrument) == '400168'}">
       <xacro:PSM_tip_006 prefix="${prefix}"
-                         parent_link="${prefix}wrist_shaft_link"/>
+                         parent_link="${prefix}shaft_link"/>
     </xacro:if>
     <!-- 049: Cadiere jaw -->
     <xacro:if value="${str(instrument) == '420049' or str(instrument) == '400049'}">
       <xacro:PSM_tip_049 prefix="${prefix}"
-                         parent_link="${prefix}wrist_shaft_link"/>
+                         parent_link="${prefix}shaft_link"/>
     </xacro:if>
     <!-- 172: Maryland wrist — currently reuses PSM_tip_006 placeholder meshes (see note in PSM_tips.urdf.xacro) -->
     <xacro:if value="${str(instrument) == '420172' or str(instrument) == '400172'}">
       <xacro:PSM_tip_172 prefix="${prefix}"
-                         parent_link="${prefix}wrist_shaft_link"/>
+                         parent_link="${prefix}shaft_link"/>
     </xacro:if>
     <!-- 117: snake tool — PSM_tip_117 is currently a kinematic stub only (no meshes, no jaw geometry, DOFs unconfirmed) -->
     <xacro:if value="${str(instrument) == '400117'}">
       <xacro:PSM_tip_117 prefix="${prefix}"
-                         parent_link="${prefix}wrist_shaft_link"/>
+                         parent_link="${prefix}shaft_link"/>
     </xacro:if>
     <!-- ECM: Si camera tip -->
     <xacro:if value="${str(instrument) == 'SF0826001'}">
       <xacro:PSM_tip_ECM prefix="${prefix}"
-                         parent_link="${prefix}wrist_shaft_link"/>
+                         parent_link="${prefix}shaft_link"/>
     </xacro:if>
     <!-- 183: cautery / no-jaw tools — PSM_tip_183 macro exists in PSM_tips.urdf.xacro but is not yet wired into this dispatch -->

File: urdf/common/PSM_tips.urdf.xacro (robot description, xacro)
@@ -3,5 +3,5 @@
   <!--
     PSM tip family macros — generation-agnostic.
-    All macros attach to ${parent_link} (= ${prefix}wrist_shaft_link).
+    All macros attach to ${parent_link} (= ${prefix}shaft_link).
     Tip families are identified by the last 3 digits of the instrument model:
       PSM_tip_006  — standard SCA wrist  (A=0.0091 m, most instruments)
@@ -17,13 +17,13 @@
   <!-- ════════════════════════════════════════════════════════════════════ -->
   <xacro:macro name="PSM_tip_006" params="prefix parent_link">
-    <!-- joint 5: wrist_pitch -->
-    <joint name="wrist_pitch" type="revolute">
-      <parent link="${parent_link}"/>
-      <child  link="${prefix}tip_006_wrist_link"/>
+    <!-- joint 5: tip_pitch -->
+    <joint name="tip_pitch" type="revolute">
+      <parent link="${parent_link}"/>
+      <child  link="${prefix}tip_006_pitch_link"/>
       <axis xyz="0 0 1"/>
       <origin rpy="-${PI_2} -${PI_2} 0" xyz="0 0 0"/>
       <limit lower="-${PI_2}" upper="${PI_2}" velocity=".4" effort="1000"/>
     </joint>
-    <link name="${prefix}tip_006_wrist_link">
+    <link name="${prefix}tip_006_pitch_link">
       <visual>
         <origin rpy="${PI_2} ${PI} 0" xyz="0.0051 0.0032 0"/>
@@ -33,13 +33,13 @@
       </visual>
     </link>
-    <!-- joint 6: wrist_yaw -->
-    <joint name="wrist_yaw" type="revolute">
-      <parent link="${prefix}tip_006_wrist_link"/>
-      <child  link="${prefix}tip_006_shaft_link"/>
+    <!-- joint 6: tip_yaw -->
+    <joint name="tip_yaw" type="revolute">
+      <parent link="${prefix}tip_006_pitch_link"/>
+      <child  link="${prefix}tip_006_yaw_link"/>
       <axis xyz="0 0 1"/>
       <origin rpy="-${PI_2} -${PI_2} 0" xyz="0.0091 0 0"/>
       <limit lower="-1.3963" upper="1.3963" velocity=".4" effort="1000"/>
     </joint>
-    <link name="${prefix}tip_006_shaft_link">
+    <link name="${prefix}tip_006_yaw_link">
       <visual>
         <origin rpy="0 0 0" xyz="0 -0.0002 -0.0025"/>
@@ -51,5 +51,5 @@
     <!-- joint 7-0: jaw (virtual centre — drives the mimics) -->
     <joint name="jaw" type="revolute">
-      <parent link="${prefix}tip_006_shaft_link"/>
+      <parent link="${prefix}tip_006_yaw_link"/>
       <child  link="${prefix}jaw_link"/>
       <axis xyz="0 0 1"/>
@@ -66,5 +66,5 @@
     <!-- jaw mimic 1 — opens +0.5× -->
     <joint name="jaw_1" type="revolute">
-      <parent link="${prefix}tip_006_shaft_link"/>
+      <parent link="${prefix}tip_006_yaw_link"/>
       <child  link="${prefix}jaw_1_link"/>
       <axis xyz="0 0 1"/>
@@ -83,5 +83,5 @@
     <!-- jaw mimic 2 — opens −0.5× (symmetric) -->
     <joint name="jaw_2" type="revolute">
-      <parent link="${prefix}tip_006_shaft_link"/>
+      <parent link="${prefix}tip_006_yaw_link"/>
       <child  link="${prefix}jaw_2_link"/>
       <axis xyz="0 0 1"/>
@@ -100,5 +100,5 @@
     <!-- tool tip reference frame -->
     <joint name="tool_tip" type="fixed">
-      <parent link="${prefix}tip_006_shaft_link"/>
+      <parent link="${prefix}tip_006_yaw_link"/>
       <child  link="${prefix}tool_tip_link"/>
       <origin rpy="0 ${PI/2} ${PI/2}" xyz="0 0.0102 0"/>
@@ -110,12 +110,12 @@
   <!-- ════════════════════════════════════════════════════════════════════ -->
   <xacro:macro name="PSM_tip_049" params="prefix parent_link">
-    <joint name="wrist_pitch" type="revolute">
-      <parent link="${parent_link}"/>
-      <child  link="${prefix}tip_049_wrist_link"/>
+    <joint name="tip_pitch" type="revolute">
+      <parent link="${parent_link}"/>
+      <child  link="${prefix}tip_049_pitch_link"/>
       <axis xyz="0 0 1"/>
       <origin rpy="-${PI_2} -${PI_2} 0" xyz="0 0 0"/>
       <limit lower="-${PI_2}" upper="${PI_2}" velocity=".4" effort="1000"/>
     </joint>
-    <link name="${prefix}tip_049_wrist_link">
+    <link name="${prefix}tip_049_pitch_link">
       <visual>
         <origin rpy="0 -${PI_2} 0" xyz="-0.0024 0 0"/>
@@ -125,12 +125,12 @@
       </visual>
     </link>
-    <joint name="wrist_yaw" type="revolute">
-      <parent link="${prefix}tip_049_wrist_link"/>
-      <child  link="${prefix}tip_049_shaft_link"/>
+    <joint name="tip_yaw" type="revolute">
+      <parent link="${prefix}tip_049_pitch_link"/>
+      <child  link="${prefix}tip_049_yaw_link"/>
       <axis xyz="0 0 1"/>
       <origin rpy="0 -${PI_2} -${PI_2}" xyz="0.0091 0 0"/>
       <limit lower="-1.3963" upper="1.3963" velocity=".4" effort="1000"/>
     </joint>
-    <link name="${prefix}tip_049_shaft_link">
+    <link name="${prefix}tip_049_yaw_link">
       <visual>
         <origin rpy="0 ${PI_2} 0" xyz="0 -0.0002 0"/>
@@ -141,5 +141,5 @@
     </link>
     <joint name="jaw" type="revolute">
-      <parent link="${prefix}tip_049_shaft_link"/>
+      <parent link="${prefix}tip_049_yaw_link"/>
       <child link="${prefix}jaw_link"/>
       <axis xyz="0 0 1"/>
@@ -154,5 +154,5 @@
     </link>
     <joint name="jaw_1" type="revolute">
-      <parent link="${prefix}tip_049_shaft_link"/>
+      <parent link="${prefix}tip_049_yaw_link"/>
       <child link="${prefix}jaw_1_link"/>
       <axis xyz="0 0 1"/>
@@ -170,5 +170,5 @@
     </link>
     <joint name="jaw_2" type="revolute">
-      <parent link="${prefix}tip_049_shaft_link"/>
+      <parent link="${prefix}tip_049_yaw_link"/>
       <child link="${prefix}jaw_2_link"/>
       <axis xyz="0 0 1"/>
@@ -186,5 +186,5 @@
     </link>
     <joint name="tool_tip" type="fixed">
-      <parent link="${prefix}tip_049_shaft_link"/>
+      <parent link="${prefix}tip_049_yaw_link"/>
       <child link="${prefix}tool_tip_link"/>
       <origin rpy="0 ${PI_2} ${PI_2}" xyz="0 0 0"/>
@@ -196,8 +196,8 @@
   <!-- ════════════════════════════════════════════════════════════════════ -->
   <xacro:macro name="PSM_tip_172" params="prefix parent_link">
-    <!-- joint 5: wrist_pitch -->
-    <joint name="wrist_pitch" type="revolute">
-      <parent link="${parent_link}"/>
-      <child  link="${prefix}tip_172_wrist_link"/>
+    <!-- joint 5: tip_pitch -->
+    <joint name="tip_pitch" type="revolute">
+      <parent link="${parent_link}"/>
+      <child  link="${prefix}tip_172_pitch_link"/>
       <axis xyz="0 0 1"/>
       <origin rpy="-${PI_2} -${PI_2} 0" xyz="0 0 0"/>
@@ -208,5 +208,5 @@
       until a dedicated Maryland wrist mesh is added to the repo.
     -->
-    <link name="${prefix}tip_172_wrist_link">
+    <link name="${prefix}tip_172_pitch_link">
       <visual>
         <origin rpy="${PI_2} ${PI} 0" xyz="0.0051 0.0032 0"/>
@@ -216,13 +216,13 @@
       </visual>
     </link>
-    <!-- joint 6: wrist_yaw (A=0.0107 — Maryland specific) -->
-    <joint name="wrist_yaw" type="revolute">
-      <parent link="${prefix}tip_172_wrist_link"/>
-      <child  link="${prefix}tip_172_shaft_link"/>
+    <!-- joint 6: tip_yaw (A=0.0107 — Maryland specific) -->
+    <joint name="tip_yaw" type="revolute">
+      <parent link="${prefix}tip_172_pitch_link"/>
+      <child  link="${prefix}tip_172_yaw_link"/>
       <axis xyz="0 0 1"/>
       <origin rpy="-${PI_2} -${PI_2} 0" xyz="0.0107 0 0"/>
       <limit lower="-1.3963" upper="1.3963" velocity=".4" effort="1000"/>
     </joint>
-    <link name="${prefix}tip_172_shaft_link">
+    <link name="${prefix}tip_172_yaw_link">
       <visual>
         <origin rpy="0 0 0" xyz="0 -0.0002 -0.0025"/>
@@ -234,5 +234,5 @@
     <!-- jaw + symmetric mimics (same as tip_006) -->
     <joint name="jaw" type="revolute">
-      <parent link="${prefix}tip_172_shaft_link"/>
+      <parent link="${prefix}tip_172_yaw_link"/>
       <child  link="${prefix}jaw_link"/>
       <axis xyz="0 0 1"/>
@@ -246,5 +246,5 @@
     </link>
     <joint name="jaw_1" type="revolute">
-      <parent link="${prefix}tip_172_shaft_link"/>
+      <parent link="${prefix}tip_172_yaw_link"/>
       <child  link="${prefix}jaw_1_link"/>
       <axis xyz="0 0 1"/>
@@ -262,5 +262,5 @@
     </link>
     <joint name="jaw_2" type="revolute">
-      <parent link="${prefix}tip_172_shaft_link"/>
+      <parent link="${prefix}tip_172_yaw_link"/>
       <child  link="${prefix}jaw_2_link"/>
       <axis xyz="0 0 1"/>
@@ -278,5 +278,5 @@
     </link>
     <joint name="tool_tip" type="fixed">
-      <parent link="${prefix}tip_172_shaft_link"/>
+      <parent link="${prefix}tip_172_yaw_link"/>
       <child  link="${prefix}tool_tip_link"/>
       <origin rpy="0 ${PI/2} ${PI/2}" xyz="0 0.0107 0"/>
@@ -295,14 +295,14 @@
       Placeholder: minimal kinematic stub so the URDF parses.
     -->
-    <joint name="wrist_pitch" type="revolute">
-      <parent link="${parent_link}"/>
-      <child  link="${prefix}tip_117_wrist_link"/>
+    <joint name="tip_pitch" type="revolute">
+      <parent link="${parent_link}"/>
+      <child  link="${prefix}tip_117_pitch_link"/>
       <axis xyz="0 0 1"/>
       <origin rpy="-${PI_2} -${PI_2} 0" xyz="0 0 0"/>
       <limit lower="-${PI_2}" upper="${PI_2}" velocity=".4" effort="1000"/>
     </joint>
-    <link name="${prefix}tip_117_wrist_link"/>
+    <link name="${prefix}tip_117_pitch_link"/>
     <joint name="jaw" type="revolute">
-      <parent link="${prefix}tip_117_wrist_link"/>
+      <parent link="${prefix}tip_117_pitch_link"/>
       <child  link="${prefix}jaw_link"/>
       <axis xyz="0 0 1"/>
@@ -312,5 +312,5 @@
     <link name="${prefix}jaw_link"/>
     <joint name="tool_tip" type="fixed">
-      <parent link="${prefix}tip_117_wrist_link"/>
+      <parent link="${prefix}tip_117_pitch_link"/>
       <child  link="${prefix}tool_tip_link"/>
       <origin rpy="0 0 0" xyz="0 0 0"/>
@@ -334,5 +334,5 @@
   <!-- ════════════════════════════════════════════════════════════════════ -->
   <xacro:macro name="PSM_tip_ECM" params="prefix parent_link">
-    <joint name="wrist_pitch" type="revolute">
+    <joint name="tip_pitch" type="revolute">
       <parent link="${parent_link}"/>
       <child  link="${prefix}tip_roll_link"/>
