Commit message: fix launch parsing error for si instrument on classic arm

File: urdf/common/psm_tools/PSM_body.urdf.xacro (robot description, xacro)
@@ -70,4 +70,10 @@
     <link name="${prefix}roll_housing_link">
       <visual>
+        <xacro:if value="${is_si}">
+          <origin rpy="0 0 1.5708" xyz="0 0 -0.0091"/>
+          <geometry>
+            <mesh filename="package://dvrk_model/meshes/instruments/Si/roll/PSM_roll_connector_8mm.stl"/>
+          </geometry>
+        </xacro:if>
         <xacro:unless value="${is_si}">
           <origin rpy="0 0 1.5708" xyz="0 0 -0.0091"/>
@@ -78,4 +84,10 @@
       </visual>
       <collision>
+        <xacro:if value="${is_si}">
+          <origin rpy="0 0 1.5708" xyz="0 0 -0.0091"/>
+          <geometry>
+            <mesh filename="package://dvrk_model/meshes/instruments/Si/roll/PSM_roll_connector_8mm.stl"/>
+          </geometry>
+        </xacro:if>
         <xacro:unless value="${is_si}">
           <origin rpy="0 0 1.5708" xyz="0 0 -0.0091"/>
@@ -93,4 +105,10 @@
     <link name="${prefix}shaft_link">
       <visual>
+        <xacro:if value="${is_si}">
+          <origin rpy="${PI_2} 0 0" xyz="0 0.00401 0"/>
+          <geometry>
+            <mesh filename="package://dvrk_model/meshes/instruments/Si/yaw/PSM_006_yaw.OBJ"/>
+          </geometry>
+        </xacro:if>
         <xacro:unless value="${is_si}">
           <origin rpy="${PI_2} 0 0" xyz="0 0.00401 0"/>
@@ -101,4 +119,10 @@
       </visual>
       <collision>
+        <xacro:if value="${is_si}">
+          <origin rpy="${PI_2} 0 0" xyz="0 0.00401 0"/>
+          <geometry>
+            <mesh filename="package://dvrk_model/meshes/instruments/Si/yaw/PSM_006_yaw.OBJ"/>
+          </geometry>
+        </xacro:if>
         <xacro:unless value="${is_si}">
           <origin rpy="${PI_2} 0 0" xyz="0 0.00401 0"/>
