Commit message: Refactor URDF files for classic and si arms to use RCM frame as reference frame, arm only or arm + SUJ.  instrument frame still broken.

File: urdf/classic_arm/ECM_base.urdf.xacro (robot description, xacro)
@@ -27,5 +27,5 @@
       <parent link="${prefix}RCM_link"/>
       <child  link="${prefix}base_link"/>
-      <origin xyz="0.0 -0.612599207482277 -0.101460" rpy="0.0 0.0 ${PI_2}"/>
+      <origin xyz="-0.612599207482277 0.0 -0.101460" rpy="0.0 0.0 0.0"/>
     </joint>
     <!-- link 0: base -->

File: urdf/classic_arm/PSM1.urdf.xacro (robot description, xacro)
@@ -14,5 +14,5 @@
   <xacro:base prefix="PSM1_"
                   parent_link="${parent_link}"
-                  xyz="-0.25 0.0 0.5" rpy="0.0 0.0 ${PI}"/>
+                  xyz="0.0 0.0 0.0" rpy="0.0 0.0 0.0"/>
   <xacro:PSM_instrument prefix="PSM1_"
                         parent_link="PSM1_tool_parent_link"

File: urdf/classic_arm/PSM2.urdf.xacro (robot description, xacro)
@@ -9,5 +9,5 @@
   <xacro:base prefix="PSM2_"
                   parent_link="${parent_link}"
-                  xyz="-0.25 0.0 0.5" rpy="0.0 0.0 ${PI}"/>
+                  xyz="0.0 0.0 0.0" rpy="0.0 0.0 0.0"/>
   <xacro:PSM_instrument prefix="PSM2_"
                         parent_link="PSM2_tool_parent_link"

File: urdf/classic_arm/PSM3.urdf.xacro (robot description, xacro)
@@ -9,5 +9,5 @@
   <xacro:base prefix="PSM3_"
                   parent_link="${parent_link}"
-                  xyz="0.50 0.0 0.5" rpy="0.0 0.0 ${-PI}"/>
+                  xyz="0.0 0.0 0.0" rpy="0.0 0.0 0.0"/>
   <xacro:PSM_instrument prefix="PSM3_"
                         parent_link="PSM3_tool_parent_link"

File: urdf/si_arm/ECM_base.urdf.xacro (robot description, xacro)
@@ -53,5 +53,5 @@
       <parent link="${prefix}RCM_link"/>
       <child  link="${prefix}base_link"/>
-      <origin xyz="-0.84316314 0.0 0.0" rpy="0.0 0.0 0.0"/>
+      <origin xyz="0.0 -0.84316314 0.0" rpy="0.0 0.0 ${PI_2}"/>
     </joint>
     <!-- link 1: yaw body -->

File: urdf/si_arm/PSM_base.urdf.xacro (robot description, xacro)
@@ -52,5 +52,5 @@
       <parent link="${prefix}RCM_link"/>
       <child  link="${prefix}base_link"/>
-      <origin xyz="-0.84316314 0.0 0.0" rpy="0.0 0.0 0.0"/>
+      <origin xyz="0.0 -0.84316314 0.0" rpy="0.0 0.0 ${PI_2}"/>
     </joint>
     <!-- link 1: yaw body -->
