Commit message: Reorganize PSM_tips.urdf by tools

File: urdf/classic_arm/ECM.urdf.xacro (robot description, xacro)
@@ -4,5 +4,5 @@
   <xacro:arg name="parent_link_" default="world"/>
   <xacro:property name="parent_link" default="$(arg parent_link_)"/>
-  <xacro:include filename="$(find dvrk_model)/urdf/Classic/ECM_base.urdf.xacro"/>
+  <xacro:include filename="$(find dvrk_model)/urdf/classic_arm/ECM_base.urdf.xacro"/>
     <xacro:include filename="$(find dvrk_model)/urdf/common/endoscope.urdf.xacro"/>
   <link name="${parent_link}"/>

File: urdf/classic_arm/MTML.urdf.xacro (robot description, xacro)
@@ -2,5 +2,5 @@
 <robot name="MTML" xmlns:xacro="http://www.ros.org/wiki/xacro">
   <!-- Macros -->
-  <xacro:include filename="$(find dvrk_model)/urdf/Classic/MTM.urdf.xacro"/>
+  <xacro:include filename="$(find dvrk_model)/urdf/classic_arm/MTM.urdf.xacro"/>
   <link name="world"/>
   <xacro:mtm_left

File: urdf/classic_arm/MTMR.urdf.xacro (robot description, xacro)
@@ -2,5 +2,5 @@
 <robot name="MTMR" xmlns:xacro="http://www.ros.org/wiki/xacro">
   <!-- Macros -->
-  <xacro:include filename="$(find dvrk_model)/urdf/Classic/MTM.urdf.xacro"/>
+  <xacro:include filename="$(find dvrk_model)/urdf/classic_arm/MTM.urdf.xacro"/>
   <link name="world"/>
   <xacro:mtm_right

File: urdf/classic_arm/PSM1.urdf.xacro (robot description, xacro)
@@ -2,15 +2,17 @@
 <robot name="PSM1" xmlns:xacro="http://www.ros.org/wiki/xacro">
   <!--
-    Si PSM1 entry point.
-    arg instrument: last 6 digits of instrument model number (default: 420006)
+    Classic PSM1 entry point.
+    arg instrument: last 6 digits of instrument model number (default: 400006)
+    arm placed at a typical setup position; adjust xyz/rpy for your rig.
   -->
-  <xacro:arg name="instrument" default="420006"/>
+  <xacro:arg name="instrument" default="400006"/>
   <xacro:arg name="parent_link_" default="world"/>
   <xacro:property name="parent_link" value="$(arg parent_link_)"/>
-  <xacro:include filename="$(find dvrk_model)/urdf/Si/PSM_base.urdf.xacro"/>
+  <xacro:include filename="$(find dvrk_model)/urdf/classic_arm/PSM_base.urdf.xacro"/>
   <xacro:include filename="$(find dvrk_model)/urdf/common/PSM_instrument.urdf.xacro"/>
   <link name="${parent_link}"/>
   <xacro:base prefix="PSM1_"
-                  parent_link="${parent_link}"/>
+                  parent_link="${parent_link}"
+                  xyz="-0.25 0.0 0.5" rpy="0.0 0.0 ${PI}"/>
   <xacro:PSM_instrument prefix="PSM1_"
                         parent_link="PSM1_tool_parent_link"

File: urdf/classic_arm/PSM1_snake.urdf.xacro (robot description, xacro)
@@ -1,6 +1,7 @@
 <?xml version="1.0" ?>
 <robot name="dvrk_psm" xmlns:xacro="http://www.ros.org/wiki/xacro">
+  <xacro:arg name="prefix" default="PSM1_"/>
   <!-- Macros -->
-  <xacro:include filename="$(find dvrk_model)/urdf/Classic/psm.urdf.xacro"/>
+  <xacro:include filename="$(find dvrk_model)/urdf/classic_arm/archive/psm.urdf.xacro"/>
   <link name="world"/>
   <xacro:psm_snake

File: urdf/classic_arm/PSM2.urdf.xacro (robot description, xacro)
@@ -1,12 +1,13 @@
 <?xml version="1.0" ?>
 <robot name="PSM2" xmlns:xacro="http://www.ros.org/wiki/xacro">
-  <xacro:arg name="instrument" default="420006"/>
+  <xacro:arg name="instrument" default="400049"/>
   <xacro:arg name="parent_link_" default="world"/>
   <xacro:property name="parent_link" value="$(arg parent_link_)"/>
-  <xacro:include filename="$(find dvrk_model)/urdf/Si/PSM_base.urdf.xacro"/>
+  <xacro:include filename="$(find dvrk_model)/urdf/classic_arm/PSM_base.urdf.xacro"/>
   <xacro:include filename="$(find dvrk_model)/urdf/common/PSM_instrument.urdf.xacro"/>
   <link name="${parent_link}"/>
   <xacro:base prefix="PSM2_"
-                  parent_link="${parent_link}"/>
+                  parent_link="${parent_link}"
+                  xyz="-0.25 0.0 0.5" rpy="0.0 0.0 ${PI}"/>
   <xacro:PSM_instrument prefix="PSM2_"
                         parent_link="PSM2_tool_parent_link"

File: urdf/classic_arm/PSM3.urdf.xacro (robot description, xacro)
@@ -1,15 +1,15 @@
 <?xml version="1.0" ?>
-<robot name="PSM2" xmlns:xacro="http://www.ros.org/wiki/xacro">
+<robot name="PSM3" xmlns:xacro="http://www.ros.org/wiki/xacro">
   <xacro:arg name="instrument" default="400049"/>
   <xacro:arg name="parent_link_" default="world"/>
   <xacro:property name="parent_link" value="$(arg parent_link_)"/>
-  <xacro:include filename="$(find dvrk_model)/urdf/Classic/PSM_base.urdf.xacro"/>
+  <xacro:include filename="$(find dvrk_model)/urdf/classic_arm/PSM_base.urdf.xacro"/>
   <xacro:include filename="$(find dvrk_model)/urdf/common/PSM_instrument.urdf.xacro"/>
   <link name="${parent_link}"/>
-  <xacro:base prefix="PSM2_"
+  <xacro:base prefix="PSM3_"
                   parent_link="${parent_link}"
-                  xyz="-0.25 0.0 0.5" rpy="0.0 0.0 ${PI}"/>
-  <xacro:PSM_instrument prefix="PSM2_"
-                        parent_link="PSM2_tool_parent_link"
+                  xyz="0.50 0.0 0.5" rpy="0.0 0.0 ${-PI}"/>
+  <xacro:PSM_instrument prefix="PSM3_"
+                        parent_link="PSM3_tool_parent_link"
                         instrument="$(arg instrument)"/>
 </robot>

File: urdf/classic_arm/archive/psm_tool.urdf.xacro (robot description, xacro)
@@ -2,8 +2,8 @@
 <robot name="dvrk_psm" xmlns:xacro="http://www.ros.org/wiki/xacro">
   <!-- Macros -->
-  <xacro:include filename="$(find dvrk_model)/urdf/Classic/psm_base.urdf.xacro"/>
-  <xacro:include filename="$(find dvrk_model)/urdf/Classic/psm_tool_sca.urdf.xacro"/>
-  <xacro:include filename="$(find dvrk_model)/urdf/Classic/psm_tool_caudier.urdf.xacro"/>
-  <xacro:include filename="$(find dvrk_model)/urdf/Classic/psm_tool_snake.urdf.xacro"/>
+  <xacro:include filename="$(find dvrk_model)/urdf/classic_arm/archive/psm_base.urdf.xacro"/>
+  <xacro:include filename="$(find dvrk_model)/urdf/classic_arm/archive/psm_tool_sca.urdf.xacro"/>
+  <xacro:include filename="$(find dvrk_model)/urdf/classic_arm/archive/psm_tool_caudier.urdf.xacro"/>
+  <xacro:include filename="$(find dvrk_model)/urdf/classic_arm/archive/psm_tool_snake.urdf.xacro"/>
   <xacro:macro name="psm_tool" params="tool_name prefix">
     <xacro:if value="${tool_name == 'sca'}">

File: urdf/common/PSM_instrument.urdf.xacro (robot description, xacro)
@@ -18,5 +18,7 @@
   -->
   <xacro:include filename="$(find dvrk_model)/urdf/common.urdf.xacro"/>
-  <xacro:include filename="$(find dvrk_model)/urdf/common/PSM_tips.urdf.xacro"/>
+  <xacro:include filename="$(find dvrk_model)/urdf/common/psm_tools/PSM_body.urdf.xacro"/>
+  <xacro:include filename="$(find dvrk_model)/urdf/common/psm_tools/PSM_006.urdf.xacro"/>
+  <xacro:include filename="$(find dvrk_model)/urdf/common/psm_tools/PSM_049.urdf.xacro"/>
   <xacro:macro name="PSM_instrument"
                params="prefix parent_link instrument">
@@ -33,130 +35,16 @@
     <xacro:property name="roll_origin" value="${shaft_length + tool_main_offset}"/>
     <xacro:property name="tip_parent_link" value="${prefix + ('roll_link' if is_si else 'shaft_link')}"/>
-    <!-- fixed joint to hold the shaft visual BEFORE the roll joint -->
-    <joint name="instrument_base_fixed" type="fixed">
-      <parent link="${parent_link}"/>
-      <child  link="${prefix}instrument_base_link"/>
-      <origin rpy="-1.5708 0 -1.5708" xyz="0 0 0"/>
-    </joint>
-    <link name="${prefix}instrument_base_link">
-      <visual>
-        <xacro:if value="${is_si}">
-          <!-- Si housing lives at the proximal tool base (not along the shaft). -->
-          <origin rpy="-1.5708 0 -1.5708" xyz="0 0 0"/>
-          <geometry>
-            <mesh filename="package://dvrk_model/meshes/instruments/Si/housing/PSM_housing.OBJ"/>
-          </geometry>
-        </xacro:if>
-        <xacro:unless value="${is_si}">
-          <origin rpy="0 0 1.5708" xyz="0 0 0.0904"/>
-          <geometry>
-            <mesh filename="package://dvrk_model/meshes/instruments/Classic/housing/PSM_housing.dae"/>
-          </geometry>
-        </xacro:unless>
-      </visual>
-      <collision>
-        <xacro:if value="${is_si}">
-          <origin rpy="0 0 0" xyz="0 0 0"/>
-          <geometry>
-            <mesh filename="package://dvrk_model/meshes/instruments/Si/housing/PSM_housing.OBJ"/>
-          </geometry>
-        </xacro:if>
-        <xacro:unless value="${is_si}">
-          <origin rpy="0 0 1.5708" xyz="0 0 0.0904"/>
-          <geometry>
-            <mesh filename="package://dvrk_model/meshes/instruments/Classic/housing/PSM_housing.dae"/>
-          </geometry>
-        </xacro:unless>
-      </collision>
-    </link>
-    <!-- joint 4: roll (outer roll of instrument inner shaft) -->
-    <joint name="roll" type="revolute">
-      <parent link="${parent_link}"/>
-      <child  link="${prefix}roll_link"/>
-      <axis xyz="0 0 1"/>
-      <origin rpy="0 0 0" xyz="0 0 ${roll_origin}"/>
-      <limit lower="-4.53786" upper="4.53786" velocity=".4" effort="1000"/>
-    </joint>
-    <!--
-      PSM_roll_link — carries the inner shaft rotation.
-      The outer shaft mesh (above) does not roll or shift.
-    -->
-    <link name="${prefix}roll_link">
-      <visual>
-        <xacro:if value="${is_si}">
-          <origin rpy="0 0 0" xyz="0 0 -0.216"/>
-          <geometry>
-            <mesh filename="package://dvrk_model/meshes/instruments/Si/roll/PSM_roll_8mm.OBJ"/>
-          </geometry>
-          <material name=""><color rgba="0.79216 0.81961 0.93333 1"/></material>
-        </xacro:if>
-      </visual>
-      <collision>
-        <xacro:if value="${is_si}">
-          <origin rpy="0 0 0" xyz="0 0 -0.216"/>
-          <geometry>
-            <mesh filename="package://dvrk_model/meshes/instruments/Si/roll/PSM_roll_8mm.OBJ"/>
-          </geometry>
-        </xacro:if>
-      </collision>
-    </link>
-    <!-- fixed joint to roll housing -->
-    <joint name="roll_fixed" type="fixed">
-      <parent link="${prefix}roll_link"/>
-      <child  link="${prefix}roll_housing_link"/>
-      <origin rpy="0 0 0" xyz="0 0 0"/>
-    </joint>
-    <link name="${prefix}roll_housing_link">
-      <visual>
-        <!-- Si: structural link only, no duplicate shaft visual here. -->
-        <xacro:unless value="${is_si}">
-          <!-- Classic roll housing at the shaft end -->
-          <origin rpy="0 0 1.5708" xyz="0 0 -0.0091"/>
-          <geometry>
-            <mesh filename="package://dvrk_model/meshes/instruments/Classic/roll/PSM_roll.dae"/>
-          </geometry>
-        </xacro:unless>
-      </visual>
-      <collision>
-        <xacro:unless value="${is_si}">
-          <origin rpy="0 0 1.5708" xyz="0 0 -0.0091"/>
-          <geometry>
-            <mesh filename="package://dvrk_model/meshes/instruments/Classic/roll/PSM_roll.dae"/>
-          </geometry>
-        </xacro:unless>
-      </collision>
-    </link>
-    <!-- fixed joint to shaft -->
-    <joint name="shaft_fixed" type="fixed">
-      <parent link="${prefix}roll_housing_link"/>
-      <child  link="${prefix}shaft_link"/>
-      <origin rpy="0 0 0" xyz="0 0 0"/>
-    </joint>
-    <link name="${prefix}shaft_link">
-      <visual>
-        <xacro:unless value="${is_si}">
-          <origin rpy="${PI_2} 0 0" xyz="0 0.00401 0"/>
-          <geometry>
-            <mesh filename="package://dvrk_model/meshes/instruments/Classic/yaw/PSM_yaw.dae"/>
-          </geometry>
-        </xacro:unless>
-      </visual>
-      <collision>
-        <xacro:unless value="${is_si}">
-          <origin rpy="${PI_2} 0 0" xyz="0 0.00401 0"/>
-          <geometry>
-            <mesh filename="package://dvrk_model/meshes/instruments/Classic/yaw/PSM_yaw.dae"/>
-          </geometry>
-        </xacro:unless>
-      </collision>
-    </link>
+    <xacro:PSM_instrument_body prefix="${prefix}"
+                   parent_link="${parent_link}"
+                   is_si="${is_si}"
+                   roll_origin="${roll_origin}"/>
     <!--
       Tip dispatch: select the correct tip+jaw macro by instrument.
       Convention: last 3 digits of the model number identify the tip family.
-        006 → standard SCA wrist (most instruments, A=0.0091)
-        049 → Cadiere jaw (same wrist, different jaw geometry)
-        172 → Maryland wrist (A=0.0107)
-        117 → snake tool (5 mm shaft, extra coupled joints)
-        183 → cautery / no-jaw tools
+        006 → standard SCA wrist (A=0.0091)
+        049 → Cadiere jaw (A=0.0091)
+      Verified common dimensions:
+        roll D  → 0.4162 Classic, 0.4670 Si
+        006 tip → tool_tip at y=0.0102
     -->
     <!-- 006: standard SCA wrist -->
@@ -170,19 +58,8 @@
     </xacro:if>
     <!-- 049: Cadiere jaw -->
-    <xacro:if value="${str(instrument) == '420049' or str(instrument) == '400049'}">
+    <xacro:if value="${str(instrument) == '400049'}">
       <xacro:PSM_tip_049 prefix="${prefix}"
                          parent_link="${tip_parent_link}"/>
     </xacro:if>
-    <!-- 172: Maryland wrist — currently reuses PSM_tip_006 placeholder meshes (see note in PSM_tips.urdf.xacro) -->
-    <xacro:if value="${str(instrument) == '420172' or str(instrument) == '400172'}">
-      <xacro:PSM_tip_172 prefix="${prefix}"
-                         parent_link="${tip_parent_link}"/>
-    </xacro:if>
-    <!-- 117: snake tool — PSM_tip_117 is currently a kinematic stub only (no meshes, no jaw geometry, DOFs unconfirmed) -->
-    <xacro:if value="${str(instrument) == '400117'}">
-      <xacro:PSM_tip_117 prefix="${prefix}"
-                         parent_link="${tip_parent_link}"/>
-    </xacro:if>
-    <!-- 183: cautery / no-jaw tools — PSM_tip_183 macro exists in PSM_tips.urdf.xacro but is not yet wired into this dispatch -->
   </xacro:macro>
 </robot>

File: urdf/si_arm/ECM.urdf.xacro (robot description, xacro)
@@ -4,5 +4,5 @@
   <xacro:arg name="parent_link_" default="world"/>
   <xacro:property name="parent_link" default="$(arg parent_link_)"/>
-  <xacro:include filename="$(find dvrk_model)/urdf/Si/ECM_base.urdf.xacro"/>
+  <xacro:include filename="$(find dvrk_model)/urdf/si_arm/ECM_base.urdf.xacro"/>
   <xacro:include filename="$(find dvrk_model)/urdf/common/endoscope.urdf.xacro"/>
   <link name="${parent_link}"/>

File: urdf/si_arm/PSM1.urdf.xacro (robot description, xacro)
@@ -1,14 +1,18 @@
 <?xml version="1.0" ?>
-<robot name="PSM3" xmlns:xacro="http://www.ros.org/wiki/xacro">
+<robot name="PSM1" xmlns:xacro="http://www.ros.org/wiki/xacro">
+  <!--
+    Si PSM1 entry point.
+    arg instrument: last 6 digits of instrument model number (default: 420006)
+  -->
   <xacro:arg name="instrument" default="420006"/>
   <xacro:arg name="parent_link_" default="world"/>
   <xacro:property name="parent_link" value="$(arg parent_link_)"/>
-  <xacro:include filename="$(find dvrk_model)/urdf/Si/PSM_base.urdf.xacro"/>
+  <xacro:include filename="$(find dvrk_model)/urdf/si_arm/PSM_base.urdf.xacro"/>
   <xacro:include filename="$(find dvrk_model)/urdf/common/PSM_instrument.urdf.xacro"/>
   <link name="${parent_link}"/>
-  <xacro:base prefix="PSM3_"
+  <xacro:base prefix="PSM1_"
                   parent_link="${parent_link}"/>
-  <xacro:PSM_instrument prefix="PSM3_"
-                        parent_link="PSM3_tool_parent_link"
+  <xacro:PSM_instrument prefix="PSM1_"
+                        parent_link="PSM1_tool_parent_link"
                         instrument="$(arg instrument)"/>
 </robot>

File: urdf/si_arm/PSM3.urdf.xacro (robot description, xacro)
@@ -1,13 +1,12 @@
 <?xml version="1.0" ?>
 <robot name="PSM3" xmlns:xacro="http://www.ros.org/wiki/xacro">
-  <xacro:arg name="instrument" default="400049"/>
+  <xacro:arg name="instrument" default="420006"/>
   <xacro:arg name="parent_link_" default="world"/>
   <xacro:property name="parent_link" value="$(arg parent_link_)"/>
-  <xacro:include filename="$(find dvrk_model)/urdf/Classic/PSM_base.urdf.xacro"/>
+  <xacro:include filename="$(find dvrk_model)/urdf/si_arm/PSM_base.urdf.xacro"/>
   <xacro:include filename="$(find dvrk_model)/urdf/common/PSM_instrument.urdf.xacro"/>
   <link name="${parent_link}"/>
   <xacro:base prefix="PSM3_"
-                  parent_link="${parent_link}"
-                  xyz="0.50 0.0 0.5" rpy="0.0 0.0 ${-PI}"/>
+                  parent_link="${parent_link}"/>
   <xacro:PSM_instrument prefix="PSM3_"
                         parent_link="PSM3_tool_parent_link"

File: urdf/si_arm/SUJ.urdf.xacro (robot description, xacro)
@@ -2,6 +2,6 @@
 <robot name="patient_cart" xmlns:xacro="http://www.ros.org/wiki/xacro">
   <xacro:include filename="$(find dvrk_model)/urdf/common.urdf.xacro"/>
-  <xacro:include filename="$(find dvrk_model)/urdf/Si/SUJ_base.urdf.xacro"/>
-  <xacro:include filename="$(find dvrk_model)/urdf/Si/SUJ_column.urdf.xacro"/>
+  <xacro:include filename="$(find dvrk_model)/urdf/si_arm/SUJ_base.urdf.xacro"/>
+  <xacro:include filename="$(find dvrk_model)/urdf/si_arm/SUJ_column.urdf.xacro"/>
   <xacro:suj_column/>
   <xacro:suj
