Commit message: Refactor ECM URDF and endoscope definitions to use adaptor_link; update joint and link references for compatibility. Added check for launch file parameters

File: urdf/classic_arm/ECM.urdf.xacro (robot description, xacro)
@@ -13,4 +13,4 @@
   <xacro:endoscope
       prefix="ECM_"
-      parent_link="ECM_roll_link"/>
+      parent_link="ECM_adaptor_link"/>
 </robot>

File: urdf/classic_arm/ECM_base.urdf.xacro (robot description, xacro)
@@ -225,4 +225,10 @@
       <limit lower="-1.552676" upper="1.566741" effort="1000" velocity="10"/>
     </joint>
+    <joint name="${prefix}adaptor_fixed" type="fixed">
+      <parent link="${prefix}roll_link"/>
+      <child  link="${prefix}adaptor_link"/>
+      <origin xyz="0.0 0.0 0.0" rpy="0.0 0.0 0.0"/>
+    </joint>
+    <link name="${prefix}adaptor_link"/>
     <!-- Alias link for backward compatibility with older rviz configs referencing remote_center_link -->
     <link name="${prefix}remote_center_link"/>

File: urdf/common/endoscopes/Classic_SD_straight.urdf.xacro (robot description, xacro)
@@ -4,18 +4,18 @@
   <!--
     Classic SD straight endoscope.
-    Attaches to ${prefix}roll_link (last link of ECM_base).
-    Provides its own mesh and a fixed endoscope_tip reference frame.
+    Attaches to ${prefix}adaptor_link.
+    Provides its own mesh and a fixed tip reference frame.
   -->
   <xacro:macro name="endoscope"
-               params="prefix:='ECM_' parent_link:='ECM_roll_link'">
-    <!-- Endoscope body: fixed to roll_link, rotates with roll -->
-    <joint name="endoscope_body" type="fixed">
+               params="prefix:='ECM_' parent_link:='ECM_adaptor_link'">
+    <!-- Endoscope body: fixed to adaptor_link, rotates with roll -->
+    <joint name="endoscope" type="fixed">
       <origin xyz="0.0 0.0 0.0" rpy="0.0 0.0 0.0"/>
       <parent link="${parent_link}"/>
-      <child  link="${prefix}endoscope_body_link"/>
+      <child  link="${prefix}endoscope_link"/>
     </joint>
-    <link name="${prefix}endoscope_body_link">
+    <link name="${prefix}endoscope_link">
       <visual>
-        <!-- z=0.010 compensates for roll_link moving 0.010 m further above RCM -->
+        <!-- z=0.010 compensates for adaptor_link moving 0.010 m further above RCM -->
         <origin xyz="0.0 0.0 0.010" rpy="0.0 0.0 0.0"/>
         <geometry>
@@ -32,10 +32,10 @@
     </link>
     <!-- Fixed transform to endoscope tip reference frame -->
-    <joint name="endoscope_tip" type="fixed">
+    <joint name="tip" type="fixed">
       <origin xyz="0.0 0.0 0.37364" rpy="0.0 0.0 0.0"/>
-      <parent link="${prefix}endoscope_body_link"/>
-      <child  link="${prefix}endoscope_tip_link"/>
+      <parent link="${prefix}endoscope_link"/>
+      <child  link="${prefix}tip_link"/>
     </joint>
-    <link name="${prefix}endoscope_tip_link"/>
+    <link name="${prefix}tip_link"/>
   </xacro:macro>
 </robot>

File: urdf/common/endoscopes/Si_straight.urdf.xacro (robot description, xacro)
@@ -4,20 +4,20 @@
   <!--
     Si straight endoscope.
-    Attaches to ${prefix}roll_link (last link of ECM_base).
+    Attaches to ${prefix}adaptor_link.
     Provides its own meshes and a fixed camera tip reference frame.
     Future variants Si_down and Si_up will add a 30-degree rotation
-    before the endoscope_tip joint.
+    before the tip joint.
   -->
   <xacro:macro name="endoscope"
-               params="prefix:='ECM_' parent_link:='ECM_roll_link'">
-    <!-- Endoscope body: housing + shaft + camera tip, fixed to roll_link -->
-    <joint name="endoscope_body" type="fixed">
+               params="prefix:='ECM_' parent_link:='ECM_adaptor_link'">
+    <!-- Endoscope body: housing + shaft + camera tip, fixed to adaptor_link -->
+    <joint name="endoscope" type="fixed">
       <origin xyz="0.0 0.0 0.0" rpy="0.0 0.0 0.0"/>
       <parent link="${parent_link}"/>
-      <child  link="${prefix}endoscope_body_link"/>
+      <child  link="${prefix}endoscope_link"/>
     </joint>
-    <link name="${prefix}endoscope_body_link">
+    <link name="${prefix}endoscope_link">
       <visual>
-        <!-- z=0.2577 compensates for roll_link moving 0.2577 m further above RCM -->
+        <!-- z=0.2577 compensates for adaptor_link moving 0.2577 m further above RCM -->
         <!-- housing -->
         <origin rpy="-1.5708 0.0 -1.5708" xyz="0.0 0.0 0.2577"/>
@@ -48,18 +48,18 @@
       </collision>
     </link>
-    <!-- Convert from roll_link into camera reference frame -->
+    <!-- Convert from adaptor_link into camera reference frame -->
     <joint name="endoscope_frame" type="fixed">
       <origin rpy="-1.5708 -1.5708 0.0" xyz="0.0 0.0 0.0"/>
-      <parent link="${prefix}endoscope_body_link"/>
+      <parent link="${prefix}endoscope_link"/>
       <child  link="${prefix}endoscope_frame_link"/>
     </joint>
     <link name="${prefix}endoscope_frame_link"/>
     <!-- Offset to physical camera tip -->
-    <joint name="endoscope_tip" type="fixed">
+    <joint name="tip" type="fixed">
       <origin xyz="0.0 0.0102 0.0" rpy="0.0 0.0 0.0"/>
       <parent link="${prefix}endoscope_frame_link"/>
-      <child  link="${prefix}endoscope_tip_link"/>
+      <child  link="${prefix}tip_link"/>
     </joint>
-    <link name="${prefix}endoscope_tip_link"/>
+    <link name="${prefix}tip_link"/>
   </xacro:macro>
 </robot>

File: urdf/si_arm/ECM.urdf.xacro (robot description, xacro)
@@ -11,4 +11,4 @@
                   parent_link="${parent_link}"/>
   <xacro:endoscope prefix="ECM_"
-                   parent_link="ECM_roll_link"/>
+                   parent_link="ECM_adaptor_link"/>
 </robot>

File: urdf/si_arm/ECM_base.urdf.xacro (robot description, xacro)
@@ -192,5 +192,5 @@
     <!-- origin z=0.2093 places roll_link exactly 0.3829 m above RCM (was 0.1252 m at z=0.4670) -->
     <joint name="roll" type="revolute">
-      <origin xyz="0.0 0.0 0.2093" rpy="0.0 0.0 0.0"/>
+      <origin xyz="0.06462752 0.0 0.2093" rpy="0.0 0.0 0.0"/>
       <parent link="${prefix}insertion_link"/>
       <child  link="${prefix}roll_link"/>
@@ -203,4 +203,10 @@
     -->
     <link name="${prefix}roll_link"/>
+    <joint name="${prefix}adaptor_fixed" type="fixed">
+      <parent link="${prefix}roll_link"/>
+      <child  link="${prefix}adaptor_link"/>
+      <origin xyz="0.0 0.0 0.0" rpy="0.0 0.0 0.0"/>
+    </joint>
+    <link name="${prefix}adaptor_link"/>
   </xacro:macro>
 </robot>
