Commit message: Fixed wrist pitch orientation and yaw placement

File: urdf/common/instruments/wrist_pitch/wrist_pitch_0167.urdf.xacro (robot description, xacro)
@@ -12,5 +12,5 @@
     <link name="${prefix}wrist_pitch_link">
       <visual>
-        <origin rpy="0.0 ${PI} -${PI_2}" xyz="-0.027915 0.0 0.0"/>
+        <origin rpy="0.0 ${PI} ${PI_2}" xyz="0.039915 0.0 0.0"/>
         <geometry>
           <mesh filename="package://dvrk_model/meshes/instruments/wrist_pitch/0167/wrist_pitch_0167.obj" scale="0.1 0.1 0.1"/>

File: urdf/common/instruments/wrist_yaw/wrist_yaw_0167.urdf.xacro (robot description, xacro)
@@ -7,5 +7,5 @@
       <child link="${prefix}wrist_yaw_link"/>
       <axis xyz="0.0 0.0 1"/>
-      <origin rpy="-${PI_2} -${PI_2} 0.0" xyz="0.0167 0.0 0.0"/>
+      <origin rpy="-${PI_2} -${PI_2} 0.0" xyz="0.011565 0.0 0.0"/>
       <limit lower="-1.39626" upper="1.39626" velocity=".4" effort="1000"/>
     </joint>

Commit message: Fix 0167 wrist pitch orientation and import roll housing with pulleys

File: urdf/common/instruments/wrist_pitch/wrist_pitch_0167.urdf.xacro (robot description, xacro)
@@ -7,5 +7,5 @@
       <child link="${prefix}wrist_pitch_link"/>
       <axis xyz="0.0 0.0 1"/>
-      <origin rpy="-${PI_2} -${PI_2} 0.0" xyz="0.0 0.0 0.0"/>
+      <origin rpy="0.0 -${PI_2} 0.0" xyz="0.0 0.0 0.0"/>
       <limit lower="-1.2217" upper="1.2217" velocity=".4" effort="1000"/>
     </joint>

Commit message: Reposition wrist pitch wrt roll

File: urdf/common/instruments/wrist_pitch/wrist_pitch_0167.urdf.xacro (robot description, xacro)
@@ -12,5 +12,5 @@
     <link name="${prefix}wrist_pitch_link">
       <visual>
-        <origin rpy="0.0 ${PI} ${PI_2}" xyz="0.039915 0.0 0.0"/>
+        <origin rpy="0.0 ${PI} ${PI_2}" xyz="0.039 0.0 0.0"/>
         <geometry>
           <mesh filename="package://dvrk_model/meshes/instruments/wrist_pitch/0167/wrist_pitch_0167.obj" scale="0.1 0.1 0.1"/>
