Commit message: Created wrist pitch and yaw frames for visualization. wrist 0112 position is fixed

File: urdf/common/instruments/wrist_pitch/wrist_pitch_0091.urdf.xacro (robot description, xacro)
@@ -17,4 +17,43 @@
         </geometry>
       </visual>
+      <!-- Uncomment this block to show wrist_pitch_link frame triad in RViz -->
+      <!--
+      <visual>
+        <origin rpy="0.0 0.0 0.0" xyz="0.0 0.0 0.0"/>
+        <geometry>
+          <sphere radius="0.0008"/>
+        </geometry>
+        <material name="wrist_pitch_frame_origin">
+          <color rgba="0.0 0.7 1.0 1.0"/>
+        </material>
+      </visual>
+      <visual>
+        <origin rpy="0.0 ${PI_2} 0.0" xyz="0.003 0.0 0.0"/>
+        <geometry>
+          <cylinder length="0.006" radius="0.00035"/>
+        </geometry>
+        <material name="wrist_pitch_frame_x">
+          <color rgba="1.0 0.0 0.0 1.0"/>
+        </material>
+      </visual>
+      <visual>
+        <origin rpy="-${PI_2} 0.0 0.0" xyz="0.0 0.003 0.0"/>
+        <geometry>
+          <cylinder length="0.006" radius="0.00035"/>
+        </geometry>
+        <material name="wrist_pitch_frame_y">
+          <color rgba="0.0 1.0 0.0 1.0"/>
+        </material>
+      </visual>
+      <visual>
+        <origin rpy="0.0 0.0 0.0" xyz="0.0 0.0 0.003"/>
+        <geometry>
+          <cylinder length="0.006" radius="0.00035"/>
+        </geometry>
+        <material name="wrist_pitch_frame_z">
+          <color rgba="0.0 0.0 1.0 1.0"/>
+        </material>
+      </visual>
+      -->
     </link>
   </xacro:macro>

File: urdf/common/instruments/wrist_pitch/wrist_pitch_0093.urdf.xacro (robot description, xacro)
@@ -17,4 +17,43 @@
         </geometry>
       </visual>
+      <!-- Uncomment this block to show wrist_pitch_link frame triad in RViz -->
+      <!--
+      <visual>
+        <origin rpy="0.0 0.0 0.0" xyz="0.0 0.0 0.0"/>
+        <geometry>
+          <sphere radius="0.0008"/>
+        </geometry>
+        <material name="wrist_pitch_frame_origin">
+          <color rgba="0.0 0.7 1.0 1.0"/>
+        </material>
+      </visual>
+      <visual>
+        <origin rpy="0.0 ${PI_2} 0.0" xyz="0.003 0.0 0.0"/>
+        <geometry>
+          <cylinder length="0.006" radius="0.00035"/>
+        </geometry>
+        <material name="wrist_pitch_frame_x">
+          <color rgba="1.0 0.0 0.0 1.0"/>
+        </material>
+      </visual>
+      <visual>
+        <origin rpy="-${PI_2} 0.0 0.0" xyz="0.0 0.003 0.0"/>
+        <geometry>
+          <cylinder length="0.006" radius="0.00035"/>
+        </geometry>
+        <material name="wrist_pitch_frame_y">
+          <color rgba="0.0 1.0 0.0 1.0"/>
+        </material>
+      </visual>
+      <visual>
+        <origin rpy="0.0 0.0 0.0" xyz="0.0 0.0 0.003"/>
+        <geometry>
+          <cylinder length="0.006" radius="0.00035"/>
+        </geometry>
+        <material name="wrist_pitch_frame_z">
+          <color rgba="0.0 0.0 1.0 1.0"/>
+        </material>
+      </visual>
+      -->
     </link>
   </xacro:macro>

File: urdf/common/instruments/wrist_pitch/wrist_pitch_0100.urdf.xacro (robot description, xacro)
@@ -17,4 +17,43 @@
         </geometry>
       </visual>
+      <!-- Uncomment this block to show wrist_pitch_link frame triad in RViz -->
+      <!--
+      <visual>
+        <origin rpy="0.0 0.0 0.0" xyz="0.0 0.0 0.0"/>
+        <geometry>
+          <sphere radius="0.0008"/>
+        </geometry>
+        <material name="wrist_pitch_frame_origin">
+          <color rgba="0.0 0.7 1.0 1.0"/>
+        </material>
+      </visual>
+      <visual>
+        <origin rpy="0.0 ${PI_2} 0.0" xyz="0.003 0.0 0.0"/>
+        <geometry>
+          <cylinder length="0.006" radius="0.00035"/>
+        </geometry>
+        <material name="wrist_pitch_frame_x">
+          <color rgba="1.0 0.0 0.0 1.0"/>
+        </material>
+      </visual>
+      <visual>
+        <origin rpy="-${PI_2} 0.0 0.0" xyz="0.0 0.003 0.0"/>
+        <geometry>
+          <cylinder length="0.006" radius="0.00035"/>
+        </geometry>
+        <material name="wrist_pitch_frame_y">
+          <color rgba="0.0 1.0 0.0 1.0"/>
+        </material>
+      </visual>
+      <visual>
+        <origin rpy="0.0 0.0 0.0" xyz="0.0 0.0 0.003"/>
+        <geometry>
+          <cylinder length="0.006" radius="0.00035"/>
+        </geometry>
+        <material name="wrist_pitch_frame_z">
+          <color rgba="0.0 0.0 1.0 1.0"/>
+        </material>
+      </visual>
+      -->
     </link>
   </xacro:macro>

File: urdf/common/instruments/wrist_pitch/wrist_pitch_0107.urdf.xacro (robot description, xacro)
@@ -17,4 +17,43 @@
         </geometry>
       </visual>
+      <!-- Uncomment this block to show wrist_pitch_link frame triad in RViz -->
+      <!--
+      <visual>
+        <origin rpy="0.0 0.0 0.0" xyz="0.0 0.0 0.0"/>
+        <geometry>
+          <sphere radius="0.0008"/>
+        </geometry>
+        <material name="wrist_pitch_frame_origin">
+          <color rgba="0.0 0.7 1.0 1.0"/>
+        </material>
+      </visual>
+      <visual>
+        <origin rpy="0.0 ${PI_2} 0.0" xyz="0.003 0.0 0.0"/>
+        <geometry>
+          <cylinder length="0.006" radius="0.00035"/>
+        </geometry>
+        <material name="wrist_pitch_frame_x">
+          <color rgba="1.0 0.0 0.0 1.0"/>
+        </material>
+      </visual>
+      <visual>
+        <origin rpy="-${PI_2} 0.0 0.0" xyz="0.0 0.003 0.0"/>
+        <geometry>
+          <cylinder length="0.006" radius="0.00035"/>
+        </geometry>
+        <material name="wrist_pitch_frame_y">
+          <color rgba="0.0 1.0 0.0 1.0"/>
+        </material>
+      </visual>
+      <visual>
+        <origin rpy="0.0 0.0 0.0" xyz="0.0 0.0 0.003"/>
+        <geometry>
+          <cylinder length="0.006" radius="0.00035"/>
+        </geometry>
+        <material name="wrist_pitch_frame_z">
+          <color rgba="0.0 0.0 1.0 1.0"/>
+        </material>
+      </visual>
+      -->
     </link>
   </xacro:macro>

File: urdf/common/instruments/wrist_pitch/wrist_pitch_0112.urdf.xacro (robot description, xacro)
@@ -12,9 +12,48 @@
     <link name="${prefix}wrist_pitch_link">
       <visual>
-        <origin rpy="0.0 ${PI_2} ${PI_2}" xyz="0.023 0.0 0.0"/>
+        <origin rpy="0.0 ${PI_2} ${PI_2}" xyz="0.02375 0.0 0.0"/>
         <geometry>
           <mesh filename="package://dvrk_model/meshes/instruments/wrist_pitch/0112/wrist_pitch_0112.obj" scale="0.1 0.1 0.1"/>
         </geometry>
       </visual>
+      <!-- Uncomment this block to show wrist_pitch_link frame triad in RViz -->
+      <!--
+      <visual>
+        <origin rpy="0.0 0.0 0.0" xyz="0.0 0.0 0.0"/>
+        <geometry>
+          <sphere radius="0.0008"/>
+        </geometry>
+        <material name="wrist_pitch_frame_origin">
+          <color rgba="0.0 0.7 1.0 1.0"/>
+        </material>
+      </visual>
+      <visual>
+        <origin rpy="0.0 ${PI_2} 0.0" xyz="0.003 0.0 0.0"/>
+        <geometry>
+          <cylinder length="0.006" radius="0.00035"/>
+        </geometry>
+        <material name="wrist_pitch_frame_x">
+          <color rgba="1.0 0.0 0.0 1.0"/>
+        </material>
+      </visual>
+      <visual>
+        <origin rpy="-${PI_2} 0.0 0.0" xyz="0.0 0.003 0.0"/>
+        <geometry>
+          <cylinder length="0.006" radius="0.00035"/>
+        </geometry>
+        <material name="wrist_pitch_frame_y">
+          <color rgba="0.0 1.0 0.0 1.0"/>
+        </material>
+      </visual>
+      <visual>
+        <origin rpy="0.0 0.0 0.0" xyz="0.0 0.0 0.003"/>
+        <geometry>
+          <cylinder length="0.006" radius="0.00035"/>
+        </geometry>
+        <material name="wrist_pitch_frame_z">
+          <color rgba="0.0 0.0 1.0 1.0"/>
+        </material>
+      </visual>
+      -->
     </link>
   </xacro:macro>

File: urdf/common/instruments/wrist_yaw/wrist_yaw_0091.urdf.xacro (robot description, xacro)
@@ -17,4 +17,43 @@
         </geometry>
       </visual>
+      <!-- Uncomment this block to show wrist_yaw_link frame triad in RViz -->
+      <!--
+      <visual>
+        <origin rpy="0.0 0.0 0.0" xyz="0.0 0.0 0.0"/>
+        <geometry>
+          <sphere radius="0.0008"/>
+        </geometry>
+        <material name="wrist_yaw_frame_origin">
+          <color rgba="1.0 0.8 0.0 1.0"/>
+        </material>
+      </visual>
+      <visual>
+        <origin rpy="0.0 ${PI_2} 0.0" xyz="0.003 0.0 0.0"/>
+        <geometry>
+          <cylinder length="0.006" radius="0.00035"/>
+        </geometry>
+        <material name="wrist_yaw_frame_x">
+          <color rgba="1.0 0.0 0.0 1.0"/>
+        </material>
+      </visual>
+      <visual>
+        <origin rpy="-${PI_2} 0.0 0.0" xyz="0.0 0.003 0.0"/>
+        <geometry>
+          <cylinder length="0.006" radius="0.00035"/>
+        </geometry>
+        <material name="wrist_yaw_frame_y">
+          <color rgba="0.0 1.0 0.0 1.0"/>
+        </material>
+      </visual>
+      <visual>
+        <origin rpy="0.0 0.0 0.0" xyz="0.0 0.0 0.003"/>
+        <geometry>
+          <cylinder length="0.006" radius="0.00035"/>
+        </geometry>
+        <material name="wrist_yaw_frame_z">
+          <color rgba="0.0 0.0 1.0 1.0"/>
+        </material>
+      </visual>
+      -->
     </link>
   </xacro:macro>

File: urdf/common/instruments/wrist_yaw/wrist_yaw_0093.urdf.xacro (robot description, xacro)
@@ -17,4 +17,43 @@
         </geometry>
       </visual>
+      <!-- Uncomment this block to show wrist_yaw_link frame triad in RViz -->
+      <!--
+      <visual>
+        <origin rpy="0.0 0.0 0.0" xyz="0.0 0.0 0.0"/>
+        <geometry>
+          <sphere radius="0.0008"/>
+        </geometry>
+        <material name="wrist_yaw_frame_origin">
+          <color rgba="1.0 0.8 0.0 1.0"/>
+        </material>
+      </visual>
+      <visual>
+        <origin rpy="0.0 ${PI_2} 0.0" xyz="0.003 0.0 0.0"/>
+        <geometry>
+          <cylinder length="0.006" radius="0.00035"/>
+        </geometry>
+        <material name="wrist_yaw_frame_x">
+          <color rgba="1.0 0.0 0.0 1.0"/>
+        </material>
+      </visual>
+      <visual>
+        <origin rpy="-${PI_2} 0.0 0.0" xyz="0.0 0.003 0.0"/>
+        <geometry>
+          <cylinder length="0.006" radius="0.00035"/>
+        </geometry>
+        <material name="wrist_yaw_frame_y">
+          <color rgba="0.0 1.0 0.0 1.0"/>
+        </material>
+      </visual>
+      <visual>
+        <origin rpy="0.0 0.0 0.0" xyz="0.0 0.0 0.003"/>
+        <geometry>
+          <cylinder length="0.006" radius="0.00035"/>
+        </geometry>
+        <material name="wrist_yaw_frame_z">
+          <color rgba="0.0 0.0 1.0 1.0"/>
+        </material>
+      </visual>
+      -->
     </link>
   </xacro:macro>

File: urdf/common/instruments/wrist_yaw/wrist_yaw_0100.urdf.xacro (robot description, xacro)
@@ -17,4 +17,43 @@
         </geometry>
       </visual>
+      <!-- Uncomment this block to show wrist_yaw_link frame triad in RViz -->
+      <!--
+      <visual>
+        <origin rpy="0.0 0.0 0.0" xyz="0.0 0.0 0.0"/>
+        <geometry>
+          <sphere radius="0.0008"/>
+        </geometry>
+        <material name="wrist_yaw_frame_origin">
+          <color rgba="1.0 0.8 0.0 1.0"/>
+        </material>
+      </visual>
+      <visual>
+        <origin rpy="0.0 ${PI_2} 0.0" xyz="0.003 0.0 0.0"/>
+        <geometry>
+          <cylinder length="0.006" radius="0.00035"/>
+        </geometry>
+        <material name="wrist_yaw_frame_x">
+          <color rgba="1.0 0.0 0.0 1.0"/>
+        </material>
+      </visual>
+      <visual>
+        <origin rpy="-${PI_2} 0.0 0.0" xyz="0.0 0.003 0.0"/>
+        <geometry>
+          <cylinder length="0.006" radius="0.00035"/>
+        </geometry>
+        <material name="wrist_yaw_frame_y">
+          <color rgba="0.0 1.0 0.0 1.0"/>
+        </material>
+      </visual>
+      <visual>
+        <origin rpy="0.0 0.0 0.0" xyz="0.0 0.0 0.003"/>
+        <geometry>
+          <cylinder length="0.006" radius="0.00035"/>
+        </geometry>
+        <material name="wrist_yaw_frame_z">
+          <color rgba="0.0 0.0 1.0 1.0"/>
+        </material>
+      </visual>
+      -->
     </link>
   </xacro:macro>

File: urdf/common/instruments/wrist_yaw/wrist_yaw_0107.urdf.xacro (robot description, xacro)
@@ -17,4 +17,43 @@
         </geometry>
       </visual>
+      <!-- Uncomment this block to show wrist_yaw_link frame triad in RViz -->
+      <!--
+      <visual>
+        <origin rpy="0.0 0.0 0.0" xyz="0.0 0.0 0.0"/>
+        <geometry>
+          <sphere radius="0.0008"/>
+        </geometry>
+        <material name="wrist_yaw_frame_origin">
+          <color rgba="1.0 0.8 0.0 1.0"/>
+        </material>
+      </visual>
+      <visual>
+        <origin rpy="0.0 ${PI_2} 0.0" xyz="0.003 0.0 0.0"/>
+        <geometry>
+          <cylinder length="0.006" radius="0.00035"/>
+        </geometry>
+        <material name="wrist_yaw_frame_x">
+          <color rgba="1.0 0.0 0.0 1.0"/>
+        </material>
+      </visual>
+      <visual>
+        <origin rpy="-${PI_2} 0.0 0.0" xyz="0.0 0.003 0.0"/>
+        <geometry>
+          <cylinder length="0.006" radius="0.00035"/>
+        </geometry>
+        <material name="wrist_yaw_frame_y">
+          <color rgba="0.0 1.0 0.0 1.0"/>
+        </material>
+      </visual>
+      <visual>
+        <origin rpy="0.0 0.0 0.0" xyz="0.0 0.0 0.003"/>
+        <geometry>
+          <cylinder length="0.006" radius="0.00035"/>
+        </geometry>
+        <material name="wrist_yaw_frame_z">
+          <color rgba="0.0 0.0 1.0 1.0"/>
+        </material>
+      </visual>
+      -->
     </link>
   </xacro:macro>

File: urdf/common/instruments/wrist_yaw/wrist_yaw_0112.urdf.xacro (robot description, xacro)
@@ -12,9 +12,48 @@
     <link name="${prefix}wrist_yaw_link">
       <visual>
-        <origin rpy="${PI} 0.0 ${PI}" xyz="-0.000236 -0.011693 0.0"/>
+        <origin rpy="${PI} 0.0 ${PI}" xyz="0.0 -0.0126 0.0"/>
         <geometry>
           <mesh filename="package://dvrk_model/meshes/instruments/wrist_yaw/0112/wrist_yaw_0112.obj" scale="0.1 0.1 0.1"/>
         </geometry>
       </visual>
+      <!-- Uncomment this block to show wrist_yaw_link frame triad in RViz -->
+      <!--
+      <visual>
+        <origin rpy="0.0 0.0 0.0" xyz="0.0 0.0 0.0"/>
+        <geometry>
+          <sphere radius="0.0008"/>
+        </geometry>
+        <material name="wrist_yaw_frame_origin">
+          <color rgba="1.0 0.8 0.0 1.0"/>
+        </material>
+      </visual>
+      <visual>
+        <origin rpy="0.0 ${PI_2} 0.0" xyz="0.003 0.0 0.0"/>
+        <geometry>
+          <cylinder length="0.006" radius="0.00035"/>
+        </geometry>
+        <material name="wrist_yaw_frame_x">
+          <color rgba="1.0 0.0 0.0 1.0"/>
+        </material>
+      </visual>
+      <visual>
+        <origin rpy="-${PI_2} 0.0 0.0" xyz="0.0 0.003 0.0"/>
+        <geometry>
+          <cylinder length="0.006" radius="0.00035"/>
+        </geometry>
+        <material name="wrist_yaw_frame_y">
+          <color rgba="0.0 1.0 0.0 1.0"/>
+        </material>
+      </visual>
+      <visual>
+        <origin rpy="0.0 0.0 0.0" xyz="0.0 0.0 0.003"/>
+        <geometry>
+          <cylinder length="0.006" radius="0.00035"/>
+        </geometry>
+        <material name="wrist_yaw_frame_z">
+          <color rgba="0.0 0.0 1.0 1.0"/>
+        </material>
+      </visual>
+      -->
     </link>
   </xacro:macro>

Commit message: Updated 0091 yaw location

File: urdf/common/instruments/wrist_pitch/wrist_pitch_0091.urdf.xacro (robot description, xacro)
@@ -12,5 +12,5 @@
     <link name="${prefix}wrist_pitch_link">
       <visual>
-        <origin rpy="0.0 ${PI_2} ${PI_2}" xyz="0.039 0.0 0.0"/>
+        <origin rpy="0.0 ${PI_2} ${PI_2}" xyz="0.0295 0.0 0.0"/>
         <geometry>
           <mesh filename="package://dvrk_model/meshes/instruments/wrist_pitch/0091/wrist_pitch_0091.obj" scale="0.1 0.1 0.1"/>
@@ -18,7 +18,6 @@
       </visual>
       <!-- Uncomment this block to show wrist_pitch_link frame triad in RViz -->
-      <!--
       <visual>
-        <origin rpy="0.0 ${PI_2} ${PI_2}" xyz="0.039 0.0 0.0"/>
+        <origin rpy="0.0 0.0 0.0" xyz="0.0 0.0 0.0"/>
         <geometry>
           <sphere radius="0.0008"/>
@@ -55,5 +54,4 @@
         </material>
       </visual>
-      -->
     </link>
   </xacro:macro>

File: urdf/common/instruments/wrist_yaw/wrist_yaw_0091.urdf.xacro (robot description, xacro)
@@ -18,5 +18,4 @@
       </visual>
       <!-- Uncomment this block to show wrist_yaw_link frame triad in RViz -->
-      <!--
       <visual>
         <origin rpy="0.0 0.0 0.0" xyz="0.0 0.0 0.0"/>
@@ -55,5 +54,4 @@
         </material>
       </visual>
-      -->
     </link>
   </xacro:macro>
