Commit message: Remove jaw zero publisher and frame display

File: urdf/common/instruments/wrist_pitch/wrist_pitch_0091.urdf.xacro (robot description, xacro)
@@ -17,41 +17,4 @@
         </geometry>
       </visual>
-      <!-- Uncomment this block to show wrist_pitch_link frame triad in RViz -->
-      <visual>
-        <origin rpy="0.0 0.0 0.0" xyz="0.0 0.0 0.0"/>
-        <geometry>
-          <sphere radius="0.0008"/>
-        </geometry>
-        <material name="wrist_pitch_frame_origin">
-          <color rgba="0.0 0.7 1.0 1.0"/>
-        </material>
-      </visual>
-      <visual>
-        <origin rpy="0.0 ${PI_2} 0.0" xyz="0.003 0.0 0.0"/>
-        <geometry>
-          <cylinder length="0.006" radius="0.00035"/>
-        </geometry>
-        <material name="wrist_pitch_frame_x">
-          <color rgba="1.0 0.0 0.0 1.0"/>
-        </material>
-      </visual>
-      <visual>
-        <origin rpy="-${PI_2} 0.0 0.0" xyz="0.0 0.003 0.0"/>
-        <geometry>
-          <cylinder length="0.006" radius="0.00035"/>
-        </geometry>
-        <material name="wrist_pitch_frame_y">
-          <color rgba="0.0 1.0 0.0 1.0"/>
-        </material>
-      </visual>
-      <visual>
-        <origin rpy="0.0 0.0 0.0" xyz="0.0 0.0 0.003"/>
-        <geometry>
-          <cylinder length="0.006" radius="0.00035"/>
-        </geometry>
-        <material name="wrist_pitch_frame_z">
-          <color rgba="0.0 0.0 1.0 1.0"/>
-        </material>
-      </visual>
     </link>
   </xacro:macro>

File: urdf/common/instruments/wrist_pitch/wrist_pitch_0093.urdf.xacro (robot description, xacro)
@@ -17,41 +17,4 @@
         </geometry>
       </visual>
-      <!-- Uncomment this block to show wrist_pitch_link frame triad in RViz -->
-      <visual>
-        <origin rpy="0.0 0.0 0.0" xyz="0.0 0.0 0.0"/>
-        <geometry>
-          <sphere radius="0.0008"/>
-        </geometry>
-        <material name="wrist_pitch_frame_origin">
-          <color rgba="0.0 0.7 1.0 1.0"/>
-        </material>
-      </visual>
-      <visual>
-        <origin rpy="0.0 ${PI_2} 0.0" xyz="0.003 0.0 0.0"/>
-        <geometry>
-          <cylinder length="0.006" radius="0.00035"/>
-        </geometry>
-        <material name="wrist_pitch_frame_x">
-          <color rgba="1.0 0.0 0.0 1.0"/>
-        </material>
-      </visual>
-      <visual>
-        <origin rpy="-${PI_2} 0.0 0.0" xyz="0.0 0.003 0.0"/>
-        <geometry>
-          <cylinder length="0.006" radius="0.00035"/>
-        </geometry>
-        <material name="wrist_pitch_frame_y">
-          <color rgba="0.0 1.0 0.0 1.0"/>
-        </material>
-      </visual>
-      <visual>
-        <origin rpy="0.0 0.0 0.0" xyz="0.0 0.0 0.003"/>
-        <geometry>
-          <cylinder length="0.006" radius="0.00035"/>
-        </geometry>
-        <material name="wrist_pitch_frame_z">
-          <color rgba="0.0 0.0 1.0 1.0"/>
-        </material>
-      </visual>
     </link>
   </xacro:macro>

File: urdf/common/instruments/wrist_pitch/wrist_pitch_0100.urdf.xacro (robot description, xacro)
@@ -17,43 +17,4 @@
         </geometry>
       </visual>
-      <!-- Uncomment this block to show wrist_pitch_link frame triad in RViz -->
-      <!--
-      <visual>
-        <origin rpy="0.0 0.0 0.0" xyz="0.0 0.0 0.0"/>
-        <geometry>
-          <sphere radius="0.0008"/>
-        </geometry>
-        <material name="wrist_pitch_frame_origin">
-          <color rgba="0.0 0.7 1.0 1.0"/>
-        </material>
-      </visual>
-      <visual>
-        <origin rpy="0.0 ${PI_2} 0.0" xyz="0.003 0.0 0.0"/>
-        <geometry>
-          <cylinder length="0.006" radius="0.00035"/>
-        </geometry>
-        <material name="wrist_pitch_frame_x">
-          <color rgba="1.0 0.0 0.0 1.0"/>
-        </material>
-      </visual>
-      <visual>
-        <origin rpy="-${PI_2} 0.0 0.0" xyz="0.0 0.003 0.0"/>
-        <geometry>
-          <cylinder length="0.006" radius="0.00035"/>
-        </geometry>
-        <material name="wrist_pitch_frame_y">
-          <color rgba="0.0 1.0 0.0 1.0"/>
-        </material>
-      </visual>
-      <visual>
-        <origin rpy="0.0 0.0 0.0" xyz="0.0 0.0 0.003"/>
-        <geometry>
-          <cylinder length="0.006" radius="0.00035"/>
-        </geometry>
-        <material name="wrist_pitch_frame_z">
-          <color rgba="0.0 0.0 1.0 1.0"/>
-        </material>
-      </visual>
-      -->
     </link>
   </xacro:macro>

File: urdf/common/instruments/wrist_pitch/wrist_pitch_0107.urdf.xacro (robot description, xacro)
@@ -17,41 +17,4 @@
         </geometry>
       </visual>
-      <!-- Uncomment this block to show wrist_pitch_link frame triad in RViz -->
-      <visual>
-        <origin rpy="0.0 0.0 0.0" xyz="0.0 0.0 0.0"/>
-        <geometry>
-          <sphere radius="0.0008"/>
-        </geometry>
-        <material name="wrist_pitch_frame_origin">
-          <color rgba="0.0 0.7 1.0 1.0"/>
-        </material>
-      </visual>
-      <visual>
-        <origin rpy="0.0 ${PI_2} 0.0" xyz="0.003 0.0 0.0"/>
-        <geometry>
-          <cylinder length="0.006" radius="0.00035"/>
-        </geometry>
-        <material name="wrist_pitch_frame_x">
-          <color rgba="1.0 0.0 0.0 1.0"/>
-        </material>
-      </visual>
-      <visual>
-        <origin rpy="-${PI_2} 0.0 0.0" xyz="0.0 0.003 0.0"/>
-        <geometry>
-          <cylinder length="0.006" radius="0.00035"/>
-        </geometry>
-        <material name="wrist_pitch_frame_y">
-          <color rgba="0.0 1.0 0.0 1.0"/>
-        </material>
-      </visual>
-      <visual>
-        <origin rpy="0.0 0.0 0.0" xyz="0.0 0.0 0.003"/>
-        <geometry>
-          <cylinder length="0.006" radius="0.00035"/>
-        </geometry>
-        <material name="wrist_pitch_frame_z">
-          <color rgba="0.0 0.0 1.0 1.0"/>
-        </material>
-      </visual>
     </link>
   </xacro:macro>

File: urdf/common/instruments/wrist_pitch/wrist_pitch_0112.urdf.xacro (robot description, xacro)
@@ -17,43 +17,4 @@
         </geometry>
       </visual>
-      <!-- Uncomment this block to show wrist_pitch_link frame triad in RViz -->
-<!--
-      <visual>
-        <origin rpy="0.0 0.0 0.0" xyz="0.0 0.0 0.0"/>
-        <geometry>
-          <sphere radius="0.0008"/>
-        </geometry>
-        <material name="wrist_pitch_frame_origin">
-          <color rgba="0.0 0.7 1.0 1.0"/>
-        </material>
-      </visual>
-      <visual>
-        <origin rpy="0.0 ${PI_2} 0.0" xyz="0.003 0.0 0.0"/>
-        <geometry>
-          <cylinder length="0.006" radius="0.00035"/>
-        </geometry>
-        <material name="wrist_pitch_frame_x">
-          <color rgba="1.0 0.0 0.0 1.0"/>
-        </material>
-      </visual>
-      <visual>
-        <origin rpy="-${PI_2} 0.0 0.0" xyz="0.0 0.003 0.0"/>
-        <geometry>
-          <cylinder length="0.006" radius="0.00035"/>
-        </geometry>
-        <material name="wrist_pitch_frame_y">
-          <color rgba="0.0 1.0 0.0 1.0"/>
-        </material>
-      </visual>
-      <visual>
-        <origin rpy="0.0 0.0 0.0" xyz="0.0 0.0 0.003"/>
-        <geometry>
-          <cylinder length="0.006" radius="0.00035"/>
-        </geometry>
-        <material name="wrist_pitch_frame_z">
-          <color rgba="0.0 0.0 1.0 1.0"/>
-        </material>
-      </visual>
-      -->
     </link>
   </xacro:macro>

File: urdf/common/instruments/wrist_yaw/wrist_yaw_0091.urdf.xacro (robot description, xacro)
@@ -17,41 +17,4 @@
         </geometry>
       </visual>
-      <!-- Uncomment this block to show wrist_yaw_link frame triad in RViz -->
-      <visual>
-        <origin rpy="0.0 0.0 0.0" xyz="0.0 0.0 0.0"/>
-        <geometry>
-          <sphere radius="0.0008"/>
-        </geometry>
-        <material name="wrist_yaw_frame_origin">
-          <color rgba="1.0 0.8 0.0 1.0"/>
-        </material>
-      </visual>
-      <visual>
-        <origin rpy="0.0 ${PI_2} 0.0" xyz="0.003 0.0 0.0"/>
-        <geometry>
-          <cylinder length="0.006" radius="0.00035"/>
-        </geometry>
-        <material name="wrist_yaw_frame_x">
-          <color rgba="1.0 0.0 0.0 1.0"/>
-        </material>
-      </visual>
-      <visual>
-        <origin rpy="-${PI_2} 0.0 0.0" xyz="0.0 0.003 0.0"/>
-        <geometry>
-          <cylinder length="0.006" radius="0.00035"/>
-        </geometry>
-        <material name="wrist_yaw_frame_y">
-          <color rgba="0.0 1.0 0.0 1.0"/>
-        </material>
-      </visual>
-      <visual>
-        <origin rpy="0.0 0.0 0.0" xyz="0.0 0.0 0.003"/>
-        <geometry>
-          <cylinder length="0.006" radius="0.00035"/>
-        </geometry>
-        <material name="wrist_yaw_frame_z">
-          <color rgba="0.0 0.0 1.0 1.0"/>
-        </material>
-      </visual>
     </link>
   </xacro:macro>

File: urdf/common/instruments/wrist_yaw/wrist_yaw_0093.urdf.xacro (robot description, xacro)
@@ -17,41 +17,4 @@
         </geometry>
       </visual>
-      <!-- Uncomment this block to show wrist_yaw_link frame triad in RViz -->
-      <visual>
-        <origin rpy="0.0 0.0 0.0" xyz="0.0 0.0 0.0"/>
-        <geometry>
-          <sphere radius="0.0008"/>
-        </geometry>
-        <material name="wrist_yaw_frame_origin">
-          <color rgba="1.0 0.8 0.0 1.0"/>
-        </material>
-      </visual>
-      <visual>
-        <origin rpy="0.0 ${PI_2} 0.0" xyz="0.003 0.0 0.0"/>
-        <geometry>
-          <cylinder length="0.006" radius="0.00035"/>
-        </geometry>
-        <material name="wrist_yaw_frame_x">
-          <color rgba="1.0 0.0 0.0 1.0"/>
-        </material>
-      </visual>
-      <visual>
-        <origin rpy="-${PI_2} 0.0 0.0" xyz="0.0 0.003 0.0"/>
-        <geometry>
-          <cylinder length="0.006" radius="0.00035"/>
-        </geometry>
-        <material name="wrist_yaw_frame_y">
-          <color rgba="0.0 1.0 0.0 1.0"/>
-        </material>
-      </visual>
-      <visual>
-        <origin rpy="0.0 0.0 0.0" xyz="0.0 0.0 0.003"/>
-        <geometry>
-          <cylinder length="0.006" radius="0.00035"/>
-        </geometry>
-        <material name="wrist_yaw_frame_z">
-          <color rgba="0.0 0.0 1.0 1.0"/>
-        </material>
-      </visual>
     </link>
   </xacro:macro>

File: urdf/common/instruments/wrist_yaw/wrist_yaw_0100.urdf.xacro (robot description, xacro)
@@ -17,43 +17,4 @@
         </geometry>
       </visual>
-      <!-- Uncomment this block to show wrist_yaw_link frame triad in RViz -->
-      <!--
-      <visual>
-        <origin rpy="0.0 0.0 0.0" xyz="0.0 0.0 0.0"/>
-        <geometry>
-          <sphere radius="0.0008"/>
-        </geometry>
-        <material name="wrist_yaw_frame_origin">
-          <color rgba="1.0 0.8 0.0 1.0"/>
-        </material>
-      </visual>
-      <visual>
-        <origin rpy="0.0 ${PI_2} 0.0" xyz="0.003 0.0 0.0"/>
-        <geometry>
-          <cylinder length="0.006" radius="0.00035"/>
-        </geometry>
-        <material name="wrist_yaw_frame_x">
-          <color rgba="1.0 0.0 0.0 1.0"/>
-        </material>
-      </visual>
-      <visual>
-        <origin rpy="-${PI_2} 0.0 0.0" xyz="0.0 0.003 0.0"/>
-        <geometry>
-          <cylinder length="0.006" radius="0.00035"/>
-        </geometry>
-        <material name="wrist_yaw_frame_y">
-          <color rgba="0.0 1.0 0.0 1.0"/>
-        </material>
-      </visual>
-      <visual>
-        <origin rpy="0.0 0.0 0.0" xyz="0.0 0.0 0.003"/>
-        <geometry>
-          <cylinder length="0.006" radius="0.00035"/>
-        </geometry>
-        <material name="wrist_yaw_frame_z">
-          <color rgba="0.0 0.0 1.0 1.0"/>
-        </material>
-      </visual>
-      -->
     </link>
   </xacro:macro>

File: urdf/common/instruments/wrist_yaw/wrist_yaw_0107.urdf.xacro (robot description, xacro)
@@ -17,41 +17,4 @@
         </geometry>
       </visual>
-      <!-- Uncomment this block to show wrist_yaw_link frame triad in RViz -->
-      <visual>
-        <origin rpy="0.0 0.0 0.0" xyz="0.0 0.0 0.0"/>
-        <geometry>
-          <sphere radius="0.0008"/>
-        </geometry>
-        <material name="wrist_yaw_frame_origin">
-          <color rgba="1.0 0.8 0.0 1.0"/>
-        </material>
-      </visual>
-      <visual>
-        <origin rpy="0.0 ${PI_2} 0.0" xyz="0.003 0.0 0.0"/>
-        <geometry>
-          <cylinder length="0.006" radius="0.00035"/>
-        </geometry>
-        <material name="wrist_yaw_frame_x">
-          <color rgba="1.0 0.0 0.0 1.0"/>
-        </material>
-      </visual>
-      <visual>
-        <origin rpy="-${PI_2} 0.0 0.0" xyz="0.0 0.003 0.0"/>
-        <geometry>
-          <cylinder length="0.006" radius="0.00035"/>
-        </geometry>
-        <material name="wrist_yaw_frame_y">
-          <color rgba="0.0 1.0 0.0 1.0"/>
-        </material>
-      </visual>
-      <visual>
-        <origin rpy="0.0 0.0 0.0" xyz="0.0 0.0 0.003"/>
-        <geometry>
-          <cylinder length="0.006" radius="0.00035"/>
-        </geometry>
-        <material name="wrist_yaw_frame_z">
-          <color rgba="0.0 0.0 1.0 1.0"/>
-        </material>
-      </visual>
     </link>
   </xacro:macro>

File: urdf/common/instruments/wrist_yaw/wrist_yaw_0112.urdf.xacro (robot description, xacro)
@@ -17,43 +17,4 @@
         </geometry>
       </visual>
-      <!-- Uncomment this block to show wrist_yaw_link frame triad in RViz -->
-<!--
-      <visual>
-        <origin rpy="0.0 0.0 0.0" xyz="0.0 0.0 0.0"/>
-        <geometry>
-          <sphere radius="0.0008"/>
-        </geometry>
-        <material name="wrist_yaw_frame_origin">
-          <color rgba="1.0 0.8 0.0 1.0"/>
-        </material>
-      </visual>
-      <visual>
-        <origin rpy="0.0 ${PI_2} 0.0" xyz="0.003 0.0 0.0"/>
-        <geometry>
-          <cylinder length="0.006" radius="0.00035"/>
-        </geometry>
-        <material name="wrist_yaw_frame_x">
-          <color rgba="1.0 0.0 0.0 1.0"/>
-        </material>
-      </visual>
-      <visual>
-        <origin rpy="-${PI_2} 0.0 0.0" xyz="0.0 0.003 0.0"/>
-        <geometry>
-          <cylinder length="0.006" radius="0.00035"/>
-        </geometry>
-        <material name="wrist_yaw_frame_y">
-          <color rgba="0.0 1.0 0.0 1.0"/>
-        </material>
-      </visual>
-      <visual>
-        <origin rpy="0.0 0.0 0.0" xyz="0.0 0.0 0.003"/>
-        <geometry>
-          <cylinder length="0.006" radius="0.00035"/>
-        </geometry>
-        <material name="wrist_yaw_frame_z">
-          <color rgba="0.0 0.0 1.0 1.0"/>
-        </material>
-      </visual>
-      -->
     </link>
   </xacro:macro>
