Commit message: Fixed 172 tips rotation

File: urdf/common/instruments/tip/tip_172.urdf.xacro (robot description, xacro)
@@ -28,8 +28,8 @@
     <link name="${prefix}jaw_1_link">
       <visual>
-        <origin xyz="0.0 0.0286 0.0" rpy="0 ${PI_2} ${PI}"/>
+        <origin xyz="0.0 0.021 0.0" rpy="0 ${PI_2} ${PI}"/>
         <geometry>
           <mesh filename="package://dvrk_model/meshes/instruments/tip/172/tip_172_1.obj"
-                scale="0.001 0.001 0.001"/>
+                scale="0.1 0.1 0.1"/>
         </geometry>
       </visual>
@@ -45,8 +45,8 @@
     <link name="${prefix}jaw_2_link">
       <visual>
-        <origin xyz="0.0 0.0286 0.0" rpy="0 ${PI_2} ${PI}"/>
+        <origin xyz="0.0 0.021 0.0" rpy="0 ${PI_2} ${PI}"/>
         <geometry>
           <mesh filename="package://dvrk_model/meshes/instruments/tip/172/tip_172_2.obj"
-                scale="0.001 0.001 0.001"/>
+                scale="0.1 0.1 0.1"/>
         </geometry>
       </visual>
@@ -55,5 +55,5 @@
       <parent link="${prefix}wrist_yaw_link"/>
       <child link="${prefix}tool_tip_link"/>
-      <origin xyz="0.0 0.0286 0.0" rpy="0 ${PI_2} ${PI_2}"/>
+      <origin xyz="0.0 0.021 0.0" rpy="0 ${PI_2} ${PI_2}"/>
     </joint>
     <link name="${prefix}tool_tip_link"/>
