Commit message: Fix wrist yaw rotation and jaw placement/hinge rotation direction

File: urdf/common/instruments/tip/tip_093.urdf.xacro (robot description, xacro)
@@ -6,5 +6,5 @@
       <parent link="${prefix}wrist_yaw_link"/>
       <child link="${prefix}jaw_link"/>
-      <axis xyz="0.0 0.0 1"/>
+      <axis xyz="1.0 0.0 0.0"/>
       <origin rpy="0.0 0.0 0.0" xyz="0.0 0.0 0.0"/>
       <limit lower="-0.349066" upper="1.39626" velocity=".4" effort="1000"/>
@@ -19,12 +19,12 @@
       <parent link="${prefix}wrist_yaw_link"/>
       <child link="${prefix}jaw_1_link"/>
-      <axis xyz="0.0 0.0 1"/>
+      <axis xyz="1.0 0.0 0.0"/>
       <origin rpy="0.0 0.0 0.0" xyz="0.0 0.0 0.0"/>
       <limit lower="-1.5707" upper="1.5707" velocity=".4" effort="1000"/>
-      <mimic joint="jaw" multiplier="-0.5"/>
+      <mimic joint="jaw" multiplier="0.5"/>
     </joint>
     <link name="${prefix}jaw_1_link">
       <visual>
-        <origin rpy="0.0 0.0 ${PI}" xyz="0.0 0.0286 0.0"/>
+        <origin rpy="0.0 ${PI_2}  ${PI}" xyz="0.0 0.0286 0.0"/>
         <geometry>
           <mesh filename="package://dvrk_model/meshes/instruments/tip/093/tip_093_1.obj" scale="0.001 0.001 0.001"/>
@@ -35,12 +35,12 @@
       <parent link="${prefix}wrist_yaw_link"/>
       <child link="${prefix}jaw_2_link"/>
-      <axis xyz="0.0 0.0 1"/>
+      <axis xyz="1.0 0.0 0.0"/>
       <origin rpy="0.0 0.0 0.0" xyz="0.0 0.0 0.0"/>
       <limit lower="-1.5707" upper="1.5707" velocity=".4" effort="1000"/>
-      <mimic joint="jaw" multiplier="0.5"/>
+      <mimic joint="jaw" multiplier="-0.5"/>
     </joint>
     <link name="${prefix}jaw_2_link">
       <visual>
-        <origin rpy="0.0 0.0 ${PI}" xyz="0.0 0.0286 0.0"/>
+        <origin rpy="0.0 ${PI_2} ${PI}" xyz="0.0 0.0286 0.0"/>
         <geometry>
           <mesh filename="package://dvrk_model/meshes/instruments/tip/093/tip_093_2.obj" scale="0.001 0.001 0.001"/>

File: urdf/common/instruments/wrist_yaw/wrist_yaw_0167.urdf.xacro (robot description, xacro)
@@ -7,10 +7,10 @@
       <child link="${prefix}wrist_yaw_link"/>
       <axis xyz="0.0 0.0 1"/>
-      <origin rpy="-${PI_2} -${PI_2} 0.0" xyz="0.011565 0.0 0.0"/>
+      <origin rpy="-${PI_2} -${PI_2} 0.0" xyz="0.0110 0.0 0.0"/>
       <limit lower="-1.39626" upper="1.39626" velocity=".4" effort="1000"/>
     </joint>
     <link name="${prefix}wrist_yaw_link">
       <visual>
-        <origin rpy="0.0 0.0 0.0" xyz="0.0 -0.027915 -0.000236"/>
+        <origin rpy="0.0 ${PI_2} 0.0" xyz="0.0 -0.02775 -0.000236"/>
         <geometry>
           <mesh filename="package://dvrk_model/meshes/instruments/wrist_yaw/0167/wrist_yaw_0167.obj" scale="0.1 0.1 0.1"/>

Commit message: fix 0167 wrist pitch and yaw rotation and placement, and 093 tool complete

File: urdf/common/instruments/tip/tip_093.urdf.xacro (robot description, xacro)
@@ -19,5 +19,5 @@
       <parent link="${prefix}wrist_yaw_link"/>
       <child link="${prefix}jaw_1_link"/>
-      <axis xyz="1.0 0.0 0.0"/>
+      <axis xyz="0.0 0.0 -1.0"/>
       <origin rpy="0.0 0.0 0.0" xyz="0.0 0.0 0.0"/>
       <limit lower="-1.5707" upper="1.5707" velocity=".4" effort="1000"/>
@@ -26,5 +26,5 @@
     <link name="${prefix}jaw_1_link">
       <visual>
-        <origin rpy="0.0 ${PI_2}  ${PI}" xyz="0.0 0.0286 0.0"/>
+        <origin rpy="0.0 0.0  ${PI}" xyz="0.0 0.0286 0.0"/>
         <geometry>
           <mesh filename="package://dvrk_model/meshes/instruments/tip/093/tip_093_1.obj" scale="0.001 0.001 0.001"/>
@@ -35,5 +35,5 @@
       <parent link="${prefix}wrist_yaw_link"/>
       <child link="${prefix}jaw_2_link"/>
-      <axis xyz="1.0 0.0 0.0"/>
+      <axis xyz="0.0 0.0 -1.0"/>
       <origin rpy="0.0 0.0 0.0" xyz="0.0 0.0 0.0"/>
       <limit lower="-1.5707" upper="1.5707" velocity=".4" effort="1000"/>
@@ -42,5 +42,5 @@
     <link name="${prefix}jaw_2_link">
       <visual>
-        <origin rpy="0.0 ${PI_2} ${PI}" xyz="0.0 0.0286 0.0"/>
+        <origin rpy="0.0 0.0 ${PI}" xyz="0.0 0.0286 0.0"/>
         <geometry>
           <mesh filename="package://dvrk_model/meshes/instruments/tip/093/tip_093_2.obj" scale="0.001 0.001 0.001"/>

File: urdf/common/instruments/wrist_pitch/wrist_pitch_0167.urdf.xacro (robot description, xacro)
@@ -7,10 +7,10 @@
       <child link="${prefix}wrist_pitch_link"/>
       <axis xyz="0.0 0.0 1"/>
-      <origin rpy="0.0 -${PI_2} 0.0" xyz="0.0 0.0 0.0"/>
+      <origin rpy="-${PI_2} -${PI_2} 0.0" xyz="0.0 0.0 0.0"/>
       <limit lower="-1.2217" upper="1.2217" velocity=".4" effort="1000"/>
     </joint>
     <link name="${prefix}wrist_pitch_link">
       <visual>
-        <origin rpy="0.0 ${PI} ${PI_2}" xyz="0.039 0.0 0.0"/>
+        <origin rpy="0.0 ${PI_2} ${PI_2}" xyz="0.039 0.0 0.0"/>
         <geometry>
           <mesh filename="package://dvrk_model/meshes/instruments/wrist_pitch/0167/wrist_pitch_0167.obj" scale="0.1 0.1 0.1"/>

File: urdf/common/instruments/wrist_yaw/wrist_yaw_0167.urdf.xacro (robot description, xacro)
@@ -12,5 +12,5 @@
     <link name="${prefix}wrist_yaw_link">
       <visual>
-        <origin rpy="0.0 ${PI_2} 0.0" xyz="0.0 -0.02775 -0.000236"/>
+        <origin rpy="${PI} 0.0 ${PI}" xyz="-0.000236 -0.02775 0.0"/>
         <geometry>
           <mesh filename="package://dvrk_model/meshes/instruments/wrist_yaw/0167/wrist_yaw_0167.obj" scale="0.1 0.1 0.1"/>

Commit message: Fix 0167 related 093 and 172 tool tip location and rotation

File: urdf/common/instruments/tip/tip_093.urdf.xacro (robot description, xacro)
@@ -16,36 +16,42 @@
       </visual>
     </link>
-    <joint name="jaw_1" type="revolute">
-      <parent link="${prefix}wrist_yaw_link"/>
-      <child link="${prefix}jaw_1_link"/>
-      <axis xyz="0.0 0.0 -1.0"/>
-      <origin rpy="0.0 0.0 0.0" xyz="0.0 0.0 0.0"/>
-      <limit lower="-1.5707" upper="1.5707" velocity=".4" effort="1000"/>
-      <mimic joint="jaw" multiplier="0.5"/>
-    </joint>
-    <link name="${prefix}jaw_1_link">
-      <visual>
-        <origin rpy="0.0 0.0  ${PI}" xyz="0.0 0.0286 0.0"/>
-        <geometry>
-          <mesh filename="package://dvrk_model/meshes/instruments/tip/093/tip_093_1.obj" scale="0.001 0.001 0.001"/>
-        </geometry>
-      </visual>
-    </link>
-    <joint name="jaw_2" type="revolute">
-      <parent link="${prefix}wrist_yaw_link"/>
-      <child link="${prefix}jaw_2_link"/>
-      <axis xyz="0.0 0.0 -1.0"/>
-      <origin rpy="0.0 0.0 0.0" xyz="0.0 0.0 0.0"/>
-      <limit lower="-1.5707" upper="1.5707" velocity=".4" effort="1000"/>
-      <mimic joint="jaw" multiplier="-0.5"/>
-    </joint>
-    <link name="${prefix}jaw_2_link">
-      <visual>
-        <origin rpy="0.0 0.0 ${PI}" xyz="0.0 0.0286 0.0"/>
-        <geometry>
-          <mesh filename="package://dvrk_model/meshes/instruments/tip/093/tip_093_2.obj" scale="0.001 0.001 0.001"/>
-        </geometry>
-      </visual>
-    </link>
+  <joint name="jaw_1" type="revolute">
+    <parent link="${prefix}wrist_yaw_link"/>
+    <child link="${prefix}jaw_1_link"/>
+    <axis xyz="0.0 0.0 -1.0"/>
+    <origin xyz="0 0 0" rpy="0 0 0"/>
+    <limit lower="-1.5707" upper="1.5707" velocity=".4" effort="1000"/>
+    <mimic joint="jaw" multiplier="0.5"/>
+  </joint>
+  <link name="${prefix}jaw_1_link">
+    <visual>
+      <origin
+        xyz="0.0 0.021 0.0" rpy="0 0 ${PI}"/>
+      <geometry>
+        <mesh
+          filename="package://dvrk_model/meshes/instruments/tip/172/tip_172_1.obj"
+          scale="0.1 0.1 0.1"/>
+      </geometry>
+    </visual>
+  </link>
+  <joint name="jaw_2" type="revolute">
+    <parent link="${prefix}wrist_yaw_link"/>
+    <child link="${prefix}jaw_2_link"/>
+    <axis xyz="0.0 0.0 -1.0"/>
+    <origin xyz="0 0 0" rpy="0 0 0"/>
+    <limit lower="-1.5707" upper="1.5707" velocity=".4" effort="1000"/>
+    <mimic joint="jaw" multiplier="-0.5"/>
+  </joint>
+  <link name="${prefix}jaw_2_link">
+    <visual>
+      <origin
+        xyz="0.0 0.021 0.0" rpy="0 0 ${PI}"/>
+      <geometry>
+        <mesh
+          filename="package://dvrk_model/meshes/instruments/tip/172/tip_172_2.obj"
+          scale="0.1 0.1 0.1"/>
+      </geometry>
+    </visual>
+  </link>
     <joint name="tool_tip" type="fixed">
       <parent link="${prefix}wrist_yaw_link"/>

File: urdf/common/instruments/tip/tip_172.urdf.xacro (robot description, xacro)
@@ -21,5 +21,5 @@
       <parent link="${prefix}wrist_yaw_link"/>
       <child link="${prefix}jaw_1_link"/>
-      <axis xyz="1.0 0.0 0.0"/>
+      <axis xyz="0.0 0.0 1.0"/>
       <origin xyz="0 0 0" rpy="0 0 0"/>
       <limit lower="-1.5707" upper="1.5707" velocity=".4" effort="1000"/>
@@ -28,5 +28,5 @@
     <link name="${prefix}jaw_1_link">
       <visual>
-        <origin xyz="0.0 0.021 0.0" rpy="0 ${PI_2} ${PI}"/>
+        <origin xyz="0.0 0.021 0.0" rpy="0 ${PI} ${PI}"/>
         <geometry>
           <mesh filename="package://dvrk_model/meshes/instruments/tip/172/tip_172_1.obj"
@@ -38,5 +38,5 @@
       <parent link="${prefix}wrist_yaw_link"/>
       <child link="${prefix}jaw_2_link"/>
-      <axis xyz="1.0 0.0 0.0"/>
+      <axis xyz="0.0 0.0 1.0"/>
       <origin xyz="0 0 0" rpy="0 0 0"/>
       <limit lower="-1.5707" upper="1.5707" velocity=".4" effort="1000"/>
@@ -45,5 +45,5 @@
     <link name="${prefix}jaw_2_link">
       <visual>
-        <origin xyz="0.0 0.021 0.0" rpy="0 ${PI_2} ${PI}"/>
+        <origin xyz="0.0 0.021 0.0" rpy="0 ${PI} ${PI}"/>
         <geometry>
           <mesh filename="package://dvrk_model/meshes/instruments/tip/172/tip_172_2.obj"

Commit message: Refactor tip_093 URDF: update jaw joint configuration and mesh references

File: urdf/common/instruments/tip/tip_093.urdf.xacro (robot description, xacro)
@@ -3,10 +3,28 @@
   <xacro:include filename="$(find dvrk_model)/urdf/common.urdf.xacro"/>
   <xacro:macro name="tip_093" params="prefix">
+    <!--
+      The ProGrasp jaw hinge is offset from wrist_yaw and this offset changes
+      as the jaw opens.  URDF mimic joints are affine, so approximate the
+      measured 7.7 mm (closed) to 5.5 mm (60 degree open) relationship with
+      a prismatic joint along the wrist-yaw Y axis:
+        distance = 0.0077 - (0.0022 / 1.0472) * jaw
+      Keep jaw as the single actuated joint; jaw_axis, jaw_1 and jaw_2 are
+      dependent joints.
+    -->
+    <joint name="jaw_axis" type="prismatic">
+      <parent link="${prefix}wrist_yaw_link"/>
+      <child link="${prefix}jaw_axis_link"/>
+      <axis xyz="0.0 1.0 0.0"/>
+      <origin rpy="0.0 0.0 0.0" xyz="0.0 0.0 0.0"/>
+      <limit lower="0.0055" upper="0.0077" velocity="0.001" effort="1000"/>
+      <mimic joint="jaw" multiplier="-0.002100845" offset="0.0077"/>
+    </joint>
+    <link name="${prefix}jaw_axis_link"/>
     <joint name="jaw" type="revolute">
-      <parent link="${prefix}wrist_yaw_link"/>
+      <parent link="${prefix}jaw_axis_link"/>
       <child link="${prefix}jaw_link"/>
       <axis xyz="1.0 0.0 0.0"/>
       <origin rpy="0.0 0.0 0.0" xyz="0.0 0.0 0.0"/>
-      <limit lower="-0.349066" upper="1.39626" velocity=".4" effort="1000"/>
+      <limit lower="0.0" upper="1.0472" velocity=".4" effort="1000"/>
     </joint>
     <link name="${prefix}jaw_link">
@@ -17,5 +35,6 @@
     </link>
   <joint name="jaw_1" type="revolute">
-    <parent link="${prefix}wrist_yaw_link"/>
+    <!-- Keep the tip hinge axes independent of the jaw-link rotation. -->
+    <parent link="${prefix}jaw_axis_link"/>
     <child link="${prefix}jaw_1_link"/>
     <axis xyz="0.0 0.0 -1.0"/>
@@ -30,11 +49,11 @@
       <geometry>
         <mesh
-          filename="package://dvrk_model/meshes/instruments/tip/172/tip_172_1.obj"
-          scale="0.1 0.1 0.1"/>
+          filename="package://dvrk_model/meshes/instruments/tip/093/tip_093_1.obj"
+          scale="0.001 0.001 0.001"/>
       </geometry>
     </visual>
   </link>
   <joint name="jaw_2" type="revolute">
-    <parent link="${prefix}wrist_yaw_link"/>
+    <parent link="${prefix}jaw_axis_link"/>
     <child link="${prefix}jaw_2_link"/>
     <axis xyz="0.0 0.0 -1.0"/>
@@ -49,6 +68,6 @@
       <geometry>
         <mesh
-          filename="package://dvrk_model/meshes/instruments/tip/172/tip_172_2.obj"
-          scale="0.1 0.1 0.1"/>
+          filename="package://dvrk_model/meshes/instruments/tip/093/tip_093_2.obj"
+          scale="0.001 0.001 0.001"/>
       </geometry>
     </visual>
