Commit message: Updated 194 instrument tool tip position

File: urdf/common/instruments/tip/tip_194.urdf.xacro (robot description, xacro)
@@ -28,5 +28,5 @@
     <link name="${prefix}jaw_1_link">
       <visual>
-        <origin rpy="0.0 0.0 ${PI}" xyz="0.0 0.0108 0.0"/>
+        <origin rpy="0.0 0.0 ${PI}" xyz="0.0 0.0127 0.0"/>
         <geometry>
           <mesh filename="package://dvrk_model/meshes/instruments/tip/194/tip_194_1.obj" scale="0.1 0.1 0.1"/>
@@ -44,5 +44,5 @@
     <link name="${prefix}jaw_2_link">
       <visual>
-        <origin rpy="0.0 0.0 ${PI}" xyz="0.0 0.0108 0.0"/>
+        <origin rpy="0.0 0.0 ${PI}" xyz="0.0 0.0127 0.0"/>
         <geometry>
           <mesh filename="package://dvrk_model/meshes/instruments/tip/194/tip_194_2.obj" scale="0.1 0.1 0.1"/>

File: urdf/common/instruments/wrist_pitch/wrist_pitch_0112.urdf.xacro (robot description, xacro)
@@ -18,5 +18,5 @@
       </visual>
       <!-- Uncomment this block to show wrist_pitch_link frame triad in RViz -->
-      <!--
+<!--
       <visual>
         <origin rpy="0.0 0.0 0.0" xyz="0.0 0.0 0.0"/>

File: urdf/common/instruments/wrist_yaw/wrist_yaw_0112.urdf.xacro (robot description, xacro)
@@ -18,5 +18,5 @@
       </visual>
       <!-- Uncomment this block to show wrist_yaw_link frame triad in RViz -->
-      <!--
+<!--
       <visual>
         <origin rpy="0.0 0.0 0.0" xyz="0.0 0.0 0.0"/>
