Commit message: Update yaw and tip position for 183

File: urdf/common/instruments/tip/tip_183.urdf.xacro (robot description, xacro)
@@ -7,10 +7,10 @@
       <child link="${prefix}jaw_link"/>
       <axis xyz="0.0 0.0 1.0"/>
-      <origin rpy="0.0 0.0 0.0" xyz="0.0 0.0 0.0"/>
+      <origin rpy="0.0 0.0 0.0" xyz="0.0 0.0038 0.0"/>
       <limit lower="0.0" upper="0.5" velocity=".4" effort="1000"/>
     </joint>
     <link name="${prefix}jaw_link">
       <visual>
-        <origin rpy="0.0 0.0 ${PI}" xyz="0.0 0.0 0.0"/>
+        <origin rpy="0.0 ${PI} ${PI}" xyz="0.0 0.0122768 -0.00015"/>
         <geometry>
           <mesh filename="package://dvrk_model/meshes/instruments/tip/183/tip_183.obj" scale="0.1 0.1 0.1"/>
@@ -21,5 +21,5 @@
       <parent link="${prefix}wrist_yaw_link"/>
       <child link="${prefix}tool_tip_link"/>
-      <origin rpy="0.0 ${PI_2} ${PI_2}" xyz="0.0 0.0123 0.0"/>
+      <origin rpy="0.0 ${PI_2} ${PI_2}" xyz="0.0 0.0160768 0.0"/>
     </joint>
     <link name="${prefix}tool_tip_link"/>

File: urdf/common/instruments/wrist_pitch/wrist_pitch_0093.urdf.xacro (robot description, xacro)
@@ -12,5 +12,5 @@
     <link name="${prefix}wrist_pitch_link">
       <visual>
-        <origin rpy="0.0 ${PI_2} ${PI_2}" xyz="0.039 -0.013864 0.0"/>
+        <origin rpy="0.0 ${PI_2} ${PI_2}" xyz="0.027066 0.0 0.0"/>
         <geometry>
           <mesh filename="package://dvrk_model/meshes/instruments/wrist_pitch/0093/wrist_pitch_0093.obj" scale="0.1 0.1 0.1"/>
@@ -18,5 +18,4 @@
       </visual>
       <!-- Uncomment this block to show wrist_pitch_link frame triad in RViz -->
-      <!--
       <visual>
         <origin rpy="0.0 0.0 0.0" xyz="0.0 0.0 0.0"/>
@@ -55,5 +54,4 @@
         </material>
       </visual>
-      -->
     </link>
   </xacro:macro>

File: urdf/common/instruments/wrist_yaw/wrist_yaw_0093.urdf.xacro (robot description, xacro)
@@ -12,5 +12,5 @@
     <link name="${prefix}wrist_yaw_link">
       <visual>
-        <origin rpy="${PI} 0.0 ${PI}" xyz="-0.000236 -0.013385 0.0"/>
+        <origin rpy="0.0 ${PI} ${PI}" xyz="-0.000236 0.017089 0.0"/>
         <geometry>
           <mesh filename="package://dvrk_model/meshes/instruments/wrist_yaw/0093/wrist_yaw_0093.obj" scale="0.1 0.1 0.1"/>
@@ -18,5 +18,4 @@
       </visual>
       <!-- Uncomment this block to show wrist_yaw_link frame triad in RViz -->
-      <!--
       <visual>
         <origin rpy="0.0 0.0 0.0" xyz="0.0 0.0 0.0"/>
@@ -55,5 +54,4 @@
         </material>
       </visual>
-      -->
     </link>
   </xacro:macro>

Commit message: Constrain 183 and 184 jaw motion to yaw link

File: urdf/common/instruments/tip/tip_183.urdf.xacro (robot description, xacro)
@@ -3,10 +3,8 @@
   <xacro:include filename="$(find dvrk_model)/urdf/common.urdf.xacro"/>
   <xacro:macro name="tip_183" params="prefix">
-    <joint name="jaw" type="revolute">
+    <joint name="jaw" type="fixed">
       <parent link="${prefix}wrist_yaw_link"/>
       <child link="${prefix}jaw_link"/>
-      <axis xyz="0.0 0.0 1.0"/>
       <origin rpy="0.0 0.0 0.0" xyz="0.0 0.0038 0.0"/>
-      <limit lower="0.0" upper="0.5" velocity=".4" effort="1000"/>
     </joint>
     <link name="${prefix}jaw_link">

File: urdf/common/instruments/tip/tip_184.urdf.xacro (robot description, xacro)
@@ -3,14 +3,12 @@
   <xacro:include filename="$(find dvrk_model)/urdf/common.urdf.xacro"/>
   <xacro:macro name="tip_184" params="prefix">
-    <joint name="jaw" type="revolute">
+    <joint name="jaw" type="fixed">
       <parent link="${prefix}wrist_yaw_link"/>
       <child link="${prefix}jaw_link"/>
-      <axis xyz="0.0 0.0 1.0"/>
-      <origin rpy="0.0 0.0 0.0" xyz="0.0 0.0 0.0"/>
-      <limit lower="0.0" upper="0.5" velocity=".4" effort="1000"/>
+      <origin rpy="0.0 0.0 0.0" xyz="0.0 0.0038 0.0"/>
     </joint>
     <link name="${prefix}jaw_link">
       <visual>
-        <origin rpy="0.0 0.0 ${PI}" xyz="0.0 0.0 0.0"/>
+        <origin rpy="0.0 ${PI} ${PI}" xyz="0.0 0.0122768 -0.00015"/>
         <geometry>
           <mesh filename="package://dvrk_model/meshes/instruments/tip/184/tip_184.obj" scale="0.1 0.1 0.1"/>
@@ -21,5 +19,5 @@
       <parent link="${prefix}wrist_yaw_link"/>
       <child link="${prefix}tool_tip_link"/>
-      <origin rpy="0.0 ${PI_2} ${PI_2}" xyz="0.0 0.0136 0.0"/>
+      <origin rpy="0.0 ${PI_2} ${PI_2}" xyz="0.0 0.0160768 0.0"/>
     </joint>
     <link name="${prefix}tool_tip_link"/>

Commit message: Updated yaw and tip 183 and 184 with pin and separated gears/tip

File: urdf/common/instruments/tip/tip_183.urdf.xacro (robot description, xacro)
@@ -6,9 +6,9 @@
       <parent link="${prefix}wrist_yaw_link"/>
       <child link="${prefix}jaw_link"/>
-      <origin rpy="0.0 0.0 0.0" xyz="0.0 0.0038 0.0"/>
+      <origin rpy="0.0 0.0 0.0" xyz="0.0 0.0 0.0"/>
     </joint>
     <link name="${prefix}jaw_link">
       <visual>
-        <origin rpy="0.0 ${PI} ${PI}" xyz="0.0 0.0122768 -0.00015"/>
+        <origin rpy="0.0 0.0 ${PI}" xyz="0.0 0.0160768 -0.00015"/>
         <geometry>
           <mesh filename="package://dvrk_model/meshes/instruments/tip/183/tip_183.obj" scale="0.1 0.1 0.1"/>

File: urdf/common/instruments/tip/tip_184.urdf.xacro (robot description, xacro)
@@ -6,9 +6,9 @@
       <parent link="${prefix}wrist_yaw_link"/>
       <child link="${prefix}jaw_link"/>
-      <origin rpy="0.0 0.0 0.0" xyz="0.0 0.0038 0.0"/>
+      <origin rpy="0.0 0.0 0.0" xyz="0.0 0.0 0.0"/>
     </joint>
     <link name="${prefix}jaw_link">
       <visual>
-        <origin rpy="0.0 ${PI} ${PI}" xyz="0.0 0.0122768 -0.00015"/>
+        <origin rpy="0.0 0.0 ${PI}" xyz="0.0 0.0160768 -0.00015"/>
         <geometry>
           <mesh filename="package://dvrk_model/meshes/instruments/tip/184/tip_184.obj" scale="0.1 0.1 0.1"/>

File: urdf/common/instruments/wrist_pitch/wrist_pitch_0093.urdf.xacro (robot description, xacro)
@@ -12,5 +12,5 @@
     <link name="${prefix}wrist_pitch_link">
       <visual>
-        <origin rpy="0.0 ${PI_2} ${PI_2}" xyz="0.027066 0.0 0.0"/>
+        <origin rpy="0.0 ${PI_2} ${PI_2}" xyz="0.026801 0.0 0.0"/>
         <geometry>
           <mesh filename="package://dvrk_model/meshes/instruments/wrist_pitch/0093/wrist_pitch_0093.obj" scale="0.1 0.1 0.1"/>

File: urdf/common/instruments/wrist_yaw/wrist_yaw_0093.urdf.xacro (robot description, xacro)
@@ -12,5 +12,5 @@
     <link name="${prefix}wrist_yaw_link">
       <visual>
-        <origin rpy="0.0 ${PI} ${PI}" xyz="-0.000236 0.017089 0.0"/>
+        <origin rpy="0.0 ${PI} ${PI}" xyz="0.0 0.0175 0.0"/>
         <geometry>
           <mesh filename="package://dvrk_model/meshes/instruments/wrist_yaw/0093/wrist_yaw_0093.obj" scale="0.1 0.1 0.1"/>
