Commit message: Complete tip 179 mesh placement

File: urdf/common/instruments/tip/tip_006.urdf.xacro (robot description, xacro)
@@ -20,5 +20,5 @@
       <child link="${prefix}jaw_1_link"/>
       <axis xyz="0.0 0.0 1"/>
-      <origin rpy="0.0 0.0 0.0" xyz="0.0 0.0 0.0"/>
+      <origin rpy="0.0 0.0 0.0" xyz="0.0 -0.01305 0.0"/>
       <limit lower="-1.5707" upper="1.5707" velocity=".4" effort="1000"/>
       <mimic joint="jaw" multiplier="0.5"/>
@@ -26,5 +26,5 @@
     <link name="${prefix}jaw_1_link">
       <visual>
-        <origin rpy="0.0 0.0 0.0" xyz="0.0 0.0 0.0"/>
+        <origin rpy="0.0 0.0 0.0" xyz="0.0 -0.01305 0.0"/>
         <geometry>
           <mesh filename="package://dvrk_model/meshes/instruments/tip/006/tip_006_1.obj"/>

File: urdf/common/instruments/tip/tip_179.urdf.xacro (robot description, xacro)
@@ -26,5 +26,8 @@
     <link name="${prefix}jaw_1_link">
       <visual>
-        <origin rpy="0.0 0.0 0.0" xyz="0.0 0.0 0.0"/>
+        <!-- Rotate tip 180 degrees about world Y (local Z) and shift hinge -->
+        <origin
+          rpy="0.0 0.0 ${PI}"
+          xyz="0.0 0.01305 0.0"/>
         <geometry>
           <mesh filename="package://dvrk_model/meshes/instruments/tip/179/tip_179_1.obj" scale="0.001 0.001 0.001"/>
@@ -42,5 +45,8 @@
     <link name="${prefix}jaw_2_link">
       <visual>
-        <origin rpy="0.0 0.0 0.0" xyz="0.0 0.0 0.0"/>
+        <!-- Rotate mirrored jaw 180 degrees about world Y (local Z) -->
+        <origin
+          rpy="0.0 0.0 ${PI}"
+          xyz="0.0 0.01305 0.0"/>
         <geometry>
           <mesh filename="package://dvrk_model/meshes/instruments/tip/179/tip_179_2.obj" scale="0.001 0.001 0.001"/>
@@ -51,5 +57,5 @@
       <parent link="${prefix}wrist_yaw_link"/>
       <child link="${prefix}tool_tip_link"/>
-      <origin rpy="0.0 ${PI_2} ${PI_2}" xyz="0.0 0.0155 0.0"/>
+      <origin rpy="0.0 ${PI_2} ${PI_2}" xyz="0.0 0.0155 -0.0016"/>
     </joint>
     <link name="${prefix}tool_tip_link"/>

Commit message: Fix change in 006 from editing the 179

File: urdf/common/instruments/tip/tip_006.urdf.xacro (robot description, xacro)
@@ -20,5 +20,5 @@
       <child link="${prefix}jaw_1_link"/>
       <axis xyz="0.0 0.0 1"/>
-      <origin rpy="0.0 0.0 0.0" xyz="0.0 -0.01305 0.0"/>
+      <origin rpy="0.0 0.0 0.0" xyz="0.0 0 0.0"/>
       <limit lower="-1.5707" upper="1.5707" velocity=".4" effort="1000"/>
       <mimic joint="jaw" multiplier="0.5"/>
@@ -26,5 +26,5 @@
     <link name="${prefix}jaw_1_link">
       <visual>
-        <origin rpy="0.0 0.0 0.0" xyz="0.0 -0.01305 0.0"/>
+        <origin rpy="0.0 0.0 0.0" xyz="0.0 0.0 0.0"/>
         <geometry>
           <mesh filename="package://dvrk_model/meshes/instruments/tip/006/tip_006_1.obj"/>

Commit message: Phase 1 detailed visual meshes used as collision meshes as proof of pipeline

File: urdf/common/instruments/tip/tip_006.urdf.xacro (robot description, xacro)
@@ -31,4 +31,10 @@
         </geometry>
       </visual>
+      <collision>
+        <origin rpy="0.0 0.0 0.0" xyz="0.0 0.0 0.0"/>
+        <geometry>
+          <mesh filename="package://dvrk_model/meshes/instruments/tip/006/tip_006_1.obj"/>
+        </geometry>
+      </collision>
     </link>
     <joint name="jaw_2" type="revolute">
@@ -47,4 +53,10 @@
         </geometry>
       </visual>
+      <collision>
+        <origin rpy="0.0 0.0 0.0" xyz="0.0 0.0 0.0"/>
+        <geometry>
+          <mesh filename="package://dvrk_model/meshes/instruments/tip/006/tip_006_2.obj"/>
+        </geometry>
+      </collision>
     </link>
     <joint name="tool_tip" type="fixed">

File: urdf/common/instruments/wrist_pitch/wrist_pitch_0091.urdf.xacro (robot description, xacro)
@@ -17,4 +17,10 @@
         </geometry>
       </visual>
+      <collision>
+        <origin rpy="0.0 ${PI_2} ${PI_2}" xyz="0.0295 0.0 0.0"/>
+        <geometry>
+          <mesh filename="package://dvrk_model/meshes/instruments/wrist_pitch/0091/wrist_pitch_0091.obj" scale="0.1 0.1 0.1"/>
+        </geometry>
+      </collision>
     </link>
   </xacro:macro>

File: urdf/common/instruments/wrist_yaw/wrist_yaw_0091.urdf.xacro (robot description, xacro)
@@ -17,4 +17,10 @@
         </geometry>
       </visual>
+      <collision>
+        <origin rpy="0.0 0.0 0.0" xyz="0.0 0.0 -0.000236"/>
+        <geometry>
+          <mesh filename="package://dvrk_model/meshes/instruments/wrist_yaw/0091/wrist_yaw_0091.obj"/>
+        </geometry>
+      </collision>
     </link>
   </xacro:macro>
