Commit message: added simple collision mesh for yaw 0091

File: urdf/common/instruments/wrist_yaw/wrist_yaw_0091.urdf.xacro (robot description, xacro)
@@ -17,4 +17,10 @@
         </geometry>
       </visual>
+      <collision>
+        <origin rpy="0.0 0.0 0.0" xyz="0.0 0.0 -0.000236"/>
+        <geometry>
+          <cylinder radius="0.005" length="0.010"/>
+        </geometry>
+      </collision>
     </link>
   </xacro:macro>
