Commit message: Update URDF models for housing and roll instruments
- Changed the mesh file for the housing_Classic instrument from housing_Classic.dae to housing_Classic_body.dae in both visual and collision elements.
- Updated the roll_4162 instrument to use roll_4670.obj instead of roll_4162.dae, adjusted the origin parameters, and modified the material name accordingly.

File: urdf/common/instruments/housing/housing_Classic.urdf.xacro (robot description, xacro)
@@ -12,5 +12,5 @@
         <origin rpy="0.0 0.0 ${PI_2}" xyz="0.0 0.0 0.0904"/>
         <geometry>
-          <mesh filename="package://dvrk_model/meshes/instruments/housing/Classic/housing_Classic.dae"/>
+          <mesh filename="package://dvrk_model/meshes/instruments/housing/Classic/housing_Classic_body.dae"/>
         </geometry>
       </visual>
@@ -18,5 +18,5 @@
         <origin rpy="0.0 0.0 ${PI_2}" xyz="0.0 0.0 0.0904"/>
         <geometry>
-          <mesh filename="package://dvrk_model/meshes/instruments/housing/Classic/housing_Classic.dae"/>
+          <mesh filename="package://dvrk_model/meshes/instruments/housing/Classic/housing_Classic_body.dae"/>
         </geometry>
       </collision>

File: urdf/common/instruments/roll/roll_4162.urdf.xacro (robot description, xacro)
@@ -12,14 +12,14 @@
     <link name="${prefix}roll_link">
       <visual>
-        <origin rpy="0.0 0.0 1.5708" xyz="0.0 0.0 -0.0091"/>
+        <origin rpy="-${PI_2} 0.0 ${PI_2}" xyz="0.0 0.0 0.02975"/>
         <geometry>
-          <mesh filename="package://dvrk_model/meshes/instruments/roll/4162/roll_4162.dae"/>
+          <mesh filename="package://dvrk_model/meshes/instruments/roll/4670/roll_4670.obj" scale="0.1 0.1 0.1"/>
         </geometry>
-        <material name="roll_4162_shaft"><color rgba="0.55 0.55 0.55 1"/></material>
+        <material name="roll_4670_shaft"><color rgba="0.55 0.55 0.55 1"/></material>
       </visual>
       <collision>
-        <origin rpy="0.0 0.0 1.5708" xyz="0.0 0.0 -0.0091"/>
+        <origin rpy="-${PI_2} 0.0 0.0" xyz="0.0 0.0 0.02975"/>
         <geometry>
-          <mesh filename="package://dvrk_model/meshes/instruments/roll/4162/roll_4162.dae"/>
+          <mesh filename="package://dvrk_model/meshes/instruments/roll/4670/roll_4670.obj" scale="0.1 0.1 0.1"/>
         </geometry>
       </collision>
