Commit message: Updatred  meshes restructure

File: urdf/common/instruments/roll/roll_4670.urdf.xacro (robot description, xacro)
@@ -12,14 +12,14 @@
     <link name="${prefix}roll_link">
       <visual>
-        <origin rpy="0.0 0.0 0.0" xyz="0.0 0.0 -0.216"/>
+        <origin rpy="-${PI_2} 0.0 0.0" xyz="0.0 0.0 0.0734"/>
         <geometry>
-          <mesh filename="package://dvrk_model/meshes/instruments/roll/4670/roll_4670.obj"/>
+          <mesh filename="package://dvrk_model/meshes/instruments/roll/4670/roll_4670.obj" scale="0.1 0.1 0.1"/>
         </geometry>
         <material name="roll_4670_shaft"><color rgba="0.55 0.55 0.55 1"/></material>
       </visual>
       <collision>
-        <origin rpy="0.0 0.0 0.0" xyz="0.0 0.0 -0.216"/>
+        <origin rpy="-${PI_2} 0.0 0.0" xyz="0.0 0.0 0.0734"/>
         <geometry>
-          <mesh filename="package://dvrk_model/meshes/instruments/roll/4670/roll_4670.obj"/>
+          <mesh filename="package://dvrk_model/meshes/instruments/roll/4670/roll_4670.obj" scale="0.1 0.1 0.1"/>
         </geometry>
       </collision>

Commit message: Updated Si roll 4670 position to match dh parameters

File: urdf/common/instruments/roll/roll_4670.urdf.xacro (robot description, xacro)
@@ -12,5 +12,5 @@
     <link name="${prefix}roll_link">
       <visual>
-        <origin rpy="-${PI_2} 0.0 0.0" xyz="0.0 0.0 0.0734"/>
+        <origin rpy="-${PI_2} 0.0 ${PI_2}" xyz="0.0 0.0 0.02975"/>
         <geometry>
           <mesh filename="package://dvrk_model/meshes/instruments/roll/4670/roll_4670.obj" scale="0.1 0.1 0.1"/>
@@ -19,5 +19,5 @@
       </visual>
       <collision>
-        <origin rpy="-${PI_2} 0.0 0.0" xyz="0.0 0.0 0.0734"/>
+        <origin rpy="-${PI_2} 0.0 0.0" xyz="0.0 0.0 0.02975"/>
         <geometry>
           <mesh filename="package://dvrk_model/meshes/instruments/roll/4670/roll_4670.obj" scale="0.1 0.1 0.1"/>

File: urdf/common/instruments/wrist_pitch/wrist_pitch_0091.urdf.xacro (robot description, xacro)
@@ -12,7 +12,7 @@
     <link name="${prefix}wrist_pitch_link">
       <visual>
-        <origin rpy="0.0 0.0 0.0" xyz="0.0 0.0 0.0"/>
+        <origin rpy="0.0 ${PI_2} ${PI_2}" xyz="0.039 0.0 0.0"/>
         <geometry>
-          <mesh filename="package://dvrk_model/meshes/instruments/wrist_pitch/0091/wrist_pitch_0091.obj"/>
+          <mesh filename="package://dvrk_model/meshes/instruments/wrist_pitch/0091/wrist_pitch_0091.obj" scale="0.1 0.1 0.1"/>
         </geometry>
       </visual>
@@ -20,5 +20,5 @@
       <!--
       <visual>
-        <origin rpy="0.0 0.0 0.0" xyz="0.0 0.0 0.0"/>
+        <origin rpy="0.0 ${PI_2} ${PI_2}" xyz="0.039 0.0 0.0"/>
         <geometry>
           <sphere radius="0.0008"/>

File: urdf/common/instruments/wrist_pitch/wrist_pitch_0107.urdf.xacro (robot description, xacro)
@@ -18,5 +18,4 @@
       </visual>
       <!-- Uncomment this block to show wrist_pitch_link frame triad in RViz -->
-      <!--
       <visual>
         <origin rpy="0.0 0.0 0.0" xyz="0.0 0.0 0.0"/>
@@ -55,5 +54,4 @@
         </material>
       </visual>
-      -->
     </link>
   </xacro:macro>

Commit message: First implementation of collision meshes for 006

File: urdf/common/instruments/roll/roll_4670.urdf.xacro (robot description, xacro)
@@ -21,5 +21,5 @@
         <origin rpy="-${PI_2} 0.0 0.0" xyz="0.0 0.0 0.02975"/>
         <geometry>
-          <mesh filename="package://dvrk_model/meshes/instruments/roll/4670/roll_4670.obj" scale="0.1 0.1 0.1"/>
+          <mesh filename="package://dvrk_model/meshes/instruments/roll/4670/roll_4670_collision.obj" scale="0.1 0.1 0.1"/>
         </geometry>
       </collision>

File: urdf/common/instruments/tip/tip_006.urdf.xacro (robot description, xacro)
@@ -34,5 +34,5 @@
         <origin rpy="0.0 0.0 0.0" xyz="0.0 0.0 0.0"/>
         <geometry>
-          <mesh filename="package://dvrk_model/meshes/instruments/tip/006/tip_006_1.obj"/>
+          <mesh filename="package://dvrk_model/meshes/instruments/tip/006/tip_006_1_collision.obj"/>
         </geometry>
       </collision>
@@ -56,5 +56,5 @@
         <origin rpy="0.0 0.0 0.0" xyz="0.0 0.0 0.0"/>
         <geometry>
-          <mesh filename="package://dvrk_model/meshes/instruments/tip/006/tip_006_2.obj"/>
+          <mesh filename="package://dvrk_model/meshes/instruments/tip/006/tip_006_2_collision.obj"/>
         </geometry>
       </collision>

File: urdf/common/instruments/wrist_pitch/wrist_pitch_0091.urdf.xacro (robot description, xacro)
@@ -20,5 +20,5 @@
         <origin rpy="0.0 ${PI_2} ${PI_2}" xyz="0.0295 0.0 0.0"/>
         <geometry>
-          <mesh filename="package://dvrk_model/meshes/instruments/wrist_pitch/0091/wrist_pitch_0091.obj" scale="0.1 0.1 0.1"/>
+          <mesh filename="package://dvrk_model/meshes/instruments/wrist_pitch/0091/wrist_pitch_0091_collision.obj" scale="0.1 0.1 0.1"/>
         </geometry>
       </collision>

File: urdf/common/instruments/wrist_yaw/wrist_yaw_0091.urdf.xacro (robot description, xacro)
@@ -17,10 +17,4 @@
         </geometry>
       </visual>
-      <collision>
-        <origin rpy="0.0 0.0 0.0" xyz="0.0 0.0 -0.000236"/>
-        <geometry>
-          <mesh filename="package://dvrk_model/meshes/instruments/wrist_yaw/0091/wrist_yaw_0091.obj"/>
-        </geometry>
-      </collision>
     </link>
   </xacro:macro>
