Commit message: remove unnecessary components in roll

File: urdf/common/instruments/roll/roll_4162.urdf.xacro (robot description, xacro)
@@ -23,16 +23,4 @@
         </geometry>
       </collision>
-      <visual>
-        <origin rpy="${PI_2} 0.0 0.0" xyz="0.0 0.00401 0.0"/>
-        <geometry>
-          <mesh filename="package://dvrk_model/meshes/instruments/roll/4162/roll_4162_yaw.dae"/>
-        </geometry>
-      </visual>
-      <collision>
-        <origin rpy="${PI_2} 0.0 0.0" xyz="0.0 0.00401 0.0"/>
-        <geometry>
-          <mesh filename="package://dvrk_model/meshes/instruments/roll/4162/roll_4162_yaw.dae"/>
-        </geometry>
-      </collision>
     </link>
   </xacro:macro>

Commit message: removed reference to roll connector

File: urdf/common/instruments/roll/roll_4162.urdf.xacro (robot description, xacro)
@@ -16,4 +16,5 @@
           <mesh filename="package://dvrk_model/meshes/instruments/roll/4162/roll_4162.dae"/>
         </geometry>
+        <material name="roll_4162_shaft"><color rgba="0.55 0.55 0.55 1"/></material>
       </visual>
       <collision>

File: urdf/common/instruments/roll/roll_4670.urdf.xacro (robot description, xacro)
@@ -16,5 +16,5 @@
           <mesh filename="package://dvrk_model/meshes/instruments/roll/4670/roll_4670.obj"/>
         </geometry>
-        <material name=""><color rgba="0.79216 0.81961 0.93333 1"/></material>
+        <material name="roll_4670_shaft"><color rgba="0.55 0.55 0.55 1"/></material>
       </visual>
       <collision>
@@ -24,16 +24,4 @@
         </geometry>
       </collision>
-      <visual>
-        <origin rpy="0.0 0.0 1.5708" xyz="0.0 0.0 -0.0091"/>
-        <geometry>
-          <mesh filename="package://dvrk_model/meshes/instruments/roll/4670/roll_4670_connector.stl"/>
-        </geometry>
-      </visual>
-      <collision>
-        <origin rpy="0.0 0.0 1.5708" xyz="0.0 0.0 -0.0091"/>
-        <geometry>
-          <mesh filename="package://dvrk_model/meshes/instruments/roll/4670/roll_4670_connector.stl"/>
-        </geometry>
-      </collision>
     </link>
   </xacro:macro>

Commit message: Temporary collision geometries to get started on dvrk_pybullet

File: urdf/common/instruments/roll/roll_4162.urdf.xacro (robot description, xacro)
@@ -22,7 +22,8 @@
       </visual>
       <collision>
-        <origin rpy="-${PI_2} 0.0 0.0" xyz="0.0 0.0 0.02975"/>
+        <!-- Mesh-aligned shaft envelope (the OBJ shaft axis is local Y). -->
+        <origin rpy="${PI} 0.0 0.0" xyz="0.0 0.0 -0.27677977"/>
         <geometry>
-          <mesh filename="package://dvrk_model/meshes/instruments/roll/4670/roll_4670.obj" scale="0.1 0.1 0.1"/>
+          <cylinder radius="0.0043725" length="0.5596247"/>
         </geometry>
       </collision>

File: urdf/common/instruments/roll/roll_4670.urdf.xacro (robot description, xacro)
@@ -22,7 +22,8 @@
       </visual>
       <collision>
-        <origin rpy="-${PI_2} 0.0 0.0" xyz="0.0 0.0 0.02975"/>
+        <!-- Mesh-aligned shaft envelope (the OBJ shaft axis is local Y). -->
+        <origin rpy="${PI} 0.0 0.0" xyz="0.0 0.0 -0.27677977"/>
         <geometry>
-          <mesh filename="package://dvrk_model/meshes/instruments/roll/4670/roll_4670.obj" scale="0.1 0.1 0.1"/>
+          <cylinder radius="0.0043725" length="0.5596247"/>
         </geometry>
       </collision>

File: urdf/common/instruments/tip/tip_006.urdf.xacro (robot description, xacro)
@@ -27,4 +27,9 @@
       <xacro:instrument_link_color add_colors="${add_colors}" kind="tip"/>
       </visual>
+      <collision>
+        <!-- Mesh-aligned jaw envelope; it follows jaw_1 directly. -->
+        <origin xyz="0.0000005 0.0036195 0.000469" rpy="0.0 0.0 0.0"/>
+        <geometry><box size="0.004825 0.012065 0.003000"/></geometry>
+      </collision>
     </link>
     <joint name="jaw_2" type="revolute">
@@ -44,4 +49,9 @@
       <xacro:instrument_link_color add_colors="${add_colors}" kind="tip"/>
       </visual>
+      <collision>
+        <!-- Mesh-aligned jaw envelope; it follows jaw_2 directly. -->
+        <origin xyz="-0.0000005 0.0036195 -0.0004945" rpy="0.0 0.0 0.0"/>
+        <geometry><box size="0.004825 0.012065 0.003000"/></geometry>
+      </collision>
     </link>
     <joint name="tool_tip" type="fixed">

File: urdf/common/instruments/wrist_pitch/wrist_pitch_0091.urdf.xacro (robot description, xacro)
@@ -18,4 +18,9 @@
       <xacro:instrument_link_color add_colors="${add_colors}" kind="pitch"/>
       </visual>
+      <collision>
+        <!-- Mesh-aligned bounding box; refine against CAD later. -->
+        <origin rpy="0.0 ${PI_2} ${PI_2}" xyz="0.0042213 -0.00001255 -0.00003155"/>
+        <geometry><box size="0.0062955 0.0145274 0.0063857"/></geometry>
+      </collision>
     </link>
   </xacro:macro>

File: urdf/common/instruments/wrist_yaw/wrist_yaw_0091.urdf.xacro (robot description, xacro)
@@ -18,4 +18,9 @@
       <xacro:instrument_link_color add_colors="${add_colors}" kind="yaw"/>
       </visual>
+      <collision>
+        <!-- Mesh-aligned bounding box; refine against CAD later. -->
+        <origin rpy="0.0 0.0 0.0" xyz="0.0000005 0.0 -0.0001145"/>
+        <geometry><box size="0.001229 0.001230 0.005461"/></geometry>
+      </collision>
     </link>
   </xacro:macro>
