Commit message: removed 0 sized boxes, EGL rendering in PyBullet replaced these with small blue cubes

File: urdf/Classic/archive/psm_tool_caudier.urdf.xacro (robot description, xacro)
@@ -59,12 +59,5 @@
     </joint>
     <!-- link 7-0: Outer open angle virtual -->
-    <link name="${prefix}tool_wrist_caudier_ee_link_0">
-      <visual>
-        <origin rpy="0 0 0" xyz="0 0 0"/>
-        <geometry>
-          <box size="0 0 0" />
-        </geometry>
-      </visual>
-    </link>
+    <link name="${prefix}tool_wrist_caudier_ee_link_0"/>
     <!-- joint 7-1: Outer open angle 1 -->
     <joint name="jaw_mimic_1" type="revolute">

File: urdf/Classic/archive/psm_tool_sca.urdf.xacro (robot description, xacro)
@@ -50,12 +50,5 @@
     </joint>
     <!-- link 7-0: Outer open angle virtual -->
-    <link name="${prefix}tool_wrist_sca_ee_link_0">
-      <visual>
-        <origin rpy="0 0 0" xyz="0 0 0"/>
-        <geometry>
-          <box size="0 0 0" />
-        </geometry>
-      </visual>
-    </link>
+    <link name="${prefix}tool_wrist_sca_ee_link_0"/>
     <!-- joint 7-1: Outer open angle 1  -->
     <joint name="jaw_mimic_1" type="revolute">

File: urdf/Classic/archive/psm_tool_snake.urdf.xacro (robot description, xacro)
@@ -81,12 +81,5 @@
     </joint>
     <!-- link 11-0: Outer open angle virtual -->
-    <link name="${prefix}tool_wrist_snake_ee_link_0">
-      <visual>
-        <origin rpy="0 0 0" xyz="0 0 0.0"/>
-        <geometry>
-          <box size="0 0 0" />
-        </geometry>
-      </visual>
-    </link>
+    <link name="${prefix}tool_wrist_snake_ee_link_0"/>
     <!-- joint 11-1: Outer open angle 1  -->
     <joint name="jaw_mimic_1" type="revolute">

File: urdf/common/instruments/tip/tip_006.urdf.xacro (robot description, xacro)
@@ -10,10 +10,5 @@
       <limit lower="-0.349066" upper="1.39626" velocity=".4" effort="1000"/>
     </joint>
-    <link name="${prefix}jaw_link">
-      <visual>
-        <origin rpy="0.0 0.0 0.0" xyz="0.0 0.0 0.0"/>
-        <geometry><box size="0 0 0"/></geometry>
-      </visual>
-    </link>
+    <link name="${prefix}jaw_link"/>
     <joint name="jaw_1" type="revolute">
       <parent link="${prefix}wrist_yaw_link"/>

File: urdf/common/instruments/tip/tip_049.urdf.xacro (robot description, xacro)
@@ -10,12 +10,5 @@
       <limit lower="-0.349066" upper="1.5708" velocity=".4" effort="1000"/>
     </joint>
-    <link name="${prefix}jaw_link">
-      <visual>
-        <origin rpy="0.0 0.0 0.0" xyz="0.0 0.0 0.0"/>
-        <geometry>
-          <box size="0 0 0"/>
-        </geometry>
-      </visual>
-    </link>
+    <link name="${prefix}jaw_link"/>
     <joint name="jaw_1" type="revolute">
       <parent link="${prefix}wrist_yaw_link"/>

File: urdf/common/instruments/tip/tip_093.urdf.xacro (robot description, xacro)
@@ -28,10 +28,5 @@
       <limit lower="0.0" upper="1.0472" velocity=".4" effort="1000"/>
     </joint>
-    <link name="${prefix}jaw_link">
-      <visual>
-        <origin rpy="0.0 0.0 0.0" xyz="0.0 0.0 0.0"/>
-        <geometry><box size="0 0 0"/></geometry>
-      </visual>
-    </link>
+    <link name="${prefix}jaw_link"/>
   <joint name="jaw_1" type="revolute">
     <!-- Keep the tip hinge axes independent of the jaw-link rotation. -->

File: urdf/common/instruments/tip/tip_172.urdf.xacro (robot description, xacro)
@@ -10,12 +10,5 @@
       <limit lower="-0.349066" upper="1.39626" velocity=".4" effort="1000"/>
     </joint>
-    <link name="${prefix}jaw_link">
-      <visual>
-        <origin xyz="0 0 0" rpy="0 0 0"/>
-        <geometry>
-          <box size="0 0 0"/>
-        </geometry>
-      </visual>
-    </link>
+    <link name="${prefix}jaw_link"/>
     <joint name="jaw_1" type="revolute">
       <parent link="${prefix}wrist_yaw_link"/>

File: urdf/common/instruments/tip/tip_179.urdf.xacro (robot description, xacro)
@@ -10,10 +10,5 @@
       <limit lower="-0.349066" upper="1.39626" velocity=".4" effort="1000"/>
     </joint>
-    <link name="${prefix}jaw_link">
-      <visual>
-        <origin rpy="0.0 0.0 0.0" xyz="0.0 0.0 0.0"/>
-        <geometry><box size="0 0 0"/></geometry>
-      </visual>
-    </link>
+    <link name="${prefix}jaw_link"/>
     <joint name="jaw_1" type="revolute">
       <parent link="${prefix}wrist_yaw_link"/>

File: urdf/common/instruments/tip/tip_194.urdf.xacro (robot description, xacro)
@@ -10,12 +10,5 @@
       <limit lower="-0.349066" upper="1.39626" velocity=".4" effort="1000"/>
     </joint>
-    <link name="${prefix}jaw_link">
-      <visual>
-        <origin rpy="0.0 0.0 0.0" xyz="0.0 0.0 0.0"/>
-        <geometry>
-          <box size="0 0 0"/>
-        </geometry>
-      </visual>
-    </link>
+    <link name="${prefix}jaw_link"/>
     <joint name="jaw_1" type="revolute">
       <parent link="${prefix}wrist_yaw_link"/>

File: urdf/common/instruments/tip/tip_309.urdf.xacro (robot description, xacro)
@@ -10,12 +10,5 @@
       <limit lower="-0.349066" upper="1.5708" velocity=".4" effort="1000"/>
     </joint>
-    <link name="${prefix}jaw_link">
-      <visual>
-        <origin rpy="0.0 0.0 0.0" xyz="0.0 0.0 0.0"/>
-        <geometry>
-          <box size="0 0 0"/>
-        </geometry>
-      </visual>
-    </link>
+    <link name="${prefix}jaw_link"/>
     <joint name="jaw_1" type="revolute">
       <parent link="${prefix}wrist_yaw_link"/>

File: urdf/common/instruments/tip/tip_327.urdf.xacro (robot description, xacro)
@@ -10,12 +10,5 @@
       <limit lower="-0.349066" upper="0.733038" velocity=".4" effort="1000"/>
     </joint>
-    <link name="${prefix}jaw_link">
-      <visual>
-        <origin xyz="0 0 0" rpy="0 0 0"/>
-        <geometry>
-          <box size="0 0 0"/>
-        </geometry>
-      </visual>
-    </link>
+    <link name="${prefix}jaw_link"/>
     <joint name="jaw_1" type="revolute">
       <parent link="${prefix}wrist_yaw_link"/>
