Commit message: Renamed link between PSM active arm and instrument adaptor_link.  Fixed for PSM Classic and Si.

File: urdf/Virtual/PSM1.urdf.xacro (robot description, xacro)
@@ -9,6 +9,8 @@
       rcm_xyz      — trocar position in world frame
       rcm_rpy      — trocar orientation in world frame
+      adaptor_offset — instrument_base offset from the RCM
   -->
   <xacro:arg name="instrument"   default="420006"/>
+  <xacro:arg name="adaptor_offset" default="0.4826"/>
   <xacro:arg name="rcm_xyz"      default="0 0 0"/>
   <xacro:arg name="rcm_rpy"      default="0 0 0"/>
@@ -18,9 +20,10 @@
   <!-- 3 virtual DOFs at the trocar — no arm geometry -->
   <xacro:base_virtual prefix="PSM1_"
+                          adaptor_offset="$(arg adaptor_offset)"
                           rcm_xyz="$(arg rcm_xyz)"
                           rcm_rpy="$(arg rcm_rpy)"/>
-  <!-- Instrument: identical to Classic/Si — attaches at PSM_tool_parent_link -->
+  <!-- Instrument: identical to Classic/Si — attaches at PSM_adaptor_link -->
   <xacro:PSM_instrument prefix="PSM1_"
-                        parent_link="PSM1_tool_parent_link"
+                        parent_link="PSM1_adaptor_link"
                         instrument="$(arg instrument)"/>
 </robot>

File: urdf/Virtual/PSM2.urdf.xacro (robot description, xacro)
@@ -2,4 +2,5 @@
 <robot name="PSM2" xmlns:xacro="http://www.ros.org/wiki/xacro">
   <xacro:arg name="instrument"   default="420006"/>
+  <xacro:arg name="adaptor_offset" default="0.4826"/>
   <xacro:arg name="rcm_xyz"      default="0 0 0"/>
   <xacro:arg name="rcm_rpy"      default="0 0 0"/>
@@ -8,8 +9,9 @@
   <link name="world"/>
   <xacro:base_virtual prefix="PSM2_"
+                          adaptor_offset="$(arg adaptor_offset)"
                           rcm_xyz="$(arg rcm_xyz)"
                           rcm_rpy="$(arg rcm_rpy)"/>
   <xacro:PSM_instrument prefix="PSM2_"
-                        parent_link="PSM2_tool_parent_link"
+                        parent_link="PSM2_adaptor_link"
                         instrument="$(arg instrument)"/>
 </robot>

File: urdf/Virtual/PSM3.urdf.xacro (robot description, xacro)
@@ -2,4 +2,5 @@
 <robot name="PSM3" xmlns:xacro="http://www.ros.org/wiki/xacro">
   <xacro:arg name="instrument"   default="420006"/>
+  <xacro:arg name="adaptor_offset" default="0.4826"/>
   <xacro:arg name="rcm_xyz"      default="0 0 0"/>
   <xacro:arg name="rcm_rpy"      default="0 0 0"/>
@@ -8,8 +9,9 @@
   <link name="world"/>
   <xacro:base_virtual prefix="PSM3_"
+                          adaptor_offset="$(arg adaptor_offset)"
                           rcm_xyz="$(arg rcm_xyz)"
                           rcm_rpy="$(arg rcm_rpy)"/>
   <xacro:PSM_instrument prefix="PSM3_"
-                        parent_link="PSM3_tool_parent_link"
+                        parent_link="PSM3_adaptor_link"
                         instrument="$(arg instrument)"/>
 </robot>

File: urdf/Virtual/PSM_base_virtual.urdf.xacro (robot description, xacro)
@@ -1,4 +1,5 @@
 <?xml version="1.0" encoding="utf-8"?>
 <robot name="dvrk_psm_virtual" xmlns:xacro="http://www.ros.org/wiki/xacro">
+  <xacro:include filename="$(find dvrk_model)/urdf/common.urdf.xacro"/>
   <!--
     Virtual PSM base — simulator variant.
@@ -12,8 +13,10 @@
     All three links share a small but non-zero inertia so physics
     simulators (Gazebo, Isaac) can integrate without singularities.
-    Output: ends at ${prefix}tool_parent_link — identical to the
+    Output: ends at ${prefix}adaptor_link — identical to the
     full Classic/Si base so PSM_instrument attaches without modification.
     Parameters:
       prefix    — arm instance prefix, e.g. "PSM1_"
+      adaptor_offset — instrument_base offset from RCM (Classic: 0.4318,
+                       Si: 0.4826)
       rcm_xyz   — trocar position in world frame (default: origin)
       rcm_rpy   — trocar orientation in world frame (default: identity)
@@ -24,4 +27,5 @@
   <xacro:macro name="base_virtual"
                params="prefix
+                       adaptor_offset:='0.4826'
                        rcm_xyz:='0 0 0'
                        rcm_rpy:='0 0 0'">
@@ -71,20 +75,20 @@
     </link>
     <!-- ── Joint 3: insertion ───────────────────────────────────────────── -->
-    <!--   Prismatic along z at the RCM. Models insertion depth.            -->
-    <!--   tool_parent_link serves as the insertion child AND the        -->
-    <!--   handoff link to PSM_instrument (same name as in Classic/Si base). -->
+    <!--   Prismatic along the PSM DH insertion axis. Models insertion depth. -->
+    <!--   adaptor_link serves as the insertion child AND the handoff link -->
+    <!--   to PSM_instrument (same name as in Classic/Si base).            -->
     <joint name="insertion" type="prismatic">
       <parent link="${prefix}RCM_pitch_link"/>
-      <child  link="${prefix}tool_parent_link"/>
+      <child  link="${prefix}adaptor_link"/>
       <axis xyz="0.0 0.0 1"/>
-      <origin xyz="0.0 0.0 0.0" rpy="0.0 0.0 0.0"/>
+      <origin xyz="0.0 0.0 ${adaptor_offset}" rpy="${PI} 0.0 ${-PI_2}"/>
       <limit lower="0.0" upper="0.240"
              effort="50" velocity="0.4"/>
     </joint>
     <!--
-      tool_parent_link — identical name to Classic/Si boundary link.
+      adaptor_link — identical name to Classic/Si boundary link.
       PSM_instrument attaches here; no change needed for any generation.
     -->
-    <link name="${prefix}tool_parent_link">
+    <link name="${prefix}adaptor_link">
       <inertial>
         <mass value="${virtual_mass}"/>

File: urdf/classic_arm/PSM1.urdf.xacro (robot description, xacro)
@@ -16,5 +16,5 @@
                   xyz="0.0 0.0 0.0" rpy="0.0 0.0 0.0"/>
   <xacro:PSM_instrument prefix="PSM1_"
-                        parent_link="PSM1_tool_parent_link"
+                        parent_link="PSM1_adaptor_link"
                         instrument="$(arg instrument)"/>
 </robot>

File: urdf/classic_arm/PSM2.urdf.xacro (robot description, xacro)
@@ -11,5 +11,5 @@
                   xyz="0.0 0.0 0.0" rpy="0.0 0.0 0.0"/>
   <xacro:PSM_instrument prefix="PSM2_"
-                        parent_link="PSM2_tool_parent_link"
+                        parent_link="PSM2_adaptor_link"
                         instrument="$(arg instrument)"/>
 </robot>

File: urdf/classic_arm/PSM3.urdf.xacro (robot description, xacro)
@@ -11,5 +11,5 @@
                   xyz="0.0 0.0 0.0" rpy="0.0 0.0 0.0"/>
   <xacro:PSM_instrument prefix="PSM3_"
-                        parent_link="PSM3_tool_parent_link"
+                        parent_link="PSM3_adaptor_link"
                         instrument="$(arg instrument)"/>
 </robot>

File: urdf/classic_arm/PSM_base.urdf.xacro (robot description, xacro)
@@ -1,4 +1,5 @@
 <?xml version="1.0" encoding="utf-8"?>
 <robot name="dvrk_psm" xmlns:xacro="http://www.ros.org/wiki/xacro">
+  <xacro:include filename="$(find dvrk_model)/urdf/common.urdf.xacro"/>
   <xacro:include filename="$(find dvrk_model)/urdf/common/RCM_visual.urdf.xacro"/>
   <!--
@@ -7,5 +8,5 @@
       Joint 2: pitch  (revolute, parallelogram linkage)
       Joint 3: insertion    (prismatic)
-    Macro output: ends at ${prefix}tool_parent_link.
+    Macro output: ends at ${prefix}adaptor_link.
     The instrument macro (PSM_instrument) attaches here and owns roll onward.
     Parameters:
@@ -155,16 +156,16 @@
     <joint name="insertion" type="prismatic">
       <parent link="${prefix}pitch_link"/>
-      <child  link="${prefix}tool_parent_link"/>
+      <child  link="${prefix}adaptor_link"/>
       <axis xyz="0.0 0.0 1"/>
-      <origin rpy="1.5708 0.0 0.0" xyz="0.0 0.4318 0.0"/>
+      <origin rpy="${PI_2} 0.0 0.0" xyz="0.0 0.4318 0.0"/>
       <limit lower="0" upper="0.240" velocity=".4" effort="1000"/>
     </joint>
     <!--
-      link 3: tool_parent_link
+      link 3: adaptor_link
       Massless boundary link — handoff point to PSM_instrument.
-      No mesh; both Si and Classic use this exact link name
-      so PSM_instrument is generation-agnostic.
+      This is the instrument_base frame from the kinematic JSON: aligned
+      with the insertion/roll axis and offset 0.4318 m from the RCM.
     -->
-    <link name="${prefix}tool_parent_link"/>
+    <link name="${prefix}adaptor_link"/>
   </xacro:macro>
 </robot>

File: urdf/common/PSM_instrument.urdf.xacro (robot description, xacro)
@@ -3,6 +3,5 @@
   <!--
     PSM instrument macro — generation-agnostic.
-    Attaches to ${parent_link} (= ${prefix}tool_parent_link from any
-    PSM_base variant: Classic, Si, or Virtual).
+    Attaches to ${parent_link} (= ${prefix}adaptor_link from the PSM base).
     DOF layout:
       Joint 4: roll         (revolute, D = shaft_length along z)
@@ -12,5 +11,5 @@
     Parameters:
       prefix        — arm instance prefix, e.g. "PSM1_"
-      parent_link   — must be ${prefix}tool_parent_link
+      parent_link   — must be ${prefix}adaptor_link
       shaft_length  — D parameter of roll joint (Classic: 0.4162, Si: 0.4670)
       instrument    — last 6 digits of instrument model number (e.g. "420006")
@@ -30,10 +29,10 @@
     <xacro:if value="${generation == 'Si'}">
       <xacro:PSM_instrument_si_roll_shaft prefix="${prefix}"
-                                          parent_link="${prefix}instrument_base_link"
+                                          parent_link="${parent_link}"
                                           roll_origin="${roll_origin}"/>
     </xacro:if>
     <xacro:if value="${generation == 'Classic'}">
       <xacro:PSM_instrument_classic_roll_shaft prefix="${prefix}"
-                                               parent_link="${prefix}instrument_base_link"
+                                               parent_link="${parent_link}"
                                                roll_origin="${roll_origin}"/>
     </xacro:if>

File: urdf/common/psm_tools/PSM_housing.urdf.xacro (robot description, xacro)
@@ -4,10 +4,10 @@
                params="prefix parent_link housing_family:=Classic">
     <xacro:property name="is_si_housing" value="${housing_family == 'Si'}"/>
-    <joint name="instrument_base_fixed" type="fixed">
+    <joint name="${prefix}instrument_housing_fixed" type="fixed">
       <parent link="${parent_link}"/>
-      <child  link="${prefix}instrument_base_link"/>
+      <child  link="${prefix}instrument_housing_link"/>
       <origin rpy="-1.5708 0.0 -1.5708" xyz="0.0 0.0 0.0"/>
     </joint>
-    <link name="${prefix}instrument_base_link">
+    <link name="${prefix}instrument_housing_link">
       <visual>
         <xacro:if value="${is_si_housing}">

File: urdf/si_arm/PSM1.urdf.xacro (robot description, xacro)
@@ -14,5 +14,5 @@
                   parent_link="${parent_link}"/>
   <xacro:PSM_instrument prefix="PSM1_"
-                        parent_link="PSM1_tool_parent_link"
+                        parent_link="PSM1_adaptor_link"
                         instrument="$(arg instrument)"/>
 </robot>

File: urdf/si_arm/PSM2.urdf.xacro (robot description, xacro)
@@ -10,5 +10,5 @@
                   parent_link="${parent_link}"/>
   <xacro:PSM_instrument prefix="PSM2_"
-                        parent_link="PSM2_tool_parent_link"
+                        parent_link="PSM2_adaptor_link"
                         instrument="$(arg instrument)"/>
 </robot>

File: urdf/si_arm/PSM3.urdf.xacro (robot description, xacro)
@@ -10,5 +10,5 @@
                   parent_link="${parent_link}"/>
   <xacro:PSM_instrument prefix="PSM3_"
-                        parent_link="PSM3_tool_parent_link"
+                        parent_link="PSM3_adaptor_link"
                         instrument="$(arg instrument)"/>
 </robot>

File: urdf/si_arm/PSM_base.urdf.xacro (robot description, xacro)
@@ -8,5 +8,5 @@
       Joint 2: pitch  (revolute, pitch, parallelogram linkage ×3)
       Joint 3: insertion (prismatic)
-    Macro output: ends at ${prefix}tool_parent_link.
+    Macro output: ends at ${prefix}adaptor_link.
     PSM_instrument attaches here and owns roll onward.
     Inertial data retained from original Si CAD export.
@@ -179,21 +179,22 @@
     </joint>
     <!--
-      joint 3: insertion (prismatic) — moved here from psm_tool.
-      Origin from original insertion_ref fixed joint (xyz 0.05061 0 0.41911)
-      combined with the insertion joint offset.
+      joint 3: insertion (prismatic)
+      The adaptor link is the instrument_base frame from PSM_Si.json.
+      This local transform keeps the adaptor on the insertion/roll axis,
+      0.4826 m from the RCM at zero insertion.
     -->
     <joint name="insertion" type="prismatic">
-      <origin xyz="0.05061 0.0 0.41911" rpy="${PI} 0.0 0.0"/>
+      <origin xyz="0.11523752 0.0 0.31095531" rpy="${PI} 0.0 ${-PI}"/>
       <parent link="${prefix}pitch_3_link"/>
-      <child  link="${prefix}tool_parent_link"/>
+      <child  link="${prefix}adaptor_link"/>
       <axis xyz="0.0 0.0 1"/>
       <limit lower="0.0" upper="0.299" velocity="0.4" effort="1000"/>
     </joint>
     <!--
-      tool_parent_link — boundary link; PSM_instrument attaches here.
-      No geometry; same name as Classic and Virtual so PSM_instrument
-      macro is generation-agnostic.
+      adaptor_link — boundary link; PSM_instrument attaches here.
+      No geometry; same name as Classic so PSM_instrument is
+      generation-agnostic.
     -->
-    <link name="${prefix}tool_parent_link"/>
+    <link name="${prefix}adaptor_link"/>
   </xacro:macro>
 </robot>

Commit message: feat: add Virtual generation support with configurable parent links, RCM parameters, and updated ROS2 launch configurations.

File: urdf/Virtual/PSM1.urdf.xacro (robot description, xacro)
@@ -7,17 +7,21 @@
                      shaft/roll geometry is selected in common/instrument
                      using the instrument code (Classic 40xxxx, Si 42xxxx)
-      rcm_xyz      — trocar position in world frame
-      rcm_rpy      — trocar orientation in world frame
+      parent_link_ — parent link for the RCM
+      rcm_xyz      — trocar position in parent link frame
+      rcm_rpy      — trocar orientation in parent link frame
       adaptor_offset — instrument_base offset from the RCM
   -->
   <xacro:arg name="instrument"   default="420006"/>
+  <xacro:arg name="parent_link_" default="world"/>
   <xacro:arg name="adaptor_offset" default="0.4826"/>
   <xacro:arg name="rcm_xyz"      default="0 0 0"/>
   <xacro:arg name="rcm_rpy"      default="0 0 0"/>
+  <xacro:property name="parent_link" value="$(arg parent_link_)"/>
   <xacro:include filename="$(find dvrk_model)/urdf/Virtual/PSM_base_virtual.urdf.xacro"/>
   <xacro:include filename="$(find dvrk_model)/urdf/common/instrument.urdf.xacro"/>
-  <link name="world"/>
+  <link name="${parent_link}"/>
   <!-- 3 virtual DOFs at the trocar — no arm geometry -->
   <xacro:base_virtual prefix="PSM1_"
+                          parent_link="${parent_link}"
                           adaptor_offset="$(arg adaptor_offset)"
                           rcm_xyz="$(arg rcm_xyz)"

File: urdf/Virtual/PSM2.urdf.xacro (robot description, xacro)
@@ -2,11 +2,14 @@
 <robot name="PSM2" xmlns:xacro="http://www.ros.org/wiki/xacro">
   <xacro:arg name="instrument"   default="420006"/>
+  <xacro:arg name="parent_link_" default="world"/>
   <xacro:arg name="adaptor_offset" default="0.4826"/>
   <xacro:arg name="rcm_xyz"      default="0 0 0"/>
   <xacro:arg name="rcm_rpy"      default="0 0 0"/>
+  <xacro:property name="parent_link" value="$(arg parent_link_)"/>
   <xacro:include filename="$(find dvrk_model)/urdf/Virtual/PSM_base_virtual.urdf.xacro"/>
   <xacro:include filename="$(find dvrk_model)/urdf/common/instrument.urdf.xacro"/>
-  <link name="world"/>
+  <link name="${parent_link}"/>
   <xacro:base_virtual prefix="PSM2_"
+                          parent_link="${parent_link}"
                           adaptor_offset="$(arg adaptor_offset)"
                           rcm_xyz="$(arg rcm_xyz)"

File: urdf/Virtual/PSM3.urdf.xacro (robot description, xacro)
@@ -2,11 +2,14 @@
 <robot name="PSM3" xmlns:xacro="http://www.ros.org/wiki/xacro">
   <xacro:arg name="instrument"   default="420006"/>
+  <xacro:arg name="parent_link_" default="world"/>
   <xacro:arg name="adaptor_offset" default="0.4826"/>
   <xacro:arg name="rcm_xyz"      default="0 0 0"/>
   <xacro:arg name="rcm_rpy"      default="0 0 0"/>
+  <xacro:property name="parent_link" value="$(arg parent_link_)"/>
   <xacro:include filename="$(find dvrk_model)/urdf/Virtual/PSM_base_virtual.urdf.xacro"/>
   <xacro:include filename="$(find dvrk_model)/urdf/common/instrument.urdf.xacro"/>
-  <link name="world"/>
+  <link name="${parent_link}"/>
   <xacro:base_virtual prefix="PSM3_"
+                          parent_link="${parent_link}"
                           adaptor_offset="$(arg adaptor_offset)"
                           rcm_xyz="$(arg rcm_xyz)"

File: urdf/Virtual/PSM_base_virtual.urdf.xacro (robot description, xacro)
@@ -2,12 +2,13 @@
 <robot name="dvrk_psm_virtual" xmlns:xacro="http://www.ros.org/wiki/xacro">
   <xacro:include filename="$(find dvrk_model)/urdf/common.urdf.xacro"/>
+  <xacro:include filename="$(find dvrk_model)/urdf/common/RCM_visual.urdf.xacro"/>
   <!--
     Virtual PSM base — simulator variant.
     Replaces the full parallelogram arm with 3 massless, geometry-free
-    joints all located at the fixed RCM (trocar) frame in world.
+    joints all located at the fixed RCM (trocar) frame.
     This is sufficient for simulation when only the instrument matters.
     DOF layout (same joint names as full model — ROS-compatible):
-      Joint 1: yaw   (revolute  z, ±π/2)
-      Joint 2: pitch (revolute  y, ±π/4)
+      Joint 1: yaw   (revolute -y, ±π/2, matching PSM Si)
+      Joint 2: pitch (revolute -x, ±π/4, matching PSM Si)
       Joint 3: insertion   (prismatic z,  0–0.240 m)
     All three links share a small but non-zero inertia so physics
@@ -19,6 +20,7 @@
       adaptor_offset — instrument_base offset from RCM (Classic: 0.4318,
                        Si: 0.4826)
-      rcm_xyz   — trocar position in world frame (default: origin)
-      rcm_rpy   — trocar orientation in world frame (default: identity)
+      parent_link — link to attach the RCM to (typically "world")
+      rcm_xyz   — trocar position in parent_link frame (default: origin)
+      rcm_rpy   — trocar orientation in parent_link frame (default: identity)
                   rpy convention: roll-pitch-yaw (radians)
   -->
@@ -27,21 +29,24 @@
   <xacro:macro name="base_virtual"
                params="prefix
+                       parent_link:='world'
                        adaptor_offset:='0.4826'
                        rcm_xyz:='0 0 0'
                        rcm_rpy:='0 0 0'">
-    <!-- Fixed anchor: world → RCM frame (trocar location) -->
+    <!-- Fixed anchor: parent_link -> RCM frame (trocar location) -->
     <joint name="${prefix}RCM_fixed" type="fixed">
-      <parent link="world"/>
+      <parent link="${parent_link}"/>
       <child  link="${prefix}RCM_link"/>
       <origin xyz="${rcm_xyz}" rpy="${rcm_rpy}"/>
     </joint>
     <!-- RCM frame link — not a DOF, just a named coordinate frame -->
-    <link name="${prefix}RCM_link"/>
+    <link name="${prefix}RCM_link">
+      <xacro:rcm_visual/>
+    </link>
     <!-- ── Joint 1: yaw ───────────────────────────────────────────── -->
-    <!--   Revolute about z at the RCM. Models the yaw of the PSM arm.      -->
+    <!--   Revolute about -y at the RCM. Models the yaw of the PSM arm (matching PSM Si). -->
     <joint name="yaw" type="revolute">
       <parent link="${prefix}RCM_link"/>
       <child  link="${prefix}RCM_yaw_link"/>
-      <axis xyz="0.0 0.0 1"/>
+      <axis xyz="0.0 -1.0 0.0"/>
       <origin xyz="0.0 0.0 0.0" rpy="0.0 0.0 0.0"/>
       <limit lower="-1.5707963" upper="1.5707963"
@@ -57,9 +62,9 @@
     </link>
     <!-- ── Joint 2: pitch ─────────────────────────────────────────── -->
-    <!--   Revolute about y at the RCM. Models the pitch of the PSM arm.    -->
+    <!--   Revolute about -x at the RCM. Models the pitch of the PSM arm (matching PSM Si). -->
     <joint name="pitch" type="revolute">
       <parent link="${prefix}RCM_yaw_link"/>
       <child  link="${prefix}RCM_pitch_link"/>
-      <axis xyz="0.0 1 0.0"/>
+      <axis xyz="-1.0 0.0 0.0"/>
       <origin xyz="0.0 0.0 0.0" rpy="0.0 0.0 0.0"/>
       <limit lower="-0.7853982" upper="0.7853982"
