Commit message: Add optional color support for virtual PSM instruments, used for tools not supporting mtl (e.g. PyBullet)

File: urdf/Virtual/PSM1.urdf.xacro (robot description, xacro)
@@ -14,4 +14,5 @@
   <xacro:arg name="instrument"   default="420006"/>
   <xacro:arg name="is_virtual"  default="true"/>
+  <xacro:arg name="add_colors" default="true"/>
   <xacro:arg name="parent_link_" default="world"/>
   <xacro:arg name="adaptor_offset" default="0.4826"/>
@@ -31,4 +32,5 @@
   <xacro:instrument prefix="PSM1_"
                         instrument="$(arg instrument)"
-                        is_virtual="$(arg is_virtual)"/>
+                        is_virtual="$(arg is_virtual)"
+                        add_colors="$(arg add_colors)"/>
 </robot>

File: urdf/Virtual/PSM2.urdf.xacro (robot description, xacro)
@@ -3,4 +3,5 @@
   <xacro:arg name="instrument"   default="420006"/>
   <xacro:arg name="is_virtual"  default="true"/>
+  <xacro:arg name="add_colors" default="true"/>
   <xacro:arg name="parent_link_" default="world"/>
   <xacro:arg name="adaptor_offset" default="0.4826"/>
@@ -18,4 +19,5 @@
   <xacro:instrument prefix="PSM2_"
                         instrument="$(arg instrument)"
-                        is_virtual="$(arg is_virtual)"/>
+                        is_virtual="$(arg is_virtual)"
+                        add_colors="$(arg add_colors)"/>
 </robot>

File: urdf/Virtual/PSM3.urdf.xacro (robot description, xacro)
@@ -3,4 +3,5 @@
   <xacro:arg name="instrument"   default="420006"/>
   <xacro:arg name="is_virtual"  default="true"/>
+  <xacro:arg name="add_colors" default="true"/>
   <xacro:arg name="parent_link_" default="world"/>
   <xacro:arg name="adaptor_offset" default="0.4826"/>
@@ -18,4 +19,5 @@
   <xacro:instrument prefix="PSM3_"
                         instrument="$(arg instrument)"
-                        is_virtual="$(arg is_virtual)"/>
+                        is_virtual="$(arg is_virtual)"
+                        add_colors="$(arg add_colors)"/>
 </robot>

File: urdf/common/instrument.urdf.xacro (robot description, xacro)
@@ -42,6 +42,27 @@
   <xacro:property name="instrument_table"
                   value="${xacro.load_yaml('$(find dvrk_model)/urdf/common/instruments/instruments.yaml')['instruments']}"/>
+  <!-- Opt-in URDF colors for the mesh-only virtual PSM instruments. -->
+  <xacro:property name="roll_color" value="0.1 0.1 0.1 1"/>
+  <xacro:property name="pitch_color" value="0.6 0.6 0.6 1"/>
+  <xacro:property name="yaw_color" value="0.5 0.5 0.5 1"/>
+  <xacro:property name="tip_color" value="0.4 0.4 0.4 1"/>
+  <xacro:macro name="instrument_link_color" params="add_colors kind">
+    <xacro:if value="${str(add_colors).lower() in ['true', '1']}">
+      <xacro:if value="${kind == 'roll'}">
+        <material name="roll_color"><color rgba="${roll_color}"/></material>
+      </xacro:if>
+      <xacro:if value="${kind == 'pitch'}">
+        <material name="pitch_color"><color rgba="${pitch_color}"/></material>
+      </xacro:if>
+      <xacro:if value="${kind == 'yaw'}">
+        <material name="yaw_color"><color rgba="${yaw_color}"/></material>
+      </xacro:if>
+      <xacro:if value="${kind == 'tip'}">
+        <material name="tip_color"><color rgba="${tip_color}"/></material>
+      </xacro:if>
+    </xacro:if>
+  </xacro:macro>
   <xacro:macro name="instrument_model"
-               params="prefix housing roll wrist_pitch wrist_yaw tip is_virtual:=false">
+               params="prefix housing roll wrist_pitch wrist_yaw tip is_virtual:=false add_colors:=false">
     <xacro:if value="${str(housing) == 'Classic' and str(is_virtual).lower() not in ['true', '1']}">
       <xacro:housing_Classic prefix="${prefix}"/>
@@ -51,68 +72,68 @@
     </xacro:if>
     <xacro:if value="${str(roll) == '4162'}">
-      <xacro:roll_4162 prefix="${prefix}"/>
+      <xacro:roll_4162 prefix="${prefix}" add_colors="${add_colors}"/>
     </xacro:if>
     <xacro:if value="${str(roll) == '4670'}">
-      <xacro:roll_4670 prefix="${prefix}"/>
+      <xacro:roll_4670 prefix="${prefix}" add_colors="${add_colors}"/>
     </xacro:if>
     <xacro:if value="${str(wrist_pitch) == '0091' or str(wrist_pitch) == '91'}">
-      <xacro:wrist_pitch_0091 prefix="${prefix}"/>
+      <xacro:wrist_pitch_0091 prefix="${prefix}" add_colors="${add_colors}"/>
     </xacro:if>
     <xacro:if value="${str(wrist_pitch) == '0093' or str(wrist_pitch) == '93'}">
-      <xacro:wrist_pitch_0093 prefix="${prefix}"/>
+      <xacro:wrist_pitch_0093 prefix="${prefix}" add_colors="${add_colors}"/>
     </xacro:if>
     <xacro:if value="${str(wrist_pitch) == '0100' or str(wrist_pitch) == '100'}">
-      <xacro:wrist_pitch_0100 prefix="${prefix}"/>
+      <xacro:wrist_pitch_0100 prefix="${prefix}" add_colors="${add_colors}"/>
     </xacro:if>
     <xacro:if value="${str(wrist_pitch) == '0107' or str(wrist_pitch) == '107'}">
-      <xacro:wrist_pitch_0107 prefix="${prefix}"/>
+      <xacro:wrist_pitch_0107 prefix="${prefix}" add_colors="${add_colors}"/>
     </xacro:if>
     <xacro:if value="${str(wrist_pitch) == '0112' or str(wrist_pitch) == '112'}">
-      <xacro:wrist_pitch_0112 prefix="${prefix}"/>
+      <xacro:wrist_pitch_0112 prefix="${prefix}" add_colors="${add_colors}"/>
     </xacro:if>
     <xacro:if value="${str(wrist_yaw) == '0091' or str(wrist_yaw) == '91'}">
-      <xacro:wrist_yaw_0091 prefix="${prefix}"/>
+      <xacro:wrist_yaw_0091 prefix="${prefix}" add_colors="${add_colors}"/>
     </xacro:if>
     <xacro:if value="${str(wrist_yaw) == '0093' or str(wrist_yaw) == '93'}">
-      <xacro:wrist_yaw_0093 prefix="${prefix}"/>
+      <xacro:wrist_yaw_0093 prefix="${prefix}" add_colors="${add_colors}"/>
     </xacro:if>
     <xacro:if value="${str(wrist_yaw) == '0100' or str(wrist_yaw) == '100'}">
-      <xacro:wrist_yaw_0100 prefix="${prefix}"/>
+      <xacro:wrist_yaw_0100 prefix="${prefix}" add_colors="${add_colors}"/>
     </xacro:if>
     <xacro:if value="${str(wrist_yaw) == '0107' or str(wrist_yaw) == '107'}">
-      <xacro:wrist_yaw_0107 prefix="${prefix}"/>
+      <xacro:wrist_yaw_0107 prefix="${prefix}" add_colors="${add_colors}"/>
     </xacro:if>
     <xacro:if value="${str(wrist_yaw) == '0112' or str(wrist_yaw) == '112'}">
-      <xacro:wrist_yaw_0112 prefix="${prefix}"/>
+      <xacro:wrist_yaw_0112 prefix="${prefix}" add_colors="${add_colors}"/>
     </xacro:if>
     <xacro:if value="${str(tip) == '006' or str(tip) == '6'}">
-      <xacro:tip_006 prefix="${prefix}"/>
+      <xacro:tip_006 prefix="${prefix}" add_colors="${add_colors}"/>
     </xacro:if>
     <xacro:if value="${str(tip) == '049' or str(tip) == '49'}">
-      <xacro:tip_049 prefix="${prefix}"/>
+      <xacro:tip_049 prefix="${prefix}" add_colors="${add_colors}"/>
     </xacro:if>
     <xacro:if value="${str(tip) == '093' or str(tip) == '93'}">
-      <xacro:tip_093 prefix="${prefix}"/>
+      <xacro:tip_093 prefix="${prefix}" add_colors="${add_colors}"/>
     </xacro:if>
     <xacro:if value="${str(tip) == '172'}">
-      <xacro:tip_172 prefix="${prefix}"/>
+      <xacro:tip_172 prefix="${prefix}" add_colors="${add_colors}"/>
     </xacro:if>
     <xacro:if value="${str(tip) == '179'}">
-      <xacro:tip_179 prefix="${prefix}"/>
+      <xacro:tip_179 prefix="${prefix}" add_colors="${add_colors}"/>
     </xacro:if>
     <xacro:if value="${str(tip) == '183'}">
-      <xacro:tip_183 prefix="${prefix}"/>
+      <xacro:tip_183 prefix="${prefix}" add_colors="${add_colors}"/>
     </xacro:if>
     <xacro:if value="${str(tip) == '184'}">
-      <xacro:tip_184 prefix="${prefix}"/>
+      <xacro:tip_184 prefix="${prefix}" add_colors="${add_colors}"/>
     </xacro:if>
     <xacro:if value="${str(tip) == '194'}">
-      <xacro:tip_194 prefix="${prefix}"/>
+      <xacro:tip_194 prefix="${prefix}" add_colors="${add_colors}"/>
     </xacro:if>
     <xacro:if value="${str(tip) == '309'}">
-      <xacro:tip_309 prefix="${prefix}"/>
+      <xacro:tip_309 prefix="${prefix}" add_colors="${add_colors}"/>
     </xacro:if>
     <xacro:if value="${str(tip) == '327'}">
-      <xacro:tip_327 prefix="${prefix}"/>
+      <xacro:tip_327 prefix="${prefix}" add_colors="${add_colors}"/>
     </xacro:if>
     <xacro:if value="${str(tip) not in ['006', '6',
@@ -126,9 +147,9 @@
                                         '309',
                                         '327']}">
-      <xacro:tip_placeholder prefix="${prefix}"/>
+      <xacro:tip_placeholder prefix="${prefix}" add_colors="${add_colors}"/>
     </xacro:if>
   </xacro:macro>
   <xacro:macro name="instrument"
-               params="prefix instrument is_virtual:=false">
+               params="prefix instrument is_virtual:=false add_colors:=false">
     <xacro:property name="model" value="${instrument_table[str(instrument)]}"/>
     <xacro:if value="${xacro.message('Using instrument ' + str(instrument) + ': ' + str(model['name'])) or False}"/>
@@ -139,5 +160,6 @@
                             wrist_yaw="${model['wrist_yaw']}"
                             tip="${model['tip']}"
-                            is_virtual="${is_virtual}"/>
+                            is_virtual="${is_virtual}"
+                            add_colors="${add_colors}"/>
   </xacro:macro>
 </robot>

File: urdf/common/instruments/roll/roll_4162.urdf.xacro (robot description, xacro)
@@ -2,5 +2,5 @@
 <robot name="dvrk_instrument_roll_4162" xmlns:xacro="http://www.ros.org/wiki/xacro">
   <xacro:include filename="$(find dvrk_model)/urdf/common.urdf.xacro"/>
-  <xacro:macro name="roll_4162" params="prefix">
+  <xacro:macro name="roll_4162" params="prefix add_colors:=false">
     <joint name="roll" type="revolute">
       <parent link="${prefix}adaptor_link"/>
@@ -16,5 +16,8 @@
           <mesh filename="package://dvrk_model/meshes/instruments/roll/4670/roll_4670.obj" scale="0.1 0.1 0.1"/>
         </geometry>
-        <material name="roll_4670_shaft"><color rgba="0.55 0.55 0.55 1"/></material>
+        <xacro:if value="${str(add_colors).lower() not in ['true', '1']}">
+          <material name="roll_4670_shaft"><color rgba="0.55 0.55 0.55 1"/></material>
+        </xacro:if>
+        <xacro:instrument_link_color add_colors="${add_colors}" kind="roll"/>
       </visual>
       <collision>

File: urdf/common/instruments/roll/roll_4670.urdf.xacro (robot description, xacro)
@@ -2,5 +2,5 @@
 <robot name="dvrk_instrument_roll_4670" xmlns:xacro="http://www.ros.org/wiki/xacro">
   <xacro:include filename="$(find dvrk_model)/urdf/common.urdf.xacro"/>
-  <xacro:macro name="roll_4670" params="prefix">
+  <xacro:macro name="roll_4670" params="prefix add_colors:=false">
     <joint name="roll" type="revolute">
       <parent link="${prefix}adaptor_link"/>
@@ -16,5 +16,8 @@
           <mesh filename="package://dvrk_model/meshes/instruments/roll/4670/roll_4670.obj" scale="0.1 0.1 0.1"/>
         </geometry>
-        <material name="roll_4670_shaft"><color rgba="0.55 0.55 0.55 1"/></material>
+        <xacro:if value="${str(add_colors).lower() not in ['true', '1']}">
+          <material name="roll_4670_shaft"><color rgba="0.55 0.55 0.55 1"/></material>
+        </xacro:if>
+        <xacro:instrument_link_color add_colors="${add_colors}" kind="roll"/>
       </visual>
       <collision>

File: urdf/common/instruments/tip/tip_006.urdf.xacro (robot description, xacro)
@@ -2,5 +2,5 @@
 <robot name="dvrk_instrument_tip_006" xmlns:xacro="http://www.ros.org/wiki/xacro">
   <xacro:include filename="$(find dvrk_model)/urdf/common.urdf.xacro"/>
-  <xacro:macro name="tip_006" params="prefix">
+  <xacro:macro name="tip_006" params="prefix add_colors:=false">
     <joint name="jaw" type="revolute">
       <parent link="${prefix}wrist_yaw_link"/>
@@ -25,4 +25,5 @@
           <mesh filename="package://dvrk_model/meshes/instruments/tip/006/tip_006_1.obj"/>
         </geometry>
+      <xacro:instrument_link_color add_colors="${add_colors}" kind="tip"/>
       </visual>
     </link>
@@ -41,4 +42,5 @@
           <mesh filename="package://dvrk_model/meshes/instruments/tip/006/tip_006_2.obj"/>
         </geometry>
+      <xacro:instrument_link_color add_colors="${add_colors}" kind="tip"/>
       </visual>
     </link>

File: urdf/common/instruments/tip/tip_049.urdf.xacro (robot description, xacro)
@@ -2,5 +2,5 @@
 <robot name="dvrk_instrument_tip_049" xmlns:xacro="http://www.ros.org/wiki/xacro">
   <xacro:include filename="$(find dvrk_model)/urdf/common.urdf.xacro"/>
-  <xacro:macro name="tip_049" params="prefix">
+  <xacro:macro name="tip_049" params="prefix add_colors:=false">
     <joint name="jaw" type="revolute">
       <parent link="${prefix}wrist_yaw_link"/>
@@ -29,4 +29,5 @@
             scale="0.1 0.1 0.1"/>
         </geometry>
+      <xacro:instrument_link_color add_colors="${add_colors}" kind="tip"/>
       </visual>
     </link>
@@ -49,4 +50,5 @@
             scale="0.1 0.1 0.1"/>
         </geometry>
+      <xacro:instrument_link_color add_colors="${add_colors}" kind="tip"/>
       </visual>
     </link>

File: urdf/common/instruments/tip/tip_093.urdf.xacro (robot description, xacro)
@@ -2,5 +2,5 @@
 <robot name="dvrk_instrument_tip_093" xmlns:xacro="http://www.ros.org/wiki/xacro">
   <xacro:include filename="$(find dvrk_model)/urdf/common.urdf.xacro"/>
-  <xacro:macro name="tip_093" params="prefix">
+  <xacro:macro name="tip_093" params="prefix add_colors:=false">
     <!--
       The ProGrasp jaw hinge is offset from wrist_yaw and this offset changes
@@ -47,4 +47,5 @@
           scale="0.001 0.001 0.001"/>
       </geometry>
+    <xacro:instrument_link_color add_colors="${add_colors}" kind="tip"/>
     </visual>
   </link>
@@ -66,4 +67,5 @@
           scale="0.001 0.001 0.001"/>
       </geometry>
+    <xacro:instrument_link_color add_colors="${add_colors}" kind="tip"/>
     </visual>
   </link>

File: urdf/common/instruments/tip/tip_172.urdf.xacro (robot description, xacro)
@@ -2,5 +2,5 @@
 <robot name="dvrk_instrument_tip_172" xmlns:xacro="http://www.ros.org/wiki/xacro">
   <xacro:include filename="$(find dvrk_model)/urdf/common.urdf.xacro"/>
-  <xacro:macro name="tip_172" params="prefix">
+  <xacro:macro name="tip_172" params="prefix add_colors:=false">
     <joint name="jaw" type="revolute">
       <parent link="${prefix}wrist_yaw_link"/>
@@ -26,4 +26,5 @@
                 scale="0.1 0.1 0.1"/>
         </geometry>
+      <xacro:instrument_link_color add_colors="${add_colors}" kind="tip"/>
       </visual>
     </link>
@@ -43,4 +44,5 @@
                 scale="0.1 0.1 0.1"/>
         </geometry>
+      <xacro:instrument_link_color add_colors="${add_colors}" kind="tip"/>
       </visual>
     </link>

File: urdf/common/instruments/tip/tip_179.urdf.xacro (robot description, xacro)
@@ -2,5 +2,5 @@
 <robot name="dvrk_instrument_tip_179" xmlns:xacro="http://www.ros.org/wiki/xacro">
   <xacro:include filename="$(find dvrk_model)/urdf/common.urdf.xacro"/>
-  <xacro:macro name="tip_179" params="prefix">
+  <xacro:macro name="tip_179" params="prefix add_colors:=false">
     <joint name="jaw" type="revolute">
       <parent link="${prefix}wrist_yaw_link"/>
@@ -28,4 +28,5 @@
           <mesh filename="package://dvrk_model/meshes/instruments/tip/179/tip_179_1.obj" scale="0.001 0.001 0.001"/>
         </geometry>
+      <xacro:instrument_link_color add_colors="${add_colors}" kind="tip"/>
       </visual>
     </link>
@@ -47,4 +48,5 @@
           <mesh filename="package://dvrk_model/meshes/instruments/tip/179/tip_179_2.obj" scale="0.001 0.001 0.001"/>
         </geometry>
+      <xacro:instrument_link_color add_colors="${add_colors}" kind="tip"/>
       </visual>
     </link>

File: urdf/common/instruments/tip/tip_183.urdf.xacro (robot description, xacro)
@@ -2,5 +2,5 @@
 <robot name="dvrk_instrument_tip_183" xmlns:xacro="http://www.ros.org/wiki/xacro">
   <xacro:include filename="$(find dvrk_model)/urdf/common.urdf.xacro"/>
-  <xacro:macro name="tip_183" params="prefix">
+  <xacro:macro name="tip_183" params="prefix add_colors:=false">
     <joint name="jaw" type="fixed">
       <parent link="${prefix}wrist_yaw_link"/>
@@ -14,4 +14,5 @@
           <mesh filename="package://dvrk_model/meshes/instruments/tip/183/tip_183.obj" scale="0.1 0.1 0.1"/>
         </geometry>
+      <xacro:instrument_link_color add_colors="${add_colors}" kind="tip"/>
       </visual>
     </link>

File: urdf/common/instruments/tip/tip_184.urdf.xacro (robot description, xacro)
@@ -2,5 +2,5 @@
 <robot name="dvrk_instrument_tip_184" xmlns:xacro="http://www.ros.org/wiki/xacro">
   <xacro:include filename="$(find dvrk_model)/urdf/common.urdf.xacro"/>
-  <xacro:macro name="tip_184" params="prefix">
+  <xacro:macro name="tip_184" params="prefix add_colors:=false">
     <joint name="jaw" type="fixed">
       <parent link="${prefix}wrist_yaw_link"/>
@@ -14,4 +14,5 @@
           <mesh filename="package://dvrk_model/meshes/instruments/tip/184/tip_184.obj" scale="0.1 0.1 0.1"/>
         </geometry>
+      <xacro:instrument_link_color add_colors="${add_colors}" kind="tip"/>
       </visual>
     </link>

File: urdf/common/instruments/tip/tip_194.urdf.xacro (robot description, xacro)
@@ -2,5 +2,5 @@
 <robot name="dvrk_instrument_tip_194" xmlns:xacro="http://www.ros.org/wiki/xacro">
   <xacro:include filename="$(find dvrk_model)/urdf/common.urdf.xacro"/>
-  <xacro:macro name="tip_194" params="prefix">
+  <xacro:macro name="tip_194" params="prefix add_colors:=false">
     <joint name="jaw" type="revolute">
       <parent link="${prefix}wrist_yaw_link"/>
@@ -25,4 +25,5 @@
           <mesh filename="package://dvrk_model/meshes/instruments/tip/194/tip_194_1.obj" scale="0.1 0.1 0.1"/>
         </geometry>
+      <xacro:instrument_link_color add_colors="${add_colors}" kind="tip"/>
       </visual>
     </link>
@@ -41,4 +42,5 @@
           <mesh filename="package://dvrk_model/meshes/instruments/tip/194/tip_194_2.obj" scale="0.1 0.1 0.1"/>
         </geometry>
+      <xacro:instrument_link_color add_colors="${add_colors}" kind="tip"/>
       </visual>
     </link>

File: urdf/common/instruments/tip/tip_309.urdf.xacro (robot description, xacro)
@@ -2,5 +2,5 @@
 <robot name="dvrk_instrument_tip_309" xmlns:xacro="http://www.ros.org/wiki/xacro">
   <xacro:include filename="$(find dvrk_model)/urdf/common.urdf.xacro"/>
-  <xacro:macro name="tip_309" params="prefix">
+  <xacro:macro name="tip_309" params="prefix add_colors:=false">
     <joint name="jaw" type="revolute">
       <parent link="${prefix}wrist_yaw_link"/>
@@ -29,4 +29,5 @@
             scale="0.1 0.1 0.1"/>
         </geometry>
+      <xacro:instrument_link_color add_colors="${add_colors}" kind="tip"/>
       </visual>
     </link>
@@ -48,4 +49,5 @@
             scale="0.1 0.1 0.1"/>
         </geometry>
+      <xacro:instrument_link_color add_colors="${add_colors}" kind="tip"/>
       </visual>
     </link>

File: urdf/common/instruments/tip/tip_327.urdf.xacro (robot description, xacro)
@@ -2,5 +2,5 @@
 <robot name="dvrk_instrument_tip_327" xmlns:xacro="http://www.ros.org/wiki/xacro">
   <xacro:include filename="$(find dvrk_model)/urdf/common.urdf.xacro"/>
-  <xacro:macro name="tip_327" params="prefix">
+  <xacro:macro name="tip_327" params="prefix add_colors:=false">
     <joint name="jaw" type="revolute">
       <parent link="${prefix}wrist_yaw_link"/>
@@ -26,4 +26,5 @@
                 scale="0.1 0.1 0.1"/>
         </geometry>
+      <xacro:instrument_link_color add_colors="${add_colors}" kind="tip"/>
       </visual>
     </link>
@@ -43,4 +44,5 @@
                 scale="0.1 0.1 0.1"/>
         </geometry>
+      <xacro:instrument_link_color add_colors="${add_colors}" kind="tip"/>
       </visual>
     </link>

File: urdf/common/instruments/tip/tip_placeholder.urdf.xacro (robot description, xacro)
@@ -2,5 +2,5 @@
 <robot name="dvrk_instrument_tip_placeholder" xmlns:xacro="http://www.ros.org/wiki/xacro">
   <xacro:include filename="$(find dvrk_model)/urdf/common.urdf.xacro"/>
-  <xacro:macro name="tip_placeholder" params="prefix">
+  <xacro:macro name="tip_placeholder" params="prefix add_colors:=false">
     <joint name="jaw" type="revolute">
       <parent link="${prefix}wrist_yaw_link"/>
@@ -14,4 +14,5 @@
         <origin rpy="0.0 0.0 0.0" xyz="0.0 0.0 0.0"/>
         <geometry><box size="0.005 0.005 0.005"/></geometry>
+        <xacro:instrument_link_color add_colors="${add_colors}" kind="tip"/>
       </visual>
     </link>
@@ -28,4 +29,5 @@
         <origin rpy="0.0 0.0 0.0" xyz="0.0 0.0025 0.0"/>
         <geometry><box size="0.005 0.005 0.005"/></geometry>
+        <xacro:instrument_link_color add_colors="${add_colors}" kind="tip"/>
       </visual>
     </link>
@@ -42,4 +44,5 @@
         <origin rpy="0.0 0.0 0.0" xyz="0.0 -0.0025 0.0"/>
         <geometry><box size="0.005 0.005 0.005"/></geometry>
+        <xacro:instrument_link_color add_colors="${add_colors}" kind="tip"/>
       </visual>
     </link>

File: urdf/common/instruments/wrist_pitch/wrist_pitch_0091.urdf.xacro (robot description, xacro)
@@ -2,5 +2,5 @@
 <robot name="dvrk_instrument_wrist_pitch_0091" xmlns:xacro="http://www.ros.org/wiki/xacro">
   <xacro:include filename="$(find dvrk_model)/urdf/common.urdf.xacro"/>
-  <xacro:macro name="wrist_pitch_0091" params="prefix">
+  <xacro:macro name="wrist_pitch_0091" params="prefix add_colors:=false">
     <joint name="wrist_pitch" type="revolute">
       <parent link="${prefix}roll_link"/>
@@ -16,4 +16,5 @@
           <mesh filename="package://dvrk_model/meshes/instruments/wrist_pitch/0091/wrist_pitch_0091.obj" scale="0.1 0.1 0.1"/>
         </geometry>
+      <xacro:instrument_link_color add_colors="${add_colors}" kind="pitch"/>
       </visual>
     </link>

File: urdf/common/instruments/wrist_pitch/wrist_pitch_0093.urdf.xacro (robot description, xacro)
@@ -2,5 +2,5 @@
 <robot name="dvrk_instrument_wrist_pitch_0093" xmlns:xacro="http://www.ros.org/wiki/xacro">
   <xacro:include filename="$(find dvrk_model)/urdf/common.urdf.xacro"/>
-  <xacro:macro name="wrist_pitch_0093" params="prefix">
+  <xacro:macro name="wrist_pitch_0093" params="prefix add_colors:=false">
     <joint name="wrist_pitch" type="revolute">
       <parent link="${prefix}roll_link"/>
@@ -16,4 +16,5 @@
           <mesh filename="package://dvrk_model/meshes/instruments/wrist_pitch/0093/wrist_pitch_0093.obj" scale="0.1 0.1 0.1"/>
         </geometry>
+      <xacro:instrument_link_color add_colors="${add_colors}" kind="pitch"/>
       </visual>
     </link>

File: urdf/common/instruments/wrist_pitch/wrist_pitch_0100.urdf.xacro (robot description, xacro)
@@ -2,5 +2,5 @@
 <robot name="dvrk_instrument_wrist_pitch_0100" xmlns:xacro="http://www.ros.org/wiki/xacro">
   <xacro:include filename="$(find dvrk_model)/urdf/common.urdf.xacro"/>
-  <xacro:macro name="wrist_pitch_0100" params="prefix">
+  <xacro:macro name="wrist_pitch_0100" params="prefix add_colors:=false">
     <joint name="wrist_pitch" type="revolute">
       <parent link="${prefix}roll_link"/>
@@ -16,4 +16,5 @@
           <mesh filename="package://dvrk_model/meshes/instruments/wrist_pitch/0100/wrist_pitch_0100.obj" scale="0.1 0.1 0.1"/>
         </geometry>
+      <xacro:instrument_link_color add_colors="${add_colors}" kind="pitch"/>
       </visual>
     </link>
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